File: 20200429/serenity-drone/pcb/CM4-CARRIER-1/CM4-CARRIER-1.kicad_sch (KiCad schematic)
At the start: 0 parts

Commit message: fix all the things
Other:
- company: Steve Griffing PE(CSE) CISSP-ISSEP CPP -> (none)
Changed lines of the file:
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@@
     (title "CM4-CARRIER-1")
     (date "2025") (rev "E")
-    (company "Steve Griffing PE(CSE) CISSP-ISSEP CPP")
     (comment_1 "Serenity-Class Tiltrotor UAV")
     (comment_2 "CC BY 4.0 creativecommons.org/licenses/by/4.0")
