File: 20200429/serenity-drone/pcb/SENSORHAT-1/SENSORHAT-1.kicad_sch (KiCad schematic)
At the start: 0 parts

Commit message: fix all the things
Other:
- company: Steve Griffing PE(CSE) CISSP-ISSEP CPP -> (none)
Changed lines of the file:
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@@
   (paper "A2")
   (title_block (title "SENSORHAT-1") (date "2026") (rev "H.1")
-    (company "Steve Griffing PE(CSE) CISSP-ISSEP CPP")
     (comment_1 "Serenity-Class Tiltrotor — 8-Node Rev H.1")
     (comment_2 "CC BY 4.0 creativecommons.org/licenses/by/4.0")
