File: serenity/kicad/COMMS-HAT-SWITCH.kicad_sch (KiCad schematic)
At the start: 0 parts

Commit message: fix all the things
Other:
- company: Steve Griffing PE(CSE) CISSP-ISSEP CPP -> (none)
Changed lines of the file:
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@@
   (paper "A2")
   (title_block (title "COMMS-HAT-SWITCH") (date "2026") (rev "I")
-    (company "Steve Griffing PE(CSE) CISSP-ISSEP CPP")
     (comment_1 "Serenity-Class Tiltrotor — 8-Node Rev I")
     (comment_2 "CC BY 4.0 creativecommons.org/licenses/by/4.0")
