File: serenity/kicad/TRIHAT-1.kicad_sch (KiCad schematic)
At the start: 0 parts

Commit message: fix all the things
Other:
- company: Steve Griffing PE(CSE) CISSP-ISSEP CPP -> (none)
Changed lines of the file:
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@@
     (title "TRIHAT-1")
     (date "2025") (rev "E")
-    (company "Steve Griffing PE(CSE) CISSP-ISSEP CPP")
     (comment_1 "SUPERSEDED by SENSORHAT-1 in Rev H — retained for reference only")
     (comment_2 "CC BY 4.0 creativecommons.org/licenses/by/4.0")
