File: serenity/kicad/CAPE-B-1.kicad_pcb (KiCad board)
At the start: 4 copper layers, 55 x 35 mm, 33 parts, among them J1 PB2I-P1-2x18, J10 Nano-Fit-4P-POWER, J11 JST-GH-4P-WINCH, J12 JST-GH-4P-LOAD-CELL, J13 1x8-NavLight-PWM, J2 PB2I-P2-2x18, J3 JST-GH-4P-CAN, J4 JST-GH-4P-RS485, J5 JST-GH-4P-1553, J6 JST-GH-6P-ETH1, J7 JST-GH-6P-ETH2, J8 JST-GH-3P-SiK, J9 JST-GH-3P-RCRS, T1 SM-1553-11, U1 RFM95W, U10 ATF16V8BQL, U11 W25Q128JV, U12 DRV8833, U13 HX711, U14 PCA9685, U2 WL1837MOD, U3 ATA6561, U4 MAX3485E, U5 DS26LV31, U6 DS26LV32, U7 DP83825I, U8 DP83825I, U9 SLB9670

Commit message: Replace generic PCB silk labels with short descriptive names
Update all F.SilkS/B.SilkS fp_text reference labels across 7 KiCad PCB
files, replacing J/U/T numeric designators with function-based names so
each component is identifiable on the board without a BOM lookup.

CAPE-A-1 / CAPE-A-1-no-comment:
  J1→PB2-P1, J2→PB2-P2, U1→IMU, U2→BARO, U3→GPS,
  U4/U5→CAN-TR/RS485, U6→1553-DRV, U7→1553-RCV, T1→1553-XFM,
  U8/U9→ETH1-PHY/ETH2-PHY, U10→TPM,
  J3→CAN-FD, J4→RS-485, J5→MIL-1553, J6→ETH1, J7→ETH2,
  J8→ESC-TLM, J9→SERVO, J10→PWR-IN

CAPE-B-1 (adds RF + payload peripherals):
  U1→LORA, U2→WIFI-BT, U10→SD-WB, U11→NOR-FLASH,
  U12→WINCH-DRV, U13→LOAD-ADC, U14→PWM-I2C,
  J8→SIK-TLM, J9→RC-RCVR, J11→WINCH, J12→LOAD-CELL, J13→NAV-LIGHT

COMMS-HAT-1 (connectors + crystal only; ICs already descriptive):
  J1→SIK-UART, J2→ETH, J3→GPIO-EXT, J4→CAN-FD,
  JP4→PWR-IN, Y1→ETH-CLK

COMMS-HAT-SWITCH:
  Y1→SW-CLK

TRIHAT-1 (superseded; ICs + inferred connector mapping):
  U1→IMU, U2→BARO, U3→GPS, U4→CAN-CTRL, U5→CAN-TR,
  U6→ETH-CTRL, U7→ETH-MAG, U8→TPM, U9→LDO, Y1→ETH-CLK,
  J-connectors mapped from net list (GPS/CAN-FD/ETH/ESC-OUT/SERVO-OUT/etc.)

CM3-CARRIER-1:
  J1→CM3-SDIMM, U1→CAN-CTRL, U1B→CAN-TR, U2→RS485,
  U3→MIL-1553, U4→ETH-CTRL, U5→USB-UART, U6→LDO, U7→HAT-EEPROM

Boards already fully descriptive (SENSORHAT-1, CM4-CARRIER-1,
CM4-CARRIER-2) are unchanged.

https://claude.ai/code/session_01GniMw4QukTVM7JMzyVjH6p
Parts:
- removed J1: PB2I-P1-2x18, PocketBeagle2:2x18_P1_Socket
- removed J10: Nano-Fit-4P-POWER, Connector_Molex_NanoFit
- removed J11: JST-GH-4P-WINCH, JST_GH_4P
- removed J12: JST-GH-4P-LOAD-CELL, JST_GH_4P
- removed J13: 1x8-NavLight-PWM, Connector_PinHeader_2.54mm
- removed J2: PB2I-P2-2x18, PocketBeagle2:2x18_P2_Socket
- removed J3: JST-GH-4P-CAN, JST_GH_4P
- removed J4: JST-GH-4P-RS485, JST_GH_4P
- removed J5: JST-GH-4P-1553, JST_GH_4P
- removed J6: JST-GH-6P-ETH1, JST_GH_6P
- removed J7: JST-GH-6P-ETH2, JST_GH_6P
- removed J8: JST-GH-3P-SiK, JST_GH_3P
- removed J9: JST-GH-3P-RCRS, JST_GH_3P
- removed T1: SM-1553-11, Package
- removed U1: RFM95W, RF_Module
- removed U10: ATF16V8BQL, Package
- removed U11: W25Q128JV, Package
- removed U12: DRV8833, Package
- removed U13: HX711, Package
- removed U14: PCA9685, Package
- removed U2: WL1837MOD, RF_Module
- removed U3: ATA6561, Package
- removed U4: MAX3485E, Package
- removed U5: DS26LV31, Package
- removed U6: DS26LV32, Package
- removed U7, U8: DP83825I, Package
- removed U9: SLB9670, Package
- added 1553-DRV: DS26LV31, Package, F.Cu at (127.0, 115.5)
- added 1553-RCV: DS26LV32, Package, F.Cu at (138.0, 115.5)
- added 1553-XFM: SM-1553-11, Package, F.Cu at (149.0, 115.5)
- added CAN-FD: JST-GH-4P-CAN, JST_GH_4P, F.Cu at (127.0, 95.5)
- added CAN-TR: ATA6561, Package, F.Cu at (127.0, 109.5)
- added ETH1: JST-GH-6P-ETH1, JST_GH_6P, F.Cu at (167.0, 95.5)
- added ETH1-PHY: DP83825I, Package, F.Cu at (146.0, 105.5)
- added ETH2: JST-GH-6P-ETH2, JST_GH_6P, F.Cu at (167.0, 102.5)
- added ETH2-PHY: DP83825I, Package, F.Cu at (165.0, 105.5)
- added LOAD-ADC: HX711, Package, F.Cu at (156.0, 115.5)
- added LOAD-CELL: JST-GH-4P-LOAD-CELL, JST_GH_4P, F.Cu at (156.0, 101.5)
- added LORA: RFM95W, RF_Module, F.Cu at (133.0, 101.5)
- added MIL-1553: JST-GH-4P-1553, JST_GH_4P, F.Cu at (127.0, 107.5)
- added NAV-LIGHT: 1x8-NavLight-PWM, Connector_PinHeader_2.54mm, F.Cu at (144.0, 95.5)
- added NOR-FLASH: W25Q128JV, Package, F.Cu at (168.0, 114.5)
- added PB2-P1: PB2I-P1-2x18, PocketBeagle2:2x18_P1_Socket, B.Cu at (148.5, 90.0)
- added PB2-P2: PB2I-P2-2x18, PocketBeagle2:2x18_P2_Socket, B.Cu at (148.5, 120.0)
- added PWM-I2C: PCA9685, Package, F.Cu at (144.0, 109.5)
- added PWR-IN: Nano-Fit-4P-POWER, Connector_Molex_NanoFit, F.Cu at (127.0, 93.5)
- added RC-RCVR: JST-GH-3P-RCRS, JST_GH_3P, F.Cu at (167.0, 114.5)
- added RS-485: JST-GH-4P-RS485, JST_GH_4P, F.Cu at (127.0, 102.5)
- added RS485: MAX3485E, Package, F.Cu at (135.0, 109.5)
- added SD-WB: ATF16V8BQL, Package, F.Cu at (160.0, 114.5)
- added SIK-TLM: JST-GH-3P-SiK, JST_GH_3P, F.Cu at (167.0, 108.5)
- added TPM: SLB9670, Package, F.Cu at (169.0, 95.5)
- added WIFI-BT: WL1837MOD, RF_Module, F.Cu at (162.0, 100.5)
- added WINCH: JST-GH-4P-WINCH, JST_GH_4P, F.Cu at (156.0, 95.5)
- added WINCH-DRV: DRV8833, Package, F.Cu at (156.0, 109.5)

Commit message: Add back-side RF/storage to CAPE-A-1; add GPIO expansion headers to CAPE-B-1
CAPE-A-1.kicad_pcb:
- Move RFM95W LoRa, WL1837MOD WiFi/BT, ATF16V8BQL CPLD write-blocker,
  W25Q128JV NOR flash, and microSD log slot to B.Cu back side
- Add nets for SPI1 bus (LoRa/NOR), SDIO bus (WiFi), and SD card signals
- Update title comment to list front/back component inventory

CAPE-B-1.kicad_pcb:
- Add 6 × JST-GH 3-pin GPIO expansion connectors (GPIO-A through GPIO-F)
  along bottom edge at 7mm spacing
- Add nets GPIO_EXP_A through GPIO_EXP_F
- Update title comment to mention GPIO expansion

https://claude.ai/code/session_01GniMw4QukTVM7JMzyVjH6p
Parts:
- added GPIO-A: JST-GH-3P-GPIO, JST_GH_3P, F.Cu at (131.0, 119.5)
- added GPIO-B: JST-GH-3P-GPIO, JST_GH_3P, F.Cu at (138.0, 119.5)
- added GPIO-C: JST-GH-3P-GPIO, JST_GH_3P, F.Cu at (145.0, 119.5)
- added GPIO-D: JST-GH-3P-GPIO, JST_GH_3P, F.Cu at (152.0, 119.5)
- added GPIO-E: JST-GH-3P-GPIO, JST_GH_3P, F.Cu at (159.0, 119.5)
- added GPIO-F: JST-GH-3P-GPIO, JST_GH_3P, F.Cu at (166.0, 119.5)
Changed lines of the file:
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@@
   (title_block
     (title "CAPE-B-1") (date "2026") (rev "M")
-    (comment 1 "Serenity-Class Tiltrotor UAV — CN Node Comms, Logging and Payload Cape")
+    (comment 1 "Serenity-Class Tiltrotor UAV — CN Node Comms, Logging, Payload and GPIO Expansion Cape")
     (comment 2 "CC BY 4.0 creativecommons.org/licenses/by/4.0")
     (comment 3 "PocketBeagle 2 Industrial (AM6254) expansion — 55x35mm 4L JLCPCB assembled")
@@
   (net 94 "SD_D3")
   (net 95 "SD_CD")
+  (net 96 "GPIO_EXP_A")
+  (net 97 "GPIO_EXP_B")
+  (net 98 "GPIO_EXP_C")
+  (net 99 "GPIO_EXP_D")
+  (net 100 "GPIO_EXP_E")
+  (net 101 "GPIO_EXP_F")
   (gr_line (start 121 87.5) (end 176 87.5) (layer "Edge.Cuts") (width 0.05))
   (gr_line (start 176 87.5) (end 176 122.5) (layer "Edge.Cuts") (width 0.05))
@@
     (pad "7" thru_hole circle (at 0 6.35) (size 1.7 1.7) (drill 1.0) (layers "*.Cu" "*.Mask"))
     (pad "8" thru_hole circle (at 0 8.89) (size 1.7 1.7) (drill 1.0) (layers "*.Cu" "*.Mask")))
+  (footprint "JST_GH_3P" (layer "F.Cu") (at 131 119.5) (property "Description" "GPIO expansion A — GND +3V3 GPIO_EXP_A")
+    (fp_text reference "GPIO-A" (at 0 -3) (layer "F.SilkS")
+      (effects (font (size 0.8 0.8) (thickness 0.15))))
+    (fp_text value "JST-GH-3P-GPIO" (at 0 3) (layer "F.Fab")
+      (effects (font (size 0.8 0.8) (thickness 0.15))))
+    (pad "1" smd rect (at -1.25 0) (size 0.8 1.6) (layers "F.Cu" "F.Paste" "F.Mask"))
+    (pad "2" smd rect (at  0.00 0) (size 0.8 1.6) (layers "F.Cu" "F.Paste" "F.Mask"))
+    (pad "3" smd rect (at  1.25 0) (size 0.8 1.6) (layers "F.Cu" "F.Paste" "F.Mask")))
+  (footprint "JST_GH_3P" (layer "F.Cu") (at 138 119.5) (property "Description" "GPIO expansion B — GND +3V3 GPIO_EXP_B")
+    (fp_text reference "GPIO-B" (at 0 -3) (layer "F.SilkS")
+      (effects (font (size 0.8 0.8) (thickness 0.15))))
+    (fp_text value "JST-GH-3P-GPIO" (at 0 3) (layer "F.Fab")
+      (effects (font (size 0.8 0.8) (thickness 0.15))))
+    (pad "1" smd rect (at -1.25 0) (size 0.8 1.6) (layers "F.Cu" "F.Paste" "F.Mask"))
+    (pad "2" smd rect (at  0.00 0) (size 0.8 1.6) (layers "F.Cu" "F.Paste" "F.Mask"))
+    (pad "3" smd rect (at  1.25 0) (size 0.8 1.6) (layers "F.Cu" "F.Paste" "F.Mask")))
+  (footprint "JST_GH_3P" (layer "F.Cu") (at 145 119.5) (property "Description" "GPIO expansion C — GND +3V3 GPIO_EXP_C")
+    (fp_text reference "GPIO-C" (at 0 -3) (layer "F.SilkS")
+      (effects (font (size 0.8 0.8) (thickness 0.15))))
+    (fp_text value "JST-GH-3P-GPIO" (at 0 3) (layer "F.Fab")
+      (effects (font (size 0.8 0.8) (thickness 0.15))))
+    (pad "1" smd rect (at -1.25 0) (size 0.8 1.6) (layers "F.Cu" "F.Paste" "F.Mask"))
+    (pad "2" smd rect (at  0.00 0) (size 0.8 1.6) (layers "F.Cu" "F.Paste" "F.Mask"))
+    (pad "3" smd rect (at  1.25 0) (size 0.8 1.6) (layers "F.Cu" "F.Paste" "F.Mask")))
+  (footprint "JST_GH_3P" (layer "F.Cu") (at 152 119.5) (property "Description" "GPIO expansion D — GND +3V3 GPIO_EXP_D")
+    (fp_text reference "GPIO-D" (at 0 -3) (layer "F.SilkS")
+      (effects (font (size 0.8 0.8) (thickness 0.15))))
+    (fp_text value "JST-GH-3P-GPIO" (at 0 3) (layer "F.Fab")
+      (effects (font (size 0.8 0.8) (thickness 0.15))))
+    (pad "1" smd rect (at -1.25 0) (size 0.8 1.6) (layers "F.Cu" "F.Paste" "F.Mask"))
+    (pad "2" smd rect (at  0.00 0) (size 0.8 1.6) (layers "F.Cu" "F.Paste" "F.Mask"))
+    (pad "3" smd rect (at  1.25 0) (size 0.8 1.6) (layers "F.Cu" "F.Paste" "F.Mask")))
+  (footprint "JST_GH_3P" (layer "F.Cu") (at 159 119.5) (property "Description" "GPIO expansion E — GND +3V3 GPIO_EXP_E")
+    (fp_text reference "GPIO-E" (at 0 -3) (layer "F.SilkS")
+      (effects (font (size 0.8 0.8) (thickness 0.15))))
+    (fp_text value "JST-GH-3P-GPIO" (at 0 3) (layer "F.Fab")
+      (effects (font (size 0.8 0.8) (thickness 0.15))))
+    (pad "1" smd rect (at -1.25 0) (size 0.8 1.6) (layers "F.Cu" "F.Paste" "F.Mask"))
+    (pad "2" smd rect (at  0.00 0) (size 0.8 1.6) (layers "F.Cu" "F.Paste" "F.Mask"))
+    (pad "3" smd rect (at  1.25 0) (size 0.8 1.6) (layers "F.Cu" "F.Paste" "F.Mask")))
+  (footprint "JST_GH_3P" (layer "F.Cu") (at 166 119.5) (property "Description" "GPIO expansion F — GND +3V3 GPIO_EXP_F")
+    (fp_text reference "GPIO-F" (at 0 -3) (layer "F.SilkS")
+      (effects (font (size 0.8 0.8) (thickness 0.15))))
+    (fp_text value "JST-GH-3P-GPIO" (at 0 3) (layer "F.Fab")
+      (effects (font (size 0.8 0.8) (thickness 0.15))))
+    (pad "1" smd rect (at -1.25 0) (size 0.8 1.6) (layers "F.Cu" "F.Paste" "F.Mask"))
+    (pad "2" smd rect (at  0.00 0) (size 0.8 1.6) (layers "F.Cu" "F.Paste" "F.Mask"))
+    (pad "3" smd rect (at  1.25 0) (size 0.8 1.6) (layers "F.Cu" "F.Paste" "F.Mask")))
 )
