File: serenity/kicad/CAPE-A-1.kicad_sch (KiCad schematic)
At the start: 13 parts, among them J1 PB2I-P1-2x18, J2 PB2I-P2-2x18, T1 SM-1553-11, U1 ICM-42688-P, U10 SLB9670, U2 BMP388, U3 SAM-M10Q, U4 ATA6561, U5 MAX3485E, U6 DS26LV31, U7 DS26LV32, U8 DP83825I, U9 DP83825I

Commit message: hopefully this doesn't breake everything
Other:
- company: (none) -> Griffing Technology LLC
Changed lines of the file:
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@@
 (kicad_sch (version 20240101) (generator eeschema)
-  (paper "A2")
+  (paper "A1")
   (title_block
-    (title "CAPE-A-1")
-    (date "2026")
-    (rev "M")
-    (comment 1 "Serenity-Class Tiltrotor UAV — FC Node Sensor and Flight Control Cape")
-    (comment 2 "CC BY 4.0 creativecommons.org/licenses/by/4.0")
-    (comment 3 "PocketBeagle 2 Industrial (AM6254) expansion — 55x35mm 4L JLCPCB assembled")
-    (comment 4 "ICM-42688-P IMU | BMP388 Baro | SAM-M10Q GPS | ATA6561 CAN FD | MAX3485E RS-485 | DS26LV31/32 1553 | DP83825I x2 ETH | SLB9670 TPM2")
-    (comment 5 "Hull: Peter Farell CC BY 4.0 | Nozzle: BamJr CC BY 4.0 | Firefly/Serenity fan-work, not officially licensed")
+    (title "CAPE-A-1") (date "2026-05-21") (rev "M") (company "Griffing Technology LLC")
+    (comment 1 "FC Node — Sensor + Flight Control Cape for Serenity UAV")
+    (comment 2 "Copyright 2026 Steve Griffing PE(CSE) CISSP-ISSEP CPP | Griffing Technology LLC")
+    (comment 3 "License: CC BY 4.0  |  creativecommons.org/licenses/by/4.0")
+    (comment 4 "Approved:                               Checked:")
   )
   (symbol (lib_id "Conn_36") (at 65.00 165.00 0)
     (unit 1) (exclude_from_sim no) (in_bom yes) (on_board yes) (dnp no)
-    (property "Reference" "J1" (at 57.00 116.55 0) (effects (font (size 1.27 1.27))))
-    (property "Value" "PB2I-P1-2x18" (at 57.00 213.45 0) (effects (font (size 1.27 1.27))))
+    (property "Reference" "J1" (at 57.00 111.25 0) (effects (font (size 1.27 1.27))))
+    (property "Value" "PB2I-P1-2x18" (at 57.00 218.75 0) (effects (font (size 1.27 1.27))))
     (property "Footprint" "" (at 0 0 0) (effects (font (size 1.27 1.27)) (hide yes)))
     (property "Datasheet" "" (at 0 0 0) (effects (font (size 1.27 1.27)) (hide yes)))
@@
   (symbol (lib_id "Conn_36") (at 65.00 430.00 0)
     (unit 1) (exclude_from_sim no) (in_bom yes) (on_board yes) (dnp no)
-    (property "Reference" "J2" (at 57.00 381.55 0) (effects (font (size 1.27 1.27))))
-    (property "Value" "PB2I-P2-2x18" (at 57.00 478.45 0) (effects (font (size 1.27 1.27))))
+    (property "Reference" "J2" (at 57.00 376.25 0) (effects (font (size 1.27 1.27))))
+    (property "Value" "PB2I-P2-2x18" (at 57.00 483.75 0) (effects (font (size 1.27 1.27))))
     (property "Footprint" "" (at 0 0 0) (effects (font (size 1.27 1.27)) (hide yes)))
     (property "Datasheet" "" (at 0 0 0) (effects (font (size 1.27 1.27)) (hide yes)))

Commit message: filled out the pcbs and schematics. also carved the nacelles to work in the proper nozzles
Parts:
- renumbered U6 to 1553-DRV, U7 to 1553-RCV, T1 to 1553-XFM, U2 to BARO, U4 to CAN-TR, U8 to ETH1-PHY, U9 to ETH2-PHY, U3 to GPS, U1 to IMU, J1 to PB2-P1, J2 to PB2-P2, U5 to RS485, U10 to TPM
Changed lines of the file:
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@@
   (symbol (lib_id "Conn_36") (at 65.00 165.00 0)
     (unit 1) (exclude_from_sim no) (in_bom yes) (on_board yes) (dnp no)
-    (property "Reference" "J1" (at 57.00 111.25 0) (effects (font (size 1.27 1.27))))
+    (property "Reference" "PB2-P1" (at 57.00 111.25 0) (effects (font (size 1.27 1.27))))
     (property "Value" "PB2I-P1-2x18" (at 57.00 218.75 0) (effects (font (size 1.27 1.27))))
     (property "Footprint" "" (at 0 0 0) (effects (font (size 1.27 1.27)) (hide yes)))
@@
   (symbol (lib_id "Conn_36") (at 65.00 430.00 0)
     (unit 1) (exclude_from_sim no) (in_bom yes) (on_board yes) (dnp no)
-    (property "Reference" "J2" (at 57.00 376.25 0) (effects (font (size 1.27 1.27))))
+    (property "Reference" "PB2-P2" (at 57.00 376.25 0) (effects (font (size 1.27 1.27))))
     (property "Value" "PB2I-P2-2x18" (at 57.00 483.75 0) (effects (font (size 1.27 1.27))))
     (property "Footprint" "" (at 0 0 0) (effects (font (size 1.27 1.27)) (hide yes)))
@@
   (symbol (lib_id "ICM-42688-P") (at 210.00 75.00 0)
     (unit 1) (exclude_from_sim no) (in_bom yes) (on_board yes) (dnp no)
-    (property "Reference" "U1" (at 210.00 62.38 0) (effects (font (size 1.27 1.27))))
+    (property "Reference" "IMU" (at 210.00 62.38 0) (effects (font (size 1.27 1.27))))
     (property "Value" "ICM-42688-P" (at 210.00 87.62 0) (effects (font (size 1.27 1.27))))
     (property "Footprint" "" (at 0 0 0) (effects (font (size 1.27 1.27)) (hide yes)))
@@
   (symbol (lib_id "BMP388") (at 310.00 75.00 0)
     (unit 1) (exclude_from_sim no) (in_bom yes) (on_board yes) (dnp no)
-    (property "Reference" "U2" (at 310.00 62.38 0) (effects (font (size 1.27 1.27))))
+    (property "Reference" "BARO" (at 310.00 62.38 0) (effects (font (size 1.27 1.27))))
     (property "Value" "BMP388" (at 310.00 87.62 0) (effects (font (size 1.27 1.27))))
     (property "Footprint" "" (at 0 0 0) (effects (font (size 1.27 1.27)) (hide yes)))
@@
   (symbol (lib_id "SAM-M10Q") (at 210.00 185.00 0)
     (unit 1) (exclude_from_sim no) (in_bom yes) (on_board yes) (dnp no)
-    (property "Reference" "U3" (at 210.00 174.92 0) (effects (font (size 1.27 1.27))))
+    (property "Reference" "GPS" (at 210.00 174.92 0) (effects (font (size 1.27 1.27))))
     (property "Value" "SAM-M10Q" (at 210.00 195.08 0) (effects (font (size 1.27 1.27))))
     (property "Footprint" "" (at 0 0 0) (effects (font (size 1.27 1.27)) (hide yes)))
@@
   (symbol (lib_id "ATA6561") (at 310.00 170.00 0)
     (unit 1) (exclude_from_sim no) (in_bom yes) (on_board yes) (dnp no)
-    (property "Reference" "U4" (at 310.00 158.65 0) (effects (font (size 1.27 1.27))))
+    (property "Reference" "CAN-TR" (at 310.00 158.65 0) (effects (font (size 1.27 1.27))))
     (property "Value" "ATA6561" (at 310.00 181.35 0) (effects (font (size 1.27 1.27))))
     (property "Footprint" "" (at 0 0 0) (effects (font (size 1.27 1.27)) (hide yes)))
@@
   (symbol (lib_id "MAX3485E") (at 210.00 260.00 0)
     (unit 1) (exclude_from_sim no) (in_bom yes) (on_board yes) (dnp no)
-    (property "Reference" "U5" (at 210.00 247.38 0) (effects (font (size 1.27 1.27))))
+    (property "Reference" "RS485" (at 210.00 247.38 0) (effects (font (size 1.27 1.27))))
     (property "Value" "MAX3485E" (at 210.00 272.62 0) (effects (font (size 1.27 1.27))))
     (property "Footprint" "" (at 0 0 0) (effects (font (size 1.27 1.27)) (hide yes)))
@@
   (symbol (lib_id "DS26LV31") (at 310.00 270.00 0)
     (unit 1) (exclude_from_sim no) (in_bom yes) (on_board yes) (dnp no)
-    (property "Reference" "U6" (at 310.00 252.30 0) (effects (font (size 1.27 1.27))))
+    (property "Reference" "1553-DRV" (at 310.00 252.30 0) (effects (font (size 1.27 1.27))))
     (property "Value" "DS26LV31" (at 310.00 287.70 0) (effects (font (size 1.27 1.27))))
     (property "Footprint" "" (at 0 0 0) (effects (font (size 1.27 1.27)) (hide yes)))
@@
   (symbol (lib_id "DS26LV32") (at 210.00 360.00 0)
     (unit 1) (exclude_from_sim no) (in_bom yes) (on_board yes) (dnp no)
-    (property "Reference" "U7" (at 210.00 344.84 0) (effects (font (size 1.27 1.27))))
+    (property "Reference" "1553-RCV" (at 210.00 344.84 0) (effects (font (size 1.27 1.27))))
     (property "Value" "DS26LV32" (at 210.00 375.16 0) (effects (font (size 1.27 1.27))))
     (property "Footprint" "" (at 0 0 0) (effects (font (size 1.27 1.27)) (hide yes)))
@@
   (symbol (lib_id "SM-1553-11") (at 310.00 360.00 0)
     (unit 1) (exclude_from_sim no) (in_bom yes) (on_board yes) (dnp no)
-    (property "Reference" "T1" (at 310.00 349.92 0) (effects (font (size 1.27 1.27))))
+    (property "Reference" "1553-XFM" (at 310.00 349.92 0) (effects (font (size 1.27 1.27))))
     (property "Value" "SM-1553-11" (at 310.00 370.08 0) (effects (font (size 1.27 1.27))))
     (property "Footprint" "" (at 0 0 0) (effects (font (size 1.27 1.27)) (hide yes)))
@@
   (symbol (lib_id "DP83825I") (at 210.00 475.00 0)
     (unit 1) (exclude_from_sim no) (in_bom yes) (on_board yes) (dnp no)
-    (property "Reference" "U8" (at 210.00 457.30 0) (effects (font (size 1.27 1.27))))
+    (property "Reference" "ETH1-PHY" (at 210.00 457.30 0) (effects (font (size 1.27 1.27))))
     (property "Value" "DP83825I" (at 210.00 492.70 0) (effects (font (size 1.27 1.27))))
     (property "Footprint" "" (at 0 0 0) (effects (font (size 1.27 1.27)) (hide yes)))
@@
   (symbol (lib_id "DP83825I") (at 360.00 475.00 0)
     (unit 1) (exclude_from_sim no) (in_bom yes) (on_board yes) (dnp no)
-    (property "Reference" "U9" (at 360.00 457.30 0) (effects (font (size 1.27 1.27))))
+    (property "Reference" "ETH2-PHY" (at 360.00 457.30 0) (effects (font (size 1.27 1.27))))
     (property "Value" "DP83825I" (at 360.00 492.70 0) (effects (font (size 1.27 1.27))))
     (property "Footprint" "" (at 0 0 0) (effects (font (size 1.27 1.27)) (hide yes)))
@@
   (symbol (lib_id "SLB9670") (at 360.00 185.00 0)
     (unit 1) (exclude_from_sim no) (in_bom yes) (on_board yes) (dnp no)
-    (property "Reference" "U10" (at 360.00 169.84 0) (effects (font (size 1.27 1.27))))
+    (property "Reference" "TPM" (at 360.00 169.84 0) (effects (font (size 1.27 1.27))))
     (property "Value" "SLB9670" (at 360.00 200.16 0) (effects (font (size 1.27 1.27))))
     (property "Footprint" "" (at 0 0 0) (effects (font (size 1.27 1.27)) (hide yes)))
