File: serenity/kicad/CAPE-B-1.kicad_sch (KiCad schematic)
At the start: 18 parts, among them J1 PB2I-P1-2x18, J2 PB2I-P2-2x18, T1 SM-1553-11, U1 RFM95W, U10 ATF16V8BQL, U11 W25Q128JV, U12 DRV8833, U13 HX711, U14 PCA9685, U2 WL1837MOD, U3 ATA6561, U4 MAX3485E, U5 DS26LV31, U6 DS26LV32, U7 DP83825I, U8 DP83825I, U9 SLB9670

Commit message: hopefully this doesn't breake everything
Other:
- company: (none) -> Griffing Technology LLC
Changed lines of the file:
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@@
 (kicad_sch (version 20240101) (generator eeschema)
-  (paper "A2")
+  (paper "A1")
   (title_block
-    (title "CAPE-B-1")
-    (date "2026")
-    (rev "M")
-    (comment 1 "Serenity-Class Tiltrotor UAV — CN Node Comms, Logging and Payload Cape")
-    (comment 2 "CC BY 4.0 creativecommons.org/licenses/by/4.0")
-    (comment 3 "PocketBeagle 2 Industrial (AM6254) expansion — 55x35mm 4L JLCPCB assembled")
-    (comment 4 "RFM95W LoRa | WL1837MOD WiFi/BT | ATA6561 CAN FD | MAX3485E RS-485 | DS26LV31/32 1553 | DP83825I x2 ETH | SLB9670 TPM2 | ATF16V8BQL CPLD | W25Q128JV NOR | DRV8833 Winch | HX711 Load Cell | PCA9685 PWM | microSD log slot")
-    (comment 5 "Hull: Peter Farell CC BY 4.0 | Nozzle: BamJr CC BY 4.0 | Firefly/Serenity fan-work, not officially licensed")
+    (title "CAPE-B-1") (date "2026-05-21") (rev "M") (company "Griffing Technology LLC")
+    (comment 1 "CN Node — Comms + Logging + Payload Cape for Serenity UAV")
+    (comment 2 "Copyright 2026 Steve Griffing PE(CSE) CISSP-ISSEP CPP | Griffing Technology LLC")
+    (comment 3 "License: CC BY 4.0  |  creativecommons.org/licenses/by/4.0")
+    (comment 4 "Approved:                               Checked:")
   )
   (symbol (lib_id "Conn_36") (at 65.00 165.00 0)
     (unit 1) (exclude_from_sim no) (in_bom yes) (on_board yes) (dnp no)
-    (property "Reference" "J1" (at 57.00 116.55 0) (effects (font (size 1.27 1.27))))
-    (property "Value" "PB2I-P1-2x18" (at 57.00 213.45 0) (effects (font (size 1.27 1.27))))
+    (property "Reference" "J1" (at 57.00 111.25 0) (effects (font (size 1.27 1.27))))
+    (property "Value" "PB2I-P1-2x18" (at 57.00 218.75 0) (effects (font (size 1.27 1.27))))
     (property "Footprint" "" (at 0 0 0) (effects (font (size 1.27 1.27)) (hide yes)))
     (property "Datasheet" "" (at 0 0 0) (effects (font (size 1.27 1.27)) (hide yes)))
@@
   (symbol (lib_id "Conn_36") (at 65.00 430.00 0)
     (unit 1) (exclude_from_sim no) (in_bom yes) (on_board yes) (dnp no)
-    (property "Reference" "J2" (at 57.00 381.55 0) (effects (font (size 1.27 1.27))))
-    (property "Value" "PB2I-P2-2x18" (at 57.00 478.45 0) (effects (font (size 1.27 1.27))))
+    (property "Reference" "J2" (at 57.00 376.25 0) (effects (font (size 1.27 1.27))))
+    (property "Value" "PB2I-P2-2x18" (at 57.00 483.75 0) (effects (font (size 1.27 1.27))))
     (property "Footprint" "" (at 0 0 0) (effects (font (size 1.27 1.27)) (hide yes)))
     (property "Datasheet" "" (at 0 0 0) (effects (font (size 1.27 1.27)) (hide yes)))

Commit message: filled out the pcbs and schematics. also carved the nacelles to work in the proper nozzles
Parts:
- renumbered U5 to 1553-DRV, U6 to 1553-RCV, T1 to 1553-XFM, U3 to CAN-TR, U7 to ETH1-PHY, U8 to ETH2-PHY, U13 to LOAD-ADC, U1 to LORA, U11 to NOR-FLASH, J1 to PB2-P1, J2 to PB2-P2, U14 to PWM-I2C, U4 to RS485, U10 to SD-WB, U9 to TPM, U2 to WIFI-BT, U12 to WINCH-DRV
Changed lines of the file:
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@@
   (symbol (lib_id "Conn_36") (at 65.00 165.00 0)
     (unit 1) (exclude_from_sim no) (in_bom yes) (on_board yes) (dnp no)
-    (property "Reference" "J1" (at 57.00 111.25 0) (effects (font (size 1.27 1.27))))
+    (property "Reference" "PB2-P1" (at 57.00 111.25 0) (effects (font (size 1.27 1.27))))
     (property "Value" "PB2I-P1-2x18" (at 57.00 218.75 0) (effects (font (size 1.27 1.27))))
     (property "Footprint" "" (at 0 0 0) (effects (font (size 1.27 1.27)) (hide yes)))
@@
   (symbol (lib_id "Conn_36") (at 65.00 430.00 0)
     (unit 1) (exclude_from_sim no) (in_bom yes) (on_board yes) (dnp no)
-    (property "Reference" "J2" (at 57.00 376.25 0) (effects (font (size 1.27 1.27))))
+    (property "Reference" "PB2-P2" (at 57.00 376.25 0) (effects (font (size 1.27 1.27))))
     (property "Value" "PB2I-P2-2x18" (at 57.00 483.75 0) (effects (font (size 1.27 1.27))))
     (property "Footprint" "" (at 0 0 0) (effects (font (size 1.27 1.27)) (hide yes)))
@@
   (symbol (lib_id "RFM95W") (at 210.00 70.00 0)
     (unit 1) (exclude_from_sim no) (in_bom yes) (on_board yes) (dnp no)
-    (property "Reference" "U1" (at 210.00 56.11 0) (effects (font (size 1.27 1.27))))
+    (property "Reference" "LORA" (at 210.00 56.11 0) (effects (font (size 1.27 1.27))))
     (property "Value" "RFM95W" (at 210.00 83.89 0) (effects (font (size 1.27 1.27))))
     (property "Footprint" "" (at 0 0 0) (effects (font (size 1.27 1.27)) (hide yes)))
@@
   (symbol (lib_id "WL1837MOD") (at 340.00 80.00 0)
     (unit 1) (exclude_from_sim no) (in_bom yes) (on_board yes) (dnp no)
-    (property "Reference" "U2" (at 340.00 63.57 0) (effects (font (size 1.27 1.27))))
+    (property "Reference" "WIFI-BT" (at 340.00 63.57 0) (effects (font (size 1.27 1.27))))
     (property "Value" "WL1837MOD" (at 340.00 96.43 0) (effects (font (size 1.27 1.27))))
     (property "Footprint" "" (at 0 0 0) (effects (font (size 1.27 1.27)) (hide yes)))
@@
   (symbol (lib_id "ATA6561") (at 210.00 170.00 0)
     (unit 1) (exclude_from_sim no) (in_bom yes) (on_board yes) (dnp no)
-    (property "Reference" "U3" (at 210.00 158.65 0) (effects (font (size 1.27 1.27))))
+    (property "Reference" "CAN-TR" (at 210.00 158.65 0) (effects (font (size 1.27 1.27))))
     (property "Value" "ATA6561" (at 210.00 181.35 0) (effects (font (size 1.27 1.27))))
     (property "Footprint" "" (at 0 0 0) (effects (font (size 1.27 1.27)) (hide yes)))
@@
   (symbol (lib_id "MAX3485E") (at 340.00 170.00 0)
     (unit 1) (exclude_from_sim no) (in_bom yes) (on_board yes) (dnp no)
-    (property "Reference" "U4" (at 340.00 157.38 0) (effects (font (size 1.27 1.27))))
+    (property "Reference" "RS485" (at 340.00 157.38 0) (effects (font (size 1.27 1.27))))
     (property "Value" "MAX3485E" (at 340.00 182.62 0) (effects (font (size 1.27 1.27))))
     (property "Footprint" "" (at 0 0 0) (effects (font (size 1.27 1.27)) (hide yes)))
@@
   (symbol (lib_id "DS26LV31") (at 210.00 275.00 0)
     (unit 1) (exclude_from_sim no) (in_bom yes) (on_board yes) (dnp no)
-    (property "Reference" "U5" (at 210.00 257.30 0) (effects (font (size 1.27 1.27))))
+    (property "Reference" "1553-DRV" (at 210.00 257.30 0) (effects (font (size 1.27 1.27))))
     (property "Value" "DS26LV31" (at 210.00 292.70 0) (effects (font (size 1.27 1.27))))
     (property "Footprint" "" (at 0 0 0) (effects (font (size 1.27 1.27)) (hide yes)))
@@
   (symbol (lib_id "DS26LV32") (at 340.00 270.00 0)
     (unit 1) (exclude_from_sim no) (in_bom yes) (on_board yes) (dnp no)
-    (property "Reference" "U6" (at 340.00 254.84 0) (effects (font (size 1.27 1.27))))
+    (property "Reference" "1553-RCV" (at 340.00 254.84 0) (effects (font (size 1.27 1.27))))
     (property "Value" "DS26LV32" (at 340.00 285.16 0) (effects (font (size 1.27 1.27))))
     (property "Footprint" "" (at 0 0 0) (effects (font (size 1.27 1.27)) (hide yes)))
@@
   (symbol (lib_id "SM-1553-11") (at 280.00 350.00 0)
     (unit 1) (exclude_from_sim no) (in_bom yes) (on_board yes) (dnp no)
-    (property "Reference" "T1" (at 280.00 339.92 0) (effects (font (size 1.27 1.27))))
+    (property "Reference" "1553-XFM" (at 280.00 339.92 0) (effects (font (size 1.27 1.27))))
     (property "Value" "SM-1553-11" (at 280.00 360.08 0) (effects (font (size 1.27 1.27))))
     (property "Footprint" "" (at 0 0 0) (effects (font (size 1.27 1.27)) (hide yes)))
@@
   (symbol (lib_id "DP83825I") (at 210.00 455.00 0)
     (unit 1) (exclude_from_sim no) (in_bom yes) (on_board yes) (dnp no)
-    (property "Reference" "U7" (at 210.00 437.30 0) (effects (font (size 1.27 1.27))))
+    (property "Reference" "ETH1-PHY" (at 210.00 437.30 0) (effects (font (size 1.27 1.27))))
     (property "Value" "DP83825I" (at 210.00 472.70 0) (effects (font (size 1.27 1.27))))
     (property "Footprint" "" (at 0 0 0) (effects (font (size 1.27 1.27)) (hide yes)))
@@
   (symbol (lib_id "DP83825I") (at 360.00 455.00 0)
     (unit 1) (exclude_from_sim no) (in_bom yes) (on_board yes) (dnp no)
-    (property "Reference" "U8" (at 360.00 437.30 0) (effects (font (size 1.27 1.27))))
+    (property "Reference" "ETH2-PHY" (at 360.00 437.30 0) (effects (font (size 1.27 1.27))))
     (property "Value" "DP83825I" (at 360.00 472.70 0) (effects (font (size 1.27 1.27))))
     (property "Footprint" "" (at 0 0 0) (effects (font (size 1.27 1.27)) (hide yes)))
@@
   (symbol (lib_id "SLB9670") (at 210.00 350.00 0)
     (unit 1) (exclude_from_sim no) (in_bom yes) (on_board yes) (dnp no)
-    (property "Reference" "U9" (at 210.00 334.84 0) (effects (font (size 1.27 1.27))))
+    (property "Reference" "TPM" (at 210.00 334.84 0) (effects (font (size 1.27 1.27))))
     (property "Value" "SLB9670" (at 210.00 365.16 0) (effects (font (size 1.27 1.27))))
     (property "Footprint" "" (at 0 0 0) (effects (font (size 1.27 1.27)) (hide yes)))
@@
   (symbol (lib_id "ATF16V8BQL") (at 380.00 280.00 0)
     (unit 1) (exclude_from_sim no) (in_bom yes) (on_board yes) (dnp no)
-    (property "Reference" "U10" (at 380.00 264.84 0) (effects (font (size 1.27 1.27))))
+    (property "Reference" "SD-WB" (at 380.00 264.84 0) (effects (font (size 1.27 1.27))))
     (property "Value" "ATF16V8BQL" (at 380.00 295.16 0) (effects (font (size 1.27 1.27))))
     (property "Footprint" "" (at 0 0 0) (effects (font (size 1.27 1.27)) (hide yes)))
@@
   (symbol (lib_id "W25Q128JV") (at 380.00 170.00 0)
     (unit 1) (exclude_from_sim no) (in_bom yes) (on_board yes) (dnp no)
-    (property "Reference" "U11" (at 380.00 154.84 0) (effects (font (size 1.27 1.27))))
+    (property "Reference" "NOR-FLASH" (at 380.00 154.84 0) (effects (font (size 1.27 1.27))))
     (property "Value" "W25Q128JV" (at 380.00 185.16 0) (effects (font (size 1.27 1.27))))
     (property "Footprint" "" (at 0 0 0) (effects (font (size 1.27 1.27)) (hide yes)))
@@
   (symbol (lib_id "DRV8833") (at 380.00 380.00 0)
     (unit 1) (exclude_from_sim no) (in_bom yes) (on_board yes) (dnp no)
-    (property "Reference" "U12" (at 380.00 364.84 0) (effects (font (size 1.27 1.27))))
+    (property "Reference" "WINCH-DRV" (at 380.00 364.84 0) (effects (font (size 1.27 1.27))))
     (property "Value" "DRV8833" (at 380.00 395.16 0) (effects (font (size 1.27 1.27))))
     (property "Footprint" "" (at 0 0 0) (effects (font (size 1.27 1.27)) (hide yes)))
@@
   (symbol (lib_id "HX711") (at 380.00 455.00 0)
     (unit 1) (exclude_from_sim no) (in_bom yes) (on_board yes) (dnp no)
-    (property "Reference" "U13" (at 380.00 442.38 0) (effects (font (size 1.27 1.27))))
+    (property "Reference" "LOAD-ADC" (at 380.00 442.38 0) (effects (font (size 1.27 1.27))))
     (property "Value" "HX711" (at 380.00 467.62 0) (effects (font (size 1.27 1.27))))
     (property "Footprint" "" (at 0 0 0) (effects (font (size 1.27 1.27)) (hide yes)))
@@
   (symbol (lib_id "PCA9685") (at 280.00 455.00 0)
     (unit 1) (exclude_from_sim no) (in_bom yes) (on_board yes) (dnp no)
-    (property "Reference" "U14" (at 280.00 439.84 0) (effects (font (size 1.27 1.27))))
+    (property "Reference" "PWM-I2C" (at 280.00 439.84 0) (effects (font (size 1.27 1.27))))
     (property "Value" "PCA9685" (at 280.00 470.16 0) (effects (font (size 1.27 1.27))))
     (property "Footprint" "" (at 0 0 0) (effects (font (size 1.27 1.27)) (hide yes)))
