File: avionics/kicad/Zoë/kicads/Zoë.kicad_pcb (KiCad board)
At the start: 4 copper layers, 55 x 35 mm, 43 parts, among them X2Y-CAN 4.7nF X2Y, X2Y-RS485 4.7nF X2Y

Commit message: Resolve TODO 0.1: rename RCRS code identifiers to 49MHZ_XCVR/XCVR-49MHZ
Code (net labels, C macros, connector/config identifiers) previously used
"RCRS" as a naming convention under the mistaken assumption the 49 MHz
link falls under FCC Part 95 Radio Control Radio Service. It's actually
governed by 47 CFR Part 15 §15.235 (REF-FCC-003) -- Part 95 was evaluated
and rejected (REF-FCC-004). User-approved rename target is frequency-
qualified "49MHZ_XCVR"/"XCVR-49MHZ" to avoid ambiguity with "Emma," the
board name that also carries LoRa.

Renamed: SI5351_RCRS_*/si5351_set_rcrs_channel() and MAL_RCRS_* firmware
macros; UART_RCRS_TX/RX KiCad net labels in the Zoe/Emma schematics and
PCBs (pure net-name text substitution, occurrence counts verified 1:1,
no geometry/placement/routing touched) and their generator scripts;
RCRS-49/TVS-RCRS/FB-RCRS component naming in Emma.md/Zoe.md and the
active current-specification files; a DTS pinctrl label and a malcolm
config key.

While auditing, also found and corrected a stale/incorrect citation in
the Cape-B-2 DTS overlay and in serenity-rev-r.jsx that still cited
"47 CFR Part 95 ... RCRS" as the governing regulation for the 49 MHz
channel plan -- the exact claim REFERENCES.md's REF-FCC-003 documents
as superseded everywhere else. Corrected to cite Part 15 Section 15.235.

Left unchanged: legitimate regulatory-term uses of "RCRS" (correctly
discussing the real FCC Part 95 RCRS designation for comparison/
rejection purposes); dated historical WBS log entries; already-archived
BOM snapshots that self-document the same correction via strikethrough;
Gerber fab output (net-name text is informational, doesn't affect the
physical board); the rcrs49_wire_post.scad filename itself (a physical-
file rename touching 7+ cross-references is separate, larger work).

ERC/DRC could not be re-verified in this environment: tools/validate_kicad.py
requires KiCad >=8 (sch erc/pcb drc CLI subcommands); only KiCad 7.0.11
was installable here (both the Ki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
Parts:
- VHF-XCVR: value JST-GH-3P-RCRS -> JST-GH-3P-XCVR-49MHZ
Connections:
- net UART_RCRS_RX renamed UART_49MHZ_XCVR_RX
- net UART_RCRS_TX renamed UART_49MHZ_XCVR_TX
Changed lines of the file:
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@@
 	(net 7 "MDC")
 	(net 8 "WINCH_IN1")
-	(net 9 "UART_RCRS_TX")
+	(net 9 "UART_49MHZ_XCVR_TX")
 	(net 10 "I2C0_SDA")
 	(net 11 "SPI1_CS_LORA")
@@
 	(net 29 "SPI1_CS_TPM")
 	(net 30 "RMII1_TX_EN")
-	(net 31 "UART_RCRS_RX")
+	(net 31 "UART_49MHZ_XCVR_RX")
 	(net 32 "RMII1_REF_CLK")
 	(net 33 "RMII1_CRS_DV")
@@
 			(layers "*.Cu" "*.Mask")
 			(remove_unused_layers no)
-			(net 31 "UART_RCRS_RX")
+			(net 31 "UART_49MHZ_XCVR_RX")
 		)
 		(pad "16" thru_hole circle
@@
 			(layers "*.Cu" "*.Mask")
 			(remove_unused_layers no)
-			(net 9 "UART_RCRS_TX")
+			(net 9 "UART_49MHZ_XCVR_TX")
 		)
 		(pad "17" thru_hole circle
@@
 			)
 		)
-		(property "Value" "JST-GH-3P-RCRS"
+		(property "Value" "JST-GH-3P-XCVR-49MHZ"
 			(at -13.25 0.5 0)
 			(layer "F.Fab")
@@
 			)
 		)
-		(property "Description" "RC Transceiver UART — GND UART_RCRS_TX UART_RCRS_RX"
+		(property "Description" "RC Transceiver UART — GND UART_49MHZ_XCVR_TX UART_49MHZ_XCVR_RX"
 			(at -5.5 -11.5 0)
 			(layer "F.Fab")
@@
 			(layers "*.Cu" "*.Mask")
 			(remove_unused_layers no)
-			(net 31 "UART_RCRS_RX")
+			(net 31 "UART_49MHZ_XCVR_RX")
 		)
 		(pad "16" thru_hole circle
@@
 			(layers "*.Cu" "*.Mask")
 			(remove_unused_layers no)
-			(net 9 "UART_RCRS_TX")
+			(net 9 "UART_49MHZ_XCVR_TX")
 		)
 		(pad "17" thru_hole circle
