File: avionics/kicad/Zoë/kicads/Zoë.kicad_pcb (KiCad board)
At the start: 4 copper layers, 55 x 35 mm, 43 parts, among them X2Y-CAN 4.7nF X2Y, X2Y-RS485 4.7nF X2Y

Commit message: lots of stuff
Parts:
- moved TVS-1553 3.96 mm to (126.6, 108.3)
- moved X2Y-CAN 3.21 mm to (124.8, 103.0)
- moved X2Y-RS485 2.82 mm to (126.0, 93.2)
Routing:
- net TMESH_P: track 2229.0 -> 0.00 mm, vias 2 -> 0
- net TMESH_N: track 2204.5 -> 0.00 mm, vias 2 -> 0
