File: avionics/kicad/Zoë/kicads/Zoë.kicad_sch (KiCad schematic)
At the start: 52 parts, among them SW1 SW_DIP_x02, X2Y_CAN 4.7nF_X2Y, X2Y_RS485 4.7nF_X2Y

Commit message: lots of stuff
Parts:
- WIFI & BT: renamed from WIFI-BT
- WINCH DRV: renamed from WINCH-DRV
- renumbered CMC_CAN to CMC-CAN, CMC_RS485 to CMC-RS485, ETH_PHY_B to ETH-PHY, X2Y_CAN to X2Y-CAN, X2Y_RS485 to X2Y-RS485
Changed lines of the file:
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@@
   (symbol (lib_id "WL1837MOD") (at 340.00 80.00 0)
     (unit 1) (exclude_from_sim no) (in_bom yes) (on_board yes) (dnp no)
-    (property "Reference" "WIFI-BT" (at 340.00 63.57 0) (effects (font (size 1.27 1.27))))
+    (property "Reference" "WIFI & BT" (at 340.00 63.57 0) (effects (font (size 1.27 1.27))))
     (property "Value" "WL1837MOD" (at 340.00 96.43 0) (effects (font (size 1.27 1.27))))
     (property "Footprint" "" (at 0 0 0) (effects (font (size 1.27 1.27)) (hide yes)))
@@
   (symbol (lib_id "DRV8833") (at 380.00 380.00 0)
     (unit 1) (exclude_from_sim no) (in_bom yes) (on_board yes) (dnp no)
-    (property "Reference" "WINCH-DRV" (at 380.00 364.84 0) (effects (font (size 1.27 1.27))))
+    (property "Reference" "WINCH DRV" (at 380.00 364.84 0) (effects (font (size 1.27 1.27))))
     (property "Value" "DRV8833" (at 380.00 395.16 0) (effects (font (size 1.27 1.27))))
     (property "Footprint" "" (at 0 0 0) (effects (font (size 1.27 1.27)) (hide yes)))
@@
   (symbol (lib_id "SRF2012") (at 225.00 170.00 0)
     (unit 1) (exclude_from_sim no) (in_bom yes) (on_board yes) (dnp no)
-    (property "Reference" "CMC_CAN" (at 225.00 163.65 0)
+    (property "Reference" "CMC-CAN" (at 225.00 163.65 0)
       (effects (font (size 1.27 1.27))))
     (property "Value" "SRF2012-100Y" (at 225.00 176.35 0)
@@
   (symbol (lib_id "SRF2012") (at 355.00 170.00 0)
     (unit 1) (exclude_from_sim no) (in_bom yes) (on_board yes) (dnp no)
-    (property "Reference" "CMC_RS485" (at 355.00 163.65 0)
+    (property "Reference" "CMC-RS485" (at 355.00 163.65 0)
       (effects (font (size 1.27 1.27))))
     (property "Value" "SRF2012-100Y" (at 355.00 176.35 0)
@@
   (symbol (lib_id "X2Y_4N7") (at 230.00 182.00 0)
     (unit 1) (exclude_from_sim no) (in_bom yes) (on_board yes) (dnp no)
-    (property "Reference" "X2Y_CAN" (at 230.00 176.92 0)
+    (property "Reference" "X2Y-CAN" (at 230.00 176.92 0)
       (effects (font (size 1.27 1.27))))
     (property "Value" "4.7nF_X2Y" (at 230.00 187.08 0)
@@
   (symbol (lib_id "X2Y_4N7") (at 360.00 182.00 0)
     (unit 1) (exclude_from_sim no) (in_bom yes) (on_board yes) (dnp no)
-    (property "Reference" "X2Y_RS485" (at 360.00 176.92 0)
+    (property "Reference" "X2Y-RS485" (at 360.00 176.92 0)
       (effects (font (size 1.27 1.27))))
     (property "Value" "4.7nF_X2Y" (at 360.00 187.08 0)
@@
   (symbol (lib_id "DP83825I") (at 350.00 680.00 0)
     (unit 1) (exclude_from_sim no) (in_bom yes) (on_board yes) (dnp no)
-    (property "Reference" "ETH_PHY_B" (at 350.00 665.00 0) (effects (font (size 1.27 1.27))))
+    (property "Reference" "ETH-PHY" (at 350.00 665.00 0) (effects (font (size 1.27 1.27))))
     (property "Value" "DP83825I" (at 350.00 695.00 0) (effects (font (size 1.27 1.27))))
     (property "Footprint" "Package_QFP:LQFP-32_7x7mm_P0.8mm" (at 0 0 0) (effects (font (size 1.27 1.27)) (hide yes)))
