File: avionics/kicad/ENC-NACELLE-1.kicad_sch (KiCad schematic)
At the start: 6 parts, among them J1 JST_GH_04P_SHLD, U1 AS5600

Commit message: physics and order
Parts:
- removed D1: PRTR5V0U2X, Package_TO_SOT_SMD:SOT-363_SC-70-6, symbol PRTR5V0U2X
- removed J1: JST_GH_04P_SHLD, Connector_JST:JST_GH_SM04B-GHS-TB_1x04-1MP_P1.25mm_Horizontal, symbol Conn_JST_GH_04P
- removed R_DIR, R_PGO: 10k, Resistor_SMD:R_0402_1005Metric, symbol R_SMD
- removed U1: AS5600, Package_SON:SOIC-8, symbol AS5600
- added C2: 1uF, Capacitor_SMD:C_0402_1005Metric, symbol C_SMD
- added P1: PIGTAIL_4W, symbol Conn_Pigtail_04
- added U1: MT6701QT, Package_DFN_QFN:QFN-16-1EP_3x3mm_P0.5mm_EP1.75x1.75mm, symbol MT6701QT
Connections:
- net +3V3: now also C1.1, C2.1, P1.3 (SDA), U1.16 (GND); no longer C1.2
- net ENC_SCL: now also P1.1 (GND), U1.11 (U)
- net ENC_SDA: now also P1.2 (+3V3), U1.12 (V)
- net GND: now also C1.2, C2.2, P1.4 (SCL), U1.13 (VDD); no longer C1.1
- no-connect marks 0 -> 7
Other:
- note added: "MAL-TILT-ENC-PCB — MT6701 nacelle tilt-angle encoder (7 x 7 mm in-house PCB)"
- note added: "MODE(14): internal 200kΩ pull-up, left OPEN = I2C/SSI (datasheet Fig-18). PUSH/OUT/Z/W/U/V unused in I2C mode (no-connect). NC pins 1-4,10. VDD=13, GND=16, SDA=6(A), SCL=7(B). Optional 6V TVS on VDD per Fig-18 (EMI)."
- note added: "P1: direct-solder 4-wire pigtail (no connector) 1=GND 2=+3V3 3=ENC_SDA 4=ENC_SCL to nacelle-control node — River (primary) / Simon (alternate). I2C pull-ups (4.7k on SDA/SCL) live at the node per datasheet Fig-18 — not on this board. Two nacelles: default addr 0x06; program one to 0x46 to share a bus, or use separate buses / TCA9548A."
- note added: "Rev R2f: pinout + I2C address VERIFIED vs Magntek MT6701 Rev.1.9 datasheet (avionics/datasheets/). 14-bit absolute angle (regs 0x03/0x04); I2C slave 0x06 default, programmable to 0x46; MODE(14) internal 200kΩ pull-up left open = I2C/SSI (datasheet Fig-18). Supersedes the Rev Q AS5600 board."
- note added: "⚠ MAGNET-TOPOLOGY DESIGN GATE (mechanical — not an electrical issue): The MT6701 is an ON-AXIS sensor. Per datasheet §6 it reads a Ø6 mm x 2.5 mm diametric CYLINDER magnet centred on the die: air gap 0.5-2.0 mm, field 200-1000 G, off-axis misalignment <= 0.3 mm. The airframe currently mounts it OFF-AXIS at R = 11 mm over a Ø22 ring (wings_s1223_revo.scad) — that is ~37x the 0.3 mm misalignment li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"
- title: ENC-NACELLE-1 — Nacelle Tilt Angle Encoder Board -> ENC-NACELLE-1 / MAL-TILT-ENC-PCB — Nacelle Tilt-Angle Encoder (MT6701)

Commit message: hall effect
Parts:
- P1: value PIGTAIL_4W -> PIGTAIL_7W; symbol Conn_Pigtail_04 -> Conn_Pigtail_07
- U1: value MT6701QT -> AK7455; footprint Package_DFN_QFN:QFN-16-1EP_3x3mm_P0.5mm_EP1.75x1.75mm -> Package_DFN_QFN:QFN-24-1EP_4x4mm_P0.5mm_EP2.6x2.6mm; symbol MT6701QT -> AK7455
Connections:
- net +3V3: now also C1.2, C2.2, P1.2 (+3V3), U1.11 (VDD); no longer C1.1, C2.1, P1.3 (SDA), U1.16 (GND)
- net GND: now also C1.1, C2.1, P1.1 (GND), U1.14 (VSS); no longer C1.2, C2.2, P1.4 (SCL)
- net ENC_ERROR: now reaches U1.15 (ERROR)
- net ENC_ERROR: now also P1.7 (ERROR)
- net ENC_MISO: now reaches U1.4 (MISO)
- net ENC_MISO: now also P1.5 (MISO)
- net ENC_MOSI: now reaches U1.5 (MOSI)
- net ENC_MOSI: now also P1.4 (MOSI)
- net ENC_SCLK: now reaches U1.6 (SCLK)
- net ENC_SCLK: now also P1.3 (SCLK)
- net ENC_CSN: now reaches U1.7 (CSN)
- net ENC_CSN: now also P1.6 (CSN)
- removed net ENC_SCL: P1.1 (GND), U1.11 (U)
- net ENC_SDA: no longer names the net of U1.12 (TEST1)
- net ENC_SDA: no longer P1.2 (+3V3)
- no-connect marks 7 -> 8
Other:
- note added: "MAL-TILT-ENC-PCB — AK7455 OFF-AXIS nacelle tilt-angle encoder (7 x 7 mm in-house PCB)"
- note added: "OFF-AXIS read (SUPPORTED by AK7455, unlike MT6701/AS5600): - Fixed IC on the wing-tip pad, off-axis beside the rotating ring on the tilt-spar hub. - Field at the IC must be 10-70 mT (Off-Axis); AK7455 alarms below ~15 mT (low-flux). - Set the sense plane via R_FIELDSEL (X-Y / X-Z / Y-Z) to match the mounting. - Ferromagnetic 4130/17-4 spar: AK7455 anomaly-field detection + error-reduction + EEPRO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"
- note added: "P1: direct-solder 7-wire pigtail (no connector) to node — River (primary) / Simon (alt). 1=GND 2=+3V3 3=SCLK 4=MOSI 5=MISO 6=CSN 7=ERROR (anomaly-field/low-flux alarm). SPI bus is SHARED port+stbd; each nacelle gets its own CSN (no address conflict). ERROR may be push-pull or open-drain — add a node-side pull-up if open-drain (verify datasheet)."
- note added: "Rev S: pinout VERIFIED vs AKM AK7455 datasheet 200800064-E-00 (avionics/datasheets/ak7455-en-datasheet-myakm.pdf). 14-bit absolute; Off-Axis (side-of-shaft) supported; 4-wire SPI + ABZ/UVW; anomaly-magnetic-field detection + error reduction (suits the ferromagnetic tilt-spar). Supersedes the on-axis MT6701 (rejected: on-axis only, cannot read a through-shaft off-axis) and the AS5600 Rev Q design."
- note added: "TEST2(13)->VSS. TEST1(12) OPEN. NC pins (8,9,10,19-24) OPEN. Back-tab/EP OPEN (do NOT ground). UVW (1,2,3) + ABZ (16,17,18) unused in SPI absolute mode -> no-connect. SPI = MISO(4) MOSI(5) SCLK(6) CSN(7). VDD(11)=+3V3, VSS(14)=GND, ERROR(15)."
- note removed: "MAL-TILT-ENC-PCB — MT6701 nacelle tilt-angle encoder (7 x 7 mm in-house PCB)"
- note removed: "MODE(14): internal 200kΩ pull-up, left OPEN = I2C/SSI (datasheet Fig-18). PUSH/OUT/Z/W/U/V unused in I2C mode (no-connect). NC pins 1-4,10. VDD=13, GND=16, SDA=6(A), SCL=7(B). Optional 6V TVS on VDD per Fig-18 (EMI)."
- note removed: "P1: direct-solder 4-wire pigtail (no connector) 1=GND 2=+3V3 3=ENC_SDA 4=ENC_SCL to nacelle-control node — River (primary) / Simon (alternate). I2C pull-ups (4.7k on SDA/SCL) live at the node per datasheet Fig-18 — not on this board. Two nacelles: default addr 0x06; program one to 0x46 to share a bus, or use separate buses / TCA9548A."
- note removed: "Rev R2f: pinout + I2C address VERIFIED vs Magntek MT6701 Rev.1.9 datasheet (avionics/datasheets/). 14-bit absolute angle (regs 0x03/0x04); I2C slave 0x06 default, programmable to 0x46; MODE(14) internal 200kΩ pull-up left open = I2C/SSI (datasheet Fig-18). Supersedes the Rev Q AS5600 board."
- note removed: "⚠ MAGNET-TOPOLOGY DESIGN GATE (mechanical — not an electrical issue): The MT6701 is an ON-AXIS sensor. Per datasheet §6 it reads a Ø6 mm x 2.5 mm diametric CYLINDER magnet centred on the die: air gap 0.5-2.0 mm, field 200-1000 G, off-axis misalignment <= 0.3 mm. The airframe currently mounts it OFF-AXIS at R = 11 mm over a Ø22 ring (wings_s1223_revo.scad) — that is ~37x the 0.3 mm misalignment li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"
- title: ENC-NACELLE-1 / MAL-TILT-ENC-PCB — Nacelle Tilt-Angle Encoder (MT6701) -> ENC-NACELLE-1 / MAL-TILT-ENC-PCB — Nacelle Tilt-Angle Encoder (AK7455, off-axis)
- moved on the sheet: C1, C2

Commit message: lots of stuff
Parts:
- P1: footprint (none) -> Serenity-Custom:Pigtail_7W_DirectSolder
Changed lines of the file:
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@@
     (property "Reference" "P1" (at 95.00 78.00 0) (effects (font (size 1.27 1.27))))
     (property "Value" "PIGTAIL_7W" (at 95.00 101.43 0) (effects (font (size 1.27 1.27))))
-    (property "Footprint" "" (at 0 0 0) (effects (font (size 1.27 1.27)) (hide yes)))
+    (property "Footprint" "Serenity-Custom:Pigtail_7W_DirectSolder" (at 0 0 0) (effects (font (size 1.27 1.27)) (hide yes)))
     (property "Datasheet" "" (at 0 0 0) (effects (font (size 1.27 1.27)) (hide yes)))
     (pin "1")
