File: avionics/kicad/ENC-NACELLE-1.kicad_pcb (KiCad board)
At the start: 2 copper layers, 7 x 14 mm, 6 parts, among them P1 PIGTAIL_7W, U1 AK7455

Commit message: just making everything shiny
Routing:
- net +3V3: track 14.1 -> 17.1 mm, vias 3 -> 4
Changed lines of the file:
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@@
+	)
+	(segment
+		(start 21.35 23.87)
+		(end 21.85 23.45)
+		(width 0.15)
+		(layer "F.Cu")
+		(net 1)
 	)
 	(segment
@@
 	(segment
 		(start 20.65 24.9)
-		(end 21 25.6)
+		(end 21.5 25.6)
 		(width 0.15)
 		(layer "F.Cu")
@@
 	)
 	(via
-		(at 21 25.6)
+		(at 21.5 25.6)
 		(size 0.6)
 		(drill 0.3)
@@
 		(net 1)
 	)
+	(via
+		(at 21.85 23.45)
+		(size 0.6)
+		(drill 0.3)
+		(layers "F.Cu" "B.Cu")
+		(net 1)
+	)
 	(segment
-		(start 21.2 26)
-		(end 21.2 29.2)
+		(start 21.35 26)
+		(end 21.35 29.2)
 		(width 0.2)
 		(layer "B.Cu")
@@
 	)
 	(segment
-		(start 21 25.6)
-		(end 21.2 26)
+		(start 21.5 25.6)
+		(end 21.35 26)
 		(width 0.2)
+		(layer "B.Cu")
+		(net 1)
+	)
+	(segment
+		(start 22.2 25.6)
+		(end 21.5 25.6)
+		(width 0.15)
+		(layer "B.Cu")
+		(net 1)
+	)
+	(segment
+		(start 21.85 23.45)
+		(end 22.2 23.87)
+		(width 0.15)
+		(layer "B.Cu")
+		(net 1)
+	)
+	(segment
+		(start 22.2 23.87)
+		(end 22.2 25.6)
+		(width 0.15)
 		(layer "B.Cu")
 		(net 1)
@@
 	(segment
 		(start 21.35 23.87)
-		(end 21 24.2)
-		(width 0.2)
+		(end 22.2 23.87)
+		(width 0.15)
 		(layer "B.Cu")
 		(net 1)
 	)
 	(segment
-		(start 21 24.2)
-		(end 21 25.6)
-		(width 0.2)
-		(layer "B.Cu")
-		(net 1)
-	)
-	(segment
-		(start 21.2 29.2)
+		(start 21.35 29.2)
 		(end 20.75 29.75)
 		(width 0.2)
