File: avionics/kicad/Kaylee/kicads/Kaylee.kicad_sch (KiCad schematic)
At the start: 99 parts

Commit message: lots of stuff
Parts:
- removed FB_6V: Wurth 742792612 600R@100MHz 2A, symbol FB_Generic
- removed J_6V: Molex Nano-Fit 4P 2.5mm servo bus, symbol Nano_Fit_4P
- removed J_SHLD_6V: PGND via-pad for 6V cable shield, symbol M3_ChassisPad
- removed L3: Wurth 744314100 10uH >=6A Isat, symbol L_Generic
- removed R_FB6_1: R for Vout=6.0V (top), symbol R_Generic
- removed R_FB6_2: R for Vout=6.0V (bot), symbol R_Generic
- removed U_BEC_6V: TPS54540DDAR 5A/40V buck 6.0V servo rail, symbol TPS54540DDAR
- added C_BOOT1, C_BOOT2, C_BOOT_SV: 100nF X7R (BOOT-SW), symbol C_Generic
- added C_COMP2_SV, C_COMPB1, C_COMPB2: C comp2 hi-f pole (verify per TPS54620 DS), symbol C_Generic
- added C_COMPA1, C_COMPA2, C_COMP_SV: C comp (verify per TPS54620 DS), symbol C_Generic
- added C_SS1, C_SS2, C_SS_SV: 10nF soft-start (verify per TPS54620 DS), symbol C_Generic
- added FB_SERVO: Wurth 742792612 600R@100MHz 2A, symbol FB_Generic
- added J_SERVO_5V: Molex Nano-Fit 4P 2.5mm SERVO-5V bus, symbol Nano_Fit_4P
- added J_SHLD_SV: PGND via-pad for SERVO-5V cable shield, symbol M3_ChassisPad
- added L4: Wurth 744314100 10uH >=6A Isat, symbol L_Generic
- added R_COMP1, R_COMP2, R_COMP_SV: R comp (verify per TPS54620 DS), symbol R_Generic
- added R_FBSV_1: R for Vout=5.0V (top), symbol R_Generic
- added R_FBSV_2: R for Vout=5.0V (bot), symbol R_Generic
- added R_VSNS: 0R Kelvin VBUS tap (VDIS), symbol R_Generic
- added U_BEC_SERVO_5V: TPS54620RGYT 6A/28V sync buck 5.0V servo rail, symbol TPS54620RGYT
- C_BEC_SV_OUT: value 100uF + 100nF output cap -> 220uF 10V electrolytic + 100nF X7R
Connections:
- net CM2_OUT_N is gone; now on net CM2_OUT_P: CM2.3 (OUT+)
- net PDB_SCL_RAW is gone; now on net PGND: D_I2C.1 (GND)
- net PDB_SDA_RAW is gone; now on net PDB_SDA: D_I2C.2 (IO1)
- net +5V: now also D_I2C.4 (VCC), J_I2C.2, R_ALERT.1, U_IS1.4 (VS), U_IS2.4 (VS), U_IS2.9 (A0), U_IS3.4 (VS), U_IS4.4 (VS), U_IS5.4 (VS), U_IS_MAIN.4 (VS), U_IS_MAIN.8 (A1)
- net 5V_AVIONICS: now also J_5V.1, J_5V.2; no longer J_5V.3, J_5V.4
- net B1: now also J_BAL.2; no longer J_BAL.6
- net B2: now also J_BAL.3; no longer J_BAL.5
- net B4: now also J_BAL.5; no longer J_BAL.3
- net B5: now also J_BAL.6; no longer J_BAL.2
- net B6: now also J_BAL.7; no longer J_BAL.1
- net BAL_GND_J: now also J_BAL.1, U_CELL.1 (VC0); no longer J_BAL.7
- net BEC5V1_RAW: now also D_OR1.1 (A1), L1.2; no longer D_OR1.2 (A2)
- net BEC5V2_RAW: now also D_OR2.1 (A1), L2.2; no longer D_OR2.2 (A2)
- net BOOT5V1: now also U_BEC_5V_1.7 (BOOT), C_BOOT1.1; no longer U_BEC_5V_1.9 (PGND)
- net BOOT5V2: now also U_BEC_5V_2.7 (BOOT), C_BOOT2.1; no longer U_BEC_5V_2.9 (PGND)
- net BQ_CAP: now also U_CELL.11 (CAP); no longer U_CELL.3 (VC2)
- net BQ_DSG_OUT: now also U_CELL.17 (DSG)
- net CM1_OUT_N: now also CM1.4 (OUT-), CM2.2 (IN-); no longer CM1.3 (OUT+), CM2.1 (IN+)
- net CM1_OUT_P: now also CM1.3 (OUT+), CM2.1 (IN+); no longer CM1.4 (OUT-), CM2.2 (IN-)
- net CM2_OUT_P: no longer CM2.4 (OUT-)
- net COMP5V1: now also C_COMPB1.1, R_COMP1.1
- net COMP5V2: now also C_COMPB2.1, R_COMP2.1
- net DSG_GATE: now also Q_BATT_DSG.1 (G); no longer Q_BATT_DSG.2 (S)
- net ESC1_CM_OUT: now also CM_ESC1.3 (OUT+), RS1.1 (F+); no longer CM_ESC1.4 (OUT-), RS1.2 (S+)
- net ESC1_FUSED: now also CM_ESC1.1 (IN+); no longer CM_ESC1.2 (IN-)
- net ESC1_RS_OUT: now also J_ESC1.1, RS1.4 (F-), U_IS1.10 (VBUS); no longer J_ESC1.2, RS1.3 (S-), U_IS1.5 (SDA)
- net ESC1_RS_SN: now also RS1.3 (S-), U_IS1.2 (IN-); no longer RS1.4 (F-), U_IS1.4 (VS)
- net ESC1_RS_SP: now also RS1.2 (S+), U_IS1.1 (IN+); no longer RS1.1 (F+), U_IS1.9 (A0)
- net ESC2_CM_OUT: now also CM_ESC2.3 (OUT+), RS2.1 (F+); no longer CM_ESC2.4 (OUT-), RS2.2 (S+)
- net ESC2_FUSED: now also CM_ESC2.1 (IN+); no longer CM_ESC2.2 (IN-)
- net ESC2_RS_OUT: now also J_ESC2.1, RS2.4 (F-), U_IS2.10 (VBUS); no longer J_ESC2.2, RS2.3 (S-), U_IS2.5 (SDA)
- net ESC2_RS_SN: now also RS2.3 (S-), U_IS2.2 (IN-); no longer RS2.4 (F-), U_IS2.4 (VS)
- net ESC2_RS_SP: now also RS2.2 (S+), U_IS2.1 (IN+); no longer RS2.1 (F+), U_IS2.9 (A0)
- net ESC3_CM_OUT: now also CM_ESC3.3 (OUT+), RS3.1 (F+); no longer CM_ESC3.4 (OUT-), RS3.2 (S+)
- net ESC3_FUSED: now also CM_ESC3.1 (IN+); no longer CM_ESC3.2 (IN-)
- net ESC3_RS_OUT: now also J_ESC3.1, RS3.4 (F-), U_IS3.10 (VBUS); no longer J_ESC3.2, RS3.3 (S-), U_IS3.5 (SDA)
- net ESC3_RS_SN: now also RS3.3 (S-), U_IS3.2 (IN-); no longer RS3.4 (F-), U_IS3.4 (VS)
- net ESC3_RS_SP: now also RS3.2 (S+), U_IS3.1 (IN+); no longer RS3.1 (F+), U_IS3.9 (A0)
- net ESC4_CM_OUT: now also CM_ESC4.3 (OUT+), RS4.1 (F+); no longer CM_ESC4.4 (OUT-), RS4.2 (S+)
- net ESC4_FUSED: now also CM_ESC4.1 (IN+); no longer CM_ESC4.2 (IN-)
- net ESC4_RS_OUT: now also J_ESC4.1, RS4.4 (F-), U_IS4.10 (VBUS); no longer J_ESC4.2, RS4.3 (S-), U_IS4.5 (SDA)
- net ESC4_RS_SN: now also RS4.3 (S-), U_IS4.2 (IN-); no longer RS4.4 (F-), U_IS4.4 (VS)
- net ESC4_RS_SP: now also RS4.2 (S+), U_IS4.1 (IN+); no longer RS4.1 (F+), U_IS4.9 (A0)
- net ESC5_CM_OUT: now also CM_ESC5.3 (OUT+), RS5.1 (F+); no longer CM_ESC5.4 (OUT-), RS5.2 (S+)
- net ESC5_FUSED: now also CM_ESC5.1 (IN+); no longer CM_ESC5.2 (IN-)
- net ESC5_RS_OUT: now also J_ESC5.1, RS5.4 (F-), U_IS5.10 (VBUS); no longer J_ESC5.2, RS5.3 (S-), U_IS5.5 (SDA)
- net ESC5_RS_SN: now also RS5.3 (S-), U_IS5.2 (IN-); no longer RS5.4 (F-), U_IS5.4 (VS)
- net ESC5_RS_SP: now also RS5.2 (S+), U_IS5.1 (IN+); no longer RS5.1 (F+), U_IS5.9 (A0)
- net FB5V1_FBK: now also U_BEC_5V_1.5 (FB); no longer U_BEC_5V_1.3 (SS)
- net FB5V1_OUT: now also U_BEC_5V_1.1 (VIN), U_BEC_5V_1.2 (EN); no longer L1.1, U_BEC_5V_1.6 (GND)
- net FB5V2_FBK: now also U_BEC_5V_2.5 (FB); no longer U_BEC_5V_2.3 (SS)
- net FB5V2_OUT: now also U_BEC_5V_2.1 (VIN), U_BEC_5V_2.2 (EN); no longer L2.1, U_BEC_5V_2.6 (GND)
- net NTC_P: now also J_NTC.1, U_CELL.9 (TS1); no longer J_NTC.2, U_CELL.5 (VC4)
- net PDB_ALERT_N: now also J_ALERT.2, U_CELL.16 (ALERT_N); no longer J_ALERT.1
- net PDB_SCL: now also D_I2C.6 (IO2), J_I2C.3, U_CELL.15 (SCL), U_IS1.6 (SCL), U_IS2.6 (SCL), U_IS3.6 (SCL), U_IS4.6 (SCL), U_IS4.9 (A0), U_IS5.6 (SCL), U_IS_MAIN.6 (SCL); no longer J_I2C.2, U_IS1.8 (A1), U_IS2.8 (A1), U_IS3.8 (A1), U_IS4.1 (IN+), U_IS4.8 (A1), U_IS5.8 (A1), U_IS_MAIN.8 (A1)
- net PDB_SDA: now also J_I2C.4, U_CELL.14 (SDA), U_IS1.5 (SDA), U_IS2.5 (SDA), U_IS3.5 (SDA), U_IS3.9 (A0), U_IS4.5 (SDA), U_IS5.5 (SDA), U_IS_MAIN.5 (SDA); no longer D_I2C.4 (VCC), J_I2C.1, U_IS1.10 (VBUS), U_IS2.10 (VBUS), U_IS3.1 (IN+), U_IS3.10 (VBUS), U_IS4.10 (VBUS), U_IS5.10 (VBUS), U_IS_MAIN.10 (VBUS)
- net RS_MAIN_SN: now also RS_MAIN.3 (S-), U_IS_MAIN.2 (IN-); no longer RS_MAIN.4 (F-), U_IS_MAIN.4 (VS)
- net RS_MAIN_SP: now also RS_MAIN.2 (S+), U_IS_MAIN.1 (IN+); no longer RS_MAIN.1 (F+), U_IS_MAIN.9 (A0)
- net SS5V1: now also U_BEC_5V_1.3 (SS), C_SS1.1; no longer U_BEC_5V_1.5 (FB)
- net SS5V2: now also U_BEC_5V_2.3 (SS), C_SS2.1; no longer U_BEC_5V_2.5 (FB)
- net SW5V1: now also L1.1, C_BOOT1.2; no longer L1.2
- net SW5V2: now also L2.1, C_BOOT2.2; no longer L2.2
- net VBAT: now also C1.1, C2.1, C3.1, C_CAP.2, C_DM1.1, C_Y1.1, D1.1 (A), Q_BATT_DSG.3 (D), RS_MAIN.1 (F+), U_CELL.10 (REGSRC), U_CELL.13 (BAT+)
- net VBAT_IN_N: now also CM1.2 (IN-), J_BATT.2; no longer CM1.1 (IN+), J_BATT.1
- net VBAT_IN_P: now also CM1.1 (IN+), J_BATT.1; no longer CM1.2 (IN-), J_BATT.2
- net VC1_R: now also U_CELL.2 (VC1); no longer U_CELL.12 (GND)
- net VC2_R: now also U_CELL.3 (VC2); no longer U_CELL.11 (CAP)
- net VC3_R: now also U_CELL.4 (VC3); no longer U_CELL.10 (REGSRC)
- net VC4_R: now also U_CELL.5 (VC4); no longer U_CELL.9 (TS1)
- net VC5_R: now also U_CELL.6 (VC5); no longer U_CELL.8 (BAL_GND)
- net VDIS: now also FB_5V1.1, FB_5V2.1, F_ESC1.1 (A), F_ESC2.1 (A), F_ESC3.1 (A), F_ESC4.1 (A), F_ESC5.1 (A), RS_MAIN.4 (F-), FB_SERVO.1, R_VSNS.1
- net VDIS_SENSE: now also U_IS_MAIN.10 (VBUS), R_VSNS.2; no longer U_IS_MAIN.5 (SDA)
- net PGND: now reaches J_PGND_BATT.1 (PGND)
- net PGND: now also C1.2, C2.2, C3.2, CM2.4 (OUT-), CM_ESC1.2 (IN-), CM_ESC1.4 (OUT-), CM_ESC2.2 (IN-), CM_ESC2.4 (OUT-), CM_ESC3.2 (IN-), CM_ESC3.4 (OUT-), CM_ESC4.2 (IN-), CM_ESC4.4 (OUT-), CM_ESC5.2 (IN-), CM_ESC5.4 (OUT-), C_5V_OUT.2, C_BEC1_IN.2, C_BEC1_OUT.2, C_BEC2_IN.2, C_BEC2_OUT.2, C_BEC_SV_IN.2, C_BEC_SV_OUT.2, C_DEC1.2, C_DEC2.2, C_DEC3.2, C_DEC4.2, C_DEC5.2, C_DM1.2, C_NTC.2, C_Y2.1, D1.2 (K), J_5V.3, J_5V.4, J_ALERT.1, J_ESC1.2, J_ESC2.2, J_ESC3.2, J_ESC4.2, J_ESC5.2, J_I2C.1, J_NTC.2, J_SHLD_5V.1 (PGND), J_SHLD_ALERT.1 (PGND), J_SHLD_ESC1.1 (PGND), J_SHLD_ESC2.1 (PGND), J_SHLD_ESC3.1 (PGND), J_SHLD_ESC4.1 (PGND), J_SHLD_ESC5.1 (PGND), J_SHLD_I2C.1 (PGND), J_SHLD_NTC.1 (PGND), Q_BATT_DSG.2 (S), R_CHGND.2, R_FB1_2.2, R_FB2_2.2, U_BEC_5V_1.6 (GND), U_BEC_5V_1.9 (PGND), U_BEC_5V_2.6 (GND), U_BEC_5V_2.9 (PGND), U_CELL.12 (GND), U_CELL.8 (BAL_GND), U_IS1.3 (GND), U_IS1.8 (A1), U_IS1.9 (A0), U_IS2.3 (GND), U_IS2.8 (A1), U_IS3.3 (GND), U_IS3.8 (A1), U_IS4.3 (GND), U_IS4.8 (A1), U_IS5.3 (GND), U_IS5.8 (A1), U_IS5.9 (A0), U_IS_MAIN.3 (GND), U_IS_MAIN.9 (A0), C_COMP2_SV.2, C_COMPA1.2, C_COMPA2.2, C_COMPB1.2, C_COMPB2.2, C_COMP_SV.2, C_SS1.2, C_SS2.2, C_SS_SV.2, J_SERVO_5V.1, J_SERVO_5V.2, J_SHLD_SV.1 (PGND), R_FBSV_2.2, U_BEC_SERVO_5V.6 (GND), U_BEC_SERVO_5V.9 (PGND)
- net 6V_SERVO renamed 5V_SERVO
- net 5V_SERVO: now also J_SERVO_5V.3, J_SERVO_5V.4, L4.2, R_FBSV_1.1
- net FB6V_OUT renamed FBSV_OUT
- net FBSV_OUT: now also FB_SERVO.2, U_BEC_SERVO_5V.1 (VIN), U_BEC_SERVO_5V.2 (EN)
- new net BOOT_SV: C_BOOT_SV.1, U_BEC_SERVO_5V.7 (BOOT)
- new net COMPRC5V1: C_COMPA1.1, R_COMP1.2
- new net COMPRC5V2: C_COMPA2.1, R_COMP2.2
- new net COMPRC_SV: C_COMP_SV.1, R_COMP_SV.2
- new net COMP_SV: C_COMP2_SV.1, R_COMP_SV.1, U_BEC_SERVO_5V.4 (COMP)
- new net FBSV_FBK: R_FBSV_1.2, R_FBSV_2.1, U_BEC_SERVO_5V.5 (FB)
- new net SS_SV: C_SS_SV.1, U_BEC_SERVO_5V.3 (SS)
- new net SW_SV: C_BOOT_SV.2, L4.1, U_BEC_SERVO_5V.8 (SW)
- no-connect marks 4 -> 5
Other:
- note added: "=== Section E: 5V Servo BEC (Rev S1 - 6V BEC retired) ==="
- note removed: "=== Section E: 6V Servo BEC ==="
