File: avionics/kicad/Kaylee/kicads/Kaylee.kicad_sch (KiCad schematic)
At the start: 115 parts

Commit message: Fleet trust module (MCU+TPM+isolated CAN-FD+RS-485) across new CAN-PERIPH-GW-1 board, Jayne, Kaylee, Emma; ISOW1412 swap on Wash/Zoë
- New stackable CAN-PERIPH-GW-1 gateway board (N_STACKS param): MSPM0G3507
  + SLB9670 TPM + ISOW1044BDFMR isolated CAN-FD + ISOW1412 isolated RS-485,
  informed by the public VimDrones ap_periph_pico/ESC S50 concept (no
  VimDrones GPL-3.0 source copied). PCB freerouted via the Specctra DSN/SES
  bridge (tools/export-specctra-dsn.py + import-specctra-ses.py +
  freerouting 2.2.4); user's manual footprint packing preserved.
- Jayne: added ISOW1412 isolated RS-485 (Section H); MSPM0G3507 pinmux
  re-verified against the real datasheet for all new assignments.
- Kaylee: full trust module added via non-destructive schematic injection
  (inject_kaylee_trust_module.py) -- gen_kaylee.py itself has drifted from
  the checked-in file and is not safe to regenerate from (tracked as an
  open item).
- Emma: SLB9670 TPM added via a dedicated header (inject_emma_tpm.py); no
  separate CAN/RS-485 needed, reaches the bus via Zoë's P1/P2 link.
- Fleet-wide ADM2795E -> ISOW1412 (integrated isolated DC-DC). While
  swapping Wash/Zoë, fixed their pre-existing broken ADM2795EBRWZ pin
  numbering and wrong ISOW1044BDFMR footprint (SOIC-16W on a 20-pin part).
- REFERENCES.md: REF-SENSOR-009/010/011 (ISOW1044/ISOW1412/SLB9670),
  ADM2795E supersession, Wash/Zoë defect history, vimdrones GPL note.
- WBS/TODO updated across avionics, airframe/wings-nacelles, and root:
  AK7455 nacelle tilt data is now bus-published by the gateway rather than
  read directly by River/Simon.

Co-Authored-By: Claude Sonnet 5 <noreply@anthropic.com>
Parts:
- added C_H_ADM1, C_H_ADM2, C_H_ISO1, C_H_TPM1: 100nF, symbol C_Generic
- added C_H_IN: 10uF, symbol C_Generic
- added C_H_ISO2, C_H_VCORE: 1uF, symbol C_Generic
- added C_H_OUT: 22uF, symbol C_Generic
- added J_CAN_IN_H: CAN-FD trunk IN (CANH/CANL/GND), symbol Conn_JST_GH_03P
- added J_CAN_OUT_H: CAN-FD trunk OUT (CANH/CANL/GND), symbol Conn_JST_GH_03P
- added J_RS485_IN_H: RS-485 trunk IN (A/B/GND), symbol Conn_JST_GH_03P
- added J_RS485_OUT_H: RS-485 trunk OUT (A/B/GND), symbol Conn_JST_GH_03P
- added J_SWD_H: SWD: DIO/CLK/NRST/GND, symbol Conn_JST_GH_04P
- added L_H1: 2.2uH, symbol L_Generic
- added R_H_485TERM, R_H_CANTERM: 120R, symbol R_Generic
- added R_H_FBB: 20k, symbol R_Generic
- added R_H_FBT, R_H_NRST, R_H_TPM_RST: 10k, symbol R_Generic
- added SJ_H_485, SJ_H_CAN: open by default, Jumper:SolderJumper-2_P1.3mm_Open_Pad1.0x1.5mm, symbol SJ_Generic
- added U_ISOCAN: TI ISOW1044BDFMR, Package_SO:SOIC-20W_7.5x12.8mm_P1.27mm, symbol Jayne_ISOW1044BDFMR
- added U_MCU: TI MSPM0G3507, Package_DFN_QFN:QFN-48-1EP_7x7mm_P0.5mm_EP5.15x5.15mm, symbol Jayne_MSPM0G3507_RGZ
- added U_REG_3V3_H: TLV62569DBVR -> +3V3, symbol TLV62569_DBV_H
- added U_RS485: TI ISOW1412, Package_SO:SOIC-20W_7.5x12.8mm_P1.27mm, symbol GW_ISOW1412
- added U_TPM: Infineon SLB9670, Package_DFN_QFN:QFN-32-1EP_5x5mm_P0.5mm_EP3.45x3.45mm, symbol Jayne_SLB9670_TPM
Connections:
- net +5V: now also C_H_IN.1, U_REG_3V3_H.1 (EN), U_REG_3V3_H.4 (VIN)
- net PDB_SCL: now also U_MCU.2 (PA1)
- net PDB_SDA: now also U_MCU.1 (PA0)
- net PGND: now also C_H_ADM1.2, C_H_IN.2, C_H_ISO1.2, C_H_OUT.2, C_H_TPM1.2, C_H_VCORE.1, C_H_VCORE.2, J_SWD_H.4, R_H_FBB.2, U_ISOCAN.10 (GND1), U_ISOCAN.4 (STB), U_ISOCAN.6 (GNDIO), U_MCU.45 (PA25), U_MCU.46 (PA26), U_MCU.47 (PA27), U_MCU.48 (VCORE), U_MCU.49 (VSS), U_MCU.7 (VSS), U_REG_3V3_H.2 (GND), U_RS485.10 (GND1), U_RS485.6 (GNDIO), U_TPM.16 (NCI/GND), U_TPM.2 (GND), U_TPM.23 (GND), U_TPM.32 (GND), U_TPM.9 (GND)
- new net: U_MCU.23 (PB9), U_TPM.6 (GPIO)
- new net: U_MCU.24 (PB14), U_TPM.7 (PP)
- new net +3V3: C_H_ADM1.1, C_H_ISO1.1, C_H_OUT.1, C_H_TPM1.1, L_H1.2, R_H_FBT.1, R_H_NRST.1, R_H_TPM_RST.1, U_ISOCAN.1 (VIO), U_ISOCAN.9 (VDD), U_MCU.41 (PB20), U_MCU.42 (PB24), U_MCU.43 (PA23), U_MCU.44 (PA24), U_MCU.6 (VDD), U_RS485.1 (VIO), U_RS485.9 (VDD), U_TPM.1 (NCI/VDD), U_TPM.14 (NCI/VDD), U_TPM.22 (VDD), U_TPM.8 (VDD)
- new net CANFD_FLT_N: U_ISOCAN.8 (EN/FLT), U_MCU.16 (PA8)
- new net CANFD_RX: U_ISOCAN.5 (RXD), U_MCU.28 (PA13)
- new net CANFD_TX: U_ISOCAN.3 (TXD), U_MCU.27 (PA12)
- new net CANTERM_MID_H: R_H_CANTERM.2, SJ_H_CAN.1
- new net CAN_H: J_CAN_IN_H.1, J_CAN_OUT_H.1, R_H_CANTERM.1, U_ISOCAN.19 (CANH)
- new net CAN_L: J_CAN_IN_H.2, J_CAN_OUT_H.2, SJ_H_CAN.2, U_ISOCAN.18 (CANL)
- new net ISO_3V3_485: C_H_ADM2.1, U_RS485.12 (VISOOUT), U_RS485.16 (VISOIN)
- new net ISO_5V_CAN: C_H_ISO2.1, U_ISOCAN.12 (VISOOUT), U_ISOCAN.13 (VSIN), U_ISOCAN.20 (VISOIN), U_TPM.31 (NCI)
- new net ISO_GND_485: C_H_ADM2.2, J_RS485_IN_H.3, J_RS485_OUT_H.3, U_RS485.11 (GND2), U_RS485.13 (MODE), U_RS485.15 (GISOIN)
- new net ISO_GND_CAN: C_H_ISO2.2, J_CAN_IN_H.3, J_CAN_OUT_H.3, U_ISOCAN.11 (GND2), U_ISOCAN.15 (GISOIN), U_ISOCAN.16 (GISOIN), U_ISOCAN.17 (GISOIN)
- new net MCU_NRST: J_SWD_H.3, R_H_NRST.2, U_MCU.4 (NRST)
- new net MCU_SWCLK: J_SWD_H.2, U_MCU.35 (PA20/SWCLK)
- new net MCU_SWDIO: J_SWD_H.1, U_MCU.34 (PA19/SWDIO)
- new net RS485_A: J_RS485_IN_H.1, J_RS485_OUT_H.1, R_H_485TERM.1, U_RS485.17 (Y), U_RS485.20 (A)
- new net RS485_B: J_RS485_IN_H.2, J_RS485_OUT_H.2, SJ_H_485.2, U_RS485.18 (Z), U_RS485.19 (B)
- new net RS485_DE: U_MCU.14 (PB2), U_RS485.3 (DE), U_RS485.5 (RE_N)
- new net RS485_FLT_N: U_MCU.15 (PB3), U_RS485.8 (EN_FLT)
- new net RS485_RX: U_MCU.26 (PB16), U_RS485.4 (R)
- new net RS485_TX: U_MCU.25 (PB15), U_RS485.2 (D)
- new net TERM485_MID_H: R_H_485TERM.2, SJ_H_485.1
- new net TPM_PIRQ: U_MCU.21 (PB7), U_MCU.9 (PA3), U_TPM.18 (PIRQ#)
- new net TPM_RESET_N: R_H_TPM_RST.2, U_MCU.13 (PA7), U_MCU.22 (PB8), U_TPM.17 (RST#)
- new net TPM_SPI_CS: U_MCU.17 (PA9), U_MCU.8 (PA2), U_TPM.20 (CS#)
- new net TPM_SPI_MISO: U_MCU.10 (PA4), U_MCU.20 (PB6), U_TPM.24 (MISO)
- new net TPM_SPI_MOSI: U_MCU.11 (PA5), U_MCU.19 (PA11), U_TPM.21 (MOSI)
- new net TPM_SPI_SCK: U_MCU.12 (PA6), U_MCU.18 (PA10), U_TPM.19 (SCLK)
- new net U_REG_H_FB: R_H_FBB.1, R_H_FBT.2, U_REG_3V3_H.5 (FB)
- new net U_REG_H_SW: L_H1.1, U_REG_3V3_H.3 (SW)
- no-connect marks 5 -> 55
Other:
- note added: "=== Section H: Trust Module (MCU+TPM+isolated CAN-FD+RS-485) ==="
