File: avionics/kicad/Kaylee/kicads/Kaylee.kicad_pcb (KiCad board)
At the start: 4 copper layers, 90 x 65 mm, 67 parts

Commit message: lots of stuff
Parts:
- removed U_BEC_6V: TPS54540DDAR, Package_SO:SOIC-8_3.9x4.9mm_P1.27mm
- added U_BEC_SERVO_5V: TPS54620 sync buck 5.0V servo rail (pkg verify), Package_DFN_QFN:Texas_RGP0020D_VQFN-20-1EP_4x4mm_P0.5mm_EP2.7x2.7mm, F.Cu at (165.5, 116.5)
- RS_1, RS_2, RS_3, RS_4, RS_MAIN, U_IS1, U_IS2, U_IS3, U_IS4, U_IS_MAIN: moved to B.Cu
- moved U_IS1 171.9 mm to (174.9, 94.0), turned to 180 degrees
- moved RS_1 165.5 mm to (166.6, 94.0), turned to 180 degrees
- moved D1 154.5 mm to (152.5, 92.5), turned to 180 degrees
- moved RS_2 140.7 mm to (156.9, 87.0), turned to 180 degrees
- moved RS_MAIN 138.3 mm to (166.4, 87.0), turned to 180 degrees
- moved U_IS_MAIN 137.2 mm to (174.9, 87.5), turned to 180 degrees
- moved U_IS2 136.3 mm to (156.5, 75.0), turned to 180 degrees
- moved F1 135.5 mm to (149.1, 107.5)
- moved J_ALERT 128.5 mm to (187.1, 115.0)
- moved U_IS3 127.8 mm to (156.9, 94.5), turned to 180 degrees
- moved C_Y2 127.5 mm to (137.5, 91.0)
- moved C_Y1 126.7 mm to (129.5, 91.0)
- moved C_BEC2_OUT 126.5 mm to (167.0, 106.5)
- moved C_BEC_SV_IN 126.4 mm to (181.0, 106.5)
- moved C_DM1 125.0 mm to (146.5, 89.5)
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- renumbered FB_6V to FB_SERVO, J_6V to J_SERVO_5V, R_FB6_1 to R_FBSV_1, R_FB6_2 to R_FBSV_2
Connections:
- C_BEC_SV_IN pad 1: BEC6V_VIN_F -> BECSV_VIN_F
- C_BEC_SV_OUT pad 1: +6V -> 5V_SERVO
- FB_SERVO pad 2: BEC6V_VIN_F -> BECSV_VIN_F
- J_SERVO_5V pad 3: +6V -> 5V_SERVO
- J_SERVO_5V pad 4: +6V -> 5V_SERVO
- L_BEC1 pad 1: BEC1_VIN_F -> BEC1_PRE_OR
- L_BEC2 pad 1: BEC2_VIN_F -> BEC2_PRE_OR
- L_BEC3 pad 1: BEC6V_VIN_F -> 5V_SERVO
- L_BEC3 pad 2: BEC6V_SW -> BECSV_SW
- R_FB1_1 pad 2: (no net) -> BEC1_FB
- R_FB1_2 pad 1: (no net) -> BEC1_FB
- R_FB2_1 pad 2: (no net) -> BEC2_FB
- R_FB2_2 pad 1: (no net) -> BEC2_FB
- R_FBSV_1 pad 1: +6V -> 5V_SERVO
- R_FBSV_1 pad 2: (no net) -> BECSV_FB
- R_FBSV_2 pad 1: (no net) -> BECSV_FB
Routing:
- added copper zone on B.Cu, net VBAT
- removed copper zone on In2.Cu, net VBAT

Commit message: fleshed out lots of pcbs
Parts:
- added C_H_ADM1: 100nF, C_0402_1005Metric, F.Cu at (107.3, 98.0)
- added C_H_ADM2: 100nF, C_0402_1005Metric, F.Cu at (107.3, 99.4)
- added C_H_IN: 10uF, C_0402_1005Metric, F.Cu at (102.5, 113.6)
- added C_H_ISO1: 100nF, C_0402_1005Metric, F.Cu at (104.9, 98.0)
- added C_H_ISO2: 1uF, C_0402_1005Metric, F.Cu at (104.9, 99.4)
- added C_H_OUT: 22uF, C_0402_1005Metric, F.Cu at (102.5, 115.0)
- added C_H_TPM1: 100nF, C_0402_1005Metric, F.Cu at (102.5, 117.8)
- added C_H_VCORE: 1uF, C_0402_1005Metric, F.Cu at (102.5, 116.4)
- added J_CAN_IN_H: CAN-FD trunk IN, JST_GH_BM03B-GHS-TBT_1x03-1MP_P1.25mm_Vertical, F.Cu at (230.0, 65.0)
- added J_CAN_OUT_H: CAN-FD trunk OUT, JST_GH_BM03B-GHS-TBT_1x03-1MP_P1.25mm_Vertical, F.Cu at (200.0, 80.0)
- added J_RS485_IN_H: RS-485 trunk IN, JST_GH_BM03B-GHS-TBT_1x03-1MP_P1.25mm_Vertical, F.Cu at (215.0, 80.0)
- added J_RS485_OUT_H: RS-485 trunk OUT, JST_GH_BM03B-GHS-TBT_1x03-1MP_P1.25mm_Vertical, F.Cu at (230.0, 80.0)
- added J_SWD_H: SWD: DIO/CLK/NRST/GND, JST_GH_BM04B-GHS-TBT_1x04-1MP_P1.25mm_Vertical, F.Cu at (215.0, 95.0)
- added L_H1: 2.2uH, L_Taiyo-Yuden_NR-20xx, F.Cu at (107.9, 87.2)
- added R_H_485TERM: 120R, R_0402_1005Metric, F.Cu at (102.5, 112.2)
- added R_H_CANTERM: 120R, R_0402_1005Metric, F.Cu at (102.5, 110.8)
- added R_H_FBB: 20k, R_0402_1005Metric, F.Cu at (102.5, 99.4)
- added R_H_FBT: 10k, R_0402_1005Metric, F.Cu at (102.5, 98.0)
- added R_H_NRST: 10k, R_0402_1005Metric, F.Cu at (102.5, 108.0)
- added R_H_TPM_RST: 10k, R_0402_1005Metric, F.Cu at (102.5, 109.4)
- added SJ_H_485: open by default, SolderJumper-2_P1.3mm_Open_Pad1.0x1.5mm, F.Cu at (126.5, 86.6)
- added SJ_H_CAN: open by default, SolderJumper-2_P1.3mm_Open_Pad1.0x1.5mm, F.Cu at (122.7, 86.6)
- added U_ISOCAN: TI ISOW1044BDFMR, SOIC-20W_7.5x12.8mm_P1.27mm, F.Cu at (200.0, 65.0)
- added U_MCU: TI MSPM0G3507, QFN-48-1EP_7x7mm_P0.5mm_EP5.15x5.15mm, F.Cu at (122.3, 93.6)
- added U_REG_3V3_H: TLV62569DBVR, SOT-23-6, F.Cu at (103.7, 87.2)
- added U_RS485: TI ISOW1412, SOIC-20W_7.5x12.8mm_P1.27mm, F.Cu at (215.0, 65.0)
- added U_TPM: Infineon SLB9670, QFN-32-1EP_5x5mm_P0.5mm_EP3.45x3.45mm, F.Cu at (105.1, 73.0)
- renumbered L_BEC1 to L1, L_BEC2 to L2, L_BEC3 to L4, RS_1 to RS1, RS_2 to RS2, RS_3 to RS3, RS_4 to RS4
Connections:
- net ESC1_SNS_N renamed ESC1_RS_SN
- net ESC1_SNS_P renamed ESC1_RS_SP
- net ESC2_SNS_N renamed ESC2_RS_SN
- net ESC2_SNS_P renamed ESC2_RS_SP
- net ESC3_SNS_N renamed ESC3_RS_SN
- net ESC3_SNS_P renamed ESC3_RS_SP
- net ESC4_SNS_N renamed ESC4_RS_SN
- net ESC4_SNS_P renamed ESC4_RS_SP
- net MAIN_SNS_N renamed RS_MAIN_SN
- net MAIN_SNS_P renamed RS_MAIN_SP
- C1 pad 1: VDIS -> VBAT
- C1 pad 2: PGND -> CM2_OUT_N
- C2 pad 1: VDIS -> VBAT
- C2 pad 2: PGND -> CM2_OUT_N
- C3 pad 1: VDIS -> VBAT
- C3 pad 2: PGND -> CM2_OUT_N
- CM1 pad 1: VDIS -> VBAT_IN_P
- CM1 pad 2: VDIS -> VBAT_IN_N
- CM1 pad 3: PGND -> CM1_OUT_P
- CM1 pad 4: PGND -> CM1_OUT_N
- CM2 pad 1: VDIS -> CM1_OUT_P
- CM2 pad 2: VDIS -> CM1_OUT_N
- CM2 pad 3: PGND -> CM2_OUT_P
- CM2 pad 4: PGND -> CM2_OUT_N
- C_BEC1_IN pad 1: BEC1_VIN_F -> FB5V1_OUT
- C_BEC1_IN pad 2: PGND -> CM2_OUT_N
- C_BEC1_OUT pad 1: BEC1_PRE_OR -> BEC5V1_RAW
- C_BEC1_OUT pad 2: PGND -> CM2_OUT_N
- C_BEC2_IN pad 1: BEC2_VIN_F -> FB5V2_OUT
- C_BEC2_IN pad 2: PGND -> CM2_OUT_N
- C_BEC2_OUT pad 1: BEC2_PRE_OR -> BEC5V2_RAW
- C_BEC2_OUT pad 2: PGND -> CM2_OUT_N
- C_BEC_SV_IN pad 1: BECSV_VIN_F -> FBSV_OUT
- C_BEC_SV_IN pad 2: PGND -> CM2_OUT_N
- C_BEC_SV_OUT pad 2: PGND -> CM2_OUT_N
- C_DM1 pad 1: VDIS -> VBAT
- C_DM1 pad 2: PGND -> CM2_OUT_N
- C_Y1 pad 1: VDIS -> VBAT
- C_Y2 pad 1: PGND -> CM2_OUT_N
- D1 pad 1: PGND -> VBAT
- D1 pad 2: VDIS -> CM2_OUT_N
- D_I2C pad 1: PGND -> CM2_OUT_N
- D_I2C pad 2: PDB_SDA_RAW -> PDB_SDA
- D_I2C pad 4: PDB_SCL -> +5V
- D_I2C pad 6: +5V -> PDB_SCL
- D_OR1 pad 1: BEC1_PRE_OR -> BEC5V1_RAW
- D_OR1 pad 3: BEC2_PRE_OR -> 5V_AVIONICS
- D_OR2 pad 1: BEC2_PRE_OR -> BEC5V2_RAW
- D_OR2 pad 3: BEC2_PRE_OR -> 5V_AVIONICS
- F1 pad 1: VDIS -> CM2_OUT_P
- F1 pad 2: VDIS -> VBAT
- FB_5V1 pad 2: BEC1_VIN_F -> FB5V1_OUT
- FB_5V2 pad 2: BEC2_VIN_F -> FB5V2_OUT
- FB_SERVO pad 2: BECSV_VIN_F -> FBSV_OUT
- F_ESC1 pad 1: VBAT -> VDIS
- F_ESC2 pad 1: VBAT -> VDIS
- F_ESC3 pad 1: VBAT -> VDIS
- F_ESC4 pad 1: VBAT -> VDIS
- J_5V pad 1: PGND -> 5V_AVIONICS
- J_5V pad 2: PGND -> 5V_AVIONICS
- J_5V pad 3: +5V -> CM2_OUT_N
- J_5V pad 4: +5V -> CM2_OUT_N
- J_ALERT pad 1: PGND -> CM2_OUT_N
- J_BATT pad 1: VDIS -> VBAT_IN_P
- J_BATT pad 2: PGND -> VBAT_IN_N
- J_ESC1 pad 2: PGND -> CM2_OUT_N
- J_ESC2 pad 2: PGND -> CM2_OUT_N
- J_ESC3 pad 2: PGND -> CM2_OUT_N
- J_ESC4 pad 2: PGND -> CM2_OUT_N
- J_I2C pad 1: PGND -> CM2_OUT_N
- J_SERVO_5V pad 1: PGND -> CM2_OUT_N
- J_SERVO_5V pad 2: PGND -> CM2_OUT_N
- L1 pad 1: BEC1_PRE_OR -> SW5V1
- L1 pad 2: BEC1_SW -> BEC5V1_RAW
- L2 pad 1: BEC2_PRE_OR -> SW5V2
- L2 pad 2: BEC2_SW -> BEC5V2_RAW
- L4 pad 1: 5V_SERVO -> SW_SV
- L4 pad 2: BECSV_SW -> 5V_SERVO
- Q_BATT_DSG pad 1: VBAT -> DSG_GATE
- Q_BATT_DSG pad 2: VBAT -> CM2_OUT_N
- RS1 pad 1: ESC1_FUSED -> ESC1_CM_OUT
- RS2 pad 1: ESC2_FUSED -> ESC2_CM_OUT
- RS3 pad 1: ESC3_FUSED -> ESC3_CM_OUT
- RS4 pad 1: ESC4_FUSED -> ESC4_CM_OUT
- RS_MAIN pad 4: VBAT -> VDIS
- R_CHGND pad 1: PGND -> CHASSIS
- R_CHGND pad 2: CHASSIS -> CM2_OUT_N
- R_DSG_G pad 1: DSG_GATE -> BQ_DSG_OUT
- R_DSG_G pad 2: PGND -> DSG_GATE
- R_FB1_1 pad 1: BEC1_PRE_OR -> BEC5V1_RAW
- R_FB1_1 pad 2: BEC1_FB -> FB5V1_FBK
- R_FB1_2 pad 1: BEC1_FB -> FB5V1_FBK
- R_FB1_2 pad 2: PGND -> CM2_OUT_N
- R_FB2_1 pad 1: BEC2_PRE_OR -> BEC5V2_RAW
- R_FB2_1 pad 2: BEC2_FB -> FB5V2_FBK
- R_FB2_2 pad 1: BEC2_FB -> FB5V2_FBK
- R_FB2_2 pad 2: PGND -> CM2_OUT_N
- R_FBSV_1 pad 2: BECSV_FB -> FBSV_FBK
- R_FBSV_2 pad 1: BECSV_FB -> FBSV_FBK
- R_FBSV_2 pad 2: PGND -> CM2_OUT_N
- U_BEC_5V_1 pad 1: BEC1_VIN_F -> FB5V1_OUT
- U_BEC_5V_1 pad 2: (no net) -> FB5V1_OUT
- U_BEC_5V_1 pad 3: (no net) -> SS5V1
- U_BEC_5V_1 pad 4: (no net) -> COMP5V1
- U_BEC_5V_1 pad 5: BEC1_SW -> FB5V1_FBK
- U_BEC_5V_1 pad 6: BEC1_SW -> CM2_OUT_N
- U_BEC_5V_1 pad 7: PGND -> BOOT5V1
- U_BEC_5V_1 pad 8: PGND -> SW5V1
- U_BEC_5V_1 pad 9: PGND -> CM2_OUT_N
- U_BEC_5V_2 pad 1: BEC2_VIN_F -> FB5V2_OUT
- U_BEC_5V_2 pad 2: (no net) -> FB5V2_OUT
- U_BEC_5V_2 pad 3: (no net) -> SS5V2
- U_BEC_5V_2 pad 4: (no net) -> COMP5V2
- U_BEC_5V_2 pad 5: BEC2_SW -> FB5V2_FBK
- U_BEC_5V_2 pad 6: BEC2_SW -> CM2_OUT_N
- U_BEC_5V_2 pad 7: PGND -> BOOT5V2
- U_BEC_5V_2 pad 8: PGND -> SW5V2
- U_BEC_5V_2 pad 9: PGND -> CM2_OUT_N
- U_BEC_SERVO_5V pad 1: BECSV_VIN_F -> FBSV_OUT
- U_BEC_SERVO_5V pad 2: (no net) -> FBSV_OUT
- U_BEC_SERVO_5V pad 3: (no net) -> SS_SV
- U_BEC_SERVO_5V pad 4: (no net) -> COMP_SV
- U_BEC_SERVO_5V pad 5: BECSV_SW -> FBSV_FBK
- U_BEC_SERVO_5V pad 6: BECSV_SW -> CM2_OUT_N
- U_BEC_SERVO_5V pad 7: PGND -> BOOT_SV
- U_BEC_SERVO_5V pad 8: PGND -> SW_SV
- U_BEC_SERVO_5V pad 9: PGND -> CM2_OUT_N
- U_IS1 pad 10: ESC1_FUSED -> ESC1_RS_OUT
- U_IS1 pad 3: PGND -> CM2_OUT_N
- U_IS1 pad 8: (no net) -> CM2_OUT_N
- U_IS1 pad 9: (no net) -> CM2_OUT_N
- U_IS2 pad 10: ESC2_FUSED -> ESC2_RS_OUT
- U_IS2 pad 3: PGND -> CM2_OUT_N
- U_IS2 pad 8: (no net) -> CM2_OUT_N
- U_IS2 pad 9: (no net) -> +5V
- U_IS3 pad 10: ESC3_FUSED -> ESC3_RS_OUT
- U_IS3 pad 3: PGND -> CM2_OUT_N
- U_IS3 pad 8: (no net) -> CM2_OUT_N
- U_IS3 pad 9: (no net) -> PDB_SDA
- U_IS4 pad 10: ESC4_FUSED -> ESC4_RS_OUT
- U_IS4 pad 3: PGND -> CM2_OUT_N
- U_IS4 pad 8: (no net) -> CM2_OUT_N
- U_IS4 pad 9: (no net) -> PDB_SCL
- U_IS_MAIN pad 10: VBAT -> VDIS_SENSE
- U_IS_MAIN pad 3: PGND -> CM2_OUT_N
- U_IS_MAIN pad 8: (no net) -> +5V
- U_IS_MAIN pad 9: (no net) -> CM2_OUT_N

Commit message: wash kaylee and firmware
Parts:
- J_CAN_IN_H, J_CAN_OUT_H, J_RS485_IN_H, J_RS485_OUT_H, J_SWD_H, U_ISOCAN, U_RS485: moved to B.Cu
- moved J_RS485_OUT_H 125.0 mm to (109.2, 112.1), turned to 180 degrees
- moved J_CAN_IN_H 110.8 mm to (129.7, 112.1), turned to 180 degrees
- moved J_RS485_IN_H 101.4 mm to (118.8, 112.0), turned to 180 degrees
- moved J_CAN_OUT_H 68.3 mm to (139.7, 112.1), turned to 180 degrees
- moved J_SWD_H 65.4 mm to (152.0, 112.5), turned to 180 degrees
- moved U_RS485 58.7 mm to (181.7, 113.3), turned to -90 degrees
- moved U_ISOCAN 58.2 mm to (167.0, 113.0), turned to -90 degrees

Commit message: wash is done, but got a reaver segfault through the chest.  kaylee's taken on more than she could handle.... and we have upgraded firmware.
Parts:
- removed FB_5V1, FB_5V2, FB_SERVO: WE-742792612, Capacitor_SMD:C_0805_2012Metric
- removed the U_BEC_SERVO_5V at (165.5, 116.5)
- added C_BIAS1: 2.2uF ceramic (BIAS to GND), C_0402_1005Metric, B.Cu at (176.5, 74.0)
- added C_BIAS2: 2.2uF ceramic (BIAS to GND), C_0402_1005Metric, B.Cu at (174.5, 74.0)
- added C_BIASSV: 2.2uF ceramic (BIAS to GND), C_0402_1005Metric, B.Cu at (172.5, 74.0)
- added C_BIAS_RCS: 2.2uF ceramic (BIAS to GND), C_0402_1005Metric, B.Cu at (172.5, 94.5)
- added C_BOOT1: 0.1uF X7R (BST-LX), C_0402_1005Metric, B.Cu at (176.5, 72.0)
- added C_BOOT2: 0.1uF X7R (BST-LX), C_0402_1005Metric, B.Cu at (174.5, 72.0)
- added C_BOOT_RCS: 0.1uF X7R (BST-LX), C_0402_1005Metric, B.Cu at (172.5, 70.5)
- added C_BOOT_SV: 0.1uF X7R (BST-LX), C_0402_1005Metric, B.Cu at (172.5, 72.0)
- added C_FF1: 50pF NP0 (feedforward), C_0402_1005Metric, B.Cu at (176.5, 76.0)
- added C_FF2: 50pF NP0 (feedforward), C_0402_1005Metric, B.Cu at (174.5, 76.0)
- added C_FFRCS: 82pF NP0 (feedforward), C_0402_1005Metric, B.Cu at (143.0, 96.0)
- added C_FFSV: 78pF NP0 (feedforward), C_0402_1005Metric, B.Cu at (172.5, 76.0)
- added C_N_BOOT: 0.47uF >=6.3V (BOOT-SW), C_0402_1005Metric, B.Cu at (143.0, 93.5)
- added C_N_IN: 0.1uF+4.7uF ceramic (PVIN bypass), CP_Radial_D10.0mm_P5.00mm, F.Cu at (150.5, 89.1)
- added C_N_OUT: 90uF eff, >=16V rated, CP_Radial_D10.0mm_P5.00mm, F.Cu at (129.5, 90.1)
- added C_N_VCC: 2.2uF ceramic (VCC to GND), C_0402_1005Metric, B.Cu at (140.0, 95.5)
- added C_RCS_IN: 0.1uF+4.7uF ceramic (SUP bypass), CP_Radial_D10.0mm_P5.00mm, F.Cu at (140.0, 90.6)
- added C_RCS_OUT: 88uF eff, CP_Radial_D10.0mm_P5.00mm, F.Cu at (170.6, 80.5)
- added J_NACELLE_12V: Molex Nano-Fit 4P 2.5mm NACELLE-12V bus (3x STS3215-C018), Molex_Nano-Fit_105309-xx04_1x04_P2.50mm_Vertical, B.Cu at (191.4, 89.8)
- added J_RCS_6V: Molex Nano-Fit 4P 2.5mm RCS-6V bus (4x RCS valve servos, fl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, Molex_Nano-Fit_105309-xx04_1x04_P2.50mm_Vertical, B.Cu at (192.0, 102.5)
- added J_WINCH_6V: Molex Nano-Fit 4P 2.5mm WINCH-6V (STS3215-C001), Molex_Nano-Fit_105309-xx04_1x04_P2.50mm_Vertical, B.Cu at (191.4, 77.2)
- added L_N: 6.8uH >=5A Isat, L_1210_3225Metric, B.Cu at (166.9, 77.0)
- added L_RCS: 2.2uH >=8A Isat, L_1210_3225Metric, B.Cu at (163.9, 72.5)
- added R_FBRCS_1: 64.9k 1% (top), R_0402_1005Metric, B.Cu at (172.0, 78.0)
- added R_FBRCS_2: 10.0k 1% (bottom), R_0402_1005Metric, B.Cu at (175.0, 78.0)
- added R_FB_N1: 100k 1% (top), R_0402_1005Metric, B.Cu at (140.0, 93.5)
- added R_FB_N2: 9.09k 1% (bottom), R_0402_1005Metric, B.Cu at (136.0, 93.5)
- added U_BEC_NACELLE_12V: LM76005 60V/5A sync buck (TI), Texas_RNP0030B_WQFN-30-1EP_4x6mm_P0.5mm_EP1.8x4.5mm, B.Cu at (162.5, 100.5)
- added U_BEC_RCS_6V: MAX42408AFOA 36V/8A sync buck (ADI), MAX42408AFOA_FC2QFN17_3.5x3.75mm, B.Cu at (175.2, 89.5)
- added U_BEC_SERVO_5V: MAX42408AFOA 36V/8A sync buck (ADI), MAX42408AFOA_FC2QFN17_3.5x3.75mm, B.Cu at (135.8, 101.0)
- D_I2C, J_5V, J_I2C, J_SERVO_5V, L4, Q_BATT_DSG, R_ALERT, R_CHGND, R_DSG_G, R_FB2_1, R_FB2_2, SJ_H_485, SJ_H_CAN, U_MCU: moved to B.Cu
- U_BEC_5V_1, U_BEC_5V_2: value TPS54620RGYT -> MAX42408AFOA 36V/8A sync buck (ADI); footprint Package_DFN_QFN:Texas_RGP0020D_VQFN-20-1EP_4x4mm_P0.5mm_EP2.7x2.7mm -> MAX42408AFOA_FC2QFN17_3.5x3.75mm; moved to B.Cu
- moved R_H_FBT 86.0 mm to (188.5, 95.5), turned to 90 degrees
- moved R_H_FBB 86.0 mm to (188.5, 97.5), turned to 90 degrees
- moved C_H_ISO2 84.0 mm to (188.5, 91.5), turned to 90 degrees
- moved C_H_ISO1 83.7 mm to (188.5, 93.5), turned to 90 degrees
- moved C_H_ADM2 82.5 mm to (189.0, 88.0), turned to 180 degrees
- moved C_H_ADM1 82.1 mm to (189.0, 89.5), turned to 180 degrees
- moved U_MCU 59.8 mm to (182.1, 93.9), turned to 180 degrees
- moved C_BEC2_OUT 55.1 mm to (114.0, 91.5)
- moved RS1 44.8 mm to (121.9, 95.0)
- moved L2 39.6 mm to (158.5, 103.5)
- moved C_Y2 37.0 mm to (169.0, 110.5)
- moved C_Y1 36.8 mm to (104.0, 117.5), turned to 90 degrees
- moved R_FB1_2 36.7 mm to (166.0, 108.5)
- moved R_FB1_1 36.0 mm to (166.0, 106.5)
- moved R_FB2_1 35.2 mm to (152.0, 100.5)
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Connections:
- net 5V_SERVO renamed SERVO_6V
- net FBSV_FBK renamed BECSV_FB
- C_BEC1_IN pad 1: FB5V1_OUT -> VDIS
- C_BEC2_IN pad 1: FB5V2_OUT -> VDIS
- C_BEC_SV_IN pad 1: FBSV_OUT -> VDIS
- L1 pad 1: SW5V1 -> U_BEC_5V_1_LX
- L2 pad 1: SW5V2 -> U_BEC_5V_2_LX
- L4 pad 1: SW_SV -> U_BEC_SERVO_5V_LX
- R_FB1_1 pad 2: FB5V1_FBK -> BEC1_FB
- R_FB1_2 pad 1: FB5V1_FBK -> BEC1_FB
- R_FB2_1 pad 2: FB5V2_FBK -> BEC2_FB
- R_FB2_2 pad 1: FB5V2_FBK -> BEC2_FB
- U_BEC_5V_1 pad 1: FB5V1_OUT -> VDIS
- U_BEC_5V_1 pad 10: PGND -> CM2_OUT_N
- U_BEC_5V_1 pad 11: BEC1_PRE_OR -> U_BEC_5V_1_BIAS
- U_BEC_5V_1 pad 12: (no net) -> BEC1_FB
- U_BEC_5V_1 pad 13: (no net) -> BEC5V1_RAW
- U_BEC_5V_1 pad 15: BEC1_VIN_F -> (no net)
- U_BEC_5V_1 pad 16: BEC1_VIN_F -> CM2_OUT_N
- U_BEC_5V_1 pad 17: BEC1_VIN_F -> (no net)
- U_BEC_5V_1 pad 2: FB5V1_OUT -> U_BEC_5V_1_BST
- U_BEC_5V_1 pad 3: SS5V1 -> VDIS
- U_BEC_5V_1 pad 4: COMP5V1 -> CM2_OUT_N
- U_BEC_5V_1 pad 5: FB5V1_FBK -> CM2_OUT_N
- U_BEC_5V_1 pad 6: CM2_OUT_N -> U_BEC_5V_1_LX
- U_BEC_5V_1 pad 7: BOOT5V1 -> CM2_OUT_N
- U_BEC_5V_1 pad 8: SW5V1 -> CM2_OUT_N
- U_BEC_5V_1 pad 9: CM2_OUT_N -> VDIS
- U_BEC_5V_2 pad 1: FB5V2_OUT -> VDIS
- U_BEC_5V_2 pad 10: PGND -> CM2_OUT_N
- U_BEC_5V_2 pad 11: BEC2_PRE_OR -> U_BEC_5V_2_BIAS
- U_BEC_5V_2 pad 12: (no net) -> BEC2_FB
- U_BEC_5V_2 pad 13: (no net) -> BEC5V2_RAW
- U_BEC_5V_2 pad 15: BEC2_VIN_F -> (no net)
- U_BEC_5V_2 pad 16: BEC2_VIN_F -> CM2_OUT_N
- U_BEC_5V_2 pad 17: BEC2_VIN_F -> (no net)
- U_BEC_5V_2 pad 2: FB5V2_OUT -> U_BEC_5V_2_BST
- U_BEC_5V_2 pad 3: SS5V2 -> VDIS
- U_BEC_5V_2 pad 4: COMP5V2 -> CM2_OUT_N
- U_BEC_5V_2 pad 5: FB5V2_FBK -> CM2_OUT_N
- U_BEC_5V_2 pad 6: CM2_OUT_N -> U_BEC_5V_2_LX
- U_BEC_5V_2 pad 7: BOOT5V2 -> CM2_OUT_N
- U_BEC_5V_2 pad 8: SW5V2 -> CM2_OUT_N
- U_BEC_5V_2 pad 9: CM2_OUT_N -> VDIS
Other:
- board size 90 x 65 mm -> 94.4 x 65 mm
- board text added: "Kaylee -- EMI-Hardened Power Distribution Board CC BY 4.0 -- July 2026 Steve Griffing, PE(CSE), CISSP-ISSEP, CPP Griffing Technology LLC github.com/Stab-Rabbit-Coding"
