File: avionics/kicad/Wash/kicads/Wash.kicad_pcb (KiCad board)
At the start: 4 copper layers, 55 x 35 mm, 46 parts, among them X2Y-CAN 4.7nF X2Y, X2Y-RS485 4.7nF X2Y

Commit message: lots of stuff
Parts:
- BARO, CMC-RS485, T-ETH, U-GPIO: moved to B.Cu
- moved C-GPIO 33.0 mm to (168.6, 115.5)
- moved U-GPIO 30.5 mm to (154.0, 97.9), turned to 180 degrees
- moved ESC-PWM 24.1 mm to (132.0, 104.0), turned to 90 degrees
- moved CMC-RS485 9.49 mm to (134.5, 94.5)
- moved X2Y-RS485 8.92 mm to (138.0, 98.2), turned to 90 degrees
- moved T-ETH 7.57 mm to (126.0, 105.5), turned to 180 degrees
- moved BARO 6.21 mm to (144.7, 94.8), turned to 180 degrees
- moved ETH1-PHY 6.01 mm to (126.5, 97.8)
- moved CMC-CAN 5.37 mm to (139.0, 95.0)
- moved TVS-CAN 3.36 mm to (130.0, 94.5)
- moved T-ETH2 3.20 mm to (126.0, 111.5), turned to 180 degrees
- moved X2Y-CAN 3.04 mm to (129.3, 97.5)
- moved TVS-RS485 1.64 mm to (136.5, 103.5), turned to -90 degrees
- moved CAN-TR 1.00 mm to (146.0, 102.5)
- moved GPIO-A 0.50 mm to (144.2, 95.0)
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Connections:
- CAN-TR pad 10: CAN_L -> GND
- CAN-TR pad 11: (no net) -> GND2_CAN
- CAN-TR pad 12: (no net) -> VCC2_CAN
- CAN-TR pad 13: (no net) -> VCC2_CAN
- CAN-TR pad 15: (no net) -> GND2_CAN
- CAN-TR pad 16: (no net) -> GND2_CAN
- CAN-TR pad 2: MCAN0_TX -> (no net)
- CAN-TR pad 3: CAN_STB -> MCAN0_TX
- CAN-TR pad 4: MCAN0_RX -> CAN_STB
- CAN-TR pad 5: (no net) -> MCAN0_RX
- CAN-TR pad 6: (no net) -> GND
- CAN-TR pad 8: GND -> (no net)
- CAN-TR pad 9: (no net) -> +3V3
- ETH1-PHY pad 1: ETH_TXP -> RMII0_TXD1
- ETH1-PHY pad 10: GND -> REXT_ETH1-PHY
- ETH1-PHY pad 11: GND -> +3V3
- ETH1-PHY pad 12: GND -> ETH_TXP
- ETH1-PHY pad 13: (no net) -> ETH_TXN
- ETH1-PHY pad 14: (no net) -> ETH_RXP
- ETH1-PHY pad 15: (no net) -> ETH_RXN
- ETH1-PHY pad 18: MDIO0 -> (no net)
- ETH1-PHY pad 19: MDC0 -> (no net)
- ETH1-PHY pad 2: ETH_TXN -> (no net)
- ETH1-PHY pad 20: PHY1_INTRN -> +3V3
- ETH1-PHY pad 21: GND2_ETH -> ETH1-PHY_CFG0
- ETH1-PHY pad 22: GND2_ETH -> PHY1_INTRN
- ETH1-PHY pad 23: (no net) -> MDC
- ETH1-PHY pad 24: (no net) -> MDIO
- ETH1-PHY pad 25: GND2_ETH -> +3V3
- ETH1-PHY pad 26: RMII0_TX_EN -> ETH1-PHY_CFG1
- ETH1-PHY pad 27: RMII0_TXD1 -> RMII0_RX_ER
- ETH1-PHY pad 28: RMII0_TXD0 -> DVDD_0P9_ETH1-PHY
- ETH1-PHY pad 29: RMII0_REF_CLK -> ETH1-PHY_PHYAD3
- ETH1-PHY pad 3: GND -> (no net)
- ETH1-PHY pad 30: RMII0_RXD0 -> ETH1-PHY_PHYAD2
- ETH1-PHY pad 31: RMII0_RXD1 -> +3V3
- ETH1-PHY pad 32: RMII0_CRS_DV -> RMII0_RXD1
- ETH1-PHY pad 33: RMII0_RX_ER -> RMII0_RXD0
- ETH1-PHY pad 34: GND2_ETH -> (no net)
- ETH1-PHY pad 35: PHY1_RSTN -> RMII0_CRS_DV
- ETH1-PHY pad 36: GND2_ETH -> DVDD_0P9_ETH1-PHY
- ETH1-PHY pad 37: (no net) -> RMII0_TX_EN
- ETH1-PHY pad 39: (no net) -> RMII0_TXD0
- ETH1-PHY pad 4: ETH_RXP -> DVDD_0P9_ETH1-PHY
- ETH1-PHY pad 40: VCC2_ETH -> +3V3
- ETH1-PHY pad 41: VCC2_ETH -> GND
- ETH1-PHY pad 49: GND -> (no net)
- ETH1-PHY pad 5: ETH_RXN -> GND
- ETH1-PHY pad 6: GND -> (no net)
- ETH1-PHY pad 7: VCC2_ETH -> PHY1_RSTN
- ETH1-PHY pad 8: VCC2_ETH -> (no net)
- ETH1-PHY pad 9: VCC2_ETH -> RMII0_REF_CLK
- ETH2-PHY pad 1: ETH2_TXP -> RMII1_TXD1
- ETH2-PHY pad 10: GND -> REXT_ETH2-PHY
- ETH2-PHY pad 11: GND -> +3V3
- ETH2-PHY pad 12: GND -> ETH2_TXP
- ETH2-PHY pad 13: (no net) -> ETH2_TXN
- ETH2-PHY pad 14: (no net) -> ETH2_RXP
- ETH2-PHY pad 15: (no net) -> ETH2_RXN
- ETH2-PHY pad 18: MDIO1 -> (no net)
- ETH2-PHY pad 19: MDC1 -> (no net)
- ETH2-PHY pad 2: ETH2_TXN -> (no net)
- ETH2-PHY pad 20: PHY2_INTRN -> +3V3
- ETH2-PHY pad 21: GND2_ETH -> ETH2-PHY_CFG0
- ETH2-PHY pad 22: GND2_ETH -> PHY2_INTRN
- ETH2-PHY pad 23: (no net) -> MDC
- ETH2-PHY pad 24: (no net) -> MDIO
- ETH2-PHY pad 25: GND2_ETH -> +3V3
- ETH2-PHY pad 26: RMII1_TX_EN -> ETH2-PHY_CFG1
- ETH2-PHY pad 27: RMII1_TXD1 -> RMII1_RX_ER
- ETH2-PHY pad 28: RMII1_TXD0 -> DVDD_0P9_ETH2-PHY
- ETH2-PHY pad 29: RMII1_REF_CLK -> ETH2-PHY_PHYAD3
- ETH2-PHY pad 3: GND -> (no net)
- ETH2-PHY pad 30: RMII1_RXD0 -> ETH2-PHY_PHYAD2
- ETH2-PHY pad 31: RMII1_RXD1 -> +3V3
- ETH2-PHY pad 32: RMII1_CRS_DV -> RMII1_RXD1
- ETH2-PHY pad 33: RMII1_RX_ER -> RMII1_RXD0
- ETH2-PHY pad 34: GND2_ETH -> (no net)
- ETH2-PHY pad 35: PHY2_RSTN -> RMII1_CRS_DV
- ETH2-PHY pad 36: GND2_ETH -> DVDD_0P9_ETH2-PHY
- ETH2-PHY pad 37: (no net) -> RMII1_TX_EN
- ETH2-PHY pad 39: (no net) -> RMII1_TXD0
- ETH2-PHY pad 4: ETH2_RXP -> DVDD_0P9_ETH2-PHY
- ETH2-PHY pad 40: VCC2_ETH -> +3V3
- ETH2-PHY pad 41: VCC2_ETH -> GND
- ETH2-PHY pad 49: GND -> (no net)
- ETH2-PHY pad 5: ETH2_RXN -> GND
- ETH2-PHY pad 6: GND -> (no net)
- ETH2-PHY pad 7: VCC2_ETH -> PHY2_RSTN
- ETH2-PHY pad 8: VCC2_ETH -> (no net)
- ETH2-PHY pad 9: VCC2_ETH -> RMII1_REF_CLK
- GPS pad 1: (no net) -> GND
- RS485 pad 10: (no net) -> GND2_RS485
- RS485 pad 11: (no net) -> RS485_A
- RS485 pad 12: (no net) -> GND2_RS485
- RS485 pad 13: (no net) -> VCC2_RS485
- RS485 pad 14: (no net) -> RS485_B
- RS485 pad 15: RS485_B -> GND2_RS485
- RS485 pad 16: (no net) -> VCC2_RS485
- RS485 pad 7: GND -> (no net)
- RS485 pad 9: (no net) -> GND2_RS485
- T-ETH pad 2: ETH_TXN -> ETH_CTD
- T-ETH pad 3: ETH_RXP -> ETH_TXN
- T-ETH pad 4: ETH_RXN -> (no net)
- T-ETH pad 5: ETH_LINE_TXP -> (no net)
- T-ETH pad 6: ETH_LINE_TXN -> ETH_RXP
- T-ETH pad 7: ETH_LINE_RXP -> ETH_CRD
- T-ETH pad 8: ETH_LINE_RXN -> ETH_RXN
- T-ETH2 pad 2: ETH2_TXN -> ETH2_CTD
- T-ETH2 pad 3: ETH2_RXP -> ETH2_TXN
- T-ETH2 pad 4: ETH2_RXN -> (no net)
- T-ETH2 pad 5: ETH2_LINE_TXP -> (no net)
- T-ETH2 pad 6: ETH2_LINE_TXN -> ETH2_RXP
- T-ETH2 pad 7: ETH2_LINE_RXP -> ETH2_CRD
- T-ETH2 pad 8: ETH2_LINE_RXN -> ETH2_RXN
- TPM pad 1: TPM_RSTN -> (no net)
- TPM pad 17: (no net) -> TPM_RSTN
- TPM pad 18: (no net) -> TPM_IRQN
- TPM pad 19: (no net) -> SPI0_CLK
- TPM pad 2: (no net) -> GND
- TPM pad 20: (no net) -> SPI0_CS_TPM
- TPM pad 22: SPI0_MISO -> +3V3
- TPM pad 23: SPI0_CLK -> GND
- TPM pad 24: TPM_IRQN -> SPI0_MISO
- TPM pad 28: SPI0_CS_TPM -> (no net)
- TPM pad 32: (no net) -> GND
- TPM pad 33: (no net) -> GND
- TPM pad 8: (no net) -> +3V3
- TPM pad 9: (no net) -> GND
Routing:
- net TMESH_P: track 2229.0 -> 0.00 mm, vias 2 -> 0
- net TMESH_N: track 2204.5 -> 0.00 mm, vias 2 -> 0
