File: avionics/kicad/Wash/kicads/Wash.kicad_pcb (KiCad board)
At the start: 4 copper layers, 55 x 35 mm, 46 parts, among them X2Y-CAN 4.7nF X2Y, X2Y-RS485 4.7nF X2Y

Commit message: Wash: complete schematic-first rebuild (ERC 0, 40/40 parts) + fix 5 latent board defects
Wash.kicad_sch was structurally corrupt and KiCad was SILENTLY TRUNCATING it at
line 1504: a stray ')))' closed the top-level form early, so ~60% of the design
sat outside the parsed document and was invisible to every ERC run ever done on
it. This is the real cause of the long-standing "PB2-P2 header appears fully
unwired" issue in Wash.md — the header was never mis-wired, it was never read.
The true ERC baseline was 275 errors, not the 48 previously recorded.

Also fixed in that file before it was superseded: a corrupted global_label
(extra paren + orphaned fragment of a deleted label), '( comment N "..." )' at
top level (only legal inside title_block), '(shape power_in)' on 4 global labels
(not a valid label shape), and C_SMD/R referenced but absent from lib_symbols —
the last of which makes kicad-cli 9.0.2 SEGFAULT (exit 139) rather than error.

Verification then showed schematic and PCB were different design generations
(only 11 of 60 refs matched, with different naming conventions). Per the
schematic-first decision in WBS.md 1.2a, gen_wash_sch.py now authors all 40 board
footprints from datasheet-transcribed pinouts at ERC = 0 errors, and is promoted
to Wash.kicad_sch; the superseded hand-authored file is archived.

Five latent electrical defects found and corrected, each verified against the OEM
datasheet in avionics/datasheets/ — the board could not have worked as netted:

  * SRF2012 common-mode chokes SHORTED the differential pair. Datasheet windings
    are 1-2 and 4-3, but the board had CAN_H on pads 1 AND 3 with CAN_L on 2 AND
    4, placing a winding straight across the pair (identically on RS-485).
  * FB1 ferrite bead had +5V on both pads — shorted out. Now PWR-IN -> +5V_IN ->
    FB1 -> +5V per Wash.md section 6.
  * RS-485 bus pins Y/Z/B/A carried no net at all, with signals sitting on
    GNDIO/VDD/GND2. Retargeted ADM2795E (16-pin) -> ISOW1412 (20-pin), which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
Parts:
- removed U-ISO-RX, U-ISO-TX: ISO7642FDWRR, SOIC-16W_7.5x10.3mm_P1.27mm
Connections:
- 1553-DRV pad 1: (no net) -> PRU_1553_TX_P
- 1553-DRV pad 10: PRU_1553_TX_P -> (no net)
- 1553-DRV pad 12: (no net) -> GND
- 1553-DRV pad 15: (no net) -> GND
- 1553-DRV pad 16: M1553_TX_N -> +3V3
- 1553-DRV pad 2: (no net) -> M1553_P
- 1553-DRV pad 4: (no net) -> M1553_TX_EN
- 1553-DRV pad 6: PRU_1553_TX_N -> M1553_N
- 1553-DRV pad 7: (no net) -> PRU_1553_TX_N
- 1553-DRV pad 8: (no net) -> GND
- 1553-DRV pad 9: (no net) -> GND
- 1553-RCV pad 1: (no net) -> M1553_N
- 1553-RCV pad 12: M1553_RX_N -> GND
- 1553-RCV pad 13: PRU_1553_RX_N -> (no net)
- 1553-RCV pad 16: (no net) -> +3V3
- 1553-RCV pad 2: (no net) -> M1553_P
- 1553-RCV pad 3: (no net) -> PRU_1553_RX_P
- 1553-RCV pad 4: (no net) -> +3V3
- 1553-RCV pad 5: (no net) -> PRU_1553_RX_N
- 1553-RCV pad 6: (no net) -> M1553_N
- 1553-RCV pad 7: (no net) -> M1553_P
- 1553-RCV pad 8: (no net) -> GND
- 1553-RCV pad 9: M1553_RX_P -> (no net)
- CAN-FD pad 1: GND -> GND2_CAN
- CAN-FD pad 2: CAN_H -> CAN_H_F
- CAN-FD pad 3: CAN_L -> CAN_L_F
- CAN-FD pad 4: +3V3 -> VCC2_CAN
- CMC-CAN pad 2: CAN_L -> CAN_H_F
- CMC-CAN pad 3: CAN_H -> CAN_L_F
- CMC-RS485 pad 2: RS485_B -> RS485_A_F
- CMC-RS485 pad 3: RS485_A -> RS485_B_F
- ESC-PWM pad MP: (no net) -> PGND
- FB1 pad 1: +5V -> +5V_IN
- IMU pad 1: SPI0_MOSI -> SPI0_MISO
- IMU pad 10: (no net) -> GND
- IMU pad 11: (no net) -> GND
- IMU pad 12: (no net) -> SPI0_CS_IMU
- IMU pad 13: (no net) -> SPI0_CLK
- IMU pad 14: IMU_INT2 -> SPI0_MOSI
- IMU pad 2: SPI0_CLK -> GND
- IMU pad 3: SPI0_CS_IMU -> GND
- IMU pad 4: (no net) -> IMU_INT1
- IMU pad 5: SPI0_MISO -> +3V3
- IMU pad 6: (no net) -> GND
- IMU pad 7: (no net) -> GND
- IMU pad 8: (no net) -> +3V3
- IMU pad 9: (no net) -> IMU_INT2
- MIL-1553 pad 1: (no net) -> BUS_1553_P
- MIL-1553 pad 2: (no net) -> BUS_1553_N
- MIL-1553 pad 3: (no net) -> GND
- MIL-1553 pad 4: (no net) -> PGND
- PWR-IN pad 1: +5V -> +5V_IN
- PWR-IN pad 2: +5V -> +5V_IN
- RS-485 pad 1: GND -> GND2_RS485
- RS-485 pad 2: RS485_A -> RS485_A_F
- RS-485 pad 3: RS485_B -> RS485_B_F
- RS-485 pad 4: +3V3 -> VCC2_RS485
- RS485 pad 10: GND2_RS485 -> GND
- RS485 pad 11: RS485_A -> GND2_RS485
- RS485 pad 12: GND2_RS485 -> VCC2_RS485
- RS485 pad 13: VCC2_RS485 -> GND2_RS485
- RS485 pad 14: RS485_B -> (no net)
- RS485 pad 17: (no net) -> RS485_A
- RS485 pad 18: (no net) -> RS485_B
- RS485 pad 19: (no net) -> RS485_B
- RS485 pad 2: GND -> RS485_TX
- RS485 pad 20: (no net) -> RS485_A
- RS485 pad 3: RS485_TX -> RS485_DE
- RS485 pad 4: RS485_DE -> RS485_RX
- RS485 pad 6: RS485_RX -> GND
- RS485 pad 8: GND -> +3V3
- RS485 pad 9: GND2_RS485 -> +3V3
- SERVO-PWM pad 7: (no net) -> +5V
- SERVO-PWM pad 8: (no net) -> GND
- TVS-1553 pad 1: GND -> BUS_1553_P
- TVS-1553 pad 2: (no net) -> PGND
- TVS-CAN pad 1: CAN_H -> CAN_H_F
- TVS-CAN pad 3: CAN_L -> CAN_L_F
- TVS-RS485 pad 1: RS485_A -> RS485_A_F
- TVS-RS485 pad 3: RS485_B -> RS485_B_F
