File: avionics/kicad/Wash/kicads/Wash_rebuild.kicad_sch (KiCad schematic)
At the start: 8 parts

Commit message: fleshed out lots of pcbs
Parts:
- added 1553-DRV: DS26LV31, symbol S_1553-DRV
- added 1553-RCV: DS26LV32AT, symbol S_1553-RCV
- RS485: value ADM2795EBRWZ -> ISOW1412DFMR
Connections:
- net +3V3: now also RS485.8 (EN/FLT), RS485.9 (VDD), 1553-DRV.16 (VCC), 1553-DRV.4 (EN), 1553-RCV.16 (VCC), 1553-RCV.4 (EN)
- net GND: now also RS485.10 (GND1), RS485.6 (GNDIO), 1553-DRV.12 (EN*), 1553-DRV.15 (DI4), 1553-DRV.8 (GND), 1553-DRV.9 (DI3), 1553-RCV.12 (EN*), 1553-RCV.8 (GND); no longer RS485.2 (GND1), RS485.8 (GND1)
- net GND2_RS485: now also RS485.11 (GND2), RS485.13 (MODE); no longer RS485.10 (GND2), RS485.12 (GND2), RS485.9 (GND2)
- net RS485_A: now also RS485.17 (Y), RS485.20 (A); no longer RS485.11 (A)
- net RS485_B: now also RS485.18 (Z), RS485.19 (B); no longer RS485.14 (B)
- net RS485_DE: now also RS485.3 (DE); no longer RS485.4 (DE)
- net RS485_RX: now also RS485.4 (R); no longer RS485.6 (RxD)
- net RS485_TX: now also RS485.2 (D); no longer RS485.3 (TxD)
- net VCC2_RS485: now also RS485.12 (VISOOUT); no longer RS485.13 (VDD2)
- new net M1553_RX_N: 1553-RCV.1 (RI1-), 1553-RCV.6 (RI2+)
- new net M1553_RX_P: 1553-RCV.2 (RI1+), 1553-RCV.7 (RI2-)
- new net M1553_TX_N: 1553-DRV.6 (DO2+)
- new net M1553_TX_P: 1553-DRV.2 (DO1+)
- new net PRU_1553_RX_N: 1553-RCV.5 (RO2)
- new net PRU_1553_RX_P: 1553-RCV.3 (RO1)
- new net PRU_1553_TX_N: 1553-DRV.7 (DI2)
- new net PRU_1553_TX_P: 1553-DRV.1 (DI1)
- no-connect marks 31 -> 44

Commit message: moved the encoder to its own folder
Changed lines of the file:
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@@
   (wire (pts (xy 95.25 538.48) (xy 97.79 538.48)) (stroke (width 0) (type default)))
   (global_label "ETH2_LINE_CT" (shape passive) (at 97.79 538.48 0) (effects (font (size 1.27 1.27)) (justify left)))
+  (symbol (lib_id "PWR_FLAG") (at 76.20 30.48 0) (unit 1)
+    (exclude_from_sim yes) (in_bom no) (on_board no) (dnp no)
+    (property "Reference" "#FLG1" (at 76.20 27.94 0) (effects (font (size 1.27 1.27)) (hide yes)))
+    (property "Value" "PWR_FLAG" (at 76.20 25.40 0) (effects (font (size 1.27 1.27))))
+    (instances (project "Wash_rebuild" (path "/a3000000-0000-0000-0000-000000000001" (reference "#FLG1") (unit 1)))))
+  (wire (pts (xy 76.20 30.48) (xy 76.20 33.02)) (stroke (width 0) (type default)))
+  (global_label "GND" (shape passive) (at 76.20 33.02 270) (effects (font (size 1.27 1.27)) (justify right)))
+  (symbol (lib_id "PWR_FLAG") (at 96.52 30.48 0) (unit 1)
+    (exclude_from_sim yes) (in_bom no) (on_board no) (dnp no)
+    (property "Reference" "#FLG2" (at 96.52 27.94 0) (effects (font (size 1.27 1.27)) (hide yes)))
+    (property "Value" "PWR_FLAG" (at 96.52 25.40 0) (effects (font (size 1.27 1.27))))
+    (instances (project "Wash_rebuild" (path "/a3000000-0000-0000-0000-000000000001" (reference "#FLG2") (unit 1)))))
+  (wire (pts (xy 96.52 30.48) (xy 96.52 33.02)) (stroke (width 0) (type default)))
+  (global_label "+3V3" (shape passive) (at 96.52 33.02 270) (effects (font (size 1.27 1.27)) (justify right)))
   (sheet_instances (path "/" (page "1")))
 )
