File: avionics/kicad/Wash/kicads/Wash.kicad_sch (KiCad schematic)
At the start: 62 parts, among them X2Y_CAN 4.7nF X2Y, X2Y_RS485 4.7nF X2Y

Commit message: Wash: complete schematic-first rebuild (ERC 0, 40/40 parts) + fix 5 latent board defects
Wash.kicad_sch was structurally corrupt and KiCad was SILENTLY TRUNCATING it at
line 1504: a stray ')))' closed the top-level form early, so ~60% of the design
sat outside the parsed document and was invisible to every ERC run ever done on
it. This is the real cause of the long-standing "PB2-P2 header appears fully
unwired" issue in Wash.md — the header was never mis-wired, it was never read.
The true ERC baseline was 275 errors, not the 48 previously recorded.

Also fixed in that file before it was superseded: a corrupted global_label
(extra paren + orphaned fragment of a deleted label), '( comment N "..." )' at
top level (only legal inside title_block), '(shape power_in)' on 4 global labels
(not a valid label shape), and C_SMD/R referenced but absent from lib_symbols —
the last of which makes kicad-cli 9.0.2 SEGFAULT (exit 139) rather than error.

Verification then showed schematic and PCB were different design generations
(only 11 of 60 refs matched, with different naming conventions). Per the
schematic-first decision in WBS.md 1.2a, gen_wash_sch.py now authors all 40 board
footprints from datasheet-transcribed pinouts at ERC = 0 errors, and is promoted
to Wash.kicad_sch; the superseded hand-authored file is archived.

Five latent electrical defects found and corrected, each verified against the OEM
datasheet in avionics/datasheets/ — the board could not have worked as netted:

  * SRF2012 common-mode chokes SHORTED the differential pair. Datasheet windings
    are 1-2 and 4-3, but the board had CAN_H on pads 1 AND 3 with CAN_L on 2 AND
    4, placing a winding straight across the pair (identically on RS-485).
  * FB1 ferrite bead had +5V on both pads — shorted out. Now PWR-IN -> +5V_IN ->
    FB1 -> +5V per Wash.md section 6.
  * RS-485 bus pins Y/Z/B/A carried no net at all, with signals sitting on
    GNDIO/VDD/GND2. Retargeted ADM2795E (16-pin) -> ISOW1412 (20-pin), which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
Parts:
- removed 1553-DRV: DS26LV31, symbol DS26LV31
- removed 1553-RCV: DS26LV32, symbol DS26LV32
- removed 1553-XFM: SM-1553-11, symbol SM-1553-11
- removed BARO: BMP388, symbol BMP388
- removed CAN-TR: ISOW1044BDFMR, Package_SO:SOIC-20W_7.5x12.8mm_P1.27mm, symbol ISOW1044BDFMR
- removed CMC_CAN, CMC_RS485, CM_ETH1, CM_ETH2: SRF2012-100Y, Inductor_SMD:L_Taiyo-Yuden_NR-20xx, symbol SRF2012-100Y
- removed C_ETH1_AVDD1, C_ETH1_IOVDD1, C_ETH2_AVDD1, C_ETH2_IOVDD1: 100nF X5R 0402, Capacitor_SMD:C_0402_1005Metric, symbol C_SMD
- removed C_ETH1_AVDD2, C_ETH2_AVDD2: 10nF X5R 0402, Capacitor_SMD:C_0402_1005Metric, symbol C_SMD
- removed C_ETH1_IOVDD2, C_ETH2_IOVDD2: 10nF 0402, Capacitor_SMD:C_0402_1005Metric, symbol C_SMD
- removed C_ETH1_IOVDD3, C_ETH2_IOVDD3: 1nF 0402, Capacitor_SMD:C_0402_1005Metric, symbol C_SMD
- removed D_1553A, D_1553B: SMAJ33CA, Diode_SMD:D_SMB, symbol SMAJ33CA
- removed D_CAN, D_RS485, D_SBUS_TVS, TVS_ETH1_RX, TVS_ETH1_TX, TVS_ETH2_RX, TVS_ETH2_TX: PRTR5V0U2X, Package_TO_SOT_SMD:SOT-363_SC-70-6, symbol PRTR5V0U2X
- removed FB_PWR: 742792512, Inductor_SMD:L_0805_2012Metric, symbol 742792512
- removed GPS: SAM-M10Q, symbol SAM-M10Q
- removed HX1188_1, HX1188_2: HX1188NL, Package_SO:SOIC-16_3.9x9.9mm_P1.27mm, symbol HX1188NL
- removed IMU: ICM-42688-P, symbol ICM-42688-P
- removed J_1553: SM04B-GHS-TB-1MP — MIL-STD-1553B, Connector_JST:JST_GH_SM04B-GHS-TB_1x04-1MP_P1.25mm_Horizontal, symbol Conn_JST_GH_04P
- removed J_485: SM03B-GHS-TB-1MP — RS-485 Bus, Connector_JST:JST_GH_SM03B-GHS-TB_1x03-1MP_P1.25mm_Horizontal, symbol Conn_JST_GH_03P_SH
- removed J_CAN: SM03B-GHS-TB-1MP — CAN FD Bus, Connector_JST:JST_GH_SM03B-GHS-TB_1x03-1MP_P1.25mm_Horizontal, symbol Conn_JST_GH_03P_SH
- removed J_ESC: SM04B-GHS-TB-1MP — EDF ESC PWM, Connector_JST:JST_GH_SM04B-GHS-TB_1x04-1MP_P1.25mm_Horizontal, symbol Conn_JST_GH_04P
- removed J_ETH1, J_ETH2: SM06B-GHS-TB-1MP, Connector_JST:JST_GH_SM06B-GHS-TB_1x06-1MP_P1.25mm_Horizontal, symbol Conn_JST_GH_06P
- removed J_GPS: SM05B-GHS-TB-1MP — u-blox M10Q GPS, Connector_JST:JST_GH_SM05B-GHS-TB_1x05-1MP_P1.25mm_Horizontal, symbol Conn_JST_GH_05P
- removed J_PWR: SM04B-GHS-TB-1MP — Power Input, Connector_JST:JST_GH_SM04B-GHS-TB_1x04-1MP_P1.25mm_Horizontal, symbol Conn_JST_GH_04P
- removed J_SBUS: Conn_JST_GH_03P, Connector_JST:JST_GH_SM03B-GHS-TB_1x03-1MP_P1.25mm_Horizontal, symbol Conn_JST_GH_03P
- removed J_SERVO: SM06B-GHS-TB-1MP — Nacelle Tilt Servos, Connector_JST:JST_GH_SM06B-GHS-TB_1x06-1MP_P1.25mm_Horizontal, symbol Conn_JST_GH_06P
- removed J_VBAT: Conn_JST_GH_02P, Connector_JST:JST_GH_SM02B-GHS-TB_1x02-1MP_P1.25mm_Horizontal, symbol Conn_JST_GH_02P
- removed PB2-P1: PB2I-P1-2x18, symbol Conn_36
- removed PB2-P2: PB2I-P2-2x18, symbol Conn_36
- removed RS485: ISOW1412, Package_SO:SOIC-20W_7.5x12.8mm_P1.27mm, symbol ISOW1412
- removed R_ETH1_RBIAS, R_ETH2_RBIAS: 49.9R 1% 0402, Resistor_SMD:R_0402_1005Metric, symbol R
- removed R_SBUS: 100R, Resistor_SMD:R_0402_1005Metric, symbol R_SMD
- removed TPM: SLB9670, symbol SLB9670
- removed U_BMON: INA219AIDR, Package_SO:SOIC-8_3.9x4.9mm_P1.27mm, symbol INA219AIDR
- removed U_BMON: INA226AIDGSR, Package_SO:SSOP-8_4.4x3mm_P0.65mm, symbol INA226AIDGSR
- removed U_ETH1_1V8, U_ETH2_1V8: TPS62933, Package_SO:SOIC-8_3.9x4.9mm_P1.27mm, symbol TPS62933
- removed U_ETH1_PHY, U_ETH2_PHY: DP83825I, Package_QFP:LQFP-32_7x7mm_P0.8mm, symbol DP83825I
- removed U_MAG: QMC5883L, Sensor_Magnetic:QMC5883L, symbol QMC5883L
- removed U_MAG: MMC5983MA, Sensor_Magnetic:MMC5983MA, symbol MMC5983MA
- removed U_SBUS: 74LVC1G14GW, Package_TO_SOT_SMD:SOT-23-5, symbol 74LVC1G14
- removed X2Y_CAN, X2Y_RS485: 4.7nF X2Y, Capacitor_SMD:C_0402_1005Metric, symbol X2Y_CAP_4N7
- added 1553-DRV: DS26LV31, symbol S_1553-DRV
- added 1553-RCV: DS26LV32AT, symbol S_1553-RCV
- added 1553-XFM: SM1553-028, symbol S_1553-XFM
- added BARO: BMP388, symbol S_BARO
- added C-GPIO: 100nF 0805, symbol S_C-GPIO
- added CAN-FD: JST SM04B-GHS-TB, symbol S_CAN-FD
- added CAN-TR: ISOW1044BDFMR, symbol S_CAN-TR
- added CMC-CAN: SRF2012-100Y, symbol S_CMC-CAN
- added CMC-RS485: SRF2012-100Y, symbol S_CMC-RS485
- added ESC-PWM: JST SM05B-GHS-TB-1MP, symbol S_ESC-PWM
- added ESC-TLM: JST SM03B-GHS-TB, symbol S_ESC-TLM
- added ETH1: JST SM04B-GHS-TB, symbol S_ETH1
- added ETH1-PHY: ADIN1300BCPZ, symbol S_ETH1-PHY
- added ETH2: JST SM04B-GHS-TB, symbol S_ETH2
- added ETH2-PHY: ADIN1300BCPZ, symbol S_ETH2-PHY
- added FB1: 742792512 600R@100MHz, symbol S_FB1
- added GPIO-A: JST SM03B-GHS-TB, symbol S_GPIO-A
- added GPIO-B: JST SM03B-GHS-TB, symbol S_GPIO-B
- added GPIO-C: JST SM03B-GHS-TB, symbol S_GPIO-C
- added GPIO-D: JST SM03B-GHS-TB, symbol S_GPIO-D
- added GPIO-E: JST SM03B-GHS-TB, symbol S_GPIO-E
- added GPIO-F: JST SM03B-GHS-TB, symbol S_GPIO-F
- added GPS: SAM-M10Q-00B, symbol S_GPS
- added IMU: ICM-42688-P, symbol S_IMU
- added MIL-1553: JST SM04B-GHS-TB, symbol S_MIL-1553
- added PB2-P1: PB2I-P1-2x18, symbol S_PB2-P1
- added PB2-P2: PB2I-P2-2x18, symbol S_PB2-P2
- added PWR-IN: Molex Nano-Fit 4P, symbol S_PWR-IN
- added RS-485: JST SM04B-GHS-TB, symbol S_RS-485
- added RS485: ISOW1412DFMR, symbol S_RS485
- added SERVO-PWM: PinHeader 2.54mm 1x08, symbol S_SERVO-PWM
- added T-ETH: 749010012A, symbol S_T-ETH
- added T-ETH2: 749010012A, symbol S_T-ETH2
- added TPM: SLB9670, symbol S_TPM
- added TVS-1553: SMAJ33CA, symbol S_TVS-1553
- added TVS-CAN: PRTR5V0U2X, symbol S_TVS-CAN
- added TVS-RS485: PRTR5V0U2X, symbol S_TVS-RS485
- added U-GPIO: PCA9555DB, symbol S_U-GPIO
- added X2Y-CAN: X2Y 4.7nF, symbol S_X2Y-CAN
- added X2Y-RS485: X2Y 4.7nF, symbol S_X2Y-RS485
Connections:
- net +3V3: now also 1553-DRV.16 (VCC), 1553-RCV.16 (VCC), 1553-RCV.4 (EN), BARO.1 (VDDIO), BARO.10 (VDD), C-GPIO.1 (P), CAN-TR.1 (VIO), CAN-TR.9 (VDD), ETH1-PHY.11 (AVDD_3P3), ETH1-PHY.20 (AVDD_3P3), ETH1-PHY.25 (VDDIO), ETH1-PHY.31 (VDDIO), ETH1-PHY.40 (VDDIO), ETH2-PHY.11 (AVDD_3P3), ETH2-PHY.20 (AVDD_3P3), ETH2-PHY.25 (VDDIO), ETH2-PHY.31 (VDDIO), ETH2-PHY.40 (VDDIO), GPIO-A.2 (+3V3), GPIO-B.2 (+3V3), GPIO-C.2 (+3V3), GPIO-D.2 (+3V3), GPIO-E.2 (+3V3), GPIO-F.2 (+3V3), GPS.2 (V_IO), GPS.3 (V_BCKP), IMU.5 (VDDIO), IMU.8 (VDD), PB2-P1.33 (P33), PB2-P1.34 (P34), RS485.1 (VIO), RS485.8 (EN/FLT), RS485.9 (VDD), TPM.22 (VDD), TPM.8 (VDD), U-GPIO.24 (VDD)
- net +5V: now also FB1.2 (OUT), PB2-P1.35 (P35), PB2-P2.35 (P35), SERVO-PWM.7 (+5V)
- net +5V_IN: now also FB1.1 (IN), PWR-IN.1 (+5V_IN), PWR-IN.2 (+5V_IN)
- net BARO_INT: now also BARO.7 (INT), PB2-P1.17 (P17)
- net CAN_STB: now also CAN-TR.4 (STB), PB2-P1.14 (P14)
- net DSHOT0: now also ESC-PWM.1 (DSHOT0), PB2-P1.6 (P6)
- net DSHOT1: now also ESC-PWM.2 (DSHOT1), PB2-P1.5 (P5)
- net DSHOT2: now also ESC-PWM.3 (DSHOT2), PB2-P1.4 (P4)
- net DSHOT3: now also ESC-PWM.4 (DSHOT3), PB2-P1.3 (P3)
- net GPS_RESETN: now also PB2-P2.9 (P9)
- net GPS_TIMEPULSE: now also GPS.7 (TIMEPULSE), PB2-P2.10 (P10)
- net IMU_INT1: now also IMU.4 (INT1), PB2-P1.19 (P19)
- net IMU_INT2: now also IMU.9 (INT2/FSYNC), PB2-P1.18 (P18)
- net MCAN0_RX: now also CAN-TR.5 (RXD), PB2-P1.15 (P15)
- net MCAN0_TX: now also CAN-TR.3 (TXD), PB2-P1.16 (P16)
- net MDC0: now also PB2-P2.18 (P18)
- net MDC1: now also PB2-P2.2 (P2)
- net MDIO0: now also PB2-P2.17 (P17)
- net MDIO1: now also PB2-P2.1 (P1)
- net PGND: now also ESC-PWM.MP (SHIELD), MIL-1553.4 (SHIELD), TVS-1553.2 (K)
- net PRU_1553_RX_N: now also 1553-RCV.5 (RO2), PB2-P1.7 (P7)
- net PRU_1553_RX_P: now also 1553-RCV.3 (RO1), PB2-P1.8 (P8)
- net PRU_1553_TX_N: now also 1553-DRV.7 (DI2), PB2-P1.9 (P9)
- net PRU_1553_TX_P: now also 1553-DRV.1 (DI1), PB2-P1.10 (P10)
- net RMII1_RXD0: now also ETH2-PHY.33 (RXD_0), PB2-P2.23 (P23)
- net RMII1_RXD1: now also ETH2-PHY.32 (RXD_1), PB2-P2.22 (P22)
- net RMII1_TXD0: now also ETH2-PHY.39 (TXD_0), PB2-P2.26 (P26)
- net RMII1_TXD1: now also ETH2-PHY.1 (TXD_1), PB2-P2.25 (P25)
- net RS485_A: now also CMC-RS485.1 (W1_IN), RS485.17 (Y), RS485.20 (A)
- net RS485_B: now also CMC-RS485.4 (W2_IN), RS485.18 (Z), RS485.19 (B)
- net RS485_DE: now also PB2-P1.11 (P11), RS485.3 (DE), RS485.5 (RE)
- net RS485_RX: now also PB2-P1.12 (P12), RS485.4 (R)
- net RS485_TX: now also PB2-P1.13 (P13), RS485.2 (D)
- net SERVO0: now also PB2-P2.8 (P8), SERVO-PWM.1 (SERVO0)
- net SERVO1: now also PB2-P2.7 (P7), SERVO-PWM.2 (SERVO1)
- net SERVO2: now also PB2-P2.6 (P6), SERVO-PWM.3 (SERVO2)
- net SERVO3: now also PB2-P2.5 (P5), SERVO-PWM.4 (SERVO3)
- net SERVO4: now also PB2-P2.4 (P4), SERVO-PWM.5 (SERVO4)
- net SERVO5: now also PB2-P2.3 (P3), SERVO-PWM.6 (SERVO5)
- net SPI0_CLK: now also BARO.2 (SCK), IMU.13 (AP_SCLK), PB2-P1.25 (P25), TPM.19 (SCLK)
- net SPI0_CS_1553: now also PB2-P1.20 (P20)
- net SPI0_CS_BARO: now also BARO.6 (CSB), PB2-P1.22 (P22)
- net SPI0_CS_IMU: now also IMU.12 (AP_CS), PB2-P1.26 (P26)
- net SPI0_CS_TPM: now also PB2-P1.21 (P21), TPM.20 (CS#)
- net SPI0_MISO: now also BARO.5 (SDO), IMU.1 (AP_SDO), PB2-P1.23 (P23), TPM.24 (MISO)
- net SPI0_MOSI: now also BARO.4 (SDI), IMU.14 (AP_SDI), PB2-P1.24 (P24), TPM.21 (MOSI)
- net TPM_IRQN: now also PB2-P2.12 (P12), TPM.18 (PIRQ#)
- net TPM_RSTN: now also PB2-P2.11 (P11), TPM.17 (RST#)
- net UART_ESC_RX: now also ESC-TLM.3 (RX), PB2-P1.29 (P29)
- net UART_ESC_TX: now also ESC-TLM.2 (TX), PB2-P1.30 (P30)
- net UART_GPS_RX: now also GPS.14 (RXD), PB2-P1.31 (P31)
- net UART_GPS_TX: now also GPS.13 (TXD), PB2-P1.32 (P32)
- new net BUS_1553_N: 1553-XFM.8 (SEC_5), MIL-1553.2 (BUS_N)
- new net BUS_1553_P: 1553-XFM.4 (SEC_1), MIL-1553.1 (BUS_P), TVS-1553.1 (A)
- new net CAN_H: CAN-TR.19 (CANH), CMC-CAN.1 (W1_IN)
- new net CAN_H_F: CAN-FD.2 (CAN_H), CMC-CAN.2 (W1_OUT), TVS-CAN.1 (IO1)
- new net CAN_L: CAN-TR.18 (CANL), CMC-CAN.4 (W2_IN)
- new net CAN_L_F: CAN-FD.3 (CAN_L), CMC-CAN.3 (W2_OUT), TVS-CAN.3 (IO2)
- new net DVDD_0P9_ETH1-PHY: ETH1-PHY.28 (DVDD_0P9), ETH1-PHY.36 (DVDD_0P9), ETH1-PHY.4 (DVDD_0P9)
- new net DVDD_0P9_ETH2-PHY: ETH2-PHY.28 (DVDD_0P9), ETH2-PHY.36 (DVDD_0P9), ETH2-PHY.4 (DVDD_0P9)
- new net ETH1-PHY_CFG0: ETH1-PHY.21 (LED_0/PHY_CFG0)
- new net ETH1-PHY_CFG1: ETH1-PHY.26 (LINK_ST/PHY_CFG1)
- new net ETH1-PHY_PHYAD2: ETH1-PHY.30 (RXD_2/PHYAD_2)
- new net ETH1-PHY_PHYAD3: ETH1-PHY.29 (RXD_3/PHYAD_3)
- new net ETH2-PHY_CFG0: ETH2-PHY.21 (LED_0/PHY_CFG0)
- new net ETH2-PHY_CFG1: ETH2-PHY.26 (LINK_ST/PHY_CFG1)
- new net ETH2-PHY_PHYAD2: ETH2-PHY.30 (RXD_2/PHYAD_2)
- new net ETH2-PHY_PHYAD3: ETH2-PHY.29 (RXD_3/PHYAD_3)
- new net ETH2_CRD: T-ETH2.7 (CRD)
- new net ETH2_CTD: T-ETH2.2 (CTD)
- new net ETH2_LINE_CT: T-ETH2.10 (CRX), T-ETH2.15 (CTX)
- new net ETH2_LINE_RXN: ETH2.4 (RXN), T-ETH2.9 (RX-)
- new net ETH2_LINE_RXP: ETH2.3 (RXP), T-ETH2.11 (RX+)
- new net ETH2_LINE_TXN: ETH2.2 (TXN), T-ETH2.14 (TX-)
- new net ETH2_LINE_TXP: ETH2.1 (TXP), T-ETH2.16 (TX+)
- new net ETH2_RXN: ETH2-PHY.15 (MDI_1_N), T-ETH2.8 (RD-)
- new net ETH2_RXP: ETH2-PHY.14 (MDI_1_P), T-ETH2.6 (RD+)
- new net ETH2_TXN: ETH2-PHY.13 (MDI_0_N), T-ETH2.3 (TD-)
- new net ETH2_TXP: ETH2-PHY.12 (MDI_0_P), T-ETH2.1 (TD+)
- new net ETH_CRD: T-ETH.7 (CRD)
- new net ETH_CTD: T-ETH.2 (CTD)
- new net ETH_LINE_CT: T-ETH.10 (CRX), T-ETH.15 (CTX)
- new net ETH_LINE_RXN: ETH1.4 (RXN), T-ETH.9 (RX-)
- new net ETH_LINE_RXP: ETH1.3 (RXP), T-ETH.11 (RX+)
- new net ETH_LINE_TXN: ETH1.2 (TXN), T-ETH.14 (TX-)
- new net ETH_LINE_TXP: ETH1.1 (TXP), T-ETH.16 (TX+)
- new net ETH_RXN: ETH1-PHY.15 (MDI_1_N), T-ETH.8 (RD-)
- new net ETH_RXP: ETH1-PHY.14 (MDI_1_P), T-ETH.6 (RD+)
- new net ETH_TXN: ETH1-PHY.13 (MDI_0_N), T-ETH.3 (TD-)
- new net ETH_TXP: ETH1-PHY.12 (MDI_0_P), T-ETH.1 (TD+)
- new net GND: 1553-DRV.12 (EN*), 1553-DRV.15 (DI4), 1553-DRV.8 (GND), 1553-DRV.9 (DI3), 1553-RCV.12 (EN*), 1553-RCV.8 (GND), BARO.3 (VSS), BARO.8 (VSS), BARO.9 (VSS), C-GPIO.2 (N), CAN-TR.10 (GND1), CAN-TR.6 (GNDIO), ESC-PWM.5 (GND), ESC-TLM.1 (GND), ETH1-PHY.41 (EP), ETH1-PHY.5 (GND), ETH2-PHY.41 (EP), ETH2-PHY.5 (GND), GPIO-A.1 (GND), GPIO-B.1 (GND), GPIO-C.1 (GND), GPIO-D.1 (GND), GPIO-E.1 (GND), GPIO-F.1 (GND), GPS.1 (GND), GPS.10 (GND), GPS.11 (GND), GPS.15 (GND), GPS.16 (GND), GPS.4 (GND), GPS.5 (GND), GPS.6 (GND), IMU.10 (RESV), IMU.11 (RESV), IMU.2 (RESV), IMU.3 (RESV), IMU.6 (GND), IMU.7 (RESV(GND)), MIL-1553.3 (GND), PB2-P1.1 (P1), PB2-P1.2 (P2), PB2-P1.36 (P36), PB2-P2.36 (P36), PWR-IN.3 (GND), PWR-IN.4 (GND), RS485.10 (GND1), RS485.6 (GNDIO), SERVO-PWM.8 (GND), TPM.2 (GND), TPM.23 (GND), TPM.32 (GND), TPM.33 (EP), TPM.9 (GND), U-GPIO.12 (VSS), U-GPIO.2 (A1), U-GPIO.21 (A0), U-GPIO.3 (A2), X2Y-CAN.1 (G1), X2Y-CAN.2 (G1), X2Y-CAN.3 (G1), X2Y-RS485.1 (G1), X2Y-RS485.2 (G1), X2Y-RS485.3 (G1)
- new net GND2_CAN: CAN-FD.1 (GND), CAN-TR.11 (GND2), CAN-TR.15 (GISOIN), CAN-TR.16 (GISOIN), CAN-TR.17 (GISOIN), TVS-CAN.2 (GND), X2Y-CAN.4 (G2)
- new net GND2_RS485: RS-485.1 (GND), RS485.11 (GND2), RS485.13 (MODE), RS485.15 (GISOIN), TVS-RS485.2 (GND), X2Y-RS485.4 (G2)
- new net GPIO_EXP_A: GPIO-A.3 (SIG), U-GPIO.4 (IO0_0)
- new net GPIO_EXP_B: GPIO-B.3 (SIG), U-GPIO.5 (IO0_1)
- new net GPIO_EXP_C: GPIO-C.3 (SIG), U-GPIO.6 (IO0_2)
- new net GPIO_EXP_D: GPIO-D.3 (SIG), U-GPIO.7 (IO0_3)
- new net GPIO_EXP_E: GPIO-E.3 (SIG), U-GPIO.8 (IO0_4)
- new net GPIO_EXP_F: GPIO-F.3 (SIG), U-GPIO.9 (IO0_5)
- new net I2C1_SCL: PB2-P1.28 (P28), U-GPIO.22 (SCL)
- new net I2C1_SDA: PB2-P1.27 (P27), U-GPIO.23 (SDA)
- new net M1553_N: 1553-DRV.6 (DO2+), 1553-RCV.1 (RI1-), 1553-RCV.6 (RI2+), 1553-XFM.3 (PRI_N)
- new net M1553_P: 1553-DRV.2 (DO1+), 1553-RCV.2 (RI1+), 1553-RCV.7 (RI2-), 1553-XFM.1 (PRI_P)
- new net M1553_TX_EN: 1553-DRV.4 (EN)
- new net MDC: ETH1-PHY.23 (MDC), ETH2-PHY.23 (MDC)
- new net MDIO: ETH1-PHY.24 (MDIO), ETH2-PHY.24 (MDIO)
- new net PHY1_INTRN: ETH1-PHY.22 (INT_N), PB2-P2.16 (P16)
- new net PHY1_RSTN: ETH1-PHY.7 (RESET_N), PB2-P2.15 (P15)
- new net PHY2_INTRN: ETH2-PHY.22 (INT_N), PB2-P2.14 (P14)
- new net PHY2_RSTN: ETH2-PHY.7 (RESET_N), PB2-P2.13 (P13)
- new net REXT_ETH1-PHY: ETH1-PHY.10 (REXT)
- new net REXT_ETH2-PHY: ETH2-PHY.10 (REXT)
- new net RMII0_CRS_DV: ETH1-PHY.35 (RX_CTL/CRS_DV), PB2-P2.29 (P29)
- new net RMII0_REF_CLK: ETH1-PHY.9 (REF_CLK), PB2-P2.27 (P27)
- new net RMII0_RXD0: ETH1-PHY.33 (RXD_0), PB2-P2.31 (P31)
- new net RMII0_RXD1: ETH1-PHY.32 (RXD_1), PB2-P2.30 (P30)
- new net RMII0_RX_ER: ETH1-PHY.27 (GP_CLK/RX_ER), PB2-P2.28 (P28)
- new net RMII0_TXD0: ETH1-PHY.39 (TXD_0), PB2-P2.34 (P34)
- new net RMII0_TXD1: ETH1-PHY.1 (TXD_1), PB2-P2.33 (P33)
- new net RMII0_TX_EN: ETH1-PHY.37 (TX_CTL/TX_EN), PB2-P2.32 (P32)
- new net RMII1_CRS_DV: ETH2-PHY.35 (RX_CTL/CRS_DV), PB2-P2.21 (P21)
- new net RMII1_REF_CLK: ETH2-PHY.9 (REF_CLK), PB2-P2.19 (P19)
- new net RMII1_RX_ER: ETH2-PHY.27 (GP_CLK/RX_ER), PB2-P2.20 (P20)
- new net RMII1_TX_EN: ETH2-PHY.37 (TX_CTL/TX_EN), PB2-P2.24 (P24)
- new net RS485_A_F: CMC-RS485.2 (W1_OUT), RS-485.2 (A), TVS-RS485.1 (IO1)
- new net RS485_B_F: CMC-RS485.3 (W2_OUT), RS-485.3 (B), TVS-RS485.3 (IO2)
- new net VCC2_CAN: CAN-FD.4 (VCC), CAN-TR.12 (VISOOUT), CAN-TR.13 (VSIN), CAN-TR.20 (VISOIN), TVS-CAN.5 (VCC)
- new net VCC2_RS485: RS-485.4 (VCC), RS485.12 (VISOOUT), RS485.16 (VISOIN), TVS-RS485.5 (VCC)
- no-connect marks 23 -> 80
Other:
- note removed: "ETH1 sub-circuit: DP83825I PHY1 + HX1188NL magnetics + TPS62933 1V8 + TVS + CMC + J_ETH1 connector"
- note removed: "ETH2 sub-circuit: DP83825I PHY2 + HX1188NL magnetics + TPS62933 1V8 + TVS + CMC + J_ETH2 connector"
- note removed: "NOTE: IN+ and IN- tied to VBAT_MON_P = voltage monitoring only. For current monitoring: insert 10 mO shunt between J_VBAT pin 1 and IN+ with IN- on shunt low side."
- company: Griffing Technology LLC -> (none)
- title: Wash — EMI-Hardened Flight Control & Sensor Cape -> (none)
