File: avionics/kicad/Jayne/kicads/Jayne.kicad_sch (KiCad schematic)
At the start: 59 parts, among them Q1 AO3400 logic-level N-MOSFET, T1 Wurth 749010012A, T1_CMC1 SRF2012-100Y, T1_CMC2 SRF2012-100Y, T1_D1 PRTR5V0U2X, T1_D2 PRTR5V0U2X, T2 Wurth 749010012A, T2_CMC1 SRF2012-100Y, T2_CMC2 SRF2012-100Y, T2_D1 PRTR5V0U2X, T2_D2 PRTR5V0U2X, U2 Microchip KSZ9477, U3 TI MSPM0G3507, U4 TI ISOW1044BDFMR, U5 Infineon SLB9670, Y1 25MHz

Commit message: Fleet trust module (MCU+TPM+isolated CAN-FD+RS-485) across new CAN-PERIPH-GW-1 board, Jayne, Kaylee, Emma; ISOW1412 swap on Wash/Zoë
- New stackable CAN-PERIPH-GW-1 gateway board (N_STACKS param): MSPM0G3507
  + SLB9670 TPM + ISOW1044BDFMR isolated CAN-FD + ISOW1412 isolated RS-485,
  informed by the public VimDrones ap_periph_pico/ESC S50 concept (no
  VimDrones GPL-3.0 source copied). PCB freerouted via the Specctra DSN/SES
  bridge (tools/export-specctra-dsn.py + import-specctra-ses.py +
  freerouting 2.2.4); user's manual footprint packing preserved.
- Jayne: added ISOW1412 isolated RS-485 (Section H); MSPM0G3507 pinmux
  re-verified against the real datasheet for all new assignments.
- Kaylee: full trust module added via non-destructive schematic injection
  (inject_kaylee_trust_module.py) -- gen_kaylee.py itself has drifted from
  the checked-in file and is not safe to regenerate from (tracked as an
  open item).
- Emma: SLB9670 TPM added via a dedicated header (inject_emma_tpm.py); no
  separate CAN/RS-485 needed, reaches the bus via Zoë's P1/P2 link.
- Fleet-wide ADM2795E -> ISOW1412 (integrated isolated DC-DC). While
  swapping Wash/Zoë, fixed their pre-existing broken ADM2795EBRWZ pin
  numbering and wrong ISOW1044BDFMR footprint (SOIC-16W on a 20-pin part).
- REFERENCES.md: REF-SENSOR-009/010/011 (ISOW1044/ISOW1412/SLB9670),
  ADM2795E supersession, Wash/Zoë defect history, vimdrones GPL note.
- WBS/TODO updated across avionics, airframe/wings-nacelles, and root:
  AK7455 nacelle tilt data is now bus-published by the gateway rather than
  read directly by River/Simon.

Co-Authored-By: Claude Sonnet 5 <noreply@anthropic.com>
Parts:
- added C_ADM1, C_ADM2: 100nF, Capacitor_SMD:C_0402_1005Metric, symbol C_Generic
- added J_RS485_IN: RS-485 trunk IN (A/B/GND), symbol Conn_JST_GH_03P
- added J_RS485_OUT: RS-485 trunk OUT (A/B/GND), symbol Conn_JST_GH_03P
- added R_485TERM: 120R, Resistor_SMD:R_0402_1005Metric, symbol R_Generic
- added SJ_485: open by default, Jumper:SolderJumper-2_P1.3mm_Open_Pad1.0x1.5mm, symbol SJ_Generic
- added U6: TI ISOW1412, Package_SO:SOIC-20W_7.5x12.8mm_P1.27mm, symbol GW_ISOW1412
Connections:
- net +3V3: now also C_ADM1.1, U6.1 (VIO), U6.9 (VDD)
- net GND: now also C_ADM1.2, U6.10 (GND1), U6.6 (GNDIO)
- net RS485_DE: now reaches U3.14 (PB2)
- net RS485_DE: now also U6.3 (DE), U6.5 (RE_N)
- net RS485_TX: now reaches U3.25 (PB15)
- net RS485_TX: now also U6.2 (D)
- net RS485_RX: now reaches U3.26 (PB16)
- net RS485_RX: now also U6.4 (R)
- new net ISO_3V3_485: C_ADM2.1, U6.12 (VISOOUT), U6.16 (VISOIN)
- new net ISO_GND_485: C_ADM2.2, J_RS485_IN.3, J_RS485_OUT.3, U6.11 (GND2), U6.13 (MODE), U6.15 (GISOIN)
- new net RS485_A: J_RS485_IN.1, J_RS485_OUT.1, R_485TERM.1, U6.17 (Y), U6.20 (A)
- new net RS485_B: J_RS485_IN.2, J_RS485_OUT.2, SJ_485.2, U6.18 (Z), U6.19 (B)
- new net RS485_FLT_N: U6.8 (EN_FLT)
- new net TERM485_MID: R_485TERM.2, SJ_485.1
- no-connect marks 271 -> 270
Other:
- note added: "=== Section H: ISOW1412 Isolated RS-485 (U6) ==="
