File: avionics/kicad/Jayne/kicads/Jayne.kicad_pcb (KiCad board)
At the start: 4 copper layers, 69.8 x 56.4 mm, 63 parts, among them Q1 AO3400 logic-level N-MOSFET, T1 Wurth 749010012A, T1_CMC1 SRF2012-100Y, T1_CMC2 SRF2012-100Y, T1_D1 PRTR5V0U2X, T1_D2 PRTR5V0U2X, T2 Wurth 749010012A, T2_CMC1 SRF2012-100Y, T2_CMC2 SRF2012-100Y, T2_D1 PRTR5V0U2X, T2_D2 PRTR5V0U2X, U2 Microchip KSZ9477, U3 TI MSPM0G3507, U4 TI ISOW1044BDFMR, U5 Infineon SLB9670, Y1 25MHz

Commit message: new branch who dis
Parts:
- added C_ADM1: 100nF, C_0402_1005Metric, F.Cu at (175.3, 124.2)
- added C_ADM2: 100nF, C_0402_1005Metric, F.Cu at (175.3, 125.7)
- added J_RS485_IN: RS-485 trunk IN (A/B/GND), JST_GH_BM03B-GHS-TBT_1x03-1MP_P1.25mm_Vertical, F.Cu at (186.1, 174.3)
- added J_RS485_OUT: RS-485 trunk OUT (A/B/GND), JST_GH_BM03B-GHS-TBT_1x03-1MP_P1.25mm_Vertical, F.Cu at (190.3, 126.9)
- added R_485TERM: 120R, R_0402_1005Metric, F.Cu at (175.3, 127.2)
- added SJ_485: open by default, SolderJumper-2_P1.3mm_Open_Pad1.0x1.5mm, F.Cu at (176.2, 175.2)
- added U6: TI ISOW1412, SOIC-20W_7.5x12.8mm_P1.27mm, F.Cu at (228.4, 130.5)
- moved R_FB1T 2.41 mm to (204.5, 161.0)
- moved R_FB3B 2.05 mm to (211.5, 161.0)
Connections:
- U3 pad 14: (no net) -> RS485_DE
- U3 pad 25: (no net) -> RS485_TX
- U3 pad 26: (no net) -> RS485_RX
- U5 pad 33: GND -> (no net)

Commit message: fleshed out lots of pcbs
Parts:
- J_RS485_IN, J_RS485_OUT: moved to B.Cu
- moved SJ_485 52.9 mm to (213.3, 137.5)
- moved U6 30.6 mm to (210.0, 155.0), turned to 90 degrees
- moved R_FB3T 16.6 mm to (229.5, 151.0)
- moved R_ISET 16.1 mm to (229.5, 152.5)
- moved U_REG_3V3_CO 14.0 mm to (227.0, 151.0)
- moved R_485TERM 13.6 mm to (188.5, 130.5)
- moved R1 13.4 mm to (230.5, 155.0)
- moved R2 13.3 mm to (233.0, 155.0)
- moved U_REG_1V2_CI 13.1 mm to (226.0, 145.5)
- moved C_ADM1 12.6 mm to (175.9, 136.8)
- moved C_ADM2 12.6 mm to (175.9, 138.3)
- moved R_NRST 11.9 mm to (224.5, 151.0)
- moved T1_D2 11.1 mm to (219.0, 148.0)
- moved J_RS485_OUT 8.81 mm to (182.5, 131.0), turned to 180 degrees
- moved J_CHASSIS_R 6.87 mm to (219.5, 145.5)
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Other:
- board text added: "Camera and Laser Sensor suite"
- board text removed: "Jayne Rev - (design exploration)"
