File: avionics/kicad/CAN-PERIPH-GW-1/kicads/CAN-PERIPH-GW-1.kicad_sch (KiCad schematic)
At the start: 32 parts, among them U1_1 TI MSPM0G3507, U2_1 Infineon SLB9670 TPM2.0, U3_1 TI ISOW1044BDFMR, U4_1 TI ISOW1412

Commit message: just making everything shiny
Parts:
- added C_ISO1_2, C_ISO1_3, C_ISO1_4, C_MCU1_2, C_MCU1_3, C_MCU1_4, C_RS1_2, C_RS1_3, C_RS1_4, C_RS2_2, C_RS2_3, C_RS2_4, C_TPM1_2, C_TPM1_3, C_TPM1_4: 100nF, Capacitor_SMD:C_0402_1005Metric, symbol C_Generic
- added C_ISO2_2, C_ISO2_3, C_ISO2_4, C_TPM2_2, C_TPM2_3, C_TPM2_4, C_VCORE_2, C_VCORE_3, C_VCORE_4: 1uF, Capacitor_SMD:C_0402_1005Metric, symbol C_Generic
- added J_CAN_IN: CAN-FD trunk IN (CANH/CANL/GND), Connector_JST:JST_GH_BM03B-GHS-TBT_1x03-1MP_P1.25mm_Vertical, symbol Conn_JST_GH_03P
- added J_ENC_2, J_ENC_3, J_ENC_4: 7W direct-solder, mates ENC-NACELLE-1 P1 pigtail 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, Serenity-Custom:Pigtail_7W_DirectSolder, symbol Pigtail_7W_DirectSolder
- added J_FLEX_2, J_FLEX_3, J_FLEX_4: 1x08 2.54mm: TX/RX/TTL/PWM/BSHOT/+5V/+3V3/GND, Connector_PinHeader_2.54mm:PinHeader_1x08_P2.54mm_Vertical, symbol PinHeader_1x08
- added J_SWD_2, J_SWD_3, J_SWD_4: SWD: DIO/CLK/NRST/GND, Connector_JST:JST_GH_BM04B-GHS-TBT_1x04-1MP_P1.25mm_Vertical, symbol Conn_JST_GH_04P
- added R_NRST_2, R_NRST_3, R_NRST_4, R_TPM_RST_2, R_TPM_RST_3, R_TPM_RST_4: 10k, Resistor_SMD:R_0402_1005Metric, symbol R_Generic
- added U1_3, U1_4: TI MSPM0G3507, Package_DFN_QFN:QFN-48-1EP_7x7mm_P0.5mm_EP5.15x5.15mm, symbol Jayne_MSPM0G3507_RGZ
- added U2_2, U2_3, U2_4: Infineon SLB9670 TPM2.0, Package_DFN_QFN:QFN-32-1EP_5x5mm_P0.5mm_EP3.45x3.45mm, symbol Jayne_SLB9670_TPM
- added U3_2, U3_3, U3_4: TI ISOW1044BDFMR, Package_SO:SOIC-20W_7.5x12.8mm_P1.27mm, symbol Jayne_ISOW1044BDFMR
- added U4_2, U4_3, U4_4: TI ISOW1412, Package_SO:SOIC-20W_7.5x12.8mm_P1.27mm, symbol GW_ISOW1412
- U1_2: renamed from J_CAN_IN; value CAN-FD trunk IN (CANH/CANL/GND) -> TI MSPM0G3507; footprint Connector_JST:JST_GH_BM03B-GHS-TBT_1x03-1MP_P1.25mm_Vertical -> Package_DFN_QFN:QFN-48-1EP_7x7mm_P0.5mm_EP5.15x5.15mm; symbol Conn_JST_GH_03P -> Jayne_MSPM0G3507_RGZ
Connections:
- net +3V3: now also U1_2.6 (VDD), C_ISO1_2.1, C_ISO1_3.1, C_ISO1_4.1, C_MCU1_2.1, C_MCU1_3.1, C_MCU1_4.1, C_RS1_2.1, C_RS1_3.1, C_RS1_4.1, C_TPM1_2.1, C_TPM1_3.1, C_TPM1_4.1, C_TPM2_2.1, C_TPM2_3.1, C_TPM2_4.1, J_ENC_2.6, J_ENC_3.6, J_ENC_4.6, J_FLEX_2.7, J_FLEX_3.7, J_FLEX_4.7, R_NRST_2.1, R_NRST_3.1, R_NRST_4.1, R_TPM_RST_2.1, R_TPM_RST_3.1, R_TPM_RST_4.1, U1_3.6 (VDD), U1_4.6 (VDD), U2_2.1 (NCI/VDD), U2_2.14 (NCI/VDD), U2_2.22 (VDD), U2_2.8 (VDD), U2_3.1 (NCI/VDD), U2_3.14 (NCI/VDD), U2_3.22 (VDD), U2_3.8 (VDD), U2_4.1 (NCI/VDD), U2_4.14 (NCI/VDD), U2_4.22 (VDD), U2_4.8 (VDD), U3_2.1 (VIO), U3_2.9 (VDD), U3_3.1 (VIO), U3_3.9 (VDD), U3_4.1 (VIO), U3_4.9 (VDD), U4_2.1 (VIO), U4_2.9 (VDD), U4_3.1 (VIO), U4_3.9 (VDD), U4_4.1 (VIO), U4_4.9 (VDD)
- net +5V: now also J_FLEX_2.6, J_FLEX_3.6, J_FLEX_4.6
- net CAN_H: now also J_CAN_IN.1, U3_2.19 (CANH), U3_3.19 (CANH), U3_4.19 (CANH); no longer U1_2.1
- net CAN_L: now also J_CAN_IN.2, U3_2.18 (CANL), U3_3.18 (CANL), U3_4.18 (CANL); no longer U1_2.2
- net GND: now also U1_2.49 (VSS), U1_2.7 (VSS), C_ISO1_2.2, C_ISO1_3.2, C_ISO1_4.2, C_MCU1_2.2, C_MCU1_3.2, C_MCU1_4.2, C_RS1_2.2, C_RS1_3.2, C_RS1_4.2, C_TPM1_2.2, C_TPM1_3.2, C_TPM1_4.2, C_TPM2_2.2, C_TPM2_3.2, C_TPM2_4.2, C_VCORE_2.2, C_VCORE_3.2, C_VCORE_4.2, J_ENC_2.1, J_ENC_3.1, J_ENC_4.1, J_FLEX_2.8, J_FLEX_3.8, J_FLEX_4.8, J_SWD_2.4, J_SWD_3.4, J_SWD_4.4, U1_3.49 (VSS), U1_3.7 (VSS), U1_4.49 (VSS), U1_4.7 (VSS), U2_2.16 (NCI/GND), U2_2.2 (GND), U2_2.23 (GND), U2_2.32 (GND), U2_2.9 (GND), U2_3.16 (NCI/GND), U2_3.2 (GND), U2_3.23 (GND), U2_3.32 (GND), U2_3.9 (GND), U2_4.16 (NCI/GND), U2_4.2 (GND), U2_4.23 (GND), U2_4.32 (GND), U2_4.9 (GND), U3_2.10 (GND1), U3_2.4 (STB), U3_2.6 (GNDIO), U3_3.10 (GND1), U3_3.4 (STB), U3_3.6 (GNDIO), U3_4.10 (GND1), U3_4.4 (STB), U3_4.6 (GNDIO), U4_2.10 (GND1), U4_2.6 (GNDIO), U4_3.10 (GND1), U4_3.6 (GNDIO), U4_4.10 (GND1), U4_4.6 (GNDIO)
- net ISO_GND_485: now also C_RS2_2.2, C_RS2_3.2, C_RS2_4.2, U4_2.11 (GND2), U4_2.13 (MODE), U4_2.15 (GISOIN), U4_3.11 (GND2), U4_3.13 (MODE), U4_3.15 (GISOIN), U4_4.11 (GND2), U4_4.13 (MODE), U4_4.15 (GISOIN)
- net ISO_GND_CAN: now also C_ISO2_2.2, C_ISO2_3.2, C_ISO2_4.2, J_CAN_IN.3, U3_2.11 (GND2), U3_2.15 (GISOIN), U3_2.16 (GISOIN), U3_2.17 (GISOIN), U3_3.11 (GND2), U3_3.15 (GISOIN), U3_3.16 (GISOIN), U3_3.17 (GISOIN), U3_4.11 (GND2), U3_4.15 (GISOIN), U3_4.16 (GISOIN), U3_4.17 (GISOIN); no longer U1_2.3
- net RS485_A: now also U4_2.17 (Y), U4_2.20 (A), U4_3.17 (Y), U4_3.20 (A), U4_4.17 (Y), U4_4.20 (A)
- net RS485_B: now also U4_2.18 (Z), U4_2.19 (B), U4_3.18 (Z), U4_3.19 (B), U4_4.18 (Z), U4_4.19 (B)
- new net CANFD_FLT_N_2: U1_2.43 (PA23), U3_2.8 (EN/FLT)
- new net CANFD_FLT_N_3: U1_3.43 (PA23), U3_3.8 (EN/FLT)
- new net CANFD_FLT_N_4: U1_4.43 (PA23), U3_4.8 (EN/FLT)
- new net CANFD_RX_2: U1_2.28 (PA13), U3_2.5 (RXD)
- new net CANFD_RX_3: U1_3.28 (PA13), U3_3.5 (RXD)
- new net CANFD_RX_4: U1_4.28 (PA13), U3_4.5 (RXD)
- new net CANFD_TX_2: U1_2.27 (PA12), U3_2.3 (TXD)
- new net CANFD_TX_3: U1_3.27 (PA12), U3_3.3 (TXD)
- new net CANFD_TX_4: U1_4.27 (PA12), U3_4.3 (TXD)
- new net ENC_ERROR_2: J_ENC_2.7, U1_2.29 (PA14)
- new net ENC_ERROR_3: J_ENC_3.7, U1_3.29 (PA14)
- new net ENC_ERROR_4: J_ENC_4.7, U1_4.29 (PA14)
- new net ENC_SPI_CS_2: J_ENC_2.2, U1_2.30 (PA15)
- new net ENC_SPI_CS_3: J_ENC_3.2, U1_3.30 (PA15)
- new net ENC_SPI_CS_4: J_ENC_4.2, U1_4.30 (PA15)
- new net ENC_SPI_MISO_2: J_ENC_2.5, U1_2.31 (PA16)
- new net ENC_SPI_MISO_3: J_ENC_3.5, U1_3.31 (PA16)
- new net ENC_SPI_MISO_4: J_ENC_4.5, U1_4.31 (PA16)
- new net ENC_SPI_MOSI_2: J_ENC_2.4, U1_2.33 (PA18)
- new net ENC_SPI_MOSI_3: J_ENC_3.4, U1_3.33 (PA18)
- new net ENC_SPI_MOSI_4: J_ENC_4.4, U1_4.33 (PA18)
- new net ENC_SPI_SCK_2: J_ENC_2.3, U1_2.32 (PA17)
- new net ENC_SPI_SCK_3: J_ENC_3.3, U1_3.32 (PA17)
- new net ENC_SPI_SCK_4: J_ENC_4.3, U1_4.32 (PA17)
- new net FLEX_BSHOT_IO_2: J_FLEX_2.5, U1_2.20 (PB6)
- new net FLEX_BSHOT_IO_3: J_FLEX_3.5, U1_3.20 (PB6)
- new net FLEX_BSHOT_IO_4: J_FLEX_4.5, U1_4.20 (PB6)
- new net FLEX_PWM_IO_2: J_FLEX_2.4, U1_2.15 (PB3)
- new net FLEX_PWM_IO_3: J_FLEX_3.4, U1_3.15 (PB3)
- new net FLEX_PWM_IO_4: J_FLEX_4.4, U1_4.15 (PB3)
- new net FLEX_TTL_GPIO_2: J_FLEX_2.3, U1_2.44 (PA24)
- new net FLEX_TTL_GPIO_3: J_FLEX_3.3, U1_3.44 (PA24)
- new net FLEX_TTL_GPIO_4: J_FLEX_4.3, U1_4.44 (PA24)
- new net FLEX_UART_RX_2: J_FLEX_2.2, U1_2.2 (PA1)
- new net FLEX_UART_RX_3: J_FLEX_3.2, U1_3.2 (PA1)
- new net FLEX_UART_RX_4: J_FLEX_4.2, U1_4.2 (PA1)
- new net FLEX_UART_TX_2: J_FLEX_2.1, U1_2.1 (PA0)
- new net FLEX_UART_TX_3: J_FLEX_3.1, U1_3.1 (PA0)
- new net FLEX_UART_TX_4: J_FLEX_4.1, U1_4.1 (PA0)
- new net ISO_3V3_485_2: C_RS2_2.1, U4_2.12 (VISOOUT), U4_2.16 (VISOIN)
- new net ISO_3V3_485_3: C_RS2_3.1, U4_3.12 (VISOOUT), U4_3.16 (VISOIN)
- new net ISO_3V3_485_4: C_RS2_4.1, U4_4.12 (VISOOUT), U4_4.16 (VISOIN)
- new net ISO_5V_CAN_2: C_ISO2_2.1, U3_2.12 (VISOOUT), U3_2.13 (VSIN), U3_2.20 (VISOIN)
- new net ISO_5V_CAN_3: C_ISO2_3.1, U3_3.12 (VISOOUT), U3_3.13 (VSIN), U3_3.20 (VISOIN)
- new net ISO_5V_CAN_4: C_ISO2_4.1, U3_4.12 (VISOOUT), U3_4.13 (VSIN), U3_4.20 (VISOIN)
- new net MCU_NRST_2: J_SWD_2.3, R_NRST_2.2, U1_2.4 (NRST)
- new net MCU_NRST_3: J_SWD_3.3, R_NRST_3.2, U1_3.4 (NRST)
- new net MCU_NRST_4: J_SWD_4.3, R_NRST_4.2, U1_4.4 (NRST)
- new net MCU_SWCLK_2: J_SWD_2.2, U1_2.35 (PA20/SWCLK)
- new net MCU_SWCLK_3: J_SWD_3.2, U1_3.35 (PA20/SWCLK)
- new net MCU_SWCLK_4: J_SWD_4.2, U1_4.35 (PA20/SWCLK)
- new net MCU_SWDIO_2: J_SWD_2.1, U1_2.34 (PA19/SWDIO)
- new net MCU_SWDIO_3: J_SWD_3.1, U1_3.34 (PA19/SWDIO)
- new net MCU_SWDIO_4: J_SWD_4.1, U1_4.34 (PA19/SWDIO)
- new net MCU_VCORE_2: C_VCORE_2.1, U1_2.48 (VCORE)
- new net MCU_VCORE_3: C_VCORE_3.1, U1_3.48 (VCORE)
- new net MCU_VCORE_4: C_VCORE_4.1, U1_4.48 (VCORE)
- new net RS485_DE_2: U1_2.14 (PB2), U4_2.3 (DE), U4_2.5 (RE_N)
- new net RS485_DE_3: U1_3.14 (PB2), U4_3.3 (DE), U4_3.5 (RE_N)
- new net RS485_DE_4: U1_4.14 (PB2), U4_4.3 (DE), U4_4.5 (RE_N)
- new net RS485_FLT_N_2: U1_2.16 (PA8), U4_2.8 (EN_FLT)
- new net RS485_FLT_N_3: U1_3.16 (PA8), U4_3.8 (EN_FLT)
- new net RS485_FLT_N_4: U1_4.16 (PA8), U4_4.8 (EN_FLT)
- new net RS485_RX_2: U1_2.26 (PB16), U4_2.4 (R)
- new net RS485_RX_3: U1_3.26 (PB16), U4_3.4 (R)
- new net RS485_RX_4: U1_4.26 (PB16), U4_4.4 (R)
- new net RS485_TX_2: U1_2.25 (PB15), U4_2.2 (D)
- new net RS485_TX_3: U1_3.25 (PB15), U4_3.2 (D)
- new net RS485_TX_4: U1_4.25 (PB15), U4_4.2 (D)
- new net TPM_PIRQ_2: U1_2.9 (PA3), U2_2.18 (PIRQ#)
- new net TPM_PIRQ_3: U1_3.9 (PA3), U2_3.18 (PIRQ#)
- new net TPM_PIRQ_4: U1_4.9 (PA3), U2_4.18 (PIRQ#)
- new net TPM_RESET_N_2: R_TPM_RST_2.2, U1_2.13 (PA7), U2_2.17 (RST#)
- new net TPM_RESET_N_3: R_TPM_RST_3.2, U1_3.13 (PA7), U2_3.17 (RST#)
- new net TPM_RESET_N_4: R_TPM_RST_4.2, U1_4.13 (PA7), U2_4.17 (RST#)
- new net TPM_SPI_CS_2: U1_2.8 (PA2), U2_2.20 (CS#)
- new net TPM_SPI_CS_3: U1_3.8 (PA2), U2_3.20 (CS#)
- new net TPM_SPI_CS_4: U1_4.8 (PA2), U2_4.20 (CS#)
- new net TPM_SPI_MISO_2: U1_2.10 (PA4), U2_2.24 (MISO)
- new net TPM_SPI_MISO_3: U1_3.10 (PA4), U2_3.24 (MISO)
- new net TPM_SPI_MISO_4: U1_4.10 (PA4), U2_4.24 (MISO)
- new net TPM_SPI_MOSI_2: U1_2.11 (PA5), U2_2.21 (MOSI)
- new net TPM_SPI_MOSI_3: U1_3.11 (PA5), U2_3.21 (MOSI)
- new net TPM_SPI_MOSI_4: U1_4.11 (PA5), U2_4.21 (MOSI)
- new net TPM_SPI_SCK_2: U1_2.12 (PA6), U2_2.19 (SCLK)
- new net TPM_SPI_SCK_3: U1_3.12 (PA6), U2_3.19 (SCLK)
- new net TPM_SPI_SCK_4: U1_4.12 (PA6), U2_4.19 (SCLK)
- no-connect marks 42 -> 165
Other:
- note added: "=== Stack 2: U1_2 MCU / U2_2 TPM / U3_2 CAN-FD / U4_2 RS-485 ==="
- note added: "=== Stack 3: U1_3 MCU / U2_3 TPM / U3_3 CAN-FD / U4_3 RS-485 ==="
- note added: "=== Stack 4: U1_4 MCU / U2_4 TPM / U3_4 CAN-FD / U4_4 RS-485 ==="
- title: CAN-PERIPH-GW-1 -- TPM-secured Dual-Isolated-Bus (CAN-FD + RS-485) Peripheral Gateway (1x stack) -> CAN-PERIPH-GW-1 -- TPM-secured Dual-Isolated-Bus (CAN-FD + RS-485) Peripheral Gateway (4x stack)
