File: avionics/kicad/CAN-PERIPH-GW-1/kicads/CAN-PERIPH-GW-1.kicad_sch (KiCad schematic)
At the start: 83 parts, among them U1_1 TI MSPM0G3507, U1_2 TI MSPM0G3507, U1_3 TI MSPM0G3507, U1_4 TI MSPM0G3507, U2_1 Infineon SLB9670 TPM2.0, U2_2 Infineon SLB9670 TPM2.0, U2_3 Infineon SLB9670 TPM2.0, U2_4 Infineon SLB9670 TPM2.0, U3_1 TI ISOW1044BDFMR, U3_2 TI ISOW1044BDFMR, U3_3 TI ISOW1044BDFMR, U3_4 TI ISOW1044BDFMR, U4_1 TI ISOW1412, U4_2 TI ISOW1412, U4_3 TI ISOW1412, U4_4 TI ISOW1412

Commit message: Rename avionics/GCS boards off Firefly character names (TODO.md §0.9 item 8)
User-directed rename to close out the last open item from the licensing audit:
Malcolm/Mal -> Skipper, Wash -> Pilot, Zoe -> XO, Kaylee -> Flight Engineer,
Emma -> Commo, Jayne -> Observer. The four avionics bay names (Shepherd's Room,
Inara's Shuttle, River's Room, Simon's Medbay) were not part of this rename.

- Physical rename of all 198 board-folder paths via git mv: KiCad schematics,
  PCBs, gerbers, scripts, companion docs, plus the 6 shared Jayne_*.kicad_sym
  symbol libraries (authored under Jayne, reused fleet-wide by Wash/Kaylee/Emma/
  CAN-PERIPH-GW-1) -> Observer_*.kicad_sym, with every sym-lib-table/
  fp-lib-table/embedded lib_symbols reference updated to match. Also caught a
  second gerber export set outside the per-board folders and 4 STL BOM
  placeholders.
- Content sweep of ~5,800 substitutions across ~330 tracked text files, using
  word-boundary regex for the safe general case plus a small set of
  hand-verified literal-substring rules for snake_case identifiers. Verified
  before running that a blanket "mal_"/"emma" substring replace would have
  corrupted real unrelated tokens already in the repo (Blender normal_z
  surface-normal variables, KiCad thermal_pads/thermal_gap/thermal_bridge_width
  settings, "washer", "piezoelectric") -- used explicit rules instead and
  confirmed all four survived intact.
- MAL-* BOM/component designators renamed to SKIPPER-* consistently, including
  inside ENC-NACELLE-1 and CAN-PERIPH-GW-1's own netlists (cross-board net
  names).
- AGENTS.md Sec 9 naming table rewritten: dropped the Firefly-quote column from
  the live table (a mutated quote next to the new name would still signal the
  original character) and added a "Naming history" subsection recording the
  former names/inspirations/quotes for attribution completeness.
- Not verified: KiCad ERC/DRC -- no kicad-cli in this build environment. Every
  renamed symbol/lib-id/net strin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
Parts:
- U1_1, U1_2, U1_3, U1_4: symbol Jayne_MSPM0G3507_RGZ -> Observer_MSPM0G3507_RGZ
- U2_1, U2_2, U2_3, U2_4: symbol Jayne_SLB9670_TPM -> Observer_SLB9670_TPM
- U3_1, U3_2, U3_3, U3_4: symbol Jayne_ISOW1044BDFMR -> Observer_ISOW1044BDFMR
Changed lines of the file:
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@@
   (title_block
     (title "CAN-PERIPH-GW-1 -- TPM-secured Dual-Isolated-Bus (CAN-FD + RS-485) Peripheral Gateway (4x stack)") (date "2026-07-26") (rev "1") (company "Griffing Technology LLC")
-    (comment 1 "Serenity UAV -- MAL-CAN-PERIPH-GW-PCB -- standalone board, not a PocketBeagle 2 Industrial cape")
+    (comment 1 "Serenity UAV -- SKIPPER-CAN-PERIPH-GW-PCB -- standalone board, not a PocketBeagle 2 Industrial cape")
     (comment 2 "Copyright 2026 Steve Griffing PE(CSE) CISSP-ISSEP CPP | Griffing Technology LLC")
     (comment 3 "License: CC BY 4.0  |  creativecommons.org/licenses/by/4.0")
@@
     (effects (font (size 1.27 1.27)))
 )
-  (symbol (lib_id "Jayne_MSPM0G3507_RGZ") (at 110.49 165.10 0)
+  (symbol (lib_id "Observer_MSPM0G3507_RGZ") (at 110.49 165.10 0)
     (unit 1) (exclude_from_sim no) (in_bom yes) (on_board yes) (dnp no)
     (property "Reference" "U1_1" (at 110.49 163.10 0)
@@
     (property "Intersheet References" "${INTERSHEET_REFS}" (at 154.92 141.19 0)
       (effects (font (size 1.016 1.016)) (hide yes))))
-  (symbol (lib_id "Jayne_SLB9670_TPM") (at 110.49 229.87 0)
+  (symbol (lib_id "Observer_SLB9670_TPM") (at 110.49 229.87 0)
     (unit 1) (exclude_from_sim no) (in_bom yes) (on_board yes) (dnp no)
     (property "Reference" "U2_1" (at 110.49 227.87 0)
@@
     (property "Intersheet References" "${INTERSHEET_REFS}" (at 148.81 232.00 0)
       (effects (font (size 1.016 1.016)) (hide yes))))
-  (symbol (lib_id "Jayne_ISOW1044BDFMR") (at 110.49 330.20 0)
+  (symbol (lib_id "Observer_ISOW1044BDFMR") (at 110.49 330.20 0)
     (unit 1) (exclude_from_sim no) (in_bom yes) (on_board yes) (dnp no)
     (property "Reference" "U3_1" (at 110.49 328.20 0)
@@
     (effects (font (size 1.27 1.27)))
 )
-  (symbol (lib_id "Jayne_MSPM0G3507_RGZ") (at 330.20 165.10 0)
+  (symbol (lib_id "Observer_MSPM0G3507_RGZ") (at 330.20 165.10 0)
     (unit 1) (exclude_from_sim no) (in_bom yes) (on_board yes) (dnp no)
     (property "Reference" "U1_2" (at 330.20 163.10 0)
@@
     (property "Intersheet References" "${INTERSHEET_REFS}" (at 374.92 141.19 0)
       (effects (font (size 1.016 1.016)) (hide yes))))
-  (symbol (lib_id "Jayne_SLB9670_TPM") (at 330.20 229.87 0)
+  (symbol (lib_id "Observer_SLB9670_TPM") (at 330.20 229.87 0)
     (unit 1) (exclude_from_sim no) (in_bom yes) (on_board yes) (dnp no)
     (property "Reference" "U2_2" (at 330.20 227.87 0)
@@
     (property "Intersheet References" "${INTERSHEET_REFS}" (at 368.81 232.00 0)
       (effects (font (size 1.016 1.016)) (hide yes))))
-  (symbol (lib_id "Jayne_ISOW1044BDFMR") (at 330.20 330.20 0)
+  (symbol (lib_id "Observer_ISOW1044BDFMR") (at 330.20 330.20 0)
     (unit 1) (exclude_from_sim no) (in_bom yes) (on_board yes) (dnp no)
     (property "Reference" "U3_2" (at 330.20 328.20 0)
@@
     (effects (font (size 1.27 1.27)))
 )
-  (symbol (lib_id "Jayne_MSPM0G3507_RGZ") (at 549.91 165.10 0)
+  (symbol (lib_id "Observer_MSPM0G3507_RGZ") (at 549.91 165.10 0)
     (unit 1) (exclude_from_sim no) (in_bom yes) (on_board yes) (dnp no)
     (property "Reference" "U1_3" (at 549.91 163.10 0)
@@
     (property "Intersheet References" "${INTERSHEET_REFS}" (at 594.92 141.19 0)
       (effects (font (size 1.016 1.016)) (hide yes))))
-  (symbol (lib_id "Jayne_SLB9670_TPM") (at 549.91 229.87 0)
+  (symbol (lib_id "Observer_SLB9670_TPM") (at 549.91 229.87 0)
     (unit 1) (exclude_from_sim no) (in_bom yes) (on_board yes) (dnp no)
     (property "Reference" "U2_3" (at 549.91 227.87 0)
@@
     (property "Intersheet References" "${INTERSHEET_REFS}" (at 588.81 232.00 0)
       (effects (font (size 1.016 1.016)) (hide yes))))
-  (symbol (lib_id "Jayne_ISOW1044BDFMR") (at 549.91 330.20 0)
+  (symbol (lib_id "Observer_ISOW1044BDFMR") (at 549.91 330.20 0)
     (unit 1) (exclude_from_sim no) (in_bom yes) (on_board yes) (dnp no)
     (property "Reference" "U3_3" (at 549.91 328.20 0)
@@
     (effects (font (size 1.27 1.27)))
 )
-  (symbol (lib_id "Jayne_MSPM0G3507_RGZ") (at 769.62 165.10 0)
+  (symbol (lib_id "Observer_MSPM0G3507_RGZ") (at 769.62 165.10 0)
     (unit 1) (exclude_from_sim no) (in_bom yes) (on_board yes) (dnp no)
     (property "Reference" "U1_4" (at 769.62 163.10 0)
@@
     (property "Intersheet References" "${INTERSHEET_REFS}" (at 814.92 141.19 0)
       (effects (font (size 1.016 1.016)) (hide yes))))
-  (symbol (lib_id "Jayne_SLB9670_TPM") (at 769.62 229.87 0)
+  (symbol (lib_id "Observer_SLB9670_TPM") (at 769.62 229.87 0)
     (unit 1) (exclude_from_sim no) (in_bom yes) (on_board yes) (dnp no)
     (property "Reference" "U2_4" (at 769.62 227.87 0)
@@
     (property "Intersheet References" "${INTERSHEET_REFS}" (at 808.81 232.00 0)
       (effects (font (size 1.016 1.016)) (hide yes))))
-  (symbol (lib_id "Jayne_ISOW1044BDFMR") (at 769.62 330.20 0)
+  (symbol (lib_id "Observer_ISOW1044BDFMR") (at 769.62 330.20 0)
     (unit 1) (exclude_from_sim no) (in_bom yes) (on_board yes) (dnp no)
     (property "Reference" "U3_4" (at 769.62 328.20 0)

Commit message: Migrate fleet TPM from Infineon SLB9670 to SLB9672
Replaces every active reference to the SLB9670 TPM with SLB9672 across
KiCad symbols/schematics/PCBs/netlists, generator scripts, firmware
device-tree overlays, and documentation (REFERENCES.md, WBS/TODO,
current-specification, graphical build guide). Archived files, frozen
revision snapshots, and the old datasheet PDF are left untouched.

- Added avionics/datasheets/SLB_9672XU20_Infineon.pdf (Infineon DS Rev
  1.3, 2024-11-18) and a new clean-room symbol/pinmap
  (Observer_SLB9672_TPM.kicad_sym, SLB9672XU2_0_pinmap.csv), replacing
  the superseded SLB9670 symbol/pinmap.
- Verified the physical footprint is unchanged (5x5mm body, 0.5mm
  pitch, 32-pin QFN, 3.6x3.6mm exposed pad per both datasheets), so the
  existing Package_DFN_QFN:QFN-32-1EP_5x5mm_P0.5mm_EP3.45x3.45mm
  footprint was reused as-is. Pin *functions* do differ (SLB9672 makes
  pins 1/14/22 the mandatory VDD pins vs 8/22 on SLB9670; pin 6 is now a
  true no-connect instead of GPIO; pins 3/4/7 are GPIO_00/01/02 instead
  of NCI/NCI/PP) -- the new symbol and every net-map/pinmap that lists
  pin functions reflect the corrected pinout.
- Populated the corrected component into Observer, Commo, Flight
  Engineer, and CAN-PERIPH-GW-1's schematics (lib_symbol block +
  instances) and into every board's PCB Value/property text. Pilot's
  and XO's own independently-authored inline TPM symbols were text-
  renamed only, preserving their pre-existing (and separately tracked)
  wrong-pin-number defect -- out of scope for this swap.
- Firmware: infineon,slb9670 -> infineon,slb9672 compatible string and
  tpm_slb9670: -> tpm_slb9672: node label in both active cape DTS
  overlays.
- REFERENCES.md REF-SENSOR-011 updated in place with validated Infineon
  URLs; new open items logged for (a) re-running kicad-cli ERC/DRC
  (unavailable in this environment) and (b) a newly-found, unrelated
  pre-existing footprint-mismatch defect on XO's placed TPM.
- PROJECT_INDEX.md / t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
Parts:
- U2_1, U2_2, U2_3, U2_4: value Infineon SLB9670 TPM2.0 -> Infineon SLB9672 TPM2.0; symbol Observer_SLB9670_TPM -> Observer_SLB9672_TPM
Changed lines of the file:
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@@
     (property "Intersheet References" "${INTERSHEET_REFS}" (at 154.92 141.19 0)
       (effects (font (size 1.016 1.016)) (hide yes))))
-  (symbol (lib_id "Observer_SLB9670_TPM") (at 110.49 229.87 0)
+  (symbol (lib_id "Observer_SLB9672_TPM") (at 110.49 229.87 0)
     (unit 1) (exclude_from_sim no) (in_bom yes) (on_board yes) (dnp no)
     (property "Reference" "U2_1" (at 110.49 227.87 0)
       (effects (font (size 1.27 1.27))))
-    (property "Value" "Infineon SLB9670 TPM2.0" (at 110.49 231.87 0)
+    (property "Value" "Infineon SLB9672 TPM2.0" (at 110.49 231.87 0)
       (effects (font (size 1.27 1.27))))
     (property "Footprint" "Package_DFN_QFN:QFN-32-1EP_5x5mm_P0.5mm_EP3.45x3.45mm" (at 0 0 0)
@@
     (property "Intersheet References" "${INTERSHEET_REFS}" (at 374.92 141.19 0)
       (effects (font (size 1.016 1.016)) (hide yes))))
-  (symbol (lib_id "Observer_SLB9670_TPM") (at 330.20 229.87 0)
+  (symbol (lib_id "Observer_SLB9672_TPM") (at 330.20 229.87 0)
     (unit 1) (exclude_from_sim no) (in_bom yes) (on_board yes) (dnp no)
     (property "Reference" "U2_2" (at 330.20 227.87 0)
       (effects (font (size 1.27 1.27))))
-    (property "Value" "Infineon SLB9670 TPM2.0" (at 330.20 231.87 0)
+    (property "Value" "Infineon SLB9672 TPM2.0" (at 330.20 231.87 0)
       (effects (font (size 1.27 1.27))))
     (property "Footprint" "Package_DFN_QFN:QFN-32-1EP_5x5mm_P0.5mm_EP3.45x3.45mm" (at 0 0 0)
@@
     (property "Intersheet References" "${INTERSHEET_REFS}" (at 594.92 141.19 0)
       (effects (font (size 1.016 1.016)) (hide yes))))
-  (symbol (lib_id "Observer_SLB9670_TPM") (at 549.91 229.87 0)
+  (symbol (lib_id "Observer_SLB9672_TPM") (at 549.91 229.87 0)
     (unit 1) (exclude_from_sim no) (in_bom yes) (on_board yes) (dnp no)
     (property "Reference" "U2_3" (at 549.91 227.87 0)
       (effects (font (size 1.27 1.27))))
-    (property "Value" "Infineon SLB9670 TPM2.0" (at 549.91 231.87 0)
+    (property "Value" "Infineon SLB9672 TPM2.0" (at 549.91 231.87 0)
       (effects (font (size 1.27 1.27))))
     (property "Footprint" "Package_DFN_QFN:QFN-32-1EP_5x5mm_P0.5mm_EP3.45x3.45mm" (at 0 0 0)
@@
     (property "Intersheet References" "${INTERSHEET_REFS}" (at 814.92 141.19 0)
       (effects (font (size 1.016 1.016)) (hide yes))))
-  (symbol (lib_id "Observer_SLB9670_TPM") (at 769.62 229.87 0)
+  (symbol (lib_id "Observer_SLB9672_TPM") (at 769.62 229.87 0)
     (unit 1) (exclude_from_sim no) (in_bom yes) (on_board yes) (dnp no)
     (property "Reference" "U2_4" (at 769.62 227.87 0)
       (effects (font (size 1.27 1.27))))
-    (property "Value" "Infineon SLB9670 TPM2.0" (at 769.62 231.87 0)
+    (property "Value" "Infineon SLB9672 TPM2.0" (at 769.62 231.87 0)
       (effects (font (size 1.27 1.27))))
     (property "Footprint" "Package_DFN_QFN:QFN-32-1EP_5x5mm_P0.5mm_EP3.45x3.45mm" (at 0 0 0)
