File: avionics/kicad/CAN-PERIPH-GW-1/kicads/CAN-PERIPH-GW-1.kicad_pcb (KiCad board)
At the start: 2 copper layers, 200.5 x 28 mm, 83 parts, among them U1_1 MSPM0G3507, U1_2 MSPM0G3507, U1_3 MSPM0G3507, U1_4 MSPM0G3507, U2_1 SLB9670, U2_2 SLB9670, U2_3 SLB9670, U2_4 SLB9670, U3_1 ISOW1044BDFMR, U3_2 ISOW1044BDFMR, U3_3 ISOW1044BDFMR, U3_4 ISOW1044BDFMR, U4_1 ISOW1412, U4_2 ISOW1412, U4_3 ISOW1412, U4_4 ISOW1412

Commit message: CAN-PERIPH-GW-1: add stack orientation option; Emma: TPM binds to PB2 host via shared SPI1, not a dedicated header
CAN-PERIPH-GW-1:
- gen_can_periph_gw_pcb.py: new STACK_ORIENTATION setting ("END_TO_END",
  default, tiles along X / short-side-to-short-side, current behavior;
  "SIDE_BY_SIDE" tiles along Y / long-side-to-long-side for a wider,
  shorter board). Both pitches verified via sandboxed N_STACKS=4 dry runs
  (0 shorts/clearance/courtyard from placement).
- Synced ATTRIBUTION_POS to the position the user hand-corrected on the
  live board (the generator's first guess ran off the board corner).

Emma:
- TPM no longer gets a dedicated J_TPM header. Per design intent, the TPM
  provides the last/first cryptographic signature for radio messages Emma
  transmits and forwards, and binds to whichever PB2-I host Emma is
  stacked on (supporting self-sufficient, non-Serenity deployments) --
  so it taps the SPI1_CS_TPM/SPI1_CLK/SPI1_MOSI/SPI1_MISO +
  TPM_IRQN/TPM_RSTN nets already reserved on Emma's own P1/P2 trunk
  instead. Removed J_TPM/lib_symbol_j_tpm_emma() from the schematic and
  from inject_emma_tpm.py; retargeted the TPM/R_TPM_RST_EMMA footprints on
  the PCB to the corrected net names. ERC/DRC 0 hard after the rewire.

Co-Authored-By: Claude Sonnet 5 <noreply@anthropic.com>
Parts:
- moved C_ISO1_1 86.8 mm to (57.1, 110.1)
- moved C_ISO1_3 86.8 mm to (157.1, 110.1)
- moved C_MCU1_4 86.8 mm to (206.7, 105.1)
- moved C_OUT 86.8 mm to (47.1, 110.1)
- moved C_RS1_4 86.8 mm to (212.7, 110.6)
- moved C_TPM1_2 86.8 mm to (130.6, 106.6)
- moved C_TPM2_2 86.8 mm to (132.1, 106.6)
- moved C_VCORE_4 86.8 mm to (213.7, 107.1)
- moved J_CAN_IN 86.8 mm to (58.1, 100.1)
- moved J_ENC_4 86.8 mm to (203.6, 114.1)
- moved J_FLEX_3 86.8 mm to (179.7, 114.1)
- moved J_FLEX_4 86.8 mm to (229.7, 114.1)
- moved J_SWD_2 86.8 mm to (137.6, 114.0)
- moved R_FBB 86.8 mm to (60.7, 107.6)
- moved R_NRST_4 86.8 mm to (207.2, 106.1)
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