File: avionics/kicad/CAN-PERIPH-GW-1/kicads/CAN-PERIPH-GW-1.kicad_pcb (KiCad board)
At the start: 2 copper layers, 200.5 x 28 mm, 83 parts, among them U1_1 MSPM0G3507, U1_2 MSPM0G3507, U1_3 MSPM0G3507, U1_4 MSPM0G3507, U2_1 SLB9670, U2_2 SLB9670, U2_3 SLB9670, U2_4 SLB9670, U3_1 ISOW1044BDFMR, U3_2 ISOW1044BDFMR, U3_3 ISOW1044BDFMR, U3_4 ISOW1044BDFMR, U4_1 ISOW1412, U4_2 ISOW1412, U4_3 ISOW1412, U4_4 ISOW1412

Commit message: commited
Parts:
- removed C_ISO1_3, C_ISO1_4, C_MCU1_3, C_MCU1_4, C_RS1_3, C_RS1_4, C_RS2_3, C_RS2_4, C_TPM1_3, C_TPM1_4: 100nF, Capacitor_SMD:C_0402_1005Metric
- removed C_ISO2_3, C_ISO2_4, C_TPM2_3, C_TPM2_4, C_VCORE_3, C_VCORE_4: 1uF, Capacitor_SMD:C_0402_1005Metric
- removed J_ENC_3, J_ENC_4: AK7455 pigtail, Serenity-Custom:Pigtail_7W_DirectSolder
- removed J_FLEX_3, J_FLEX_4: UART/TTL/PWM/BSHOT, Connector_PinHeader_2.54mm:PinHeader_1x08_P2.54mm_Vertical
- removed J_SWD_3, J_SWD_4: SWD, Connector_JST:JST_GH_BM04B-GHS-TBT_1x04-1MP_P1.25mm_Vertical
- removed R_NRST_3, R_NRST_4, R_TPM_RST_3, R_TPM_RST_4: 10k, Resistor_SMD:R_0402_1005Metric
- removed U1_3, U1_4: MSPM0G3507, Package_DFN_QFN:QFN-48-1EP_7x7mm_P0.5mm_EP5.15x5.15mm
- removed U2_3, U2_4: SLB9670, Package_DFN_QFN:QFN-32-1EP_5x5mm_P0.5mm_EP3.45x3.45mm
- removed U3_3, U3_4: ISOW1044BDFMR, Package_SO:SOIC-20W_7.5x12.8mm_P1.27mm
- removed U4_3, U4_4: ISOW1412, Package_SO:SOIC-20W_7.5x12.8mm_P1.27mm
- U1_2, U2_2: moved to F.Cu
- moved J_SWD_2 53.0 mm to (86.0, 102.0)
- moved R_TPM_RST_2 45.0 mm to (90.0, 95.5)
- moved J_SWD_1 40.8 mm to (48.5, 102.5)
- moved C_TPM1_2 40.7 mm to (91.5, 95.5)
- moved C_TPM2_2 40.7 mm to (93.0, 95.5)
- moved C_RS2_2 38.0 mm to (91.5, 93.0), turned to 90 degrees
- moved U4_2 35.5 mm to (99.5, 99.0), turned to 180 degrees
- moved U2_2 33.2 mm to (85.3, 95.0), turned to 0 degrees
- moved C_ISO2_2 32.9 mm to (93.0, 93.0), turned to 90 degrees
- moved J_FLEX_2 29.7 mm to (100.6, 108.0)
- moved SJ2 26.7 mm to (63.5, 100.5)
- moved C_VCORE_2 23.0 mm to (92.5, 98.0)
- moved C_RS1_2 22.3 mm to (92.5, 101.0)
- moved U1_2 21.7 mm to (99.1, 95.9), turned to 0 degrees
- moved R_485TERM 20.9 mm to (65.8, 100.5), turned to -90 degrees
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Routing:
- net FLEX_PWM_IO_2: track 5.00 -> 21.2 mm, vias 0 -> 3
- net ENC_ERROR_2: track 16.1 -> 0.00 mm, vias 3 -> 0
- net RS485_DE_1: track 3.97 -> 0.00 mm
- net ISO_5V_CAN_2: track 36.4 -> 40.4 mm
- net +3V3: track 632.3 -> 635.0 mm
- net CANTERM_MID: track 2.72 -> 0.00 mm
Other:
- board size 200.5 x 28 mm -> 64.3 x 19.5 mm
- board text added: "TPM-Secured CAN-FD/RS-485 Gateway CC BY 4.0 — July 2026 Griffing Technology LLC github.com/Stab-Rabbit-Coding"
- board text removed: "TPM-Secured CAN-FD/RS-485 Gateway For the PocketBeagle2 fleet CC BY 4.0 — July 2026 Steve Griffing PE(CSE), CISSP-ISSEP, CPP Griffing Technology LLC github.com/Stab-Rabbit-Coding"
