File: avionics/kicad/CAN-PERIPH-GW-1/kicads/CAN-PERIPH-GW-1.kicad_pcb (KiCad board)
At the start: 2 copper layers, 64.3 x 19.5 mm, 49 parts, among them U1_1 MSPM0G3507, U1_2 MSPM0G3507, U2_1 SLB9670, U2_2 SLB9670, U3_1 ISOW1044BDFMR, U3_2 ISOW1044BDFMR, U4_1 ISOW1412, U4_2 ISOW1412

Commit message: Migrate fleet TPM from Infineon SLB9670 to SLB9672
Replaces every active reference to the SLB9670 TPM with SLB9672 across
KiCad symbols/schematics/PCBs/netlists, generator scripts, firmware
device-tree overlays, and documentation (REFERENCES.md, WBS/TODO,
current-specification, graphical build guide). Archived files, frozen
revision snapshots, and the old datasheet PDF are left untouched.

- Added avionics/datasheets/SLB_9672XU20_Infineon.pdf (Infineon DS Rev
  1.3, 2024-11-18) and a new clean-room symbol/pinmap
  (Observer_SLB9672_TPM.kicad_sym, SLB9672XU2_0_pinmap.csv), replacing
  the superseded SLB9670 symbol/pinmap.
- Verified the physical footprint is unchanged (5x5mm body, 0.5mm
  pitch, 32-pin QFN, 3.6x3.6mm exposed pad per both datasheets), so the
  existing Package_DFN_QFN:QFN-32-1EP_5x5mm_P0.5mm_EP3.45x3.45mm
  footprint was reused as-is. Pin *functions* do differ (SLB9672 makes
  pins 1/14/22 the mandatory VDD pins vs 8/22 on SLB9670; pin 6 is now a
  true no-connect instead of GPIO; pins 3/4/7 are GPIO_00/01/02 instead
  of NCI/NCI/PP) -- the new symbol and every net-map/pinmap that lists
  pin functions reflect the corrected pinout.
- Populated the corrected component into Observer, Commo, Flight
  Engineer, and CAN-PERIPH-GW-1's schematics (lib_symbol block +
  instances) and into every board's PCB Value/property text. Pilot's
  and XO's own independently-authored inline TPM symbols were text-
  renamed only, preserving their pre-existing (and separately tracked)
  wrong-pin-number defect -- out of scope for this swap.
- Firmware: infineon,slb9670 -> infineon,slb9672 compatible string and
  tpm_slb9670: -> tpm_slb9672: node label in both active cape DTS
  overlays.
- REFERENCES.md REF-SENSOR-011 updated in place with validated Infineon
  URLs; new open items logged for (a) re-running kicad-cli ERC/DRC
  (unavailable in this environment) and (b) a newly-found, unrelated
  pre-existing footprint-mismatch defect on XO's placed TPM.
- PROJECT_INDEX.md / t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
Parts:
- U2_1, U2_2: value SLB9670 -> SLB9672
Changed lines of the file:
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@@
 			)
 		)
-		(property "Value" "SLB9670"
+		(property "Value" "SLB9672"
 			(at 0 3.83 0)
 			(layer "F.Fab")
@@
 			)
 		)
-		(property "Value" "SLB9670"
+		(property "Value" "SLB9672"
 			(at 0 -3.83 0)
 			(layer "B.Fab")
