File: avionics/kicad/Observer/kicads/Observer.kicad_pcb (KiCad board)
At the start: 4 copper layers, 69.8 x 56.4 mm, 63 parts, among them Q1 AO3400 logic-level N-MOSFET, T1 Wurth 749010012A, T1_CMC1 SRF2012-100Y, T1_CMC2 SRF2012-100Y, T1_D1 PRTR5V0U2X, T1_D2 PRTR5V0U2X, T2 Wurth 749010012A, T2_CMC1 SRF2012-100Y, T2_CMC2 SRF2012-100Y, T2_D1 PRTR5V0U2X, T2_D2 PRTR5V0U2X, U2 Microchip KSZ9477, U3 TI MSPM0G3519-Q1, U4 TI ISOW1044BDFMR, U5 Infineon SLB 9672AU2.0, Y1 25MHz

Commit message: Apply the exposed-pad corrections in place instead of rebuilding footprints
Rebuilding U3/U5 and the gateway TPMs from the KiCad library discarded
whatever the board author had tuned on those placed instances (mask
margins, pad clearance overrides, zone connections). On Observer that
turned a no-op land correction into ~180 new clearance /
solder_mask_bridge / shorting violations.

The same-pad-count swaps now edit the placed block directly, changing
only the library reference, the Value and the thermal pad size (plus the
exposed pad's net where it had none). Observer is back to its baseline
DRC of 289 with the RGZ0048F 4.1 mm pad and the SLB9672 3.6 mm pad
correctly applied.

Also corrects the DRC figures recorded earlier: they had been measured on
copies taken outside the project directory, so the sibling .kicad_pro
custom rules and netclasses were missing and the numbers were wrong.
Measured in place: Observer 289 -> 289, gateway 743 -> 804 (+61
clearance in the MCU area, pending the manual re-route).

Co-Authored-By: Claude Opus 5 <noreply@anthropic.com>
Parts:
- J_CAM_DS: footprint Observer:DS_Camera_9P -> Jayne:DS_Camera_9P
- J_LASER_DS: footprint Observer:DS_Laser_2P -> Jayne:DS_Laser_2P
- J_TOF_DS: footprint Observer:DS_ToF_4P -> Jayne:DS_ToF_4P
- T1, T2: footprint Observer:Wurth_749010012A_10-100BASE-TX -> Jayne:Wurth_749010012A_10-100BASE-TX
- U2: footprint Observer:TQFP-128-1EP_KSZ9477_14x14mm_P0.4mm_EP10x10 -> Jayne:TQFP-128-1EP_KSZ9477_14x14mm_P0.4mm_EP10x10
- U_SOM: footprint Observer:phyCORE-AM62x_PCM071_2xBTH-060 -> Jayne:phyCORE-AM62x_PCM071_2xBTH-060
Other:
- board text added: "Jayne Rev - (design exploration)"
- board text removed: "Observer Rev - (design exploration)"

Commit message: docs(avionics): Wurth usage notice + uncrewed-only statement on 5 boards; catalogue REF-SENSOR-022..040
Owner decision 2026-09-26: retain the Wurth parts. The Wurth datasheet
usage notice is quoted verbatim [REF-SENSOR-028: Wurth 749010012A data
sheet rev 004.000 p.1] with an 'intended for use only on uncrewed
aircraft' statement in each Wurth-bearing board's .md, as a schematic
text item and PCB Cmts.User text, and in title-block comments 8/9
(tools/add_board_notices.py, idempotent). ERC/DRC/parity counts
unchanged on all five boards (kicad-cli 9.0.2).

REFERENCES.md: REF-SENSOR-022/023/025-030/033/038/040 were cited by
board schematics and generator scripts but never catalogued; entries
added with URLs validated 2026-09-26, unreachable ones marked
'requires verification'.

AI-authored: Claude Opus 5.5 (Anthropic).

Co-Authored-By: Claude Opus 5.5 <noreply@anthropic.com>
Other:
- board text added: "WÜRTH ELEKTRONIK USAGE NOTICE (verbatim, 749010012A data sheet rev 004.000 p.1; applies to Würth parts on this board: 749010012A): This electronic component has been designed and developed for usage in general electronic equipment only. This product is not authorized for use in equipment where a higher safety standard and reliability standard is especially required or where a failure of the produ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"
Changed lines of the file:
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@@
 		(comment 3 "1.0 × 2.75 in (25.4 × 69.85 mm) 4-layer FR4, DOUBLE-SIDED, EMI-hardened — see gen_Jayne_pcb.py docstring")
 		(comment 4 "SoM end-state: real footprints (PCM-071 2xBTH-060, TQFP-128-EP, VQFN, SOIC-20W); see gen_Jayne_carrier_pcb.py")
+		(comment 8 "Wurth parts (749010012A): see Wurth usage notice on this page [USAGE-NOTICE-2026-09-26]")
+		(comment 9 "Intended for use ONLY on uncrewed aircraft")
 	)
 	(layers
@@
 	)
 	(embedded_fonts no)
+	(gr_text "WÜRTH ELEKTRONIK USAGE NOTICE (verbatim, 749010012A data sheet rev 004.000 p.1; applies to Würth\nparts on this board: 749010012A):\n\nThis electronic component has been designed and developed for usage in general electronic equipment\nonly. This product is not authorized for use in equipment where a higher safety standard and\nreliability standard is especially required or where a failure of the product is reasonably expected\nto cause severe personal injury or death, unless the parties have executed an agreement specifically\ngoverning such use. Moreover Würth Elektronik eiSos GmbH & Co KG products are neither designed nor\nintended for use in areas such as military, aerospace, aviation, nuclear control, submarine,\ntransportation, transportation signal, disaster prevention, medical, public information network\netc.. Würth Elektronik eiSos GmbH & Co KG must be informed about the intent of such usage before the\ndesign-in stage. In addition, sufficient reliability evaluation checks for safety must be performed\non every electronic component which is used in electrical circuits that require high safety and\nreliability functions or performance.\n\nINTENDED USE: The Serenity-UAV avionics, including this board, are intended for use only on uncrewed\naircraft.\n[USAGE-NOTICE-2026-09-26]"
+		(at 248.74 123.17 0)
+		(layer "Cmts.User")
+		(effects (font (size 0.8 0.8) (thickness 0.1)) (justify left top))
+	)
 )

Commit message: fix(avionics): TLV62569 -> TLV62569PDRLR and TLV75725 -> TLV75725PDRVR package swaps; regulator circuit fixes; stale-component cleanup
Owner-approved swaps (2026-09-26, avionics/WBS.md U7.1e) using the
datasheet-verified SecureControllers library via ${SECURE_CONTROLLERS_LIB}:
- CAN-PERIPH-GW-1 U_REG_3V3, Observer U_REG_3V3/U_REG_1V2, Flight
  Engineer U_REG_3V3_H -> TLV62569PDRLR (SOT-563, 1.6 x 1.6 mm).
  Pins remapped by name; the old symbols had FB/PG swapped (gateway,
  Observer) or sat on a 3-pad SOT-23 (Flight Engineer).
- Observer U_REG_2V5 -> TLV75725PDRVR (WSON-6 2x2, EP to GND).
- Feedback dividers per TLV62569 Sec. 8.2.2.2 Eq. 2 (VFB 0.6 V):
  gateway 10k/20k (0.9 V!) -> 453k/100k = 3.318 V; Observer placeholders
  -> 453k/100k (3V3) and 100k/100k (1V2).
- Flight Engineer: EN was tied to its own 3V3 output and FB straight to
  +3V3 (would regulate at 0.6 V); EN -> +5V, added R_H_FBT 453k /
  R_H_FBB 100k. Parity 2 -> 0, ERC 0.
- tools/kicad_prune_stale.py: parity-driven removal of stale electrical
  footprints and only the copper they orphan; mounting holes are marked
  board_only + renumbered (Commo parity 93 -> 86, Observer 21 -> 17).
- New tools kicad_relink.py / kicad_add_part.py / kicad_set_value.py;
  SecureControllers entries added to every board's lib tables.

Sources: TI TLV62569 (SLVSDG1C) Pin Functions, Sec. 8.2.2.2; TI TLV757P
Fig. 4-3, Pin Functions, DRV0006A.

AI-authored: Claude Opus 5.5 (Anthropic).

Co-Authored-By: Claude Opus 5.5 <noreply@anthropic.com>
Parts:
- R_FB1B, R_FB3B: value R_fbbot -> 100k 1%
- R_FB1T: value R_fbtop -> 100k 1%
- R_FB3T: value R_fbtop -> 453k 1%
- U_REG_1V2: value TLV62569 -> +1V2 -> TLV62569PDRLR; footprint Package_TO_SOT_SMD:SOT-23-6 -> Package_TO_SOT_SMD:SOT-563
- U_REG_2V5: value TLV75725 -> +2V5 -> TLV75725PDRVR; footprint Package_TO_SOT_SMD:SOT-23-5 -> Package_SON:WSON-6-1EP_2x2mm_P0.65mm_EP1x1.6mm
- U_REG_3V3: value TLV62569 -> +3V3 -> TLV62569PDRLR; footprint Package_TO_SOT_SMD:SOT-23-6 -> Package_TO_SOT_SMD:SOT-563
Connections:
- U_REG_1V2 pad 1: +5V -> U_REG_1V2_FB
- U_REG_1V2 pad 3: U_REG_1V2_SW -> +5V
- U_REG_1V2 pad 4: +5V -> U_REG_1V2_SW
- U_REG_1V2 pad 5: U_REG_1V2_FB -> +5V
- U_REG_2V5 pad 1: +3V3 -> +2V5
- U_REG_2V5 pad 2: GND -> (no net)
- U_REG_2V5 pad 3: +3V3 -> GND
- U_REG_2V5 pad 4: (no net) -> +3V3
- U_REG_2V5 pad 5: +2V5 -> (no net)
- U_REG_3V3 pad 1: +5V -> U_REG_3V3_FB
- U_REG_3V3 pad 3: U_REG_3V3_SW -> +5V
- U_REG_3V3 pad 4: +5V -> U_REG_3V3_SW
- U_REG_3V3 pad 5: U_REG_3V3_FB -> +5V

Commit message: fix(avionics): PRTR5V0U2X package/pinout fix on all 12 instances, 5 boards
Owner-approved 2026-09-26 (avionics/WBS.md U7.2). Per Nexperia
PRTR5V0U2X datasheet Table 2 (SOT143B: 1=GND, 2=I/O1, 3=I/O2, 4=VCC),
relinked via tools/kicad_relink.py --rewire (same footprint position/
rotation preserved, only package + pin-to-net correspondence corrected):

- Pilot TVS-CAN, TVS-RS485; TACCO TVS-CAN, TVS-RS485; FlightEngineer
  D_I2C: straightforward SOT-363->SOT-143 swap with existing GND/VCC
  nets carried over unchanged (5 instances).
- Observer T1_D1/T1_D2/T2_D1/T2_D2 (Ethernet magnetics ESD) and D5
  (CAN-FD), Commo 'ANT TVS' and 'UART TVS': these had no VCC net at
  all in the original (wrong-package) design -- VCC tied to the local
  GND/PGND net as a conservative fallback (line-to-line and
  line-to-ground clamping preserved; the rail-clamp direction is
  inert). This is a judgment call, not a datasheet requirement --
  flagged for review, not a silent assumption (7 instances).

ERC unchanged (0/0/0/0/154-pre-existing) on all 5 boards; DRC/parity
flat or improved except one new courtyard-overlap warning on Pilot
(TVS-CAN vs C-IN1, mechanical only) left unresolved rather than guess
a nudge direction without full layout context.

AI-authored: Claude Sonnet 5 (Anthropic).

Co-Authored-By: Claude Sonnet 5 <noreply@anthropic.com>
Parts:
- D5: value PRTR5V0U2X (CAN) -> PRTR5V0U2X; footprint Package_TO_SOT_SMD:SOT-363_SC-70-6 -> Package_TO_SOT_SMD:SOT-143
- T1_D1, T1_D2, T2_D1, T2_D2: footprint Package_TO_SOT_SMD:SOT-363_SC-70-6 -> Package_TO_SOT_SMD:SOT-143
Connections:
- D5 pad 1: CANFD_H -> PGND
- D5 pad 2: CANFD_L -> CANFD_H
- D5 pad 3: PGND -> CANFD_L
- D5 pad 4: (no net) -> PGND
- T1_D1 pad 1: ETH_IN_TXP -> GND
- T1_D1 pad 2: ETH_IN_TXN -> ETH_IN_TXP
- T1_D1 pad 3: GND -> ETH_IN_TXN
- T1_D1 pad 4: (no net) -> GND
- T1_D2 pad 1: ETH_IN_RXP -> GND
- T1_D2 pad 2: ETH_IN_RXN -> ETH_IN_RXP
- T1_D2 pad 3: GND -> ETH_IN_RXN
- T1_D2 pad 4: (no net) -> GND
- T2_D1 pad 1: ETH_OUT_TXP -> GND
- T2_D1 pad 2: ETH_OUT_TXN -> ETH_OUT_TXP
- T2_D1 pad 3: GND -> ETH_OUT_TXN
- T2_D1 pad 4: (no net) -> GND
- T2_D2 pad 1: ETH_OUT_RXP -> GND
- T2_D2 pad 2: ETH_OUT_RXN -> ETH_OUT_RXP
- T2_D2 pad 3: GND -> ETH_OUT_RXN
- T2_D2 pad 4: (no net) -> GND
