File: avionics/kicad/XO/kicads/XO.kicad_pcb (KiCad board)
At the start: 4 copper layers, 55 x 35 mm, 43 parts, among them X2Y-CAN 4.7nF X2Y, X2Y-RS485 4.7nF X2Y

Commit message: Migrate fleet TPM from Infineon SLB9670 to SLB9672
Replaces every active reference to the SLB9670 TPM with SLB9672 across
KiCad symbols/schematics/PCBs/netlists, generator scripts, firmware
device-tree overlays, and documentation (REFERENCES.md, WBS/TODO,
current-specification, graphical build guide). Archived files, frozen
revision snapshots, and the old datasheet PDF are left untouched.

- Added avionics/datasheets/SLB_9672XU20_Infineon.pdf (Infineon DS Rev
  1.3, 2024-11-18) and a new clean-room symbol/pinmap
  (Observer_SLB9672_TPM.kicad_sym, SLB9672XU2_0_pinmap.csv), replacing
  the superseded SLB9670 symbol/pinmap.
- Verified the physical footprint is unchanged (5x5mm body, 0.5mm
  pitch, 32-pin QFN, 3.6x3.6mm exposed pad per both datasheets), so the
  existing Package_DFN_QFN:QFN-32-1EP_5x5mm_P0.5mm_EP3.45x3.45mm
  footprint was reused as-is. Pin *functions* do differ (SLB9672 makes
  pins 1/14/22 the mandatory VDD pins vs 8/22 on SLB9670; pin 6 is now a
  true no-connect instead of GPIO; pins 3/4/7 are GPIO_00/01/02 instead
  of NCI/NCI/PP) -- the new symbol and every net-map/pinmap that lists
  pin functions reflect the corrected pinout.
- Populated the corrected component into Observer, Commo, Flight
  Engineer, and CAN-PERIPH-GW-1's schematics (lib_symbol block +
  instances) and into every board's PCB Value/property text. Pilot's
  and XO's own independently-authored inline TPM symbols were text-
  renamed only, preserving their pre-existing (and separately tracked)
  wrong-pin-number defect -- out of scope for this swap.
- Firmware: infineon,slb9670 -> infineon,slb9672 compatible string and
  tpm_slb9670: -> tpm_slb9672: node label in both active cape DTS
  overlays.
- REFERENCES.md REF-SENSOR-011 updated in place with validated Infineon
  URLs; new open items logged for (a) re-running kicad-cli ERC/DRC
  (unavailable in this environment) and (b) a newly-found, unrelated
  pre-existing footprint-mismatch defect on XO's placed TPM.
- PROJECT_INDEX.md / t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
Parts:
- TPM: value SLB9670 -> SLB9672
Changed lines of the file:
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@@
 		(comment 2 "CC BY 4.0 creativecommons.org/licenses/by/4.0")
 		(comment 3 "PocketBeagle 2 Industrial (AM6254) expansion — 55x35mm 4L JLCPCB assembled")
-		(comment 4 "F: ISOW1044BDFMR CAN FD (iso) | ADM2795EBRWZ RS-485 (iso) | DS26LV31/32 1553 | ADIN1300+ISO7642 ETH (iso) | SLB9670 TPM2 | DRV8833 Winch | HX711 Load Cell | PCA9685 PWM | B: RFM95W LoRa | WL1837MOD WiFi/BT | ATF16V8BQL CPLD | W25Q128JV NOR | microSD log slot | EMI: SRF2012 CMC | PRTR5V0U2X TVS | SMAJ33CA 1553 | 742792512 FB")
+		(comment 4 "F: ISOW1044BDFMR CAN FD (iso) | ADM2795EBRWZ RS-485 (iso) | DS26LV31/32 1553 | ADIN1300+ISO7642 ETH (iso) | SLB9672 TPM2 | DRV8833 Winch | HX711 Load Cell | PCA9685 PWM | B: RFM95W LoRa | WL1837MOD WiFi/BT | ATF16V8BQL CPLD | W25Q128JV NOR | microSD log slot | EMI: SRF2012 CMC | PRTR5V0U2X TVS | SMAJ33CA 1553 | 742792512 FB")
 		(comment 5 "Hull: misubisu CC BY 4.0 | Nozzle: BamJr CC BY 4.0 | Firefly/Serenity fan-work, not officially licensed")
 	)
@@
 			)
 		)
-		(property "Value" "SLB9670"
+		(property "Value" "SLB9672"
 			(at -13 -0.84 0)
 			(layer "B.Fab")
@@
 			)
 		)
-		(pad "SLB9670" smd rect
+		(pad "SLB9672" smd rect
 			(at 0 0)
 			(size 2.65 2.65)

Commit message: feat(avionics): XO schematic-first rebuild to ERC 0; PCB placement in progress
Replaces XO's legacy schematic/PCB (169 sch refs vs 43 PCB footprints, 564
ERC violations) with a fresh generator pipeline matching Pilot's method
(gen_xo_sch.py / gen_xo_footprints.py / gen_xo_pcb.py), all datasheet-verified.

Fleet-shared blocks reused verbatim from Pilot (same parts, same pin tables,
_B_-suffixed nets per XO.md's own documented bus-sharing rationale): ISOW1044
CAN-FD, ISOW1412 RS-485, HI-1573 + PM-DB2791S MIL-STD-1553B (retires the
DS26LV31/32 + fake "SM-1553-11" defect, same fix as Pilot), SLB9672 TPM,
DP83825I Ethernet PHY x1 (single PHY per WBS.md "XO: 1x PHY (RMII0)" —
resolves a 3-way doc contradiction over whether XO has Ethernet in favor of
WBS's more authoritative, more recent "restored at Rev R" entry).

New XO-unique blocks, each pin table transcribed from its own OEM datasheet:
RFD900x SiK UHF radio, RFM95W LoRa module, WL1837MOD WiFi+BT (~14 of 100
balls carry a net this pass, a disclosed scope calibration), TPS63031 RF
buck-boost rail, W25Q128JV SPI NOR flash, ATF16V8BQL used as a logging
write-block interlock (JEDEC fuse map is a firmware deliverable, out of
scope here), three antenna filter/ESD chains, microSD slot.

Two part-number defects found in XO.md's own antenna-filter BOM and
corrected (flagged, not silently fixed): Johanson "0915LP15B0100E" and
"2450BP15B050E" do not exist in Johanson's catalog (confirmed against their
product listings) — substituted with the closest real parts found
(0915LP15B026E, 2450BP15E0100); NEEDS owner confirmation. XO.md's cited
microSD connector "Molex 503182-1852" could not be verified real —
replaced with the confirmed-real Connector_Card:microSD_HC_Molex_104031-0811
already in KiCad's system library. RCLAMP0502B's datasheet PDF could not be
obtained from any source tried; its footprint is a reasonable SOD-882
estimate, not pixel-verified — flagged for a real datasheet fetch.

ERC 0 confirmed (kicad-cli sch erc --sev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
Parts:
- removed 1553-DRV: DS26LV31, SOIC-16_3.9x9.9mm_P1.27mm
- removed 1553-RCV: DS26LV32, SOIC-16_3.9x9.9mm_P1.27mm
- removed the 1553-XFM at (146.0, 113.5)
- removed ? (x4): , MountingHole:MountingHole_2.7mm_M2.5
- removed CAN-FD: JST-GH-4P-CAN, JST_GH_4P
- removed the CAN-TR at (136.6, 111.8)
- removed the CMC-CAN at (143.8, 100.3)
- removed the ETH-PHY at (128.5, 97.2)
- removed the J-ETH at (124.6, 110.0)
- removed LOAD-ADC: HX711, SOIC-16_3.9x9.9mm_P1.27mm
- removed LOAD-CELL: JST-GH-4P-LOAD-CELL, JST_GH_4P
- removed Log microSD NON-X: microSD-Log, Connector_Card:microSD_HC_Molex_104031-0811
- removed MIL-1553: JST-GH-4P-1553, JST_GH_4P
- removed NAV-LIGHT PWM: 1x8-NavLight-PWM, Connector_PinHeader_2.54mm
- removed the NOR-FLASH at (169.1, 96.5)
- removed PB2-P1-TOP: PB2I-P1-2x18, 2x18_P1_Socket
- removed PB2-P2-TOP: PB2I-P2-2x18, 2x18_P2_Socket
- removed PWM-I2C: PCA9685, HTSSOP-28-1EP_4.4x9.7mm_P0.65mm_EP2.75x6.2mm
- removed the PWR-IN at (126.8, 116.0)
- removed RS-485: JST-GH-4P-RS485, JST_GH_4P
- removed SIK-TLM: JST-GH-3P-SiK, JST_GH_3P
- removed T-ETH1: 749010012A, ETH_XFMR_8P_5x3.5mm
- removed the TPM at (163.3, 96.7)
- removed TVS-1553: SMAJ33CA, DO-214AC_SMA
- removed the TVS-CAN at (154.2, 102.5)
- removed U-ISO-RX, U-ISO-TX: ISO7642FDWRR, SOIC-16W_7.5x10.3mm_P1.27mm
- removed VHF-XCVR: JST-GH-3P-XCVR-49MHZ, JST_GH_3P
- removed WIFI & BT: WL1837MOD, RF_Module
- removed WINCH: JST-GH-4P-WINCH, JST_GH_4P
- removed WINCH DRV: DRV8833, HTSSOP-16-1EP_4.4x5mm_P0.65mm_EP3.4x5mm
- removed the X2Y-CAN at (124.8, 103.0)
- removed uSD-X-Blk: ATF16V8BQL, PLCC-20
- added 1553-XCVR: HI-1573PCI, Package_DFN_QFN:QFN-44-1EP_7x7mm_P0.5mm_EP5.2x5.2mm, B.Cu at (170.8, 97.3)
- added 1553-XFM: PM-DB2791S, Serenity-Custom:Xfmr_1553_SMD_0.40in_8pin, F.Cu at (152.1, 111.6)
- added C-1553A: 100nF, Capacitor_SMD:C_0402_1005Metric, F.Cu at (301.0, 97.5)
- added C-1553B: 100nF, Capacitor_SMD:C_0402_1005Metric, F.Cu at (304.0, 97.5)
- added C-1553C: 10uF 6.3V X5R, Capacitor_SMD:C_0805_2012Metric, F.Cu at (217.0, 97.5)
- added C-1V8-IN: 1uF, Capacitor_SMD:C_0402_1005Metric, B.Cu at (126.5, 95.2)
- added C-1V8-OUT: 1uF, Capacitor_SMD:C_0402_1005Metric, B.Cu at (147.0, 116.0)
- added C-25M: 100nF, Capacitor_SMD:C_0402_1005Metric, F.Cu at (144.2, 117.0)
- added C-3V3-HF: 100nF, Capacitor_SMD:C_0402_1005Metric, B.Cu at (174.8, 114.6)
- added C-3V3-IN: 10uF 10V X5R, Capacitor_SMD:C_0805_2012Metric, F.Cu at (144.1, 94.5)
- added C-3V3-O1: 22uF 6.3V X5R, Capacitor_SMD:C_0805_2012Metric, B.Cu at (148.1, 113.5)
- added C-3V3-O2: 22uF 6.3V X5R, Capacitor_SMD:C_0805_2012Metric, B.Cu at (137.1, 94.8)
- added C-485-1: 10nF, Capacitor_SMD:C_0201_0603Metric, F.Cu at (140.8, 106.8)
- added C-485-2: 10uF 10V X5R, Capacitor_SMD:C_0805_2012Metric, B.Cu at (133.3, 94.8)
- added C-485-3: 100nF, Capacitor_SMD:C_0402_1005Metric, F.Cu at (295.0, 97.5)
- added C-485-4: 10nF, Capacitor_SMD:C_0201_0603Metric, F.Cu at (139.0, 106.8)
- added C-485-5: 10uF 10V X5R, Capacitor_SMD:C_0805_2012Metric, F.Cu at (214.0, 97.5)
- added C-485-6: 100nF, Capacitor_SMD:C_0402_1005Metric, F.Cu at (298.0, 97.5)
- added C-BS: 10nF 2kV, Capacitor_SMD:C_1808_4520Metric, B.Cu at (147.6, 103.4)
- added C-BST: 100nF, Capacitor_SMD:C_0402_1005Metric, F.Cu at (307.0, 97.5)
- added C-CAN1: 10nF, Capacitor_SMD:C_0201_0603Metric, F.Cu at (137.0, 106.7)
- added C-CAN2: 10uF 10V X5R, Capacitor_SMD:C_0805_2012Metric, F.Cu at (123.8, 94.5)
- added C-CAN3: 100nF, Capacitor_SMD:C_0402_1005Metric, F.Cu at (310.0, 97.5)
- added C-CAN4: 10nF, Capacitor_SMD:C_0201_0603Metric, F.Cu at (134.7, 106.8)
- added C-CAN5: 10uF 10V X5R, Capacitor_SMD:C_0805_2012Metric, B.Cu at (129.4, 94.8)
- added C-CAN6: 100nF, Capacitor_SMD:C_0402_1005Metric, B.Cu at (126.5, 93.9)
- added C-FLASH1: 100nF, Capacitor_SMD:C_0402_1005Metric, F.Cu at (313.0, 97.5)
- added C-IN1: 47uF 10V X5R, Capacitor_SMD:C_1210_3225Metric, F.Cu at (173.3, 109.9)
- added C-IN2: 10uF 10V X5R, Capacitor_SMD:C_0805_2012Metric, F.Cu at (220.0, 97.5)
- added C-IN3: 100nF, Capacitor_SMD:C_0402_1005Metric, F.Cu at (316.0, 97.5)
- added C-LORA1: 100nF, Capacitor_SMD:C_0402_1005Metric, F.Cu at (319.0, 97.5)
- added C-PHY-A1: 10nF, Capacitor_SMD:C_0201_0603Metric, B.Cu at (174.7, 116.5)
- added C-PHY-A2: 100nF, Capacitor_SMD:C_0402_1005Metric, F.Cu at (322.0, 97.5)
- added C-PHY-A3: 1uF, Capacitor_SMD:C_0402_1005Metric, F.Cu at (325.0, 97.5)
- added C-PHY-CRD1: 100nF, Capacitor_SMD:C_0402_1005Metric, F.Cu at (328.0, 97.5)
- added C-PHY-CRD2: 1uF, Capacitor_SMD:C_0402_1005Metric, F.Cu at (331.0, 97.5)
- added C-PHY-CTD1: 100nF, Capacitor_SMD:C_0402_1005Metric, F.Cu at (334.0, 97.5)
- added C-PHY-CTD2: 1uF, Capacitor_SMD:C_0402_1005Metric, F.Cu at (337.0, 97.5)
- added C-PLD1: 100nF, Capacitor_SMD:C_0402_1005Metric, F.Cu at (340.0, 97.5)
- added C-RF-IN1: 10uF 10V X5R, Capacitor_SMD:C_0805_2012Metric, F.Cu at (223.0, 97.5)
- added C-RF-IN2: 100nF, Capacitor_SMD:C_0402_1005Metric, F.Cu at (343.0, 97.5)
- added C-RF-O1: 22uF 6.3V X5R, Capacitor_SMD:C_0805_2012Metric, F.Cu at (226.0, 97.5)
- added C-RF-O2: 22uF 6.3V X5R, Capacitor_SMD:C_0805_2012Metric, F.Cu at (229.0, 97.5)
- added C-SIK1: 10uF 10V X5R, Capacitor_SMD:C_0805_2012Metric, B.Cu at (123.6, 94.7)
- added C-SIK2: 100nF, Capacitor_SMD:C_0402_1005Metric, F.Cu at (346.0, 97.5)
- added C-SS: 10nF, Capacitor_SMD:C_0201_0603Metric, B.Cu at (155.3, 99.1)
- added C-TPM1: 1uF, Capacitor_SMD:C_0402_1005Metric, F.Cu at (349.0, 97.5)
- added C-TPM2: 100nF, Capacitor_SMD:C_0402_1005Metric, F.Cu at (352.0, 97.5)
- added C-TPM3: 100nF, Capacitor_SMD:C_0402_1005Metric, F.Cu at (355.0, 97.5)
- added C-TPM4: 100nF, Capacitor_SMD:C_0402_1005Metric, F.Cu at (358.0, 97.5)
- added C-WIFI1: 100nF, Capacitor_SMD:C_0402_1005Metric, F.Cu at (361.0, 97.5)
- added C-WIFI2: 10uF 6.3V X5R, Capacitor_SMD:C_0805_2012Metric, F.Cu at (232.0, 97.5)
- added CAN-TR: ISOW1044BDFMR, Package_SO:SOIC-20W_7.5x12.8mm_P1.27mm, F.Cu at (136.6, 99.5)
- added CMC-CAN: SRF2012-100Y, Serenity-Custom:Bourns_SRF2012_4T, B.Cu at (172.7, 109.5)
- added D-ANT-LORA: RCLAMP0502B, Serenity-Custom:RCLAMP0502B_SOD882, F.Cu at (286.0, 97.5)
- added D-ANT-SIK: RCLAMP0502B, Serenity-Custom:RCLAMP0502B_SOD882, F.Cu at (289.0, 97.5)
- added D-ANT-WIFI: RCLAMP0502B, Serenity-Custom:RCLAMP0502B_SOD882, F.Cu at (292.0, 97.5)
- added ETH-PHY: DP83825IRHBR, Package_DFN_QFN:Texas_RMQ0024A_WQFN-24-1EP_3x3mm_P0.4mm_EP1.9x1.9mm, F.Cu at (168.5, 115.5)
- added FB-SDIO1: 742792510, Inductor_SMD:L_0805_2012Metric, F.Cu at (238.0, 97.5)
- added FB-SDIO2: 742792510, Inductor_SMD:L_0805_2012Metric, F.Cu at (241.0, 97.5)
- added FB-SDIO3: 742792510, Inductor_SMD:L_0805_2012Metric, F.Cu at (244.0, 97.5)
- added FB-SDIO4: 742792510, Inductor_SMD:L_0805_2012Metric, F.Cu at (247.0, 97.5)
- added FB-SDIO5: 742792510, Inductor_SMD:L_0805_2012Metric, F.Cu at (250.0, 97.5)
- added FB-SDIO6: 742792510, Inductor_SMD:L_0805_2012Metric, F.Cu at (253.0, 97.5)
- added FB-SIK1: 742792510, Inductor_SMD:L_0805_2012Metric, F.Cu at (256.0, 97.5)
- added FB-SIK2: 742792510, Inductor_SMD:L_0805_2012Metric, F.Cu at (128.6, 93.4)
- added FB-SIK3: 742792510, Inductor_SMD:L_0805_2012Metric, F.Cu at (259.0, 97.5)
- added FB-SIK4: 742792510, Inductor_SMD:L_0805_2012Metric, F.Cu at (262.0, 97.5)
- added FL-LORA: 0915LP15B026E, Serenity-Custom:Johanson_0915LP15B026E_SMD4, F.Cu at (274.0, 97.5)
- added FL-SIK: 0915LP15B026E, Serenity-Custom:Johanson_0915LP15B026E_SMD4, F.Cu at (277.0, 97.5)
- added FL-WIFI: 2450BP15E0100, Serenity-Custom:Johanson_2450BP15E0100_SMD4, F.Cu at (280.0, 97.5)
- added H1: M2.5 PGND, Serenity-Custom:MountingHole_2.7mm_M2.5_PGND_Ring, F.Cu at (124.0, 90.5)
- added H2: M2.5 PGND, Serenity-Custom:MountingHole_2.7mm_M2.5_PGND_Ring, F.Cu at (173.0, 90.5)
- added H3: M2.5 PGND, Serenity-Custom:MountingHole_2.7mm_M2.5_PGND_Ring, F.Cu at (124.0, 119.5)
- added H4: M2.5 PGND, Serenity-Custom:MountingHole_2.7mm_M2.5_PGND_Ring, F.Cu at (173.0, 119.5)
- added J-1553: SM04B-GHS-TB, Connector_JST:JST_GH_SM04B-GHS-TB_1x04-1MP_P1.25mm_Horizontal, F.Cu at (128.4, 111.9)
- added J-485: SM03B-GHS-TB, Connector_JST:JST_GH_SM03B-GHS-TB_1x03-1MP_P1.25mm_Horizontal, B.Cu at (150.2, 96.4)
- added J-CAN: SM03B-GHS-TB, Connector_JST:JST_GH_SM03B-GHS-TB_1x03-1MP_P1.25mm_Horizontal, B.Cu at (170.8, 105.0)
- added J-ETH: SM04B-GHS-TB, Connector_JST:JST_GH_SM04B-GHS-TB_1x04-1MP_P1.25mm_Horizontal, B.Cu at (161.1, 96.4)
- added J-FAN: SM03B-GHS-TB, Connector_JST:JST_GH_SM03B-GHS-TB_1x03-1MP_P1.25mm_Horizontal, F.Cu at (190.0, 97.5)
- added J-SD: microSD push-pull, Connector_Card:microSD_HC_Molex_104031-0811, F.Cu at (152.2, 99.1)
- added J-SIK-ANT: U.FL-R-SMT-1, Connector_Coaxial:U.FL_Hirose_U.FL-R-SMT-1_Vertical, F.Cu at (205.0, 97.5)
- added J-SMA-LORA: MMCX vertical, Connector_Coaxial:MMCX_Molex_73415-1471_Vertical, F.Cu at (196.0, 97.5)
- added J-SMA-SIK: MMCX vertical, Connector_Coaxial:MMCX_Molex_73415-1471_Vertical, F.Cu at (199.0, 97.5)
- added J-SMA-WIFI: MMCX vertical, Connector_Coaxial:MMCX_Molex_73415-1471_Vertical, F.Cu at (202.0, 97.5)
- added L-3V3: 3.3uH 2.25A, Serenity-Custom:L_WE-MAPI_3015, F.Cu at (208.0, 97.5)
- added L-RF1: 2.2uH 3A, Inductor_SMD:L_0805_2012Metric, F.Cu at (268.0, 97.5)
- added L-RF2: 2.2uH 3A, Inductor_SMD:L_0805_2012Metric, F.Cu at (271.0, 97.5)
- added LORA: RFM95W, Serenity-Custom:HopeRF_RFM95W_Castellated_16, B.Cu at (157.8, 108.4)
- added NOR-FLASH: W25Q128JVSIQ, Package_SO:SOIC-8_3.9x4.9mm_P1.27mm, B.Cu at (170.4, 113.9)
- added PWR-IN: Nano-Fit 4P, Serenity-Custom:Molex_NanoFit_1x04_Horizontal, F.Cu at (165.3, 109.9)
- added R-1553N: 55R 2%, Resistor_SMD:R_0603_1608Metric, F.Cu at (129.5, 100.1)
- added R-1553P: 55R 2%, Resistor_SMD:R_0603_1608Metric, F.Cu at (129.6, 96.8)
- added R-485T: 120R, Resistor_SMD:R_0603_1608Metric, B.Cu at (155.3, 97.0)
- added R-AD0: 2.49k, Resistor_SMD:R_0201_0603Metric, F.Cu at (132.9, 106.8)
- added R-BSR: 75R, Resistor_SMD:R_0402_1005Metric, F.Cu at (174.2, 113.0)
- added R-BST: 75R, Resistor_SMD:R_0402_1005Metric, F.Cu at (174.7, 114.8)
- added R-CANT: 120R, Resistor_SMD:R_0603_1608Metric, F.Cu at (283.0, 97.5)
- added R-EN3: 100k, Resistor_SMD:R_0201_0603Metric, B.Cu at (146.4, 112.3)
- added R-FB3H: 100k 1%, Resistor_SMD:R_0201_0603Metric, B.Cu at (146.3, 109.3)
- added R-FB3L: 32.4k 1%, Resistor_SMD:R_0201_0603Metric, B.Cu at (148.7, 116.2)
- added R-FLASH-WP: 10k, Resistor_SMD:R_0201_0603Metric, B.Cu at (146.4, 114.5)
- added R-LORA-C: 33R, Resistor_SMD:R_0402_1005Metric, B.Cu at (155.6, 94.3)
- added R-LORA-M1: 33R, Resistor_SMD:R_0402_1005Metric, B.Cu at (145.3, 94.8)
- added R-LORA-M2: 33R, Resistor_SMD:R_0402_1005Metric, B.Cu at (144.1, 94.7)
- added R-LORA-N: 33R, Resistor_SMD:R_0402_1005Metric, B.Cu at (174.8, 112.4)
- added R-LORA-RST: 10k, Resistor_SMD:R_0201_0603Metric, F.Cu at (364.0, 97.5)
- added R-PGND: 0R, Resistor_SMD:R_0805_2012Metric, F.Cu at (235.0, 97.5)
- added R-RBIAS: 6.49k 1%, Resistor_SMD:R_0201_0603Metric, F.Cu at (367.0, 97.5)
- added R-TPM10: 10k, Resistor_SMD:R_0201_0603Metric, F.Cu at (370.0, 97.5)
- added R-TPMCS: 10k, Resistor_SMD:R_0201_0603Metric, F.Cu at (373.0, 97.5)
- added R-WIFI-EN: 10k, Resistor_SMD:R_0201_0603Metric, F.Cu at (122.2, 113.7)
- added SD-WB: ATF16V8BQL-15XI, Package_SO:TSSOP-20_4.4x6.5mm_P0.65mm, F.Cu at (187.0, 97.5)
- added SIK: RFD900x, Serenity-Custom:RFDesign_RFD900x_2x8_THT, B.Cu at (133.8, 106.4)
- added T-ETH: 749010012A, Serenity-Custom:Wurth_749010012A_WE-LAN, F.Cu at (184.0, 97.5)
- added TPM: SLB9672XU20, Package_DFN_QFN:QFN-32-1EP_5x5mm_P0.5mm_EP3.6x3.6mm, F.Cu at (193.0, 97.5)
- added TVS-1553N: SMAJ33CA, Diode_SMD:D_SMA, F.Cu at (126.8, 98.0)
- added TVS-1553P: SMAJ33CA, Diode_SMD:D_SMA, F.Cu at (162.5, 115.5)
- added TVS-CAN: PRTR5V0U2X, Package_TO_SOT_SMD:SOT-143, F.Cu at (173.2, 105.2)
- added U-1V8: TLV75718PDBVR, Package_TO_SOT_SMD:SOT-89-3, F.Cu at (128.0, 104.4)
- added U-3V3: TPS62933DRLR, Package_TO_SOT_SMD:SOT-583-8, F.Cu at (173.8, 94.9)
- added U-3V3RF: TPS63031DSKR, Serenity-Custom:TPS6303x_VSON-10_2p5, F.Cu at (211.0, 97.5)
- added WIFI: WL1837MOD, Serenity-Custom:WL1837MOD_MOC_100, F.Cu at (136.9, 112.4)
- added X-25M: 25MHz 3.3V, Oscillator:Oscillator_SMD_ECS_2520MV-xxx-xx-4Pin_2.5x2.0mm, F.Cu at (172.4, 115.3)
- added X2Y-CAN: 4.7nF X2Y, Serenity-Custom:X2Y_0805_4T, B.Cu at (140.8, 94.5)
- CMC-RS485: footprint Bourns_SRF2012_4T -> Serenity-Custom:Bourns_SRF2012_4T; moved to B.Cu
- FB1: value 742792512 -> 742792510; footprint C_0805_2012Metric -> Inductor_SMD:L_0805_2012Metric
- PB2-P1: footprint PocketBeagle2:2x18_P1_Socket -> Serenity-Custom:PocketBeagle2_2x18_P1_Socket
- PB2-P2: footprint PocketBeagle2:2x18_P2_Socket -> Serenity-Custom:PocketBeagle2_2x18_P2_Socket
- RS485: value ADM2795EBRWZ -> ISOW1412DFMR; footprint SOIC-20W_7.5x12.8mm_P1.27mm -> Package_SO:SOIC-20W_7.5x12.8mm_P1.27mm; moved to F.Cu
- TVS-RS485: footprint SOT-363_SC-88 -> Package_TO_SOT_SMD:SOT-143; moved to F.Cu
- X2Y-RS485: footprint X2Y_Cap_4T_0402 -> Serenity-Custom:X2Y_0805_4T
- moved FB1 141.8 mm to (265.0, 97.5), turned to 0 degrees
- moved X2Y-RS485 48.2 mm to (173.5, 101.7)
- moved TVS-RS485 23.8 mm to (173.4, 98.3), turned to 0 degrees
- moved RS485 19.5 mm to (165.5, 99.5), turned to 0 degrees
- moved CMC-RS485 6.40 mm to (147.9, 109.0), turned to 90 degrees
Connections:
- CMC-RS485 pad 1: RS485_A -> RS485_B_A
- CMC-RS485 pad 2: RS485_B -> RS485_B_A_F
- CMC-RS485 pad 3: RS485_A -> RS485_B_B_F
- CMC-RS485 pad 4: RS485_B -> RS485_B_B
- FB1 pad 1: +5V -> +5V_IN
- PB2-P1 pad 10: RS485_RX -> PRU_1553B_TX_P
- PB2-P1 pad 11: RS485_TX -> RS485_B_DE
- PB2-P1 pad 12: CAN_STB -> RS485_B_RX
- PB2-P1 pad 13: MCAN1_RX -> RS485_B_TX
- PB2-P1 pad 14: MCAN1_TX -> CAN_B_STB
- PB2-P1 pad 15: UART_49MHZ_XCVR_RX -> MCAN0_B_RX
- PB2-P1 pad 16: UART_49MHZ_XCVR_TX -> MCAN0_B_TX
- PB2-P1 pad 17: UART_SIK_RX -> SD_CD
- PB2-P1 pad 18: UART_SIK_TX -> (no net)
- PB2-P1 pad 19: LORA_RESETN -> (no net)
- PB2-P1 pad 20: LORA_DIO0 -> M1553B_TX_INH
- PB2-P1 pad 21: SPI1_CS_TPM -> SPI0_B_CS_TPM
- PB2-P1 pad 22: SPI1_CS_NOR -> SPI0_B_CS_FLASH
- PB2-P1 pad 23: SPI1_MISO -> SPI0_B_MISO
- PB2-P1 pad 24: SPI1_MOSI -> SPI0_B_MOSI
- PB2-P1 pad 25: SPI1_CLK -> SPI0_B_CLK
- PB2-P1 pad 26: SPI1_CS_LORA -> SPI0_B_CS_LORA
- PB2-P1 pad 27: SDIO_D3 -> (no net)
- PB2-P1 pad 28: SDIO_D2 -> (no net)
- PB2-P1 pad 29: SDIO_D1 -> (no net)
- PB2-P1 pad 3: I2C0_SDA -> (no net)
- PB2-P1 pad 30: SDIO_D0 -> (no net)
- PB2-P1 pad 31: SDIO_CMD -> UART_SIK_RX
- PB2-P1 pad 32: SDIO_CLK -> UART_SIK_TX
- PB2-P1 pad 33: +3V3 -> +3V3_PB2
- PB2-P1 pad 34: +3V3 -> +3V3_PB2
- PB2-P1 pad 4: I2C0_SCL -> (no net)
- PB2-P1 pad 5: PRU_1553_RX_N -> (no net)
- PB2-P1 pad 6: PRU_1553_RX_P -> (no net)
- PB2-P1 pad 7: PRU_1553_TX_N -> PRU_1553B_RX_N
- PB2-P1 pad 8: PRU_1553_TX_P -> PRU_1553B_RX_P
- PB2-P1 pad 9: RS485_DE -> PRU_1553B_TX_N
- PB2-P2 pad 1: SERVO7 -> SDIO_D2
- PB2-P2 pad 10: WINCH_IN1 -> WIFI_IRQ
- PB2-P2 pad 11: TPM_RSTN -> TPM_B_RSTN
- PB2-P2 pad 12: TPM_IRQN -> TPM_B_IRQN
- PB2-P2 pad 13: PHY2_RSTN -> PLD_I3
- PB2-P2 pad 14: PHY2_INTRN -> PLD_I4
- PB2-P2 pad 17: MDIO -> MDIO0
- PB2-P2 pad 18: MDC -> MDC0
- PB2-P2 pad 19: RMII1_REF_CLK -> SDIO_CLK
- PB2-P2 pad 2: SERVO6 -> SDIO_D3
- PB2-P2 pad 20: RMII1_RX_ER -> SDIO_CMD
- PB2-P2 pad 21: RMII1_CRS_DV -> SDIO_D0
- PB2-P2 pad 22: RMII1_RXD1 -> SDIO_D1
- PB2-P2 pad 23: RMII1_RXD0 -> PLD_I5
- PB2-P2 pad 24: RMII1_TX_EN -> PLD_I6
- PB2-P2 pad 25: RMII1_TXD1 -> PLD_I7
- PB2-P2 pad 26: RMII1_TXD0 -> PLD_I8
- PB2-P2 pad 27: RMII0_REF_CLK -> LORA_DIO0
- PB2-P2 pad 3: PWM_CH3 -> SIK_CTS
- PB2-P2 pad 4: PWM_CH2 -> SIK_RTS
- PB2-P2 pad 5: PWM_CH1 -> FAN_PWM_B
- PB2-P2 pad 6: PWM_CH0 -> PLD_CLK
- PB2-P2 pad 7: LOAD_CELL_DOUT -> PLD_I1
- PB2-P2 pad 8: LOAD_CELL_SCK -> PLD_I2
- PB2-P2 pad 9: WINCH_IN2 -> WIFI_EN
- RS485 pad 10: (no net) -> GND
- RS485 pad 11: VCC2_RS485 -> GND2_RS485B
- RS485 pad 12: GND2_RS485 -> VCC2_RS485B
- RS485 pad 13: GND2_RS485 -> GND2_RS485B
- RS485 pad 14: RS485_A -> (no net)
- RS485 pad 15: RS485_B -> GND2_RS485B
- RS485 pad 16: (no net) -> VCC2_RS485B
- RS485 pad 17: (no net) -> RS485_B_A
- RS485 pad 18: GND2_RS485 -> RS485_B_B
- RS485 pad 19: GND2_RS485 -> RS485_B_B
- RS485 pad 2: GND -> RS485_B_TX
- RS485 pad 20: VCC2_RS485 -> RS485_B_A
- RS485 pad 3: RS485_TX -> RS485_B_DE
- RS485 pad 4: RS485_DE -> RS485_B_RX
- RS485 pad 5: RS485_DE -> RS485_B_DE
- RS485 pad 6: RS485_RX -> GND
- RS485 pad 7: GND -> (no net)
- RS485 pad 8: GND -> +3V3
- RS485 pad 9: (no net) -> +5V
- TVS-RS485 pad 1: RS485_A -> RS485_B_A_F
- TVS-RS485 pad 2: GND2_RS485 -> GND2_RS485B
- TVS-RS485 pad 3: RS485_B -> RS485_B_B_F
- TVS-RS485 pad 4: (no net) -> VCC2_RS485B
- X2Y-RS485 pad 3: GND -> GND2_RS485B
- X2Y-RS485 pad 4: GND2_RS485 -> GND2_RS485B
Routing:
- added copper zone on In4.Cu, net +3V3
- added copper zone on In1.Cu, net GND
- added copper zone on In1.Cu, net GND2_CANB
- added copper zone on In1.Cu, net GND2_RS485B
Other:
- copper layers 4 -> 6
- board text added: "ISOLATED CAN-FD | RS-485"
- board text added: "XO Rev S2 Griffing Technology LLC CC BY 4.0"
- board text removed: "Resillient Communications Cape For the PocketBeagle2 CC BY 4.0 — May 2026 Steve Griffing PE(CSE), CISSP-ISSEP, CPP Griffing Technology LLC github.com/Stab-Rabbit-Coding"
- board text removed: "TAMPER EVIDENT MESH"

Commit message: fix(avionics): XO drop duplicate LoRa (RFM95W) — Commo already carries it
Per the owner: Commo already has its own LoRa radio, so RFM95W on XO was
fleet-level duplicate capability, not a unique function. Removing it is
de-duplication, not the kind of capability loss flagged earlier in this
rebuild (unlike, say, dropping WiFi/BT or SiK, which nothing else on the
fleet provides).

Removed: LORA (RFM95W) itself, its SPI series-resistor filtering (R-LORA-M1/
M2/C/N), 3.3V bypass (C-LORA1), reset pull-up (R-LORA-RST), and its antenna
filter/ESD/jack chain (FL-LORA, D-ANT-LORA, J-SMA-LORA). Freed two PB2 header
ball positions (was LORA_DIO0 and SPI0_B_CS_LORA) left explicitly None rather
than reassigned.

ERC 0 confirmed (121 parts, 664 pins, down from 131/700).

Area impact: 3833 -> 3497 mm^2, i.e. 99.6% -> 90.8% of the 3850 mm^2
two-sided theoretical ceiling. Regenerated the PCB (owner has closed KiCad,
so this run is safe): auto-placer result improved from 56/131 unplaced to
43/121 unplaced -- real progress, but the board still isn't fully placed.
Next lever (another subsystem cut, a small board-length increase, or manual
placement) is an open decision for the owner.

Co-Authored-By: Claude Sonnet 5 <noreply@anthropic.com>
Parts:
- removed the C-1553C at (217.0, 97.5)
- removed the C-3V3-IN at (144.1, 94.5)
- removed C-LORA1: 100nF, Capacitor_SMD:C_0402_1005Metric
- removed D-ANT-LORA: RCLAMP0502B, Serenity-Custom:RCLAMP0502B_SOD882
- removed FL-LORA: 0915LP15B026E, Serenity-Custom:Johanson_0915LP15B026E_SMD4
- removed J-SIK-ANT: U.FL-R-SMT-1, Connector_Coaxial:U.FL_Hirose_U.FL-R-SMT-1_Vertical
- removed J-SMA-LORA: MMCX vertical, Connector_Coaxial:MMCX_Molex_73415-1471_Vertical
- removed LORA: RFM95W, Serenity-Custom:HopeRF_RFM95W_Castellated_16
- removed the R-485T at (155.3, 97.0)
- removed the R-CANT at (283.0, 97.5)
- removed R-LORA-C, R-LORA-M1, R-LORA-M2, R-LORA-N: 33R, Resistor_SMD:R_0402_1005Metric
- removed R-LORA-RST: 10k, Resistor_SMD:R_0201_0603Metric
- removed the SIK at (133.8, 106.4)
- added C-1553C: 10uF 6.3V X5R, Capacitor_SMD:C_0603_1608Metric, B.Cu at (173.9, 97.4)
- added C-3V3-IN: 10uF 10V X5R, Capacitor_SMD:C_0603_1608Metric, F.Cu at (250.0, 97.5)
- added R-485T: 120R, Resistor_SMD:R_0402_1005Metric, B.Cu at (170.1, 116.3)
- added R-CANT: 120R, Resistor_SMD:R_0402_1005Metric, B.Cu at (126.5, 93.7)
- added SIK: RFD900ux-SMT, Serenity-Custom:RFDesign_RFD900ux_SMT, B.Cu at (136.9, 105.7)
- C-1553A, C-1553B, C-25M, C-485-1, C-485-3, C-485-6, C-CAN1, C-CAN3, C-FLASH1, C-IN3, C-PHY-A2, C-PHY-A3, C-PHY-CRD2, C-PHY-CTD1, C-PHY-CTD2, C-PLD1, C-TPM1, C-TPM2, CAN-TR, J-FAN, R-BSR, R-BST, WIFI: moved to B.Cu
- C-3V3-HF, C-BS, C-PHY-A1, C-SS, CMC-CAN, CMC-RS485, J-485, J-CAN, J-ETH, R-EN3, R-FB3H, R-FB3L, R-FLASH-WP: moved to F.Cu
- C-3V3-O1, C-3V3-O2, C-485-2: footprint Capacitor_SMD:C_0805_2012Metric -> Capacitor_SMD:C_0603_1608Metric; moved to F.Cu
- C-485-5, C-CAN5, C-IN2, C-RF-IN1, C-RF-O1, C-RF-O2, C-SIK1: footprint Capacitor_SMD:C_0805_2012Metric -> Capacitor_SMD:C_0603_1608Metric
- C-CAN2, C-WIFI2: footprint Capacitor_SMD:C_0805_2012Metric -> Capacitor_SMD:C_0603_1608Metric; moved to B.Cu
- FB-SDIO1: footprint Inductor_SMD:L_0805_2012Metric -> Inductor_SMD:L_1812_4532Metric; moved to B.Cu
- FB-SDIO2, FB-SDIO3, FB-SDIO4, FB-SDIO5, FB-SDIO6, FB-SIK1, FB-SIK2, FB-SIK3, FB-SIK4, FB1: footprint Inductor_SMD:L_0805_2012Metric -> Inductor_SMD:L_1812_4532Metric
- L-RF1, L-RF2: footprint Inductor_SMD:L_0805_2012Metric -> Inductor_SMD:L_Wuerth_MAPI-3015
- moved C-PLD1 209.3 mm to (130.8, 93.6)
- moved R-WIFI-EN 194.5 mm to (316.0, 97.5), turned to 0 degrees
- moved C-PHY-A3 181.8 mm to (143.2, 93.8)
- moved C-PHY-A2 181.1 mm to (140.9, 93.6)
- moved C-IN3 181.1 mm to (135.0, 93.8)
- moved C-TPM2 178.5 mm to (174.3, 113.8)
- moved C-TPM1 175.4 mm to (174.3, 112.7)
- moved C-PHY-CTD1 170.9 mm to (163.4, 107.8)
- moved C-PHY-CTD2 163.6 mm to (174.0, 111.0), turned to 90 degrees
- moved C-CAN3 163.3 mm to (146.7, 93.8)
- moved C-485-3 162.2 mm to (132.8, 93.8)
- moved C-485-6 159.3 mm to (138.8, 93.8)
- moved R-FLASH-WP 158.5 mm to (304.0, 97.5), turned to 0 degrees
- moved C-PHY-CRD2 157.2 mm to (174.3, 109.3)
- moved C-PHY-CRD1 154.0 mm to (174.4, 108.6)
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Connections:
- PB2-P1 pad 26: SPI0_B_CS_LORA -> (no net)
- PB2-P2 pad 27: LORA_DIO0 -> (no net)

Commit message: feat(avionics): rebuild XO schematic with mLRS (Wio-E5) replacing SiK, ERC 0
Relocates XO's SiK radio (RFD900ux-SMT) to Commo and fills the freed slot
with mLRS firmware on a Seeed Wio-E5 (STM32WLE5) module, per this
session's ce-ideate analysis: XO+Commo need path diversity between a
SiK-class link and a LoRa-family link, and mLRS on Wio-E5 is the
closest like-for-like replacement for what SiK provided (MAVLink-
transparent telemetry + bidirectional RC + frequency hopping) without
collapsing that diversity, now that SiK itself has moved to Commo. A
second TPS62933 (U-1V8RF) shares the RF 1.8V rail instead of adding a
separate LDO. Also folds in the Murata Type2EL (WL1837MOD replacement)
tri-radio footprint work. kicad-cli sch erc: 0 violations. PCB
regenerated to 143 footprints/135 nets, 86.1% of the 2-sided area
ceiling, 0 schematic-parity issues against the netlist.

Co-Authored-By: Claude Sonnet 5 <noreply@anthropic.com>
Parts:
- removed C-1V8-IN, C-1V8-OUT: 1uF, Capacitor_SMD:C_0402_1005Metric
- removed C-SIK1: 10uF 10V X5R, Capacitor_SMD:C_0603_1608Metric
- removed C-SIK2, C-WIFI1: 100nF, Capacitor_SMD:C_0402_1005Metric
- removed C-WIFI2: 10uF 6.3V X5R, Capacitor_SMD:C_0603_1608Metric
- removed D-ANT-SIK, D-ANT-WIFI: RCLAMP0502B, Serenity-Custom:RCLAMP0502B_SOD882
- removed FB-SIK1, FB-SIK2, FB-SIK3, FB-SIK4: 742792510, Inductor_SMD:L_1812_4532Metric
- removed FL-SIK: 0915LP15B026E, Serenity-Custom:Johanson_0915LP15B026E_SMD4
- removed FL-WIFI: 2450BP15E0100, Serenity-Custom:Johanson_2450BP15E0100_SMD4
- removed J-SMA-SIK, J-SMA-WIFI: MMCX vertical, Connector_Coaxial:MMCX_Molex_73415-1471_Vertical
- removed R-WIFI-EN: 10k, Resistor_SMD:R_0201_0603Metric
- removed SIK: RFD900ux-SMT, Serenity-Custom:RFDesign_RFD900ux_SMT
- removed U-1V8: TLV75718PDBVR, Package_TO_SOT_SMD:SOT-89-3
- removed WIFI: WL1837MOD, Serenity-Custom:WL1837MOD_MOC_100
- added C-1V8RF-HF: 100nF, Capacitor_SMD:C_0402_1005Metric, F.Cu at (235.0, 97.5)
- added C-1V8RF-IN: 10uF 10V X5R, Capacitor_SMD:C_0603_1608Metric, F.Cu at (220.0, 97.5)
- added C-1V8RF-O1: 22uF 6.3V X5R, Capacitor_SMD:C_0603_1608Metric, B.Cu at (174.3, 106.7)
- added C-1V8RF-O2: 22uF 6.3V X5R, Capacitor_SMD:C_0603_1608Metric, B.Cu at (174.4, 110.0)
- added C-ANT-SANT: 10pF, Capacitor_SMD:C_0201_0603Metric, B.Cu at (172.8, 97.9)
- added C-ANT-SH1: DNP, Capacitor_SMD:C_0402_1005Metric, F.Cu at (134.4, 93.0)
- added C-ANT-SH2: DNP, Capacitor_SMD:C_0402_1005Metric, F.Cu at (135.7, 116.8)
- added C-BST18: 100nF, Capacitor_SMD:C_0402_1005Metric, B.Cu at (164.6, 104.0)
- added C-SS18: 10nF, Capacitor_SMD:C_0201_0603Metric, F.Cu at (295.0, 97.5)
- added C-WIOE5-IN: 4.7uF, Capacitor_SMD:C_0603_1608Metric, B.Cu at (148.5, 105.0)
- added C-WIOE5-SH1: DNP, Capacitor_SMD:C_0201_0603Metric, F.Cu at (175.0, 102.5)
- added C-WIOE5-SH2: DNP, Capacitor_SMD:C_0201_0603Metric, F.Cu at (163.0, 117.0)
- added C-ZB-18-1: 100nF, Capacitor_SMD:C_0402_1005Metric, B.Cu at (146.0, 116.4)
- added C-ZB-18-2: 100nF, Capacitor_SMD:C_0402_1005Metric, F.Cu at (277.0, 97.5)
- added C-ZB-33-1: 100nF, Capacitor_SMD:C_0402_1005Metric, F.Cu at (280.0, 97.5)
- added C-ZB-33-2: 100nF, Capacitor_SMD:C_0402_1005Metric, F.Cu at (283.0, 97.5)
- added C-ZB-SDVIO: 100nF, Capacitor_SMD:C_0402_1005Metric, F.Cu at (286.0, 97.5)
- added C-ZB-VIO: 100nF, Capacitor_SMD:C_0402_1005Metric, F.Cu at (289.0, 97.5)
- added D-ANT-RADIO: RCLAMP0502B, Serenity-Custom:RCLAMP0502B_SOD882, F.Cu at (129.4, 94.0)
- added D-ANT-WIOE5: RCLAMP0502B, Serenity-Custom:RCLAMP0502B_SOD882, F.Cu at (152.2, 93.4)
- added FB-WIOE5-1: 742792510, Inductor_SMD:L_1812_4532Metric, F.Cu at (143.3, 96.5)
- added FB-WIOE5-2: 742792510, Inductor_SMD:L_1812_4532Metric, F.Cu at (143.2, 114.5)
- added J-ANT-RADIO: MMCX vertical, Connector_Coaxial:MMCX_Molex_73415-1471_Vertical, F.Cu at (133.1, 96.2)
- added J-ANT-WIOE5: MMCX vertical, Connector_Coaxial:MMCX_Molex_73415-1471_Vertical, F.Cu at (172.9, 95.2)
- added J-WIOE5-SWD: SM04B-GHS-TB, Connector_JST:JST_GH_SM04B-GHS-TB_1x04-1MP_P1.25mm_Horizontal, F.Cu at (125.0, 98.2)
- added L-1V8RF: 3.3uH 2.25A, Serenity-Custom:L_WE-MAPI_3015, F.Cu at (172.8, 106.4)
- added L-ANT-SER: 0R link, Resistor_SMD:R_0402_1005Metric, F.Cu at (132.2, 93.0)
- added L-WIOE5-SER: 0R link, Resistor_SMD:R_0402_1005Metric, F.Cu at (161.4, 94.6)
- added LED-WIOE5-G: Green, LED_SMD:LED_0603_1608Metric, F.Cu at (152.1, 116.7)
- added LED-WIOE5-R: Red, LED_SMD:LED_0603_1608Metric, F.Cu at (144.7, 93.4)
- added R-EN18: 100k, Resistor_SMD:R_0201_0603Metric, B.Cu at (174.5, 97.9)
- added R-FB18H: 40.2k 1%, Resistor_SMD:R_0201_0603Metric, F.Cu at (307.0, 97.5)
- added R-FB18L: 32.4k 1%, Resistor_SMD:R_0201_0603Metric, F.Cu at (310.0, 97.5)
- added R-WIOE5-LEDG: 1k, Resistor_SMD:R_0201_0603Metric, B.Cu at (149.4, 113.8)
- added R-WIOE5-LEDR: 1k, Resistor_SMD:R_0201_0603Metric, F.Cu at (157.9, 117.1)
- added R-WIOE5-RST: 22k, Resistor_SMD:R_0201_0603Metric, B.Cu at (167.6, 115.1)
- added R-WIOE5-SWCLK: 22R, Resistor_SMD:R_0201_0603Metric, B.Cu at (125.2, 116.5)
- added R-WIOE5-SWDIO: 22R, Resistor_SMD:R_0201_0603Metric, B.Cu at (141.7, 116.3)
- added SW-WIOE5-BOOT: PTS125Sx43, Button_Switch_SMD:SW_Push_1P1T_NO_CK_PTS125Sx43PSMTR, F.Cu at (148.5, 105.0)
- added U-1V8RF: TPS62933DRLR, Package_TO_SOT_SMD:SOT-583-8, F.Cu at (214.0, 97.5)
- added WIFI-BT-ZB: LBES5PL2EL-923, Serenity-Custom:Murata_Type2EL_LGA107, B.Cu at (167.7, 98.0)
- added WIOE5: Wio-E5, Serenity-Custom:Seeed_WioE5_QFN28, F.Cu at (163.7, 102.5)
- C-25M, C-CAN1, C-CAN5, C-IN3, C-PHY-A3, C-PHY-CRD2, C-PHY-CTD1, C-PHY-CTD2, C-PLD1, C-TPM1, C-TPM2, FB-SDIO1, J-FAN, NOR-FLASH, R-485T, X2Y-CAN: moved to F.Cu
- C-485-2, C-485-4, C-485-5, C-BS, C-RF-IN1, C-RF-O1, CMC-RS485, FB-SDIO2, J-485, J-ETH, J-SD, R-1553N, R-1553P, R-TPMCS, RS485, SD-WB, T-ETH, X2Y-RS485: moved to B.Cu
- moved R-TPM10 150.2 mm to (161.1, 117.1)
- moved R-TPMCS 143.0 mm to (171.3, 116.4)
- moved R-RBIAS 141.5 mm to (165.6, 92.9)
- moved R-FLASH-WP 139.4 mm to (166.0, 117.1)
- moved C-PLD1 128.3 mm to (259.0, 97.5)
- moved C-PHY-A3 100.9 mm to (244.0, 97.5)
- moved C-RF-O1 95.2 mm to (167.1, 104.1)
- moved C-TPM2 95.1 mm to (268.0, 97.5)
- moved C-TPM1 92.0 mm to (265.0, 97.5)
- moved C-PHY-CTD1 90.2 mm to (253.0, 97.5)
- moved C-RF-IN1 88.9 mm to (170.4, 104.1)
- moved C-PHY-CTD2 83.1 mm to (256.0, 97.5), turned to 0 degrees
- moved L-3V3 82.8 mm to (139.0, 114.6)
- moved CMC-CAN 76.8 mm to (164.3, 94.6)
- moved C-PHY-CRD2 76.6 mm to (250.0, 97.5)
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Connections:
- PB2-P1 pad 26: (no net) -> SPI0_B_CS_ZB
- PB2-P1 pad 27: (no net) -> ZB_SPI_INT
- PB2-P1 pad 3: (no net) -> BT_UART_TX
- PB2-P1 pad 31: UART_SIK_RX -> UART_WIOE5_RX
- PB2-P1 pad 32: UART_SIK_TX -> UART_WIOE5_TX
- PB2-P1 pad 4: (no net) -> BT_UART_RX
- PB2-P1 pad 5: (no net) -> BT_UART_RTS
- PB2-P1 pad 6: (no net) -> BT_UART_CTS
- PB2-P2 pad 3: SIK_CTS -> (no net)
- PB2-P2 pad 4: SIK_RTS -> (no net)
