File: avionics/kicad/XO/kicads/XO.kicad_sch (KiCad schematic)
At the start: 131 parts, among them X2Y-CAN 4.7nF X2Y, X2Y-RS485 4.7nF X2Y

Commit message: fix(avionics): XO drop duplicate LoRa (RFM95W) — Commo already carries it
Per the owner: Commo already has its own LoRa radio, so RFM95W on XO was
fleet-level duplicate capability, not a unique function. Removing it is
de-duplication, not the kind of capability loss flagged earlier in this
rebuild (unlike, say, dropping WiFi/BT or SiK, which nothing else on the
fleet provides).

Removed: LORA (RFM95W) itself, its SPI series-resistor filtering (R-LORA-M1/
M2/C/N), 3.3V bypass (C-LORA1), reset pull-up (R-LORA-RST), and its antenna
filter/ESD/jack chain (FL-LORA, D-ANT-LORA, J-SMA-LORA). Freed two PB2 header
ball positions (was LORA_DIO0 and SPI0_B_CS_LORA) left explicitly None rather
than reassigned.

ERC 0 confirmed (121 parts, 664 pins, down from 131/700).

Area impact: 3833 -> 3497 mm^2, i.e. 99.6% -> 90.8% of the 3850 mm^2
two-sided theoretical ceiling. Regenerated the PCB (owner has closed KiCad,
so this run is safe): auto-placer result improved from 56/131 unplaced to
43/121 unplaced -- real progress, but the board still isn't fully placed.
Next lever (another subsystem cut, a small board-length increase, or manual
placement) is an open decision for the owner.

Co-Authored-By: Claude Sonnet 5 <noreply@anthropic.com>
Parts:
- removed C-485-1: 10nF, Capacitor_SMD:C_0201_0603Metric, symbol XO:S_C-485-1
- removed C-LORA1: 100nF, Capacitor_SMD:C_0402_1005Metric, symbol XO:S_C-LORA1
- removed D-ANT-LORA: RCLAMP0502B, Serenity-Custom:RCLAMP0502B_SOD882, symbol XO:S_D-ANT-LORA
- removed FL-LORA: 0915LP15B026E, Serenity-Custom:Johanson_0915LP15B026E_SMD4, symbol XO:S_FL-LORA
- removed J-ETH: SM04B-GHS-TB, Connector_JST:JST_GH_SM04B-GHS-TB_1x04-1MP_P1.25mm_Horizontal, symbol XO:S_J-ETH
- removed J-SMA-LORA: MMCX vertical, Connector_Coaxial:MMCX_Molex_73415-1471_Vertical, symbol XO:S_J-SMA-LORA
- removed R-LORA-C: 33R, Resistor_SMD:R_0402_1005Metric, symbol XO:S_R-LORA-C
- removed R-LORA-M1: 33R, Resistor_SMD:R_0402_1005Metric, symbol XO:S_R-LORA-M1
- removed R-LORA-M2: 33R, Resistor_SMD:R_0402_1005Metric, symbol XO:S_R-LORA-M2
- removed R-LORA-N: 33R, Resistor_SMD:R_0402_1005Metric, symbol XO:S_R-LORA-N
- removed R-LORA-RST: 10k, Resistor_SMD:R_0201_0603Metric, symbol XO:S_R-LORA-RST
- removed WIFI: WL1837MOD, Serenity-Custom:WL1837MOD_MOC_100, symbol XO:S_WIFI
- removed X2Y-CAN: 4.7nF X2Y, Serenity-Custom:X2Y_0805_4T, symbol XO:S_X2Y-CAN
- removed X2Y-RS485: 4.7nF X2Y, Serenity-Custom:X2Y_0805_4T, symbol XO:S_X2Y-RS485
- added CMC-CAN: SRF2012-100Y, Serenity-Custom:Bourns_SRF2012_4T, symbol XO:S_CMC-CAN
- added CMC-RS485: SRF2012-100Y, Serenity-Custom:Bourns_SRF2012_4T, symbol XO:S_CMC-RS485
- added TVS-CAN: PRTR5V0U2X, Package_TO_SOT_SMD:SOT-143, symbol XO:S_TVS-CAN
- added TVS-RS485: PRTR5V0U2X, Package_TO_SOT_SMD:SOT-143, symbol XO:S_TVS-RS485
- C-485-1: renamed from TVS-CAN; value PRTR5V0U2X -> 10nF; footprint Package_TO_SOT_SMD:SOT-143 -> Capacitor_SMD:C_0201_0603Metric; symbol XO:S_TVS-CAN -> XO:S_C-485-1; MPN PRTR5V0U2X,315 -> (none)
- J-ETH: renamed from TVS-RS485; value PRTR5V0U2X -> SM04B-GHS-TB; footprint Package_TO_SOT_SMD:SOT-143 -> Connector_JST:JST_GH_SM04B-GHS-TB_1x04-1MP_P1.25mm_Horizontal; symbol XO:S_TVS-RS485 -> XO:S_J-ETH; MPN PRTR5V0U2X,315 -> SM04B-GHS-TB(LF)(SN)
- WIFI: renamed from LORA; value RFM95W -> WL1837MOD; footprint Serenity-Custom:HopeRF_RFM95W_Castellated_16 -> Serenity-Custom:WL1837MOD_MOC_100; symbol XO:S_LORA -> XO:S_WIFI; MPN RFM95W-915S2 -> WL1837MOD
- X2Y-CAN: renamed from CMC-CAN; value SRF2012-100Y -> 4.7nF X2Y; footprint Serenity-Custom:Bourns_SRF2012_4T -> Serenity-Custom:X2Y_0805_4T; symbol XO:S_CMC-CAN -> XO:S_X2Y-CAN; MPN SRF2012-121YA -> CX0805MRX7R0BB472
- X2Y-RS485: renamed from CMC-RS485; value SRF2012-100Y -> 4.7nF X2Y; footprint Serenity-Custom:Bourns_SRF2012_4T -> Serenity-Custom:X2Y_0805_4T; symbol XO:S_CMC-RS485 -> XO:S_X2Y-RS485; MPN SRF2012-121YA -> CX0805MRX7R0BB472
Connections:
- net LORA_ANT_RF is gone; now on net GND: WIFI.9 (GND)
- net LORA_RESETN is gone; now on net SDIO_CMD_F: WIFI.6 (WL_SDIO_CMD)
- net +1V8_IO: now also WIFI.38 (VIO)
- net +3V3_RF: now also WIFI.46 (VBAT_IN), WIFI.47 (VBAT_IN); no longer WIFI.13 (3.3V)
- net +5V: now also C-485-1.1 (P)
- net CAN_B_H: now also CMC-CAN.1 (W1_IN); no longer X2Y-CAN.1 (W1_IN)
- net CAN_B_H_F: now also CMC-CAN.2 (W1_OUT), TVS-CAN.1 (IO1); no longer C-485-1.1 (IO1), X2Y-CAN.2 (W1_OUT)
- net CAN_B_L: now also CMC-CAN.4 (W2_IN); no longer X2Y-CAN.4 (W2_IN)
- net CAN_B_L_F: now also CMC-CAN.3 (W2_OUT), TVS-CAN.3 (IO2); no longer C-485-1.3 (IO2), X2Y-CAN.3 (W2_OUT)
- net ETHB_LINE_RXN: now also J-ETH.4 (RXN)
- net ETHB_LINE_RXP: now also J-ETH.3 (RXP)
- net ETHB_LINE_TXN: now also J-ETH.2 (TXN)
- net ETHB_LINE_TXP: now also J-ETH.1 (TXP)
- net GND: now also C-485-1.2 (N), WIFI.15 (GND), WIFI.17 (GND), WIFI.41 (BT_EN), WIFI.7 (GND), X2Y-CAN.1 (A), X2Y-CAN.2 (B), X2Y-RS485.1 (A), X2Y-RS485.2 (B); no longer WIFI.10 (GND), WIFI.8 (GND)
- net GND2_CANB: now also X2Y-CAN.3 (G1), X2Y-CAN.4 (G2), TVS-CAN.2 (GND); no longer C-485-1.2 (GND)
- net GND2_RS485B: now also X2Y-RS485.3 (G1), X2Y-RS485.4 (G2), TVS-RS485.2 (GND); no longer J-ETH.2 (GND)
- net PGND: now also J-ETH.MP (SHIELD)
- net RS485_B_A: now also CMC-RS485.1 (W1_IN); no longer X2Y-RS485.1 (W1_IN)
- net RS485_B_A_F: now also CMC-RS485.2 (W1_OUT), TVS-RS485.1 (IO1); no longer J-ETH.1 (IO1), X2Y-RS485.2 (W1_OUT)
- net RS485_B_B: now also CMC-RS485.4 (W2_IN); no longer X2Y-RS485.4 (W2_IN)
- net RS485_B_B_F: now also CMC-RS485.3 (W2_OUT), TVS-RS485.3 (IO2); no longer J-ETH.3 (IO2), X2Y-RS485.3 (W2_OUT)
- net SDIO_CLK_F: now also WIFI.8 (WL_SDIO_CLK)
- net SDIO_D0_F: now also WIFI.10 (WL_SDIO_D0)
- net SDIO_D1_F: now also WIFI.11 (WL_SDIO_D1)
- net SDIO_D2_F: now also WIFI.12 (WL_SDIO_D2)
- net SDIO_D3_F: now also WIFI.13 (WL_SDIO_D3)
- net VCC2_CANB: now also TVS-CAN.4 (VCC); no longer C-485-1.4 (VCC)
- net VCC2_RS485B: now also TVS-RS485.4 (VCC); no longer J-ETH.4 (VCC)
- net WIFI_ANT_RF: now also WIFI.32 (RF_ANT1)
- net WIFI_EN: now also WIFI.40 (WLAN_EN)
- net WIFI_IRQ: now also WIFI.14 (WLAN_IRQ)
- net LORA_DIO0: no longer names the net of PB2-P2.27 (P27)
- net LORA_DIO0: no longer WIFI.14 (DIO0)
- net SPI0_B_CLK_F: no longer names the net of WIFI.4 (NC)
- net SPI0_B_CS_LORA: no longer names the net of PB2-P1.26 (P26)
- net SPI0_B_CS_LORA_F: no longer names the net of WIFI.5 (NC)
- net SPI0_B_MISO_F: no longer names the net of WIFI.2 (NC)
- net SPI0_B_MOSI_F: no longer names the net of WIFI.3 (NC)
- no-connect marks 176 -> 173
Other:
- moved on the sheet: X2Y-CAN, X2Y-RS485

Commit message: feat(avionics): rebuild XO schematic with mLRS (Wio-E5) replacing SiK, ERC 0
Relocates XO's SiK radio (RFD900ux-SMT) to Commo and fills the freed slot
with mLRS firmware on a Seeed Wio-E5 (STM32WLE5) module, per this
session's ce-ideate analysis: XO+Commo need path diversity between a
SiK-class link and a LoRa-family link, and mLRS on Wio-E5 is the
closest like-for-like replacement for what SiK provided (MAVLink-
transparent telemetry + bidirectional RC + frequency hopping) without
collapsing that diversity, now that SiK itself has moved to Commo. A
second TPS62933 (U-1V8RF) shares the RF 1.8V rail instead of adding a
separate LDO. Also folds in the Murata Type2EL (WL1837MOD replacement)
tri-radio footprint work. kicad-cli sch erc: 0 violations. PCB
regenerated to 143 footprints/135 nets, 86.1% of the 2-sided area
ceiling, 0 schematic-parity issues against the netlist.

Co-Authored-By: Claude Sonnet 5 <noreply@anthropic.com>
Parts:
- removed C-1V8-IN: 1uF, Capacitor_SMD:C_0402_1005Metric, symbol XO:S_C-1V8-IN
- removed C-1V8-OUT: 1uF, Capacitor_SMD:C_0402_1005Metric, symbol XO:S_C-1V8-OUT
- removed C-3V3-HF: 100nF, Capacitor_SMD:C_0402_1005Metric, symbol XO:S_C-3V3-HF
- removed C-3V3-IN: 10uF 10V X5R, Capacitor_SMD:C_0603_1608Metric, symbol XO:S_C-3V3-IN
- removed C-IN1: 47uF 10V X5R, Capacitor_SMD:C_1210_3225Metric, symbol XO:S_C-IN1
- removed C-IN2: 10uF 10V X5R, Capacitor_SMD:C_0603_1608Metric, symbol XO:S_C-IN2
- removed C-IN3: 100nF, Capacitor_SMD:C_0402_1005Metric, symbol XO:S_C-IN3
- removed C-SIK1: 10uF 10V X5R, Capacitor_SMD:C_0603_1608Metric, symbol XO:S_C-SIK1
- removed C-SIK2: 100nF, Capacitor_SMD:C_0402_1005Metric, symbol XO:S_C-SIK2
- removed C-WIFI1: 100nF, Capacitor_SMD:C_0402_1005Metric, symbol XO:S_C-WIFI1
- removed C-WIFI2: 10uF 6.3V X5R, Capacitor_SMD:C_0603_1608Metric, symbol XO:S_C-WIFI2
- removed D-ANT-SIK: RCLAMP0502B, Serenity-Custom:RCLAMP0502B_SOD882, symbol XO:S_D-ANT-SIK
- removed D-ANT-WIFI: RCLAMP0502B, Serenity-Custom:RCLAMP0502B_SOD882, symbol XO:S_D-ANT-WIFI
- removed FB-SIK1: 742792510, Inductor_SMD:L_1812_4532Metric, symbol XO:S_FB-SIK1
- removed FB-SIK2: 742792510, Inductor_SMD:L_1812_4532Metric, symbol XO:S_FB-SIK2
- removed FB-SIK3: 742792510, Inductor_SMD:L_1812_4532Metric, symbol XO:S_FB-SIK3
- removed FB-SIK4: 742792510, Inductor_SMD:L_1812_4532Metric, symbol XO:S_FB-SIK4
- removed FB1: 742792510, Inductor_SMD:L_1812_4532Metric, symbol XO:S_FB1
- removed FL-SIK: 0915LP15B026E, Serenity-Custom:Johanson_0915LP15B026E_SMD4, symbol XO:S_FL-SIK
- removed FL-WIFI: 2450BP15E0100, Serenity-Custom:Johanson_2450BP15E0100_SMD4, symbol XO:S_FL-WIFI
- removed J-SMA-SIK: MMCX vertical, Connector_Coaxial:MMCX_Molex_73415-1471_Vertical, symbol XO:S_J-SMA-SIK
- removed J-SMA-WIFI: MMCX vertical, Connector_Coaxial:MMCX_Molex_73415-1471_Vertical, symbol XO:S_J-SMA-WIFI
- removed R-EN3: 100k, Resistor_SMD:R_0201_0603Metric, symbol XO:S_R-EN3
- removed R-PGND: 0R, Resistor_SMD:R_0805_2012Metric, symbol XO:S_R-PGND
- removed R-WIFI-EN: 10k, Resistor_SMD:R_0201_0603Metric, symbol XO:S_R-WIFI-EN
- removed TVS-RS485: PRTR5V0U2X, Package_TO_SOT_SMD:SOT-143, symbol XO:S_TVS-RS485
- removed WIFI: WL1837MOD, Serenity-Custom:WL1837MOD_MOC_100, symbol XO:S_WIFI
- added C-1V8RF-HF: 100nF, Capacitor_SMD:C_0402_1005Metric, symbol XO:S_C-1V8RF-HF
- added C-1V8RF-IN: 10uF 10V X5R, Capacitor_SMD:C_0603_1608Metric, symbol XO:S_C-1V8RF-IN
- added C-1V8RF-O2: 22uF 6.3V X5R, Capacitor_SMD:C_0603_1608Metric, symbol XO:S_C-1V8RF-O2
- added C-3V3-O2: 22uF 6.3V X5R, Capacitor_SMD:C_0603_1608Metric, symbol XO:S_C-3V3-O2
- added C-ANT-SANT: 10pF, Capacitor_SMD:C_0201_0603Metric, symbol XO:S_C-ANT-SANT
- added C-ANT-SH1: DNP, Capacitor_SMD:C_0402_1005Metric, symbol XO:S_C-ANT-SH1
- added C-ANT-SH2: DNP, Capacitor_SMD:C_0402_1005Metric, symbol XO:S_C-ANT-SH2
- added C-BS: 10nF 2kV, Capacitor_SMD:C_1808_4520Metric, symbol XO:S_C-BS
- added C-BST18: 100nF, Capacitor_SMD:C_0402_1005Metric, symbol XO:S_C-BST18
- added C-PHY-CTD2: 1uF, Capacitor_SMD:C_0402_1005Metric, symbol XO:S_C-PHY-CTD2
- added C-RF-IN1: 10uF 10V X5R, Capacitor_SMD:C_0603_1608Metric, symbol XO:S_C-RF-IN1
- added C-RF-IN2: 100nF, Capacitor_SMD:C_0402_1005Metric, symbol XO:S_C-RF-IN2
- added C-RF-O1: 22uF 6.3V X5R, Capacitor_SMD:C_0603_1608Metric, symbol XO:S_C-RF-O1
- added C-RF-O2: 22uF 6.3V X5R, Capacitor_SMD:C_0603_1608Metric, symbol XO:S_C-RF-O2
- added C-SS18: 10nF, Capacitor_SMD:C_0201_0603Metric, symbol XO:S_C-SS18
- added C-WIOE5-IN: 4.7uF, Capacitor_SMD:C_0603_1608Metric, symbol XO:S_C-WIOE5-IN
- added C-WIOE5-SH1: DNP, Capacitor_SMD:C_0201_0603Metric, symbol XO:S_C-WIOE5-SH1
- added C-WIOE5-SH2: DNP, Capacitor_SMD:C_0201_0603Metric, symbol XO:S_C-WIOE5-SH2
- added C-ZB-18-1: 100nF, Capacitor_SMD:C_0402_1005Metric, symbol XO:S_C-ZB-18-1
- added C-ZB-18-2: 100nF, Capacitor_SMD:C_0402_1005Metric, symbol XO:S_C-ZB-18-2
- added C-ZB-33-1: 100nF, Capacitor_SMD:C_0402_1005Metric, symbol XO:S_C-ZB-33-1
- added C-ZB-33-2: 100nF, Capacitor_SMD:C_0402_1005Metric, symbol XO:S_C-ZB-33-2
- added C-ZB-SDVIO: 100nF, Capacitor_SMD:C_0402_1005Metric, symbol XO:S_C-ZB-SDVIO
- added C-ZB-VIO: 100nF, Capacitor_SMD:C_0402_1005Metric, symbol XO:S_C-ZB-VIO
- added D-ANT-RADIO: RCLAMP0502B, Serenity-Custom:RCLAMP0502B_SOD882, symbol XO:S_D-ANT-RADIO
- added D-ANT-WIOE5: RCLAMP0502B, Serenity-Custom:RCLAMP0502B_SOD882, symbol XO:S_D-ANT-WIOE5
- added FB-WIOE5-1: 742792510, Inductor_SMD:L_1812_4532Metric, symbol XO:S_FB-WIOE5-1
- added FB-WIOE5-2: 742792510, Inductor_SMD:L_1812_4532Metric, symbol XO:S_FB-WIOE5-2
- added J-ANT-RADIO: MMCX vertical, Connector_Coaxial:MMCX_Molex_73415-1471_Vertical, symbol XO:S_J-ANT-RADIO
- added J-ANT-WIOE5: MMCX vertical, Connector_Coaxial:MMCX_Molex_73415-1471_Vertical, symbol XO:S_J-ANT-WIOE5
- added J-WIOE5-SWD: SM04B-GHS-TB, Connector_JST:JST_GH_SM04B-GHS-TB_1x04-1MP_P1.25mm_Horizontal, symbol XO:S_J-WIOE5-SWD
- added L-1V8RF: 3.3uH 2.25A, Serenity-Custom:L_WE-MAPI_3015, symbol XO:S_L-1V8RF
- added L-ANT-SER: 0R link, Resistor_SMD:R_0402_1005Metric, symbol XO:S_L-ANT-SER
- added L-RF1: 2.2uH 3A, Inductor_SMD:L_Wuerth_MAPI-3015, symbol XO:S_L-RF1
- added L-RF2: 2.2uH 3A, Inductor_SMD:L_Wuerth_MAPI-3015, symbol XO:S_L-RF2
- added L-WIOE5-SER: 0R link, Resistor_SMD:R_0402_1005Metric, symbol XO:S_L-WIOE5-SER
- added LED-WIOE5-G: Green, LED_SMD:LED_0603_1608Metric, symbol XO:S_LED-WIOE5-G
- added LED-WIOE5-R: Red, LED_SMD:LED_0603_1608Metric, symbol XO:S_LED-WIOE5-R
- added R-EN18: 100k, Resistor_SMD:R_0201_0603Metric, symbol XO:S_R-EN18
- added R-FB18H: 40.2k 1%, Resistor_SMD:R_0201_0603Metric, symbol XO:S_R-FB18H
- added R-FB18L: 32.4k 1%, Resistor_SMD:R_0201_0603Metric, symbol XO:S_R-FB18L
- added R-WIOE5-LEDG: 1k, Resistor_SMD:R_0201_0603Metric, symbol XO:S_R-WIOE5-LEDG
- added R-WIOE5-LEDR: 1k, Resistor_SMD:R_0201_0603Metric, symbol XO:S_R-WIOE5-LEDR
- added R-WIOE5-RST: 22k, Resistor_SMD:R_0201_0603Metric, symbol XO:S_R-WIOE5-RST
- added R-WIOE5-SWCLK: 22R, Resistor_SMD:R_0201_0603Metric, symbol XO:S_R-WIOE5-SWCLK
- added R-WIOE5-SWDIO: 22R, Resistor_SMD:R_0201_0603Metric, symbol XO:S_R-WIOE5-SWDIO
- added SW-WIOE5-BOOT: PTS125Sx43, Button_Switch_SMD:SW_Push_1P1T_NO_CK_PTS125Sx43PSMTR, symbol XO:S_SW-WIOE5-BOOT
- added WIFI-BT-ZB: LBES5PL2EL-923, Serenity-Custom:Murata_Type2EL_LGA107, symbol XO:S_WIFI-BT-ZB
- added WIOE5: Wio-E5, Serenity-Custom:Seeed_WioE5_QFN28, symbol XO:S_WIOE5
- C-1V8RF-O1: renamed from X2Y-CAN; value 4.7nF X2Y -> 22uF 6.3V X5R; footprint Serenity-Custom:X2Y_0805_4T -> Capacitor_SMD:C_0603_1608Metric; symbol XO:S_X2Y-CAN -> XO:S_C-1V8RF-O1; MPN CX0805MRX7R0BB472 -> (none)
- C-3V3-HF: renamed from U-1V8; value TLV75718PDBVR -> 100nF; footprint Package_TO_SOT_SMD:SOT-89-3 -> Capacitor_SMD:C_0402_1005Metric; symbol XO:S_U-1V8 -> XO:S_C-3V3-HF; MPN TLV75718PDBVR -> (none)
- C-3V3-IN: renamed from C-RF-O2; value 22uF 6.3V X5R -> 10uF 10V X5R; symbol XO:S_C-RF-O2 -> XO:S_C-3V3-IN
- C-IN1: renamed from L-RF1; value 2.2uH 3A -> 47uF 10V X5R; footprint Inductor_SMD:L_Wuerth_MAPI-3015 -> Capacitor_SMD:C_1210_3225Metric; symbol XO:S_L-RF1 -> XO:S_C-IN1; MPN LPS3015-222MRC -> (none)
- C-IN2: renamed from L-RF2; value 2.2uH 3A -> 10uF 10V X5R; footprint Inductor_SMD:L_Wuerth_MAPI-3015 -> Capacitor_SMD:C_0603_1608Metric; symbol XO:S_L-RF2 -> XO:S_C-IN2; MPN LPS3015-222MRC -> (none)
- C-IN3: renamed from C-RF-IN1; value 10uF 10V X5R -> 100nF; footprint Capacitor_SMD:C_0603_1608Metric -> Capacitor_SMD:C_0402_1005Metric; symbol XO:S_C-RF-IN1 -> XO:S_C-IN3
- FB1: renamed from C-3V3-O2; value 22uF 6.3V X5R -> 742792510; footprint Capacitor_SMD:C_0603_1608Metric -> Inductor_SMD:L_1812_4532Metric; symbol XO:S_C-3V3-O2 -> XO:S_FB1; MPN (none) -> 742792510
- R-EN3: renamed from C-RF-O1; value 22uF 6.3V X5R -> 100k; footprint Capacitor_SMD:C_0603_1608Metric -> Resistor_SMD:R_0201_0603Metric; symbol XO:S_C-RF-O1 -> XO:S_R-EN3
- R-PGND: renamed from C-RF-IN2; value 100nF -> 0R; footprint Capacitor_SMD:C_0402_1005Metric -> Resistor_SMD:R_0805_2012Metric; symbol XO:S_C-RF-IN2 -> XO:S_R-PGND
- TVS-RS485: renamed from C-PHY-CTD2; value 1uF -> PRTR5V0U2X; footprint Capacitor_SMD:C_0402_1005Metric -> Package_TO_SOT_SMD:SOT-143; symbol XO:S_C-PHY-CTD2 -> XO:S_TVS-RS485; MPN (none) -> PRTR5V0U2X,315
- U-1V8RF: renamed from SIK; value RFD900ux-SMT -> TPS62933DRLR; footprint Serenity-Custom:RFDesign_RFD900ux_SMT -> Package_TO_SOT_SMD:SOT-583-8; symbol XO:S_SIK -> XO:S_U-1V8RF; MPN RFD900UX-SMT -> TPS62933DRLR
- X2Y-CAN: renamed from C-BS; value 10nF 2kV -> 4.7nF X2Y; footprint Capacitor_SMD:C_1808_4520Metric -> Serenity-Custom:X2Y_0805_4T; symbol XO:S_C-BS -> XO:S_X2Y-CAN; MPN (none) -> CX0805MRX7R0BB472
Connections:
- net +1V8_IO is gone; now on net GND: C-3V3-HF.2 (N)
- net +3V3: now also C-3V3-O2.1 (P), C-ZB-VIO.1 (P), WIFI-BT-ZB.24 (RF_CNTL4), WIFI-BT-ZB.25 (RF_CNTL3/CONFIG_XOSC_SEL), WIFI-BT-ZB.54 (VIO), WIFI-BT-ZB.55 (CONFIG_HOST[0]), WIFI-BT-ZB.56 (CONFIG_HOST[1]); no longer C-3V3-HF.3 (IN), FB1.1 (P)
- net +3V3_RF: now also C-RF-O1.1 (P), C-RF-O2.1 (P), C-WIOE5-IN.1 (P), C-ZB-33-1.1 (P), C-ZB-33-2.1 (P), J-WIOE5-SWD.1 (VTREF), L-RF2.2 (B), R-WIOE5-LEDR.1 (A), R-WIOE5-RST.1 (A), WIFI-BT-ZB.12 (AVDD33_1), WIFI-BT-ZB.13 (AVDD33_2), WIOE5.1 (VCC); no longer C-3V3-IN.1 (P), C-IN2.2 (B), R-EN3.1 (P)
- net +5V: now also C-3V3-HF.1 (P), C-3V3-IN.1 (P), C-IN2.1 (P), FB1.2 (OUT), R-EN3.1 (A), U-1V8RF.3 (VIN), C-1V8RF-HF.1 (P), C-1V8RF-IN.1 (P), C-RF-IN1.1 (P), C-RF-IN2.1 (P), L-RF1.2 (B), R-EN18.1 (A); no longer C-IN1.2 (B), R-PGND.1 (P)
- net +5V_IN: now also C-IN1.1 (P), FB1.1 (IN)
- net ETHB_BS: now also C-BS.1 (P); no longer X2Y-CAN.1 (P)
- net ETHB_CTD: now also C-PHY-CTD2.1 (P); no longer TVS-RS485.1 (P)
- net GND: now also C-IN1.2 (N), C-IN2.2 (N), R-PGND.1 (A), U-1V8RF.1 (RT), U-1V8RF.4 (GND), X2Y-CAN.1 (A), X2Y-CAN.2 (B), C-1V8RF-HF.2 (N), C-1V8RF-IN.2 (N), C-1V8RF-O2.2 (N), C-3V3-O2.2 (N), C-ANT-SH1.2 (B), C-ANT-SH2.2 (B), C-PHY-CTD2.2 (N), C-RF-IN1.2 (N), C-RF-IN2.2 (N), C-RF-O1.2 (N), C-RF-O2.2 (N), C-SS18.2 (N), C-WIOE5-IN.2 (N), C-WIOE5-SH1.2 (B), C-WIOE5-SH2.2 (B), C-ZB-18-1.2 (N), C-ZB-18-2.2 (N), C-ZB-33-1.2 (N), C-ZB-33-2.2 (N), C-ZB-SDVIO.2 (N), C-ZB-VIO.2 (N), J-WIOE5-SWD.4 (GND), LED-WIOE5-G.2 (K), R-FB18L.2 (B), SW-WIOE5-BOOT.2 (B), WIFI-BT-ZB.1 (GND), WIFI-BT-ZB.100 (GND), WIFI-BT-ZB.101 (GND), WIFI-BT-ZB.102 (GND), WIFI-BT-ZB.103 (GND), WIFI-BT-ZB.104 (GND), WIFI-BT-ZB.105 (GND), WIFI-BT-ZB.106 (GND), WIFI-BT-ZB.107 (GND), WIFI-BT-ZB.11 (GND), WIFI-BT-ZB.14 (GND), WIFI-BT-ZB.16 (GND), WIFI-BT-ZB.17 (GND), WIFI-BT-ZB.19 (GND), WIFI-BT-ZB.2 (GND), WIFI-BT-ZB.20 (GND), WIFI-BT-ZB.21 (GND), WIFI-BT-ZB.22 (GND), WIFI-BT-ZB.28 (GND), WIFI-BT-ZB.29 (GND), WIFI-BT-ZB.32 (GND), WIFI-BT-ZB.39 (GND), WIFI-BT-ZB.41 (GND), WIFI-BT-ZB.43 (GND), WIFI-BT-ZB.53 (GND), WIFI-BT-ZB.62 (GND), WIFI-BT-ZB.67 (GND), WIFI-BT-ZB.68 (GND), WIFI-BT-ZB.71 (GND), WIFI-BT-ZB.81 (GND), WIFI-BT-ZB.82 (GND), WIFI-BT-ZB.83 (GND), WIFI-BT-ZB.84 (GND), WIFI-BT-ZB.85 (GND), WIFI-BT-ZB.86 (GND), WIFI-BT-ZB.87 (GND), WIFI-BT-ZB.88 (GND), WIFI-BT-ZB.89 (GND), WIFI-BT-ZB.9 (GND), WIFI-BT-ZB.90 (GND), WIFI-BT-ZB.91 (GND), WIFI-BT-ZB.92 (GND), WIFI-BT-ZB.93 (GND), WIFI-BT-ZB.94 (GND), WIFI-BT-ZB.95 (GND), WIFI-BT-ZB.96 (GND), WIFI-BT-ZB.97 (GND), WIFI-BT-ZB.98 (GND), WIFI-BT-ZB.99 (GND), WIOE5.14 (GND), WIOE5.16 (GND), WIOE5.2 (GND), WIOE5.22 (GND), WIOE5.29 (PAD_GND); no longer C-1V8RF-O1.1 (A), C-3V3-HF.1 (GND), FB1.2 (N), R-EN3.2 (N), R-PGND.2 (N), TVS-RS485.2 (N), U-1V8RF.11 (GND), U-1V8RF.12 (GND), U-1V8RF.14 (GND), U-1V8RF.15 (GND), U-1V8RF.17 (GND), U-1V8RF.18 (GND), U-1V8RF.20 (GND), U-1V8RF.29 (GND_THERMAL1), U-1V8RF.30 (GND_THERMAL2), U-1V8RF.8 (GND), U-1V8RF.9 (GND)
- net GND2_CANB: now also X2Y-CAN.3 (G1), X2Y-CAN.4 (G2); no longer C-1V8RF-O1.3 (G1), C-1V8RF-O1.4 (G2)
- net GND2_RS485B: now also TVS-RS485.2 (GND)
- net PGND: now also R-PGND.2 (B), C-BS.2 (N), D-ANT-RADIO.2 (K), D-ANT-WIOE5.2 (K), J-ANT-RADIO.2 (SHIELD), J-ANT-WIOE5.2 (SHIELD); no longer X2Y-CAN.2 (N)
- net RF_SW1: now also L-RF1.1 (A); no longer C-IN1.1 (A)
- net RF_SW2: now also L-RF2.1 (A); no longer C-IN2.1 (A)
- net RS485_B_A_F: now also TVS-RS485.1 (IO1)
- net RS485_B_B_F: now also TVS-RS485.3 (IO2)
- net SDIO_CLK_F: now also WIFI-BT-ZB.44 (SD_CLK)
- net SDIO_CMD_F: now also WIFI-BT-ZB.42 (SD_CMD)
- net SDIO_D0_F: now also WIFI-BT-ZB.48 (SD_DAT0)
- net SDIO_D1_F: now also WIFI-BT-ZB.45 (SD_DAT1)
- net SDIO_D2_F: now also WIFI-BT-ZB.47 (SD_DAT2)
- net SDIO_D3_F: now also WIFI-BT-ZB.46 (SD_DAT3)
- net SPI0_B_CLK: now also WIFI-BT-ZB.8 (SPI_CLK)
- net SPI0_B_MISO: now also WIFI-BT-ZB.6 (SPI_RXD)
- net SPI0_B_MOSI: now also WIFI-BT-ZB.7 (SPI_TXD)
- net U3V3_EN: now also R-EN3.2 (B)
- net VCC2_RS485B: now also TVS-RS485.4 (VCC)
- net WIFI_EN: now also WIFI-BT-ZB.10 (PDn)
- net WIFI_IRQ: now also WIFI-BT-ZB.72 (SD_INT)
- net U1V8RF_EN: now reaches U-1V8RF.2 (EN)
- net U1V8RF_EN: now also R-EN18.2 (B)
- net SW_1V8RF: now reaches U-1V8RF.5 (SW)
- net SW_1V8RF: now also C-BST18.2 (N), L-1V8RF.1 (A)
- net BST_1V8RF: now reaches U-1V8RF.6 (BST)
- net BST_1V8RF: now also C-BST18.1 (P)
- net SS_1V8RF: now reaches U-1V8RF.7 (SS/PG)
- net SS_1V8RF: now also C-SS18.1 (P)
- net SPI0_B_CS_ZB: now reaches PB2-P1.26 (P26)
- net SPI0_B_CS_ZB: now also WIFI-BT-ZB.4 (SPI_FRM)
- net ZB_SPI_INT: now reaches PB2-P1.27 (P27)
- net ZB_SPI_INT: now also WIFI-BT-ZB.5 (SPI_INT)
- net BT_UART_TX: now reaches PB2-P1.3 (P3)
- net BT_UART_TX: now also WIFI-BT-ZB.49 (UART_TX)
- net BT_UART_RX: now reaches PB2-P1.4 (P4)
- net BT_UART_RX: now also WIFI-BT-ZB.51 (UART_RX)
- net BT_UART_RTS: now reaches PB2-P1.5 (P5)
- net BT_UART_RTS: now also WIFI-BT-ZB.52 (UART_RTS)
- net BT_UART_CTS: now reaches PB2-P1.6 (P6)
- net BT_UART_CTS: now also WIFI-BT-ZB.50 (UART_CTS)
- removed net SIK_ANT_RF: U-1V8RF.13 (ANT1)
- net SIK_CTS: no longer names the net of PB2-P2.3 (P3)
- removed net SIK_CTS_F: U-1V8RF.28 (CTS)
- net SIK_RTS: no longer names the net of PB2-P2.4 (P4)
- net SIK_RTS: no longer U-1V8RF.27 (RTS)
- removed net SIK_VCC_F: U-1V8RF.19 (+5V)
- net UART_SIK_RX renamed UART_WIOE5_RX
- net UART_WIOE5_RX: now also FB-WIOE5-1.1 (IN)
- removed net UART_SIK_RX_F: U-1V8RF.25 (RX)
- net UART_SIK_TX renamed UART_WIOE5_TX
- net UART_WIOE5_TX: now also FB-WIOE5-2.1 (IN)
- removed net UART_SIK_TX_F: U-1V8RF.26 (TX)
- new net +1V8_RF: C-1V8RF-O1.1 (P), C-1V8RF-O2.1 (P), C-ZB-18-1.1 (P), C-ZB-18-2.1 (P), C-ZB-SDVIO.1 (P), L-1V8RF.2 (B), R-FB18H.1 (A), WIFI-BT-ZB.30 (AVDD18_2), WIFI-BT-ZB.31 (AVDD18_1), WIFI-BT-ZB.40 (SD_VIO)
- new net FB_1V8RF: R-FB18H.2 (B), R-FB18L.1 (A), U-1V8RF.8 (FB)
- new net RADIO_ANT1_IN: C-ANT-SANT.2 (B), WIFI-BT-ZB.18 (BT_15.4_IN)
- new net RADIO_ANT1_OUT: C-ANT-SANT.1 (A), WIFI-BT-ZB.23 (ANT1)
- new net RADIO_ANT_F: C-ANT-SH2.1 (A), D-ANT-RADIO.1 (A), J-ANT-RADIO.1 (RF), L-ANT-SER.2 (B)
- new net RADIO_ANT_RF: C-ANT-SH1.1 (A), L-ANT-SER.1 (A), WIFI-BT-ZB.15 (ANT0)
- new net UART_WIOE5_RX_F: FB-WIOE5-1.2 (OUT), WIOE5.18 (PA3)
- new net UART_WIOE5_TX_F: FB-WIOE5-2.2 (OUT), WIOE5.19 (PA2)
- new net WIOE5_ANT_F: C-WIOE5-SH2.1 (A), D-ANT-WIOE5.1 (A), J-ANT-WIOE5.1 (RF), L-WIOE5-SER.2 (B)
- new net WIOE5_ANT_RF: C-WIOE5-SH1.1 (A), L-WIOE5-SER.1 (A), WIOE5.15 (RFIO)
- new net WIOE5_BOOT_BTN: SW-WIOE5-BOOT.1 (A), WIOE5.24 (PB13)
- new net WIOE5_LEDG_A: LED-WIOE5-G.1 (A), R-WIOE5-LEDG.2 (B)
- new net WIOE5_LEDR_A: LED-WIOE5-R.1 (A), R-WIOE5-LEDR.2 (B)
- new net WIOE5_LED_G: R-WIOE5-LEDG.1 (A), WIOE5.6 (PA15)
- new net WIOE5_LED_R: LED-WIOE5-R.2 (K), WIOE5.11 (PB5)
- new net WIOE5_RST: R-WIOE5-RST.2 (B), WIOE5.17 (RST)
- new net WIOE5_SWCLK: R-WIOE5-SWCLK.1 (A), WIOE5.4 (PA14)
- new net WIOE5_SWCLK_HDR: J-WIOE5-SWD.3 (SWCLK), R-WIOE5-SWCLK.2 (B)
- new net WIOE5_SWDIO: R-WIOE5-SWDIO.1 (A), WIOE5.3 (PA13)
- new net WIOE5_SWDIO_HDR: J-WIOE5-SWD.2 (SWDIO), R-WIOE5-SWDIO.2 (B)
- no-connect marks 173 -> 115
Other:
- moved on the sheet: C-3V3-IN, C-IN1, C-IN2, C-IN3, FB1, R-EN3, R-PGND
