File: avionics/kicad/Commo/kicads/Commo.kicad_sch (KiCad schematic)
At the start: 77 parts, among them U1 ByA 100nF +3V3 U1-VDDA Bypass, U1 ByB 100nF +3V3 U1-VDD Bypass

Commit message: fix(avionics): Commo lib_id prefix corruption crashing kicad-cli; add missing XO RFD900ux footprint
Commo.kicad_sch had no sym-lib-table/fp-lib-table and used bare (unprefixed)
lib_ids (e.g. "S_+5V_Bead") instead of "Commo:S_+5V_Bead" — prefixing only the
instance lib_id references without also prefixing the matching embedded
lib_symbols cache-key definitions produced a state that segfaulted
`kicad-cli sch erc` outright. Fixed both the instance references and the
embedded cache keys together (matching gen_pilot_sch.py/gen_xo_sch.py's own
convention), extracted the embedded lib_symbols block into a companion
Commo.kicad_sym, and added the missing sym-lib-table/fp-lib-table. Also fixed
4 bare TPM-injection symbols (SLB9672_TPM, R_Generic_TPM, C_Generic_TPM,
PWR_FLAG_TPM) the same way.

ERC: 127 -> 48 violations (all 79 lib_symbol_issues resolved; 43
global_label_dangling + 5 endpoint_off_grid remain, not yet fixed).

Also adds avionics/kicad/Serenity-Custom.pretty/RFDesign_RFD900ux_SMT.kicad_mod
and avionics/datasheets/hm-trp.pdf, which were used by 71d2f09 (XO RFD900x ->
RFD900ux-SMT swap) but not staged in that commit.

Co-Authored-By: Claude Sonnet 5 <noreply@anthropic.com>
Parts:
- +3V 100n: symbol S_+3V_100n -> Commo:S_+3V_100n
- +3V 100u: symbol S_+3V_100u -> Commo:S_+3V_100u
- +3V 10n: symbol S_+3V_10n -> Commo:S_+3V_10n
- +3V 10u: symbol S_+3V_10u -> Commo:S_+3V_10u
- +5V 100n: symbol S_+5V_100n -> Commo:S_+5V_100n
- +5V 100u: symbol S_+5V_100u -> Commo:S_+5V_100u
- +5V Bead: symbol S_+5V_Bead -> Commo:S_+5V_Bead
- 1.2k C: symbol S_1.2k_C -> Commo:S_1.2k_C
- 1.2k R: symbol S_1.2k_R -> Commo:S_1.2k_R
- 2.2k C: symbol S_2.2k_C -> Commo:S_2.2k_C
- 2.2k R: symbol S_2.2k_R -> Commo:S_2.2k_R
- 49M DDS: symbol S_49M_DDS -> Commo:S_49M_DDS
- AFSK Cp: symbol S_AFSK_Cp -> Commo:S_AFSK_Cp
- ANT CMC: symbol S_ANT_CMC -> Commo:S_ANT_CMC
- ANT RPSMA: symbol S_ANT_RPSMA -> Commo:S_ANT_RPSMA
- ANT TVS: symbol S_ANT_TVS -> Commo:S_ANT_TVS
- C1 120p: symbol S_C1_120p -> Commo:S_C1_120p
- C2 180p: symbol S_C2_180p -> Commo:S_C2_180p
- C3 120p: symbol S_C3_120p -> Commo:S_C3_120p
- CMP By: symbol S_CMP_By -> Commo:S_CMP_By
- C_INV: symbol S_C_INV -> Commo:S_C_INV
- C_MUX: symbol S_C_MUX -> Commo:S_C_MUX
- C_TPM_EMMA1: symbol C_Generic_TPM -> Commo:C_Generic_TPM
- DAC By: symbol S_DAC_By -> Commo:S_DAC_By
- ETH-PHY: symbol S_ETH-PHY -> Commo:S_ETH-PHY
- GND X2Y: symbol S_GND_X2Y -> Commo:S_GND_X2Y
- INV1: symbol S_INV1 -> Commo:S_INV1
- J-ETH: symbol S_J-ETH -> Commo:S_J-ETH
- L1 100n: symbol S_L1_100n -> Commo:S_L1_100n
- L2 180n: symbol S_L2_180n -> Commo:S_L2_180n
- L3 180n: symbol S_L3_180n -> Commo:S_L3_180n
- LDO 3V3: symbol S_LDO_3V3 -> Commo:S_LDO_3V3
- LDO By: symbol S_LDO_By -> Commo:S_LDO_By
- LNA: symbol S_LNA -> Commo:S_LNA
- LNA By: symbol S_LNA_By -> Commo:S_LNA_By
- LoRa: symbol S_LoRa -> Commo:S_LoRa
- MUX1: symbol S_MUX1 -> Commo:S_MUX1
- OSC By: symbol S_OSC_By -> Commo:S_OSC_By
- PA 100mW: symbol S_PA_100mW -> Commo:S_PA_100mW
- PA By: symbol S_PA_By -> Commo:S_PA_By
- PA By2: symbol S_PA_By2 -> Commo:S_PA_By2
- PA Cb1: symbol S_PA_Cb1 -> Commo:S_PA_Cb1
- PA Cb2: symbol S_PA_Cb2 -> Commo:S_PA_Cb2
- PA Drvr: symbol S_PA_Drvr -> Commo:S_PA_Drvr
- PA Rb1: symbol S_PA_Rb1 -> Commo:S_PA_Rb1
- PA Rb2: symbol S_PA_Rb2 -> Commo:S_PA_Rb2
- PA Rc1: symbol S_PA_Rc1 -> Commo:S_PA_Rc1
- PA Re: symbol S_PA_Re -> Commo:S_PA_Re
- PB2-P1: symbol S_PB2-P1 -> Commo:S_PB2-P1
- PB2-P2: symbol S_PB2-P2 -> Commo:S_PB2-P2
- PGND 10n: symbol S_PGND_10n -> Commo:S_PGND_10n
- PTT Bead: symbol S_PTT_Bead -> Commo:S_PTT_Bead
- RSSI Hi: symbol S_RSSI_Hi -> Commo:S_RSSI_Hi
- RSSI Lo: symbol S_RSSI_Lo -> Commo:S_RSSI_Lo
- RSSI_CBY: symbol S_RSSI_CBY -> Commo:S_RSSI_CBY
- RSSI_CMP: symbol S_RSSI_CMP -> Commo:S_RSSI_CMP
- RSSI_RH: symbol S_RSSI_RH -> Commo:S_RSSI_RH
- RSSI_RL: symbol S_RSSI_RL -> Commo:S_RSSI_RL
- RX Bead: symbol S_RX_Bead -> Commo:S_RX_Bead
- RX Demod: symbol S_RX_Demod -> Commo:S_RX_Demod
- R_MODE: symbol S_R_MODE -> Commo:S_R_MODE
- R_TPM_RST_EMMA: symbol R_Generic_TPM -> Commo:R_Generic_TPM
- S1: symbol S_S1 -> Commo:S_S1
- SMA ESD: symbol S_SMA_ESD -> Commo:S_SMA_ESD
- SW By: symbol S_SW_By -> Commo:S_SW_By
- T-ETH: symbol S_T-ETH -> Commo:S_T-ETH
- T/R Sw: symbol S_T_R_Sw -> Commo:S_T_R_Sw
- TCXO 25M: symbol S_TCXO_25M -> Commo:S_TCXO_25M
- TPM: symbol SLB9672_TPM -> Commo:SLB9672_TPM
- TX Bead: symbol S_TX_Bead -> Commo:S_TX_Bead
- TX DAC: symbol S_TX_DAC -> Commo:S_TX_DAC
- Th Hi: symbol S_Th_Hi -> Commo:S_Th_Hi
- Th Lo: symbol S_Th_Lo -> Commo:S_Th_Lo
- U1 ByA: symbol S_U1_ByA -> Commo:S_U1_ByA
- U1 ByB: symbol S_U1_ByB -> Commo:S_U1_ByB
- UART CMC: symbol S_UART_CMC -> Commo:S_UART_CMC
- UART TVS: symbol S_UART_TVS -> Commo:S_UART_TVS

Commit message: feat(avionics): swap Commo's LoRa (RFM95W) for SiK (RFD900ux-SMT), ERC 0
Completes the other half of the XO<->Commo radio relocation: Commo
gains the SiK link SiK-side via a new one-off script
(swap_lora_for_sik.py) that does direct S-expression surgery rather
than re-running gen_commo_sch.py, which is PCB-first and already
confirmed drifted from the real board. Also fixes two pre-existing
circuit bugs the swap's ERC cleanup exposed: the T/R switch's antenna
pin was on a differently-named net one row away from the working ANT
filter chain (merged); and the PA final transistor's emitter pin was
wired straight to GND, bypassing its own degeneration resistor
(rewired onto PA_EMIT). DDS_FSYNC (the TX DAC's SPI chip-select,
previously unrouted) now uses the exact PB2 pin the LoRa->SiK swap
freed (ex-SPI1_CS_LORA), by explicit owner decision. kicad-cli sch
erc: 0 violations (down from 45).

PCB synced to match (schematic driving PCB, not the reverse): old
RFM95W footprint removed, 8 new SIK-chain footprints added with nets
matched 1:1 against the real schematic pin table. Along the way DRC
caught a real geometry bug in the shared RFDesign_RFD900ux_SMT
footprint (pad pitch/axis swap causing adjacent castellated pins to
short) -- fixed against RFD900ux DataSheet v1.2.pdf Table 6-1 and
confirmed via DRC. Residual: Commo's existing hand-placed layout has
no contiguous free region for the 21x29mm SIK module without touching
ETH-PHY/T-ETH -- flagged in WBS.md as needing a real floorplan pass,
not silently left implicit.

Co-Authored-By: Claude Sonnet 5 <noreply@anthropic.com>
Parts:
- removed LoRa: RFM95W, symbol Commo:S_LoRa
- added C-SIK-SH1: DNP, symbol Commo:S_C_SIK_SH1
- added C-SIK-SH2: DNP, symbol Commo:S_C_SIK_SH2
- added C-SIK1: 10uF 10V X5R, symbol Commo:S_C_SIK1
- added C-SIK2: 100nF, symbol Commo:S_C_SIK2
- added D-ANT-SIK: RCLAMP0502B, symbol Commo:S_D_ANT_SIK
- added J-ANT-SIK: MMCX vertical, symbol Commo:S_J_ANT_SIK
- added L-SIK-SER: 0R link, symbol Commo:S_L_SIK_SER
- added SIK: RFD900ux-SMT, symbol Commo:S_SIK
Connections:
- net RF_ANT_SW is gone; now on net ANT: T/R Sw.1 (ANT)
- net SPI1_CS_LORA is gone; now on net DDS_FSYNC: PB2-P1.26 (DDS_FSYNC)
- net GND: now also C-SIK-SH1.2 (B), C-SIK-SH2.2 (B), C-SIK1.2 (N), C-SIK2.2 (N), D-ANT-SIK.2 (K), J-ANT-SIK.2 (SHIELD), SIK.11 (GND), SIK.12 (GND), SIK.14 (GND), SIK.15 (GND), SIK.17 (GND), SIK.18 (GND), SIK.20 (GND), SIK.29 (GND), SIK.30 (GND), SIK.8 (GND), SIK.9 (GND); no longer PA 100mW.2 (GND)
- net PA_EMIT: now also PA 100mW.2 (GND)
- net UART_SIK_RX: now also SIK.25 (UART_SIK_RX)
- net UART_SIK_TX: now also SIK.26 (UART_SIK_TX)
- net CAN_STB: no longer names the net of PB2-P1.12 (CAN_STB)
- net I2C0_SCL: no longer names the net of PB2-P1.4 (I2C0_SCL)
- net I2C0_SDA: no longer names the net of PB2-P1.3 (I2C0_SDA)
- net LOAD_CELL_DOUT: no longer names the net of PB2-P2.7 (LOAD_CELL_DOUT)
- net LOAD_CELL_SCK: no longer names the net of PB2-P2.8 (LOAD_CELL_SCK)
- net LORA_DIO0 renamed SIK_CTS
- net SIK_CTS: now also SIK.28 (SIK_CTS)
- net LORA_RESETN renamed SIK_RTS
- net SIK_RTS: now also SIK.27 (SIK_RTS)
- net MCAN1_RX: no longer names the net of PB2-P1.13 (MCAN1_RX)
- net MCAN1_TX: no longer names the net of PB2-P1.14 (MCAN1_TX)
- net PHY1_INTRN: no longer names the net of PB2-P2.16 (PHY1_INTRN)
- net PHY1_RSTN: no longer names the net of PB2-P2.15 (PHY1_RSTN)
- net PRU_1553_RX_N: no longer names the net of PB2-P1.5 (PRU_1553_RX_N)
- net PRU_1553_RX_P: no longer names the net of PB2-P1.6 (PRU_1553_RX_P)
- net PRU_1553_TX_N: no longer names the net of PB2-P1.7 (PRU_1553_TX_N)
- net PRU_1553_TX_P: no longer names the net of PB2-P1.8 (PRU_1553_TX_P)
- net PWM_CH0: no longer names the net of PB2-P2.6 (PWM_CH0)
- net PWM_CH1: no longer names the net of PB2-P2.5 (PWM_CH1)
- net PWM_CH2: no longer names the net of PB2-P2.4 (PWM_CH2)
- net PWM_CH3: no longer names the net of PB2-P2.3 (PWM_CH3)
- net RMII0_CRS_DV: no longer names the net of PB2-P2.29 (RMII0_CRS_DV)
- net RMII0_REF_CLK: no longer names the net of PB2-P2.27 (RMII0_REF_CLK)
- net RMII0_RXD0: no longer names the net of PB2-P2.31 (RMII0_RXD0)
- net RMII0_RXD1: no longer names the net of PB2-P2.30 (RMII0_RXD1)
- net RMII0_RX_ER: no longer names the net of PB2-P2.28 (RMII0_RX_ER)
- net RMII0_TXD0: no longer names the net of PB2-P2.34 (RMII0_TXD0)
- net RMII0_TXD1: no longer names the net of PB2-P2.33 (RMII0_TXD1)
- net RMII0_TX_EN: no longer names the net of PB2-P2.32 (RMII0_TX_EN)
- net RS485_DE: no longer names the net of PB2-P1.9 (RS485_DE)
- net RS485_RX: no longer names the net of PB2-P1.10 (RS485_RX)
- net RS485_TX: no longer names the net of PB2-P1.11 (RS485_TX)
- net SDIO_CLK: no longer names the net of PB2-P1.32 (SDIO_CLK)
- net SDIO_CMD: no longer names the net of PB2-P1.31 (SDIO_CMD)
- net SDIO_D0: no longer names the net of PB2-P1.30 (SDIO_D0)
- net SDIO_D1: no longer names the net of PB2-P1.29 (SDIO_D1)
- net SDIO_D2: no longer names the net of PB2-P1.28 (SDIO_D2)
- net SDIO_D3: no longer names the net of PB2-P1.27 (SDIO_D3)
- net SPI1_CS_NOR: no longer names the net of PB2-P1.22 (SPI1_CS_NOR)
- net WINCH_IN1: no longer names the net of PB2-P2.10 (WINCH_IN1)
- net WINCH_IN2: no longer names the net of PB2-P2.9 (WINCH_IN2)
- new net SIK_ANT_F: C-SIK-SH2.1 (A), D-ANT-SIK.1 (A), J-ANT-SIK.1 (RF), L-SIK-SER.2 (B)
- new net SIK_ANT_RF: C-SIK-SH1.1 (A), L-SIK-SER.1 (A), SIK.13 (SIK_ANT_RF)
- new net SIK_VCC: C-SIK1.1 (P), C-SIK2.1 (P), SIK.19 (SIK_VCC)
- no-connect marks 43 -> 85
Other:
- note added: "SiK RFD900ux-SMT (915 MHz UHF telemetry -- relocated from XO 2026-09-21, see avionics/WBS.md)"
- note removed: "LoRa 915 MHz (RFM95W, SPI via PB2-P1)"
- moved on the sheet: R_TPM_RST_EMMA
