File: avionics/kicad/Commo/kicads/Commo.kicad_sch (KiCad schematic)
At the start: 84 parts, among them U1 ByA 100nF +3V3 U1-VDDA Bypass, U1 ByB 100nF +3V3 U1-VDD Bypass

Commit message: fix(avionics): PRTR5V0U2X package/pinout fix on all 12 instances, 5 boards
Owner-approved 2026-09-26 (avionics/WBS.md U7.2). Per Nexperia
PRTR5V0U2X datasheet Table 2 (SOT143B: 1=GND, 2=I/O1, 3=I/O2, 4=VCC),
relinked via tools/kicad_relink.py --rewire (same footprint position/
rotation preserved, only package + pin-to-net correspondence corrected):

- Pilot TVS-CAN, TVS-RS485; TACCO TVS-CAN, TVS-RS485; FlightEngineer
  D_I2C: straightforward SOT-363->SOT-143 swap with existing GND/VCC
  nets carried over unchanged (5 instances).
- Observer T1_D1/T1_D2/T2_D1/T2_D2 (Ethernet magnetics ESD) and D5
  (CAN-FD), Commo 'ANT TVS' and 'UART TVS': these had no VCC net at
  all in the original (wrong-package) design -- VCC tied to the local
  GND/PGND net as a conservative fallback (line-to-line and
  line-to-ground clamping preserved; the rail-clamp direction is
  inert). This is a judgment call, not a datasheet requirement --
  flagged for review, not a silent assumption (7 instances).

ERC unchanged (0/0/0/0/154-pre-existing) on all 5 boards; DRC/parity
flat or improved except one new courtyard-overlap warning on Pilot
(TVS-CAN vs C-IN1, mechanical only) left unresolved rather than guess
a nudge direction without full layout context.

AI-authored: Claude Sonnet 5 (Anthropic).

Co-Authored-By: Claude Sonnet 5 <noreply@anthropic.com>
Parts:
- ANT TVS: footprint (none) -> Package_TO_SOT_SMD:SOT-143; symbol Commo:S_ANT_TVS -> SecureControllers:PRTR5V0U2X
- UART TVS: value PRTR5V0U2X Dual TVS 5.5V UART-TX/RX ESD -> PRTR5V0U2X; footprint (none) -> Package_TO_SOT_SMD:SOT-143; symbol Commo:S_UART_TVS -> SecureControllers:PRTR5V0U2X
Connections:
- net GND: no longer ANT TVS.3 (GND), ANT TVS.6 (GND), UART TVS.3 (GND), UART TVS.6 (GND)
- net RF_TX: now also ANT TVS.3 (IO2); no longer ANT TVS.5 (RF_TX)
- net UART_49MHZ_XCVR_TX: now also UART TVS.3 (IO2); no longer UART TVS.5 (UART_49MHZ_XCVR_TX)
Changed lines of the file:
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@@
   (wire (pts (xy 364.49 427.99) (xy 368.30 427.99)) (stroke (width 0) (type default)))
   (global_label "ANT" (shape passive) (at 368.30 427.99 0) (effects (font (size 1.27 1.27)) (justify left)))
-  (symbol (lib_id "Commo:S_ANT_TVS") (at 444.50 429.26 0) (unit 1)
-    (exclude_from_sim no) (in_bom yes) (on_board yes) (dnp no)
+  (symbol (lib_id "SecureControllers:PRTR5V0U2X") (at 444.50 429.26 0) (unit 1)
+    (exclude_from_sim no) (in_bom yes) (on_board yes) (dnp no)
+    (property "Datasheet" "https://assets.nexperia.com/documents/data-sheet/PRTR5V0U2X.pdf" (at 444.50 429.26 0) (effects (font (size 1.27 1.27)) (hide yes)))
+    (property "Footprint" "Package_TO_SOT_SMD:SOT-143" (at 444.50 429.26 0) (effects (font (size 1.27 1.27)) (hide yes)))
     (property "Reference" "ANT TVS" (at 444.50 421.64 0) (effects (font (size 1.27 1.27))))
     (property "Value" "PRTR5V0U2X" (at 444.50 436.88 0) (effects (font (size 1.27 1.27))))
@@
     (instances (project "Commo" (path "/49030000-0000-0000-0000-000000000001" (reference "ANT TVS") (unit 1))))
   )
-  (wire (pts (xy 429.26 425.45) (xy 425.45 425.45)) (stroke (width 0) (type default)))
-  (global_label "GND" (shape passive) (at 425.45 425.45 180) (effects (font (size 1.27 1.27)) (justify right)))
-  (wire (pts (xy 429.26 427.99) (xy 425.45 427.99)) (stroke (width 0) (type default)))
-  (global_label "ANT" (shape passive) (at 425.45 427.99 180) (effects (font (size 1.27 1.27)) (justify right)))
-  (wire (pts (xy 429.26 430.53) (xy 425.45 430.53)) (stroke (width 0) (type default)))
-  (global_label "GND" (shape passive) (at 425.45 430.53 180) (effects (font (size 1.27 1.27)) (justify right)))
-  (wire (pts (xy 459.74 425.45) (xy 463.55 425.45)) (stroke (width 0) (type default)))
-  (global_label "GND" (shape passive) (at 463.55 425.45 0) (effects (font (size 1.27 1.27)) (justify left)))
-  (wire (pts (xy 459.74 427.99) (xy 463.55 427.99)) (stroke (width 0) (type default)))
-  (global_label "RF_TX" (shape passive) (at 463.55 427.99 0) (effects (font (size 1.27 1.27)) (justify left)))
-  (wire (pts (xy 459.74 430.53) (xy 463.55 430.53)) (stroke (width 0) (type default)))
-  (global_label "GND" (shape passive) (at 463.55 430.53 0) (effects (font (size 1.27 1.27)) (justify left)))
   (symbol (lib_id "Commo:S_SMA_ESD") (at 539.75 429.26 0) (unit 1)
     (exclude_from_sim no) (in_bom yes) (on_board yes) (dnp no)
@@
   (wire (pts (xy 78.74 734.06) (xy 82.55 734.06)) (stroke (width 0) (type default)))
   (global_label "UART_49MHZ_XCVR_TX" (shape passive) (at 82.55 734.06 0) (effects (font (size 1.27 1.27)) (justify left)))
-  (symbol (lib_id "Commo:S_UART_TVS") (at 158.75 734.06 0) (unit 1)
-    (exclude_from_sim no) (in_bom yes) (on_board yes) (dnp no)
+  (symbol (lib_id "SecureControllers:PRTR5V0U2X") (at 158.75 734.06 0) (unit 1)
+    (exclude_from_sim no) (in_bom yes) (on_board yes) (dnp no)
+    (property "Datasheet" "https://assets.nexperia.com/documents/data-sheet/PRTR5V0U2X.pdf" (at 158.75 734.06 0) (effects (font (size 1.27 1.27)) (hide yes)))
+    (property "Footprint" "Package_TO_SOT_SMD:SOT-143" (at 158.75 734.06 0) (effects (font (size 1.27 1.27)) (hide yes)))
     (property "Reference" "UART TVS" (at 158.75 726.44 0) (effects (font (size 1.27 1.27))))
-    (property "Value" "PRTR5V0U2X  Dual TVS 5.5V  UART-TX/RX ESD" (at 158.75 741.68 0) (effects (font (size 1.27 1.27))))
+    (property "Value" "PRTR5V0U2X" (at 158.75 741.68 0) (effects (font (size 1.27 1.27))))
     (pin "1")
     (pin "2")
@@
     (instances (project "Commo" (path "/49030000-0000-0000-0000-000000000001" (reference "UART TVS") (unit 1))))
   )
-  (wire (pts (xy 143.51 730.25) (xy 139.70 730.25)) (stroke (width 0) (type default)))
-  (global_label "GND" (shape passive) (at 139.70 730.25 180) (effects (font (size 1.27 1.27)) (justify right)))
-  (wire (pts (xy 143.51 732.79) (xy 139.70 732.79)) (stroke (width 0) (type default)))
-  (global_label "UART_49MHZ_XCVR_RX" (shape passive) (at 139.70 732.79 180) (effects (font (size 1.27 1.27)) (justify right)))
-  (wire (pts (xy 143.51 735.33) (xy 139.70 735.33)) (stroke (width 0) (type default)))
-  (global_label "GND" (shape passive) (at 139.70 735.33 180) (effects (font (size 1.27 1.27)) (justify right)))
-  (wire (pts (xy 173.99 730.25) (xy 177.80 730.25)) (stroke (width 0) (type default)))
-  (global_label "GND" (shape passive) (at 177.80 730.25 0) (effects (font (size 1.27 1.27)) (justify left)))
-  (wire (pts (xy 173.99 732.79) (xy 177.80 732.79)) (stroke (width 0) (type default)))
-  (global_label "UART_49MHZ_XCVR_TX" (shape passive) (at 177.80 732.79 0) (effects (font (size 1.27 1.27)) (justify left)))
-  (wire (pts (xy 173.99 735.33) (xy 177.80 735.33)) (stroke (width 0) (type default)))
-  (global_label "GND" (shape passive) (at 177.80 735.33 0) (effects (font (size 1.27 1.27)) (justify left)))
   (symbol (lib_id "Commo:S_TX_Bead") (at 254.00 734.06 0) (unit 1)
     (exclude_from_sim no) (in_bom yes) (on_board yes) (dnp no)
@@
     (effects (font (size 1.27 1.27)))
 )
+  (global_label "ANT" (shape bidirectional) (at 434.3400 424.1800 180)
+    (effects (font (size 1.27 1.27)))
+)
+  (global_label "RF_TX" (shape bidirectional) (at 434.3400 426.7200 180)
+    (effects (font (size 1.27 1.27)))
+)
+  (global_label "GND" (shape bidirectional) (at 444.5000 439.4200 270)
+    (effects (font (size 1.27 1.27)))
+)
+  (global_label "GND" (shape bidirectional) (at 444.5000 419.1000 90)
+    (effects (font (size 1.27 1.27)))
+)
+  (global_label "UART_49MHZ_XCVR_RX" (shape bidirectional) (at 148.5900 728.9800 180)
+    (effects (font (size 1.27 1.27)))
+)
+  (global_label "UART_49MHZ_XCVR_TX" (shape bidirectional) (at 148.5900 731.5200 180)
+    (effects (font (size 1.27 1.27)))
+)
+  (global_label "GND" (shape bidirectional) (at 158.7500 744.2200 270)
+    (effects (font (size 1.27 1.27)))
+)
+  (global_label "GND" (shape bidirectional) (at 158.7500 723.9000 90)
+    (effects (font (size 1.27 1.27)))
+)
