File: avionics/kicad/Commo/kicads/Commo.kicad_pcb (KiCad board)
At the start: 4 copper layers, 55 x 35 mm, 88 parts, among them U1 ByA 100nF +3V3 U1-VDDA Bypass, U1 ByB 100nF +3V3 U1-VDD Bypass

Commit message: scrub away the cape-a and cape-b labels for Pilot and TACCO
Other:
- board text added: "J1 6P HDR TACCO I/F"
- board text removed: "J1 6P HDR CAPE-B I/F"
Changed lines of the file:
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@@
 		)
 	)
-	(gr_text "J1 6P HDR\nCAPE-B I/F"
+	(gr_text "J1 6P HDR\nTACCO I/F"
 		(at 120 104.5 0)
 		(layer "F.Fab")

Commit message: cleaned up stuff
Parts:
- moved ETH-PHY 24.3 mm to (148.5, 123.5)
- moved T-ETH 22.5 mm to (147.0, 108.5), turned to 180 degrees
- moved C-SIK-SH2 21.0 mm to (104.5, 117.0), turned to -90 degrees
- moved C-SIK-SH1 17.9 mm to (104.5, 115.0), turned to 90 degrees
- moved J-ANT-SIK 14.2 mm to (102.5, 121.0)
- moved RSSI_CBY 13.8 mm to (142.5, 107.0), turned to 90 degrees
- moved C-SIK2 13.0 mm to (104.5, 113.0), turned to 90 degrees
- moved L-SIK-SER 12.9 mm to (104.5, 111.0), turned to 90 degrees
- moved C_TPM_EMMA1 12.4 mm to (141.0, 107.0), turned to 90 degrees
- moved RSSI_CMP 12.4 mm to (141.0, 111.0), turned to 0 degrees
- moved RSSI_RL 9.21 mm to (138.0, 107.0), turned to 90 degrees
- moved R_TPM_RST_EMMA 8.51 mm to (139.5, 107.0), turned to 90 degrees
- moved C-SIK1 7.50 mm to (104.0, 108.0), turned to 90 degrees
- moved RSSI_RH 6.71 mm to (136.5, 107.0), turned to 90 degrees
- moved SIK 5.00 mm to (120.0, 117.5)
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Routing:
- net RSSI_REF: vias 0 -> 1
- net RSSI_ANA: vias 1 -> 3
- net GND: vias 81 -> 79
- net +5V_FILT: vias 2 -> 1
Other:
- board text added: "49 MHz AX.25 KISS and 915MHz SiK COMMO EMI Hardened Sub GHZ XCVR FCC 47 CFR Part 15 15.235 49.830-49.890 MHz AFSK 1200bd FCC ID: PENDING CERTIFICATION Complies w/ FCC Pt.15: (1) may not cause harmful interference (2) must accept any interference received CERN OHWL-P 4.0 September 2026 Steve Griffing, PE(CSE), CISSP-ISSEP, CPP Griffing Technology LLC github.com/Stab-Rabbit-Coding"
- board text removed: "49 MHz AX.25 KISS Transceiver XCVR-49MHZ-2 Rev 2 — EMI-Hardened FCC 47 CFR Part 15 15.235 49.830-49.890 MHz AFSK 1200bd FCC ID: PENDING CERTIFICATION Complies w/ FCC Pt.15: (1) may not cause harmful interference (2) must accept any interference received CC BY 4.0 — June 2026 Steve Griffing PE(CSE), CISSP-ISSEP, CPP Griffing Technology LLC github.com/Stab-Rabbit-Coding"
