File: avionics/kicad/TACCO/kicads/TACCO.kicad_sch (KiCad schematic)
At the start: 170 parts, among them X2Y-CAN 4.7nF X2Y, X2Y-RS485 4.7nF X2Y

Commit message: TACCO: SSM-DV-LC rails, redrawn isolation band, single TPS63031 inductor (WIP placement)
- PB2 rails -> Samtec SSM-118-L-DV-LC SMT sockets (footprint from samtec_ssm_footprint.pdf
  Rev D Fig. 4, -LC clip holes as through-board anchors); WBS R3 owner decision 2026-10-05.
- Isolation band redrawn: transceivers top face, bus connectors at the bottom edge; band on
  F.Cu + inner layers only, B.Cu beneath it limited to B-routable parts.
- TPS63031 fix: one inductor across L1-L2 per tps63031.pdf (L-RF2 removed).
- Placer: children after their anchor parent; THT/NPTH holes checked against the opposite
  face's copper.
- Docs: WBS, TACCO.md §13a, CONCEPTS.md, PB2 learning docs corrected for 4.80 mm rails.

Placement is not yet closed: the committed board still has parts parked off-outline; routing
and fab outputs follow once a full placement is found.

Co-Authored-By: Claude Opus 5.5 <noreply@anthropic.com>
Claude-Session: https://claude.ai/code/session_01YLwDy53g1VCBzNBwW4moUC
Parts:
- removed CMC-CAN: SRF2012-100Y, Serenity-Custom:Bourns_SRF2012_4T, symbol TACCO:S_CMC-CAN
- removed CMC-RS485: SRF2012-100Y, Serenity-Custom:Bourns_SRF2012_4T, symbol TACCO:S_CMC-RS485
- removed H1: M2.5 PGND, Serenity-Custom:MountingHole_2.7mm_M2.5_PGND_Ring, symbol TACCO:S_H1
- removed J-1553: SM04B-GHS-TB, Connector_JST:JST_GH_SM04B-GHS-TB_1x04-1MP_P1.25mm_Horizontal, symbol TACCO:S_J-1553
- removed J-485: SM03B-GHS-TB, Connector_JST:JST_GH_SM03B-GHS-TB_1x03-1MP_P1.25mm_Horizontal, symbol TACCO:S_J-485
- removed J-CAN: SM03B-GHS-TB, Connector_JST:JST_GH_SM03B-GHS-TB_1x03-1MP_P1.25mm_Horizontal, symbol TACCO:S_J-CAN
- removed J-FAN: SM03B-GHS-TB, Connector_JST:JST_GH_SM03B-GHS-TB_1x03-1MP_P1.25mm_Horizontal, symbol TACCO:S_J-FAN
- removed J-MLRS-SWD: TC2030-IDC-NL pads, Connector:Tag-Connect_TC2030-IDC-NL_2x03_P1.27mm_Vertical, symbol TACCO:S_J-MLRS-SWD
- removed RFSW-MLRS: PE4259, Package_TO_SOT_SMD:SOT-363_SC-70-6, symbol TACCO:S_RFSW-MLRS
- removed X-25M: 25MHz 3.3V, Oscillator:Oscillator_SMD_ECS_2520MV-xxx-xx-4Pin_2.5x2.0mm, symbol TACCO:S_X-25M
- removed X-50M: 50MHz 3.3V, Oscillator:Oscillator_SMD_ECS_2520MV-xxx-xx-4Pin_2.5x2.0mm, symbol TACCO:S_X-50M
- removed X-MLRS: TG2520SMN 32MHz 1.8V clipped-sine, Oscillator:Oscillator_SMD_SeikoEpson_TG2520SMN-xxx-xxxxxx-4Pin_2.5x2.0mm, symbol TACCO:S_X-MLRS
- added C-1553A: 100nF, Capacitor_SMD:C_0402_1005Metric, symbol TACCO:S_C-1553A
- added C-25M: 100nF, Capacitor_SMD:C_0402_1005Metric, symbol TACCO:S_C-25M
- added C-485-1: 10nF, Capacitor_SMD:C_0201_0603Metric, symbol TACCO:S_C-485-1
- added C-50M: 100nF, Capacitor_SMD:C_0402_1005Metric, symbol TACCO:S_C-50M
- added C-MLRS-SH1: DNP, Capacitor_SMD:C_0201_0603Metric, symbol TACCO:S_C-MLRS-SH1
- added C-MLRS-TCXO: 100nF, Capacitor_SMD:C_0402_1005Metric, symbol TACCO:S_C-MLRS-TCXO
- added C-ZB-33-1: 100nF 6.3V X5R, Capacitor_SMD:C_0201_0603Metric, symbol TACCO:S_C-ZB-33-1
- added R-485T: 120R, Resistor_SMD:R_0402_1005Metric, symbol TACCO:S_R-485T
- added R-BST: 75R, Resistor_SMD:R_0402_1005Metric, symbol TACCO:S_R-BST
- added R-CANT: 120R, Resistor_SMD:R_0402_1005Metric, symbol TACCO:S_R-CANT
- added SW-MLRS: KMR2 tact, Button_Switch_SMD:SW_Push_1P1T_NO_CK_KMR2, symbol TACCO:S_SW-MLRS
- C-1553B: renamed from C-1553A; symbol TACCO:S_C-1553A -> TACCO:S_C-1553B
- C-1553C: renamed from C-1553B; value 100nF -> 10uF 6.3V X5R; footprint Capacitor_SMD:C_0402_1005Metric -> Capacitor_SMD:C_0603_1608Metric; symbol TACCO:S_C-1553B -> TACCO:S_C-1553C
- C-1553D: renamed from C-1553C; value 10uF 6.3V X5R -> 100nF; footprint Capacitor_SMD:C_0603_1608Metric -> Capacitor_SMD:C_0402_1005Metric; symbol TACCO:S_C-1553C -> TACCO:S_C-1553D
- C-485-2: renamed from C-485-1; value 10nF -> 10uF 10V X5R; footprint Capacitor_SMD:C_0201_0603Metric -> Capacitor_SMD:C_0603_1608Metric; symbol TACCO:S_C-485-1 -> TACCO:S_C-485-2
- C-485-3: renamed from C-485-2; value 10uF 10V X5R -> 100nF; footprint Capacitor_SMD:C_0603_1608Metric -> Capacitor_SMD:C_0402_1005Metric; symbol TACCO:S_C-485-2 -> TACCO:S_C-485-3
- C-485-4: renamed from C-485-3; value 100nF -> 10nF; footprint Capacitor_SMD:C_0402_1005Metric -> Capacitor_SMD:C_0201_0603Metric; symbol TACCO:S_C-485-3 -> TACCO:S_C-485-4
- C-485-5: renamed from C-485-4; value 10nF -> 10uF 10V X5R; footprint Capacitor_SMD:C_0201_0603Metric -> Capacitor_SMD:C_0603_1608Metric; symbol TACCO:S_C-485-4 -> TACCO:S_C-485-5
- C-485-6: renamed from C-485-5; value 10uF 10V X5R -> 100nF; footprint Capacitor_SMD:C_0603_1608Metric -> Capacitor_SMD:C_0402_1005Metric; symbol TACCO:S_C-485-5 -> TACCO:S_C-485-6
- C-ANT-SANT: renamed from J-ANT-RADIO; value MMCX vertical -> 10pF; footprint Connector_Coaxial:MMCX_Molex_73415-1471_Vertical -> Capacitor_SMD:C_0201_0603Metric; symbol TACCO:S_J-ANT-RADIO -> TACCO:S_C-ANT-SANT; MPN 73415-1471 -> (none)
- C-ANT-SH1: renamed from J-ANT-MLRS; value MMCX vertical -> DNP; footprint Connector_Coaxial:MMCX_Molex_73415-1471_Vertical -> Capacitor_SMD:C_0402_1005Metric; symbol TACCO:S_J-ANT-MLRS -> TACCO:S_C-ANT-SH1; MPN 73415-1471 -> (none)
- C-ANT-SH2: renamed from L-ANT-SER; value 0R link -> DNP; footprint Resistor_SMD:R_0402_1005Metric -> Capacitor_SMD:C_0402_1005Metric; symbol TACCO:S_L-ANT-SER -> TACCO:S_C-ANT-SH2
- C-BS: renamed from R-BSR; value 75R -> 10nF 2kV; footprint Resistor_SMD:R_0402_1005Metric -> Capacitor_SMD:C_1808_4520Metric; symbol TACCO:S_R-BSR -> TACCO:S_C-BS
- C-CAN1: renamed from C-RF-O2; value 22uF 6.3V X5R -> 10nF; footprint Capacitor_SMD:C_0603_1608Metric -> Capacitor_SMD:C_0201_0603Metric; symbol TACCO:S_C-RF-O2 -> TACCO:S_C-CAN1
- C-CAN2: renamed from C-CAN1; value 10nF -> 10uF 10V X5R; footprint Capacitor_SMD:C_0201_0603Metric -> Capacitor_SMD:C_0603_1608Metric; symbol TACCO:S_C-CAN1 -> TACCO:S_C-CAN2
- C-CAN3: renamed from C-CAN2; value 10uF 10V X5R -> 100nF; footprint Capacitor_SMD:C_0603_1608Metric -> Capacitor_SMD:C_0402_1005Metric; symbol TACCO:S_C-CAN2 -> TACCO:S_C-CAN3
- C-CAN4: renamed from C-CAN3; value 100nF -> 10nF; footprint Capacitor_SMD:C_0402_1005Metric -> Capacitor_SMD:C_0201_0603Metric; symbol TACCO:S_C-CAN3 -> TACCO:S_C-CAN4
- C-CAN5: renamed from C-CAN4; value 10nF -> 10uF 10V X5R; footprint Capacitor_SMD:C_0201_0603Metric -> Capacitor_SMD:C_0603_1608Metric; symbol TACCO:S_C-CAN4 -> TACCO:S_C-CAN5
- C-CAN6: renamed from C-CAN5; value 10uF 10V X5R -> 100nF; footprint Capacitor_SMD:C_0603_1608Metric -> Capacitor_SMD:C_0402_1005Metric; symbol TACCO:S_C-CAN5 -> TACCO:S_C-CAN6
- C-FLASH1: renamed from C-ZB-SDVIO; value 100nF 6.3V X5R -> 100nF; footprint Capacitor_SMD:C_0201_0603Metric -> Capacitor_SMD:C_0402_1005Metric; symbol TACCO:S_C-ZB-SDVIO -> TACCO:S_C-FLASH1
- C-MLRS-BULK: renamed from C-MLRS-SMPS; value 100nF -> 4.7uF; footprint Capacitor_SMD:C_0402_1005Metric -> Capacitor_SMD:C_0603_1608Metric; symbol TACCO:S_C-MLRS-SMPS -> TACCO:S_C-MLRS-BULK
- C-MLRS-HSE: renamed from C-MLRS-TCXO; value 100nF -> 10pF C0G; symbol TACCO:S_C-MLRS-TCXO -> TACCO:S_C-MLRS-HSE
- C-MLRS-RST: renamed from R-MLRS-RST; value 22k -> 100nF; footprint Resistor_SMD:R_0201_0603Metric -> Capacitor_SMD:C_0402_1005Metric; symbol TACCO:S_R-MLRS-RST -> TACCO:S_C-MLRS-RST
- C-MLRS-RX1: renamed from L-MLRS-RX2; footprint Inductor_SMD:L_0402_1005Metric -> Capacitor_SMD:C_0402_1005Metric; symbol TACCO:S_L-MLRS-RX2 -> TACCO:S_C-MLRS-RX1
- C-MLRS-RXN: renamed from C-MLRS-RXP; symbol TACCO:S_C-MLRS-RXP -> TACCO:S_C-MLRS-RXN
- C-MLRS-RXP: renamed from C-MLRS-TX2; symbol TACCO:S_C-MLRS-TX2 -> TACCO:S_C-MLRS-RXP
- C-MLRS-SH2: renamed from L-MLRS-SER; value 0R link -> DNP; footprint Resistor_SMD:R_0402_1005Metric -> Capacitor_SMD:C_0201_0603Metric; symbol TACCO:S_L-MLRS-SER -> TACCO:S_C-MLRS-SH2
- C-MLRS-SMPS: renamed from C-MLRS-VBAT; symbol TACCO:S_C-MLRS-VBAT -> TACCO:S_C-MLRS-SMPS
- C-MLRS-TX0: renamed from L-MLRS-PA; footprint Inductor_SMD:L_0402_1005Metric -> Capacitor_SMD:C_0402_1005Metric; symbol TACCO:S_L-MLRS-PA -> TACCO:S_C-MLRS-TX0
- C-MLRS-TX1: renamed from L-MLRS-TX1; footprint Inductor_SMD:L_0402_1005Metric -> Capacitor_SMD:C_0402_1005Metric; symbol TACCO:S_L-MLRS-TX1 -> TACCO:S_C-MLRS-TX1
- C-MLRS-TX2: renamed from L-MLRS-TX2; footprint Inductor_SMD:L_0402_1005Metric -> Capacitor_SMD:C_0402_1005Metric; symbol TACCO:S_L-MLRS-TX2 -> TACCO:S_C-MLRS-TX2
- C-MLRS-VBAT: renamed from C-MLRS-VDDRF; symbol TACCO:S_C-MLRS-VDDRF -> TACCO:S_C-MLRS-VBAT
- C-MLRS-VDD1: renamed from R-TPM10; value 10k -> 100nF; footprint Resistor_SMD:R_0201_0603Metric -> Capacitor_SMD:C_0402_1005Metric; symbol TACCO:S_R-TPM10 -> TACCO:S_C-MLRS-VDD1
- C-MLRS-VDD2: renamed from C-MLRS-VDD1; symbol TACCO:S_C-MLRS-VDD1 -> TACCO:S_C-MLRS-VDD2
- C-MLRS-VDDA1: renamed from C-MLRS-VDD2; symbol TACCO:S_C-MLRS-VDD2 -> TACCO:S_C-MLRS-VDDA1
- C-MLRS-VDDA2: renamed from C-MLRS-VDDA1; value 100nF -> 1uF; symbol TACCO:S_C-MLRS-VDDA1 -> TACCO:S_C-MLRS-VDDA2
- C-MLRS-VDDPA1: renamed from C-MLRS-BULK; value 4.7uF -> 100nF; footprint Capacitor_SMD:C_0603_1608Metric -> Capacitor_SMD:C_0402_1005Metric; symbol TACCO:S_C-MLRS-BULK -> TACCO:S_C-MLRS-VDDPA1
- C-MLRS-VDDPA2: renamed from C-MLRS-VDDPA1; value 100nF -> 4.7uF; footprint Capacitor_SMD:C_0402_1005Metric -> Capacitor_SMD:C_0603_1608Metric; symbol TACCO:S_C-MLRS-VDDPA1 -> TACCO:S_C-MLRS-VDDPA2
- C-MLRS-VDDRF: renamed from C-MLRS-VDDA2; value 1uF -> 100nF; symbol TACCO:S_C-MLRS-VDDA2 -> TACCO:S_C-MLRS-VDDRF
- C-MLRS-VFB: renamed from C-MLRS-VDDPA2; value 4.7uF -> 470nF; footprint Capacitor_SMD:C_0603_1608Metric -> Capacitor_SMD:C_0402_1005Metric; symbol TACCO:S_C-MLRS-VDDPA2 -> TACCO:S_C-MLRS-VFB
- C-MLRS-VRPA: renamed from L-MLRS-SMPS; value 15uH -> 100nF VERIFY AN5457; footprint Inductor_SMD:L_0603_1608Metric -> Capacitor_SMD:C_0402_1005Metric; symbol TACCO:S_L-MLRS-SMPS -> TACCO:S_C-MLRS-VRPA
- C-PHY-A1: renamed from R-AD0; value 2.49k -> 10nF; footprint Resistor_SMD:R_0201_0603Metric -> Capacitor_SMD:C_0201_0603Metric; symbol TACCO:S_R-AD0 -> TACCO:S_C-PHY-A1
- C-PHY-A2: renamed from C-PHY-A1; value 10nF -> 100nF; footprint Capacitor_SMD:C_0201_0603Metric -> Capacitor_SMD:C_0402_1005Metric; symbol TACCO:S_C-PHY-A1 -> TACCO:S_C-PHY-A2
- C-PHY-A3: renamed from C-PHY-A2; value 100nF -> 1uF; symbol TACCO:S_C-PHY-A2 -> TACCO:S_C-PHY-A3
- C-PHY-CRD1: renamed from C-PHY-CTD2; value 1uF -> 100nF; symbol TACCO:S_C-PHY-CTD2 -> TACCO:S_C-PHY-CRD1
- C-PHY-CRD2: renamed from C-PHY-CRD1; value 100nF -> 1uF; symbol TACCO:S_C-PHY-CRD1 -> TACCO:S_C-PHY-CRD2
- C-PHY-CTD1: renamed from C-PHY-A3; value 1uF -> 100nF; symbol TACCO:S_C-PHY-A3 -> TACCO:S_C-PHY-CTD1
- C-PHY-CTD2: renamed from C-PHY-CTD1; value 100nF -> 1uF; symbol TACCO:S_C-PHY-CTD1 -> TACCO:S_C-PHY-CTD2
- C-PLD1: renamed from R-FLASH-WP; value 10k -> 100nF; footprint Resistor_SMD:R_0201_0603Metric -> Capacitor_SMD:C_0402_1005Metric; symbol TACCO:S_R-FLASH-WP -> TACCO:S_C-PLD1
- C-RF-IN1: renamed from L-RF2; value 2.2uH 3A -> 10uF 10V X5R; footprint Inductor_SMD:L_Wuerth_MAPI-3015 -> Capacitor_SMD:C_0603_1608Metric; symbol TACCO:S_L-RF2 -> TACCO:S_C-RF-IN1; MPN LPS3015-222MRC -> (none)
- C-RF-IN2: renamed from C-RF-IN1; value 10uF 10V X5R -> 100nF; footprint Capacitor_SMD:C_0603_1608Metric -> Capacitor_SMD:C_0402_1005Metric; symbol TACCO:S_C-RF-IN1 -> TACCO:S_C-RF-IN2
- C-RF-O1: renamed from C-RF-IN2; value 100nF -> 22uF 6.3V X5R; footprint Capacitor_SMD:C_0402_1005Metric -> Capacitor_SMD:C_0603_1608Metric; symbol TACCO:S_C-RF-IN2 -> TACCO:S_C-RF-O1
- C-RF-O2: renamed from C-RF-O1; symbol TACCO:S_C-RF-O1 -> TACCO:S_C-RF-O2
- C-TPM1: renamed from C-50M; value 100nF -> 1uF; symbol TACCO:S_C-50M -> TACCO:S_C-TPM1
- C-TPM2: renamed from C-TPM1; value 1uF -> 100nF 6.3V X5R; footprint Capacitor_SMD:C_0402_1005Metric -> Capacitor_SMD:C_0201_0603Metric; symbol TACCO:S_C-TPM1 -> TACCO:S_C-TPM2
- C-TPM3: renamed from C-TPM2; symbol TACCO:S_C-TPM2 -> TACCO:S_C-TPM3
- C-TPM4: renamed from C-TPM3; symbol TACCO:S_C-TPM3 -> TACCO:S_C-TPM4
- C-ZB-18-1: renamed from C-ZB-33-2; symbol TACCO:S_C-ZB-33-2 -> TACCO:S_C-ZB-18-1
- C-ZB-18-2: renamed from C-ZB-18-1; symbol TACCO:S_C-ZB-18-1 -> TACCO:S_C-ZB-18-2
- C-ZB-33-2: renamed from C-ZB-33-1; symbol TACCO:S_C-ZB-33-1 -> TACCO:S_C-ZB-33-2
- C-ZB-SDVIO: renamed from C-ZB-VIO; symbol TACCO:S_C-ZB-VIO -> TACCO:S_C-ZB-SDVIO
- C-ZB-VIO: renamed from C-ZB-18-2; symbol TACCO:S_C-ZB-18-2 -> TACCO:S_C-ZB-VIO
- CMC-CAN: renamed from C-CAN6; value 100nF -> SRF2012-100Y; footprint Capacitor_SMD:C_0402_1005Metric -> Serenity-Custom:Bourns_SRF2012_4T; symbol TACCO:S_C-CAN6 -> TACCO:S_CMC-CAN; MPN (none) -> SRF2012-121YA
- CMC-RS485: renamed from C-485-6; value 100nF -> SRF2012-100Y; footprint Capacitor_SMD:C_0402_1005Metric -> Serenity-Custom:Bourns_SRF2012_4T; symbol TACCO:S_C-485-6 -> TACCO:S_CMC-RS485; MPN (none) -> SRF2012-121YA
- D-ANT-MLRS: renamed from C-MLRS-SH2; value DNP -> RCLAMP0502B; footprint Capacitor_SMD:C_0201_0603Metric -> Serenity-Custom:RCLAMP0502B_SOD882; symbol TACCO:S_C-MLRS-SH2 -> TACCO:S_D-ANT-MLRS; MPN (none) -> RCLAMP0502BTCL
- D-ANT-RADIO: renamed from C-ANT-SH2; value DNP -> RCLAMP0502B; footprint Capacitor_SMD:C_0402_1005Metric -> Serenity-Custom:RCLAMP0502B_SOD882; symbol TACCO:S_C-ANT-SH2 -> TACCO:S_D-ANT-RADIO; MPN (none) -> RCLAMP0502BTCL
- FB-MLRS-1: renamed from R-MLRS-BOOT0; value 10k -> 600R@100MHz 0402; footprint Resistor_SMD:R_0201_0603Metric -> Inductor_SMD:L_0402_1005Metric; symbol TACCO:S_R-MLRS-BOOT0 -> TACCO:S_FB-MLRS-1
- FB-MLRS-2: renamed from FB-MLRS-1; symbol TACCO:S_FB-MLRS-1 -> TACCO:S_FB-MLRS-2
- H1: renamed from C-ANT-SANT; value 10pF -> M2.5 PGND; footprint Capacitor_SMD:C_0201_0603Metric -> Serenity-Custom:MountingHole_2.7mm_M2.5_PGND_Ring; symbol TACCO:S_C-ANT-SANT -> TACCO:S_H1
- J-1553: renamed from TVS-1553N; value SMAJ33CA -> SM04B-GHS-TB; footprint Diode_SMD:D_SMA -> Connector_JST:JST_GH_SM04B-GHS-TB_1x04-1MP_P1.25mm_Horizontal; symbol TACCO:S_TVS-1553N -> TACCO:S_J-1553; MPN SMAJ33CA -> SM04B-GHS-TB(LF)(SN)
- J-485: renamed from R-485T; value 120R -> SM03B-GHS-TB; footprint Resistor_SMD:R_0402_1005Metric -> Connector_JST:JST_GH_SM03B-GHS-TB_1x03-1MP_P1.25mm_Horizontal; symbol TACCO:S_R-485T -> TACCO:S_J-485; MPN (none) -> SM03B-GHS-TB(LF)(SN); now fitted
- J-ANT-MLRS: renamed from D-ANT-MLRS; value RCLAMP0502B -> MMCX vertical; footprint Serenity-Custom:RCLAMP0502B_SOD882 -> Connector_Coaxial:MMCX_Molex_73415-1471_Vertical; symbol TACCO:S_D-ANT-MLRS -> TACCO:S_J-ANT-MLRS; MPN RCLAMP0502BTCL -> 73415-1471
- J-ANT-RADIO: renamed from D-ANT-RADIO; value RCLAMP0502B -> MMCX vertical; footprint Serenity-Custom:RCLAMP0502B_SOD882 -> Connector_Coaxial:MMCX_Molex_73415-1471_Vertical; symbol TACCO:S_D-ANT-RADIO -> TACCO:S_J-ANT-RADIO; MPN RCLAMP0502BTCL -> 73415-1471
- J-CAN: renamed from R-CANT; value 120R -> SM03B-GHS-TB; footprint Resistor_SMD:R_0402_1005Metric -> Connector_JST:JST_GH_SM03B-GHS-TB_1x03-1MP_P1.25mm_Horizontal; symbol TACCO:S_R-CANT -> TACCO:S_J-CAN; MPN (none) -> SM03B-GHS-TB(LF)(SN); now fitted
- J-FAN: renamed from C-PLD1; value 100nF -> SM03B-GHS-TB; footprint Capacitor_SMD:C_0402_1005Metric -> Connector_JST:JST_GH_SM03B-GHS-TB_1x03-1MP_P1.25mm_Horizontal; symbol TACCO:S_C-PLD1 -> TACCO:S_J-FAN; MPN (none) -> SM03B-GHS-TB(LF)(SN)
- J-MLRS-SWD: renamed from R-MLRS-SWCLK; value 22R -> TC2030-IDC-NL pads; footprint Resistor_SMD:R_0201_0603Metric -> Connector:Tag-Connect_TC2030-IDC-NL_2x03_P1.27mm_Vertical; symbol TACCO:S_R-MLRS-SWCLK -> TACCO:S_J-MLRS-SWD; now not fitted
- L-ANT-SER: renamed from C-ANT-SH1; value DNP -> 0R link; footprint Capacitor_SMD:C_0402_1005Metric -> Resistor_SMD:R_0402_1005Metric; symbol TACCO:S_C-ANT-SH1 -> TACCO:S_L-ANT-SER
- L-MLRS-PA: renamed from LED-MLRS-R; value Red -> VERIFY AN5457; footprint LED_SMD:LED_0603_1608Metric -> Inductor_SMD:L_0402_1005Metric; symbol TACCO:S_LED-MLRS-R -> TACCO:S_L-MLRS-PA
- L-MLRS-RX1: renamed from C-MLRS-RXN; footprint Capacitor_SMD:C_0402_1005Metric -> Inductor_SMD:L_0402_1005Metric; symbol TACCO:S_C-MLRS-RXN -> TACCO:S_L-MLRS-RX1
- L-MLRS-RX2: renamed from L-MLRS-RX1; symbol TACCO:S_L-MLRS-RX1 -> TACCO:S_L-MLRS-RX2
- L-MLRS-SER: renamed from C-MLRS-SH1; value DNP -> 0R link; footprint Capacitor_SMD:C_0201_0603Metric -> Resistor_SMD:R_0402_1005Metric; symbol TACCO:S_C-MLRS-SH1 -> TACCO:S_L-MLRS-SER
- L-MLRS-SMPS: renamed from C-MLRS-VFB; value 470nF -> 15uH; footprint Capacitor_SMD:C_0402_1005Metric -> Inductor_SMD:L_0603_1608Metric; symbol TACCO:S_C-MLRS-VFB -> TACCO:S_L-MLRS-SMPS
- L-MLRS-TX1: renamed from C-MLRS-TX0; footprint Capacitor_SMD:C_0402_1005Metric -> Inductor_SMD:L_0402_1005Metric; symbol TACCO:S_C-MLRS-TX0 -> TACCO:S_L-MLRS-TX1
- L-MLRS-TX2: renamed from C-MLRS-TX1; footprint Capacitor_SMD:C_0402_1005Metric -> Inductor_SMD:L_0402_1005Metric; symbol TACCO:S_C-MLRS-TX1 -> TACCO:S_L-MLRS-TX2
- L-RF1: value 2.2uH 3A -> 1.5uH; MPN LPS3015-222MRC -> LPS3015-152MRC
- LED-MLRS-G: renamed from R-MLRS-LEDG; value 1k -> Green; footprint Resistor_SMD:R_0201_0603Metric -> LED_SMD:LED_0603_1608Metric; symbol TACCO:S_R-MLRS-LEDG -> TACCO:S_LED-MLRS-G
- LED-MLRS-R: renamed from R-MLRS-LEDR; value 1k -> Red; footprint Resistor_SMD:R_0201_0603Metric -> LED_SMD:LED_0603_1608Metric; symbol TACCO:S_R-MLRS-LEDR -> TACCO:S_LED-MLRS-R
- PB2-P1: footprint Serenity-Custom:PocketBeagle2_2x18_P1_Socket -> Serenity-Custom:PocketBeagle2_2x18_P1_SSM-DV-LC; MPN (none) -> SSM-118-L-DV-LC
- PB2-P2: footprint Serenity-Custom:PocketBeagle2_2x18_P2_Socket -> Serenity-Custom:PocketBeagle2_2x18_P2_SSM-DV-LC; MPN (none) -> SSM-118-L-DV-LC
- R-1553IRQ: renamed from C-1553D; value 100nF -> 10k; footprint Capacitor_SMD:C_0402_1005Metric -> Resistor_SMD:R_0402_1005Metric; symbol TACCO:S_C-1553D -> TACCO:S_R-1553IRQ
- R-1553N: renamed from R-1553P; symbol TACCO:S_R-1553P -> TACCO:S_R-1553N
- R-1553P: renamed from C-PHY-CRD2; value 1uF -> 55R 2%; footprint Capacitor_SMD:C_0402_1005Metric -> Resistor_SMD:R_0603_1608Metric; symbol TACCO:S_C-PHY-CRD2 -> TACCO:S_R-1553P
- R-AD0: renamed from R-RBIAS; value 6.49k 1% -> 2.49k; symbol TACCO:S_R-RBIAS -> TACCO:S_R-AD0
- R-BSR: renamed from R-BST; symbol TACCO:S_R-BST -> TACCO:S_R-BSR
- R-FLASH-WP: renamed from C-FLASH1; value 100nF -> 10k; footprint Capacitor_SMD:C_0402_1005Metric -> Resistor_SMD:R_0201_0603Metric; symbol TACCO:S_C-FLASH1 -> TACCO:S_R-FLASH-WP
- R-MLRS-BOOT0: renamed from C-MLRS-RST; value 100nF -> 10k; footprint Capacitor_SMD:C_0402_1005Metric -> Resistor_SMD:R_0201_0603Metric; symbol TACCO:S_C-MLRS-RST -> TACCO:S_R-MLRS-BOOT0
- R-MLRS-LEDG: renamed from SW-MLRS; value KMR2 tact -> 1k; footprint Button_Switch_SMD:SW_Push_1P1T_NO_CK_KMR2 -> Resistor_SMD:R_0201_0603Metric; symbol TACCO:S_SW-MLRS -> TACCO:S_R-MLRS-LEDG
- R-MLRS-LEDR: renamed from LED-MLRS-G; value Green -> 1k; footprint LED_SMD:LED_0603_1608Metric -> Resistor_SMD:R_0201_0603Metric; symbol TACCO:S_LED-MLRS-G -> TACCO:S_R-MLRS-LEDR
- R-MLRS-RST: renamed from C-MLRS-HSE; value 10pF C0G -> 22k; footprint Capacitor_SMD:C_0402_1005Metric -> Resistor_SMD:R_0201_0603Metric; symbol TACCO:S_C-MLRS-HSE -> TACCO:S_R-MLRS-RST
- R-MLRS-SWCLK: renamed from R-MLRS-SWDIO; symbol TACCO:S_R-MLRS-SWDIO -> TACCO:S_R-MLRS-SWCLK
- R-MLRS-SWDIO: renamed from FB-MLRS-2; value 600R@100MHz 0402 -> 22R; footprint Inductor_SMD:L_0402_1005Metric -> Resistor_SMD:R_0201_0603Metric; symbol TACCO:S_FB-MLRS-2 -> TACCO:S_R-MLRS-SWDIO
- R-RBIAS: renamed from C-25M; value 100nF -> 6.49k 1%; footprint Capacitor_SMD:C_0402_1005Metric -> Resistor_SMD:R_0201_0603Metric; symbol TACCO:S_C-25M -> TACCO:S_R-RBIAS
- R-TPM10: renamed from R-TPMCS; symbol TACCO:S_R-TPMCS -> TACCO:S_R-TPM10
- R-TPMCS: renamed from C-TPM4; value 100nF 6.3V X5R -> 10k; footprint Capacitor_SMD:C_0201_0603Metric -> Resistor_SMD:R_0201_0603Metric; symbol TACCO:S_C-TPM4 -> TACCO:S_R-TPMCS
- RFSW-MLRS: renamed from C-MLRS-RX1; value VERIFY AN5457 -> PE4259; footprint Capacitor_SMD:C_0402_1005Metric -> Package_TO_SOT_SMD:SOT-363_SC-70-6; symbol TACCO:S_C-MLRS-RX1 -> TACCO:S_RFSW-MLRS; MPN (none) -> PE4259-63
- TVS-1553N: renamed from TVS-1553P; symbol TACCO:S_TVS-1553P -> TACCO:S_TVS-1553N
- TVS-1553P: renamed from R-1553N; value 55R 2% -> SMAJ33CA; footprint Resistor_SMD:R_0603_1608Metric -> Diode_SMD:D_SMA; symbol TACCO:S_R-1553N -> TACCO:S_TVS-1553P; MPN (none) -> SMAJ33CA
- X-25M: renamed from C-BS; value 10nF 2kV -> 25MHz 3.3V; footprint Capacitor_SMD:C_1808_4520Metric -> Oscillator:Oscillator_SMD_ECS_2520MV-xxx-xx-4Pin_2.5x2.0mm; symbol TACCO:S_C-BS -> TACCO:S_X-25M; MPN (none) -> ECS-2520MV-250-BN-TR
- X-50M: renamed from R-1553IRQ; value 10k -> 50MHz 3.3V; footprint Resistor_SMD:R_0402_1005Metric -> Oscillator:Oscillator_SMD_ECS_2520MV-xxx-xx-4Pin_2.5x2.0mm; symbol TACCO:S_R-1553IRQ -> TACCO:S_X-50M; MPN (none) -> ECS-2520MV-500-BN-TR
- X-MLRS: renamed from C-MLRS-VRPA; value 100nF VERIFY AN5457 -> TG2520SMN 32MHz 1.8V clipped-sine; footprint Capacitor_SMD:C_0402_1005Metric -> Oscillator:Oscillator_SMD_SeikoEpson_TG2520SMN-xxx-xxxxxx-4Pin_2.5x2.0mm; symbol TACCO:S_C-MLRS-VRPA -> TACCO:S_X-MLRS
Connections:
- net +1V8_RF: now also C-ZB-18-1.1 (P), C-ZB-SDVIO.1 (P); no longer C-FLASH1.1 (P), C-ZB-VIO.1 (P)
- net +3V3: now also C-485-3.1 (P), C-CAN3.1 (P), C-FLASH1.1 (P), C-ZB-VIO.1 (P), R-AD0.1 (A), X-25M.4 (VDD), X-50M.4 (VDD), C-1553A.1 (P), C-25M.1 (P), C-50M.1 (P); no longer C-485-4.1 (P), C-CAN4.1 (P), C-MLRS-VDD1.1 (A), C-PHY-CTD1.1 (P), C-ZB-SDVIO.1 (P), J-FAN.1 (P), R-RBIAS.1 (P), X-50M.1 (A)
- net +3V3_RF: now also C-MLRS-VDD1.1 (P), C-RF-O1.1 (P), J-MLRS-SWD.1 (VTREF), R-MLRS-LEDR.1 (A), R-MLRS-RST.1 (A), C-ZB-33-1.1 (P); no longer C-CAN1.1 (P), C-MLRS-RST.1 (A), C-MLRS-VFB.1 (P), C-RF-IN1.2 (B), C-ZB-18-1.1 (P), LED-MLRS-R.1 (A)
- net +5V: now also C-CAN1.1 (P), C-RF-IN1.1 (P), J-FAN.2 (+5V), C-485-1.1 (P); no longer C-485-3.1 (P), C-CAN3.1 (P), C-RF-O1.1 (P), L-RF1.2 (B)
- net BUS_1553_B_N: now also J-1553.2 (BUS_N), R-1553N.2 (B), TVS-1553N.1 (A); no longer J-1553.1 (A), TVS-1553P.2 (B)
- net BUS_1553_B_P: now also J-1553.1 (BUS_P), R-1553P.2 (B), TVS-1553P.1 (A); no longer R-1553N.2 (B), TVS-1553N.1 (A)
- net CAN_B_H: now also CMC-CAN.1 (W1_IN)
- net CAN_B_H_F: now also CMC-CAN.2 (W1_OUT), R-CANT.1 (A)
- net CAN_B_L: now also CMC-CAN.4 (W2_IN)
- net CAN_B_L_F: now also CMC-CAN.3 (W2_OUT), R-CANT.2 (B)
- net ETH-PHY_RBIAS: now also R-RBIAS.1 (A); no longer R-AD0.1 (A)
- net ETHB_BS: now also C-BS.1 (P), R-BST.2 (B); no longer C-BS.2 (B), X-25M.1 (P)
- net ETHB_CRD: now also C-PHY-CRD1.1 (P); no longer R-1553P.1 (P)
- net ETHB_CTD: now also C-PHY-CTD1.1 (P); no longer C-PHY-CRD1.1 (P)
- net ETHB_LINE_CRX: now also R-BSR.1 (A); no longer C-BS.1 (A)
- net ETHB_LINE_CTX: now also R-BST.1 (A); no longer R-BSR.1 (A)
- net FAN_PWM_B: now also J-FAN.3 (FAN_PWM)
- net FLASH_WP_N: now also R-FLASH-WP.2 (B); no longer C-PLD1.2 (B)
- net GND: now also C-ANT-SH1.2 (B), C-ANT-SH2.2 (B), C-MLRS-RST.2 (N), C-MLRS-SH2.2 (B), C-MLRS-TX1.2 (B), C-MLRS-TX2.2 (B), C-MLRS-VDD1.2 (N), C-MLRS-VRPA.2 (N), C-PHY-A1.2 (N), C-PLD1.2 (N), C-RF-IN1.2 (N), J-1553.3 (GND), J-FAN.1 (GND), J-MLRS-SWD.5 (GND), L-MLRS-RX2.2 (B), LED-MLRS-G.2 (K), X-25M.2 (GND), X-50M.2 (GND), C-1553A.2 (N), C-25M.2 (N), C-485-1.2 (N), C-50M.2 (N), C-MLRS-SH1.2 (B), C-MLRS-TCXO.2 (N), C-ZB-33-1.2 (N), SW-MLRS.2 (B); no longer C-485-4.2 (N), C-CAN4.2 (N), C-MLRS-HSE.2 (N), C-MLRS-RXP.2 (B), D-ANT-MLRS.2 (B), D-ANT-RADIO.2 (B), FB-MLRS-1.2 (B), J-FAN.2 (N), L-ANT-SER.2 (B), L-MLRS-SER.2 (B), L-MLRS-SMPS.2 (N), L-MLRS-TX2.2 (B), R-1553IRQ.2 (N), R-1553P.2 (N), R-AD0.2 (B), R-FLASH-WP.2 (N), R-MLRS-LEDG.2 (B), R-MLRS-LEDR.2 (K), R-TPMCS.2 (N)
- net GND2_CANB: now also C-CAN4.2 (N), J-CAN.3 (GND); no longer CMC-CAN.2 (N)
- net GND2_RS485B: now also C-485-4.2 (N), J-485.3 (GND); no longer CMC-RS485.2 (N)
- net M1553B_IRQN: now also R-1553IRQ.2 (B); no longer X-50M.2 (B)
- net M1553B_MCLK: now also X-50M.3 (OUT)
- net M1553B_SEC_N: now also R-1553N.1 (A); no longer TVS-1553P.1 (A)
- net M1553B_SEC_P: now also R-1553P.1 (A); no longer R-1553N.1 (A)
- net MLRS_ANT_F: now also C-MLRS-SH2.1 (A), L-MLRS-SER.2 (B); no longer C-ANT-SH1.1 (RF), C-MLRS-SH2.2 (B)
- net MLRS_ANT_RF: now also RFSW-MLRS.5 (RFC), C-MLRS-SH1.1 (A); no longer C-MLRS-SH2.1 (A)
- net MLRS_BOOT0: now also R-MLRS-BOOT0.1 (A); no longer FB-MLRS-1.1 (A)
- net MLRS_BTN: now also SW-MLRS.1 (A); no longer R-MLRS-LEDG.1 (A)
- net MLRS_HSE_IN: now also C-MLRS-HSE.2 (B); no longer R-MLRS-RST.2 (B)
- net MLRS_LEDG_A: now also LED-MLRS-G.1 (A), R-MLRS-LEDG.2 (B); no longer LED-MLRS-G.2 (B), R-MLRS-LEDR.1 (A)
- net MLRS_LEDR_A: now also LED-MLRS-R.1 (A), R-MLRS-LEDR.2 (B); no longer L-MLRS-PA.1 (A), LED-MLRS-R.2 (B)
- net MLRS_LED_G: now also R-MLRS-LEDG.1 (A); no longer LED-MLRS-G.1 (A)
- net MLRS_LED_R: now also LED-MLRS-R.2 (K); no longer L-MLRS-PA.2 (K)
- net MLRS_RFI_N: now also C-MLRS-RXN.1 (A); no longer L-MLRS-RX1.1 (A)
- net MLRS_RFI_P: now also C-MLRS-RXP.1 (A); no longer C-MLRS-RXN.1 (A)
- net MLRS_RFO_HP: now also C-MLRS-TX0.1 (A), L-MLRS-PA.2 (B); no longer C-MLRS-TX0.2 (B), L-MLRS-TX1.1 (A)
- net MLRS_RF_RX_EN: now also RFSW-MLRS.4 (CTRL)
- net MLRS_RF_TX_EN: now also RFSW-MLRS.6 (CTRLB)
- net MLRS_RST: now also C-MLRS-RST.1 (P), J-MLRS-SWD.3 (nRESET), R-MLRS-RST.2 (B); no longer C-MLRS-RST.2 (B), R-MLRS-BOOT0.1 (P)
- net MLRS_RX1: now also C-MLRS-RXP.2 (B), L-MLRS-RX1.1 (A); no longer C-MLRS-RXN.2 (B), L-MLRS-RX2.1 (A)
- net MLRS_RX2: now also C-MLRS-RXN.2 (B), L-MLRS-RX2.1 (A); no longer C-MLRS-RX1.1 (A), L-MLRS-RX1.2 (B)
- net MLRS_RX_F: now also C-MLRS-RX1.1 (A), L-MLRS-RX1.2 (B); no longer L-MLRS-RX2.2 (B)
- net MLRS_SWCLK: now also R-MLRS-SWCLK.1 (A); no longer J-MLRS-SWD.1 (A)
- net MLRS_SWCLK_HDR: now also J-MLRS-SWD.4 (SWCLK), R-MLRS-SWCLK.2 (B); no longer J-MLRS-SWD.2 (B)
- net MLRS_SWDIO: now also R-MLRS-SWDIO.1 (A); no longer R-MLRS-SWCLK.1 (A)
- net MLRS_SWDIO_HDR: now also J-MLRS-SWD.2 (SWDIO), R-MLRS-SWDIO.2 (B); no longer R-MLRS-SWCLK.2 (B)
- net MLRS_TCXO_OUT: now also C-MLRS-HSE.1 (A), X-MLRS.3 (OUT); no longer R-MLRS-RST.1 (A)
- net MLRS_TX1: now also C-MLRS-TX0.2 (B), L-MLRS-TX1.1 (A); no longer C-MLRS-TX1.1 (A), L-MLRS-TX1.2 (B)
- net MLRS_TX2: now also C-MLRS-TX1.1 (A), L-MLRS-TX1.2 (B); no longer C-MLRS-TX1.2 (B), C-MLRS-TX2.1 (A)
- net MLRS_TX_F: now also C-MLRS-TX2.1 (A), L-MLRS-TX2.2 (B), RFSW-MLRS.3 (RF2); no longer C-MLRS-RXP.1 (A), C-MLRS-TX2.2 (B)
- net MLRS_VDDTCXO: now also X-MLRS.4 (VCC), C-MLRS-TCXO.1 (P); no longer C-MLRS-HSE.1 (P)
- net MLRS_VFB: now also C-MLRS-VFB.1 (P), L-MLRS-SMPS.2 (B); no longer C-MLRS-VRPA.2 (B), L-MLRS-SMPS.1 (P)
- net MLRS_VLX: now also L-MLRS-SMPS.1 (A); no longer C-MLRS-VRPA.1 (A)
- net MLRS_VR_PA: now also C-MLRS-VRPA.1 (P), L-MLRS-PA.1 (A); no longer C-MLRS-TX0.1 (A), X-MLRS.1 (P)
- net PGND: now also C-BS.2 (N), D-ANT-MLRS.2 (K), D-ANT-RADIO.2 (K), H1.1 (PGND), J-1553.4 (SHIELD), J-1553.MP (SHIELD), J-485.MP (SHIELD), J-CAN.MP (SHIELD), TVS-1553P.2 (K); no longer C-ANT-SANT.2 (SHIELD), C-ANT-SH1.2 (SHIELD), J-1553.2 (K), X-25M.2 (N)
- net PHY_XI_25M: now also X-25M.3 (OUT)
- net RADIO_ANT1_IN: now also C-ANT-SANT.2 (B); no longer H1.2 (B)
- net RADIO_ANT1_OUT: now also C-ANT-SANT.1 (A); no longer H1.1 (A)
- net RADIO_ANT_F: now also C-ANT-SH2.1 (A), L-ANT-SER.2 (B); no longer C-ANT-SANT.1 (RF), C-ANT-SH2.2 (B)
- net RADIO_ANT_RF: now also C-ANT-SH1.1 (A); no longer C-ANT-SH2.1 (A)
- net RF_SW2: now also L-RF1.2 (B); no longer C-RF-IN1.1 (A)
- net RMII2_RXD0: now also R-AD0.2 (B); no longer C-PHY-A1.2 (B)
- net RS485_B_A: now also CMC-RS485.1 (W1_IN)
- net RS485_B_A_F: now also CMC-RS485.2 (W1_OUT), R-485T.1 (A)
- net RS485_B_B: now also CMC-RS485.4 (W2_IN)
- net RS485_B_B_F: now also CMC-RS485.3 (W2_OUT), R-485T.2 (B)
- net SPI0_B_CS_TPM: now also R-TPMCS.2 (B); no longer R-TPM10.2 (B)
- net TPM_B_P10_PU: now also R-TPM10.2 (B); no longer C-MLRS-VDD1.2 (B)
- net UART_WIOE5_RX: now also FB-MLRS-1.1 (IN); no longer FB-MLRS-2.1 (IN)
- net UART_WIOE5_RX_F: now also FB-MLRS-1.2 (OUT); no longer FB-MLRS-2.2 (OUT)
- net UART_WIOE5_TX: now also FB-MLRS-2.1 (IN); no longer R-MLRS-SWDIO.1 (IN)
- net UART_WIOE5_TX_F: now also FB-MLRS-2.2 (OUT); no longer R-MLRS-SWDIO.2 (OUT)
- net VCC2_CANB: now also C-CAN4.1 (P); no longer CMC-CAN.1 (P)
- net VCC2_RS485B: now also C-485-4.1 (P); no longer CMC-RS485.1 (P)
Other:
- moved on the sheet: C-1553B, C-1553C, C-1553D, C-ANT-SANT, C-ANT-SH1, C-ANT-SH2, C-BS, C-FLASH1, C-MLRS-BULK, C-MLRS-HSE, C-MLRS-RST, C-MLRS-RX1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

Commit message: TACCO: antenna jacks to Hirose U.FL SMT; seeded placement-order what-if
Owner 2026-10-05: J-ANT-RADIO / J-ANT-MLRS move from through-hole MMCX to U.FL-R-SMT-1(10)
to free bottom-face area; WBS records the strain-relief requirement. Generator gains a
what-if 'seed' to search placement orders. 1553-XCVR still parked off-outline (KiCad
validator: 0 hard).

Co-Authored-By: Claude Opus 5.5 <noreply@anthropic.com>
Claude-Session: https://claude.ai/code/session_01YLwDy53g1VCBzNBwW4moUC
Parts:
- J-ANT-MLRS, J-ANT-RADIO: value MMCX vertical -> U.FL; footprint Connector_Coaxial:MMCX_Molex_73415-1471_Vertical -> Connector_Coaxial:U.FL_Hirose_U.FL-R-SMT-1_Vertical; MPN 73415-1471 -> U.FL-R-SMT-1(10)
Changed lines of the file:
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@@
     (exclude_from_sim no) (in_bom yes) (on_board yes) (dnp no)
     (property "Reference" "J-ANT-MLRS" (at 520.70 298.45 0) (effects (font (size 1.27 1.27))))
-    (property "Value" "MMCX vertical" (at 520.70 306.07 0) (effects (font (size 1.27 1.27))))
-    (property "Footprint" "Connector_Coaxial:MMCX_Molex_73415-1471_Vertical" (at 520.70 302.26 0) (effects (font (size 1.27 1.27)) (hide yes)))
-    (property "Datasheet" "mLRS antenna jack — same vertical-MMCX board-area rationale as the WiFi/BT/802.15.4 jack" (at 520.70 302.26 0) (effects (font (size 1.27 1.27)) (hide yes)))
-    (property "MPN" "73415-1471" (at 520.70 302.26 0) (effects (font (size 1.27 1.27)) (hide yes)))
+    (property "Value" "U.FL" (at 520.70 306.07 0) (effects (font (size 1.27 1.27))))
+    (property "Footprint" "Connector_Coaxial:U.FL_Hirose_U.FL-R-SMT-1_Vertical" (at 520.70 302.26 0) (effects (font (size 1.27 1.27)) (hide yes)))
+    (property "Datasheet" "mLRS antenna jack — Hirose U.FL SMT (owner 2026-10-05: replaces the through-hole MMCX, whose pins blocked both faces; KiCad library land, Hirose drawing to be archived; cable needs a tie-down/adhesive strain relief)" (at 520.70 302.26 0) (effects (font (size 1.27 1.27)) (hide yes)))
+    (property "MPN" "U.FL-R-SMT-1(10)" (at 520.70 302.26 0) (effects (font (size 1.27 1.27)) (hide yes)))
     (pin "1")
     (pin "2")
@@
     (exclude_from_sim no) (in_bom yes) (on_board yes) (dnp no)
     (property "Reference" "J-ANT-RADIO" (at 520.70 400.05 0) (effects (font (size 1.27 1.27))))
-    (property "Value" "MMCX vertical" (at 520.70 407.67 0) (effects (font (size 1.27 1.27))))
-    (property "Footprint" "Connector_Coaxial:MMCX_Molex_73415-1471_Vertical" (at 520.70 403.86 0) (effects (font (size 1.27 1.27)) (hide yes)))
-    (property "Datasheet" "Shared WiFi/BT/802.15.4 antenna jack (SANT mode) — was WiFi-only J-SMA-WIFI; Type2EL's single ANT0 feed now serves all three radios, so XO drops from needing (at minimum) two antenna jacks/chains down to one" (at 520.70 403.86 0) (effects (font (size 1.27 1.27)) (hide yes)))
-    (property "MPN" "73415-1471" (at 520.70 403.86 0) (effects (font (size 1.27 1.27)) (hide yes)))
+    (property "Value" "U.FL" (at 520.70 407.67 0) (effects (font (size 1.27 1.27))))
+    (property "Footprint" "Connector_Coaxial:U.FL_Hirose_U.FL-R-SMT-1_Vertical" (at 520.70 403.86 0) (effects (font (size 1.27 1.27)) (hide yes)))
+    (property "Datasheet" "Hirose U.FL SMT (owner 2026-10-05, replaces through-hole MMCX 73415-1471). Shared WiFi/BT/802.15.4 antenna jack (SANT mode) — was WiFi-only J-SMA-WIFI; Type2EL's single ANT0 feed now serves all three radios, so XO drops from needing (at minimum) two antenna jacks/chains down to one" (at 520.70 403.86 0) (effects (font (size 1.27 1.27)) (hide yes)))
+    (property "MPN" "U.FL-R-SMT-1(10)" (at 520.70 403.86 0) (effects (font (size 1.27 1.27)) (hide yes)))
     (pin "1")
     (pin "2")

Commit message: TACCO: male TSM-118-04-L-DV-LC rails and PB2-I height budget (owner 2026-10-05)
The PB2-I carries female receptacles (3.0 mm tall), so the cape needs male pins: Samtec
TSM-DV land per samtec_tsm-dv-footprint.pdf Rev F, -04 shortest post, -LC clip holes; the
unusable SSM-DV socket footprints are removed. Placer gains a bottom-face height budget
(5.54 mm stack gap, 0.5 mm margin, reduced over the PB2-I microSD and JST). T-ETH moves to
the top face, J-SD to the bottom, PWR-IN off the P1 rail. 1553-XFM still unplaced
(KiCad validator: 0 hard). Pilot rails follow.

Co-Authored-By: Claude Opus 5.5 <noreply@anthropic.com>
Claude-Session: https://claude.ai/code/session_01YLwDy53g1VCBzNBwW4moUC
Parts:
- PB2-P1: footprint Serenity-Custom:PocketBeagle2_2x18_P1_SSM-DV-LC -> Serenity-Custom:PocketBeagle2_2x18_P1_TSM-DV-LC; MPN SSM-118-L-DV-LC -> TSM-118-04-L-DV-LC
- PB2-P2: footprint Serenity-Custom:PocketBeagle2_2x18_P2_SSM-DV-LC -> Serenity-Custom:PocketBeagle2_2x18_P2_TSM-DV-LC; MPN SSM-118-L-DV-LC -> TSM-118-04-L-DV-LC
Changed lines of the file:
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@@
     (property "Reference" "PB2-P1" (at 139.70 420.37 0) (effects (font (size 1.27 1.27))))
     (property "Value" "PB2I-P1-2x18" (at 139.70 473.71 0) (effects (font (size 1.27 1.27))))
-    (property "Footprint" "Serenity-Custom:PocketBeagle2_2x18_P1_SSM-DV-LC" (at 139.70 447.04 0) (effects (font (size 1.27 1.27)) (hide yes)))
-    (property "Datasheet" "PocketBeagle 2 P1/P2 expansion rails (XO map); Samtec SSM-DV SMT socket, -LC locking clip (manual placement per drawing note 8) [REF-SENSOR-023]" (at 139.70 447.04 0) (effects (font (size 1.27 1.27)) (hide yes)))
-    (property "MPN" "SSM-118-L-DV-LC" (at 139.70 447.04 0) (effects (font (size 1.27 1.27)) (hide yes)))
+    (property "Footprint" "Serenity-Custom:PocketBeagle2_2x18_P1_TSM-DV-LC" (at 139.70 447.04 0) (effects (font (size 1.27 1.27)) (hide yes)))
+    (property "Datasheet" "PocketBeagle 2 P1/P2 expansion rails (XO map); Samtec TSM-DV SMT male strip, -04 post, -LC locking clip (manual placement) [REF-SENSOR-023]" (at 139.70 447.04 0) (effects (font (size 1.27 1.27)) (hide yes)))
+    (property "MPN" "TSM-118-04-L-DV-LC" (at 139.70 447.04 0) (effects (font (size 1.27 1.27)) (hide yes)))
     (pin "1")
     (pin "2")
@@
     (property "Reference" "PB2-P2" (at 139.70 486.41 0) (effects (font (size 1.27 1.27))))
     (property "Value" "PB2I-P2-2x18" (at 139.70 539.75 0) (effects (font (size 1.27 1.27))))
-    (property "Footprint" "Serenity-Custom:PocketBeagle2_2x18_P2_SSM-DV-LC" (at 139.70 513.08 0) (effects (font (size 1.27 1.27)) (hide yes)))
-    (property "Datasheet" "PocketBeagle 2 P1/P2 expansion rails (XO map); Samtec SSM-DV SMT socket, -LC locking clip (manual placement per drawing note 8) [REF-SENSOR-023]" (at 139.70 513.08 0) (effects (font (size 1.27 1.27)) (hide yes)))
-    (property "MPN" "SSM-118-L-DV-LC" (at 139.70 513.08 0) (effects (font (size 1.27 1.27)) (hide yes)))
+    (property "Footprint" "Serenity-Custom:PocketBeagle2_2x18_P2_TSM-DV-LC" (at 139.70 513.08 0) (effects (font (size 1.27 1.27)) (hide yes)))
+    (property "Datasheet" "PocketBeagle 2 P1/P2 expansion rails (XO map); Samtec TSM-DV SMT male strip, -04 post, -LC locking clip (manual placement) [REF-SENSOR-023]" (at 139.70 513.08 0) (effects (font (size 1.27 1.27)) (hide yes)))
+    (property "MPN" "TSM-118-04-L-DV-LC" (at 139.70 513.08 0) (effects (font (size 1.27 1.27)) (hide yes)))
     (pin "1")
     (pin "2")

Commit message: TACCO: Molex 105162-0001 microSD header; rip-up-and-repair placement pass
Owner 2026-10-05: J-SD becomes the Molex 105162-0001 1.45 mm microSD header (land from
SD-105162-001 sheet 2, pad positions cross-checked against the Molex/Ultra Librarian model;
drawing and product spec archived). Rated -40 to +85 C. Placer gains a rip-up-and-repair
pass; 1553-XFM and MLRS-MCU are pinned on the bottom face. L-1V8RF still unplaced (KiCad
validator: 0 hard).

Co-Authored-By: Claude Opus 5.5 <noreply@anthropic.com>
Claude-Session: https://claude.ai/code/session_01YLwDy53g1VCBzNBwW4moUC
Parts:
- J-SD: value microSD push-pull -> microSD header 1.45H; footprint Connector_Card:microSD_HC_Molex_104031-0811 -> Serenity-Custom:microSD_Molex_105162-0001; MPN 104031-0811 -> 105162-0001
Connections:
- net GND: now also J-SD.G (SHELL); no longer J-SD.10 (SW-COM), J-SD.3 (VSS1)
- net SD_CD: now also J-SD.9 (DET); no longer J-SD.11 (SW-NC)

Commit message: TACCO: +1V8_RF LDO (TLV75718P) closes placement; all 163 parts placed, DRC 0, parity 0
Owner 2026-10-05: the WiFi module's 1.8 V buck (TPS62933, 3015 inductor, bootstrap,
soft-start, EN pull-up, FB divider) becomes a TLV75718PDBVR SOT-23-5 LDO from +3V3_RF per
tlv757p.pdf. Generator uses PLACEMENT_SEED 1 (shortest wirelength of five clean orderings).
Pre-route DRC: 0 errors, schematic parity 0; ERC unchanged.

Co-Authored-By: Claude Opus 5.5 <noreply@anthropic.com>
Claude-Session: https://claude.ai/code/session_01YLwDy53g1VCBzNBwW4moUC
Parts:
- removed C-BST18: 100nF, Capacitor_SMD:C_0402_1005Metric, symbol TACCO:S_C-BST18
- removed C-SS18: 10nF, Capacitor_SMD:C_0201_0603Metric, symbol TACCO:S_C-SS18
- removed J-SD: microSD header 1.45H, Serenity-Custom:microSD_Molex_105162-0001, symbol TACCO:S_J-SD
- removed L-1V8RF: 3.3uH 2.25A, Serenity-Custom:L_WE-MAPI_3015, symbol TACCO:S_L-1V8RF
- removed R-EN18: 100k, Resistor_SMD:R_0201_0603Metric, symbol TACCO:S_R-EN18
- removed R-FB18H: 40.2k 1%, Resistor_SMD:R_0201_0603Metric, symbol TACCO:S_R-FB18H
- removed R-FB18L: 32.4k 1%, Resistor_SMD:R_0201_0603Metric, symbol TACCO:S_R-FB18L
- added C-ZB-18-2: 100nF 6.3V X5R, Capacitor_SMD:C_0201_0603Metric, symbol TACCO:S_C-ZB-18-2
- J-SD: renamed from C-ZB-18-2; value 100nF 6.3V X5R -> microSD header 1.45H; footprint Capacitor_SMD:C_0201_0603Metric -> Serenity-Custom:microSD_Molex_105162-0001; symbol TACCO:S_C-ZB-18-2 -> TACCO:S_J-SD; MPN (none) -> 105162-0001
- U-1V8RF: value TPS62933DRLR -> TLV75718PDBVR; footprint Package_TO_SOT_SMD:SOT-583-8 -> Package_TO_SOT_SMD:SOT-23-5; MPN TPS62933DRLR -> TLV75718PDBVR
Connections:
- net SW_1V8RF is gone; now on net +1V8_RF: U-1V8RF.5 (OUT)
- net U1V8RF_EN is gone; now on net GND: U-1V8RF.2 (GND)
- net +1V8_RF: now also C-ZB-18-2.1 (P); no longer J-SD.1 (P)
- net +3V3: now also J-SD.4 (VDD)
- net +3V3_RF: now also C-1V8RF-HF.1 (P), C-1V8RF-IN.1 (P), U-1V8RF.1 (IN), U-1V8RF.3 (EN)
- net +5V: no longer C-1V8RF-HF.1 (P), C-1V8RF-IN.1 (P), U-1V8RF.3 (VIN)
- net GND: now also J-SD.6 (VSS), J-SD.G (SHELL), C-ZB-18-2.2 (N); no longer J-SD.2 (N), U-1V8RF.1 (RT), U-1V8RF.4 (GND)
- net SD_CD: now also J-SD.9 (DET)
- removed net BST_1V8RF: U-1V8RF.6 (BST)
- removed net FB_1V8RF: U-1V8RF.8 (FB)
- removed net SS_1V8RF: U-1V8RF.7 (SS/PG)
- no-connect marks 145 -> 146
