File: avionics/kicad/Pilot/kicads/Pilot.kicad_sch (KiCad schematic)
At the start: 124 parts, among them X2Y-CAN 4.7nF X2Y, X2Y-RS485 4.7nF X2Y

Commit message: Pilot sch: GNSS off-board for ISOW §13.1 (117 parts, ERC 0); WBS puck item
Owner decision 2026-10-12: move the MAX-M10S off the cape to isolated CAN-FD
GPS pucks in the two dorsal GPS cups.  The two ISOW §13.1 4 mm metal-free
bubbles [REF-SENSOR-009/010] fit only in the strip between the PB2 rail pads
and displace the buck, IMU/BARO, GPS and 1553 transceiver; there is no other
area for all of them on 55 x 35 mm.

- Removed GPS, R-ANT, C-ANT, L-ANT, J-ANT, C-GPS1/2; P1-31/32 and P2-9/10 NC.
- avionics/WBS.md: §13.1 re-floorplan item (with PGND perimeter fence, owner
  2026-10-12) and the GPS-puck item.  Envelope from a scratch run of the
  tools/cargo_layout_fit.py geometry: O28 x 8 mm under each cup, 4 mm aft.
  The isolated puck (owner choice) still has to be proved to fit.
- TODO.md files regenerated from WBS.md.

Co-Authored-By: Claude Opus 5.5 (1M context) <noreply@anthropic.com>
Parts:
- removed C-485-1: 10nF, Capacitor_SMD:C_0201_0603Metric, symbol Pilot:S_C-485-1
- removed C-ANT: 10nF X7R, Capacitor_SMD:C_0402_1005Metric, symbol Pilot:S_C-ANT
- removed C-GPS1: 10uF 6.3V X5R, Capacitor_SMD:C_0805_2012Metric, symbol Pilot:S_C-GPS1
- removed C-GPS2: 100nF, Capacitor_SMD:C_0402_1005Metric, symbol Pilot:S_C-GPS2
- removed ETH1-PHY: DP83825IRMQR, Package_DFN_QFN:Texas_RMQ0024A_WQFN-24-1EP_3x3mm_P0.4mm_EP1.9x1.9mm, symbol Pilot:S_ETH1-PHY
- removed H2: M2.5 PGND, Serenity-Custom:MountingHole_2.7mm_M2.5_PGND_Ring, symbol Pilot:S_H2
- removed J-ANT: U.FL-R-SMT-1, Connector_Coaxial:U.FL_Hirose_U.FL-R-SMT-1_Vertical, symbol Pilot:S_J-ANT
- removed L-ANT: 27nH, Inductor_SMD:L_0402_1005Metric, symbol Pilot:S_L-ANT
- removed R-ANT: 10R, Resistor_SMD:R_0201_0603Metric, symbol Pilot:S_R-ANT
- removed R-BS2T: 75R, Resistor_SMD:R_0402_1005Metric, symbol Pilot:S_R-BS2T
- removed R-P2-AD0: 2.49k, Resistor_SMD:R_0201_0603Metric, symbol Pilot:S_R-P2-AD0
- removed X2Y-CAN: 4.7nF X2Y, Serenity-Custom:X2Y_0805_4T, symbol Pilot:S_X2Y-CAN
- removed X2Y-RS485: 4.7nF X2Y, Serenity-Custom:X2Y_0805_4T, symbol Pilot:S_X2Y-RS485
- added C-TPM1: 1uF, Capacitor_SMD:C_0402_1005Metric, symbol Pilot:S_C-TPM1
- added CMC-CAN: SRF2012-100Y, Serenity-Custom:Bourns_SRF2012_4T, symbol Pilot:S_CMC-CAN
- added CMC-RS485: SRF2012-100Y, Serenity-Custom:Bourns_SRF2012_4T, symbol Pilot:S_CMC-RS485
- added H4: M2.5 PGND, Serenity-Custom:MountingHole_2.7mm_M2.5_PGND_Ring, symbol Pilot:S_H4
- added TVS-CAN: PRTR5V0U2X, Package_TO_SOT_SMD:SOT-363_SC-70-6, symbol Pilot:S_TVS-CAN
- added TVS-RS485: PRTR5V0U2X, Package_TO_SOT_SMD:SOT-363_SC-70-6, symbol Pilot:S_TVS-RS485
- C-485-1: renamed from TVS-CAN; value PRTR5V0U2X -> 10nF; footprint Package_TO_SOT_SMD:SOT-363_SC-70-6 -> Capacitor_SMD:C_0201_0603Metric; symbol Pilot:S_TVS-CAN -> Pilot:S_C-485-1; MPN PRTR5V0U2X,115 -> (none)
- ETH1: renamed from TVS-RS485; value PRTR5V0U2X -> SM04B-GHS-TB; footprint Package_TO_SOT_SMD:SOT-363_SC-70-6 -> Connector_JST:JST_GH_SM04B-GHS-TB_1x04-1MP_P1.25mm_Horizontal; symbol Pilot:S_TVS-RS485 -> Pilot:S_ETH1; MPN PRTR5V0U2X,115 -> SM04B-GHS-TB(LF)(SN)
- ETH1-PHY: renamed from GPS; value MAX-M10S-00B -> DP83825IRMQR; footprint RF_GPS:ublox_MAX -> Package_DFN_QFN:Texas_RMQ0024A_WQFN-24-1EP_3x3mm_P0.4mm_EP1.9x1.9mm; symbol Pilot:S_GPS -> Pilot:S_ETH1-PHY; MPN MAX-M10S-00B -> DP83825IRMQR
- H2: renamed from C-TPM1; value 1uF -> M2.5 PGND; footprint Capacitor_SMD:C_0402_1005Metric -> Serenity-Custom:MountingHole_2.7mm_M2.5_PGND_Ring; symbol Pilot:S_C-TPM1 -> Pilot:S_H2
- R-BS2T: renamed from ETH1; value SM04B-GHS-TB -> 75R; footprint Connector_JST:JST_GH_SM04B-GHS-TB_1x04-1MP_P1.25mm_Horizontal -> Resistor_SMD:R_0402_1005Metric; symbol Pilot:S_ETH1 -> Pilot:S_R-BS2T; MPN SM04B-GHS-TB(LF)(SN) -> (none)
- R-P2-AD0: renamed from H4; value M2.5 PGND -> 2.49k; footprint Serenity-Custom:MountingHole_2.7mm_M2.5_PGND_Ring -> Resistor_SMD:R_0201_0603Metric; symbol Pilot:S_H4 -> Pilot:S_R-P2-AD0
- X2Y-CAN: renamed from CMC-CAN; value SRF2012-100Y -> 4.7nF X2Y; footprint Serenity-Custom:Bourns_SRF2012_4T -> Serenity-Custom:X2Y_0805_4T; symbol Pilot:S_CMC-CAN -> Pilot:S_X2Y-CAN; MPN SRF2012-121YA -> CX0805MRX7R0BB472
- X2Y-RS485: renamed from CMC-RS485; value SRF2012-100Y -> 4.7nF X2Y; footprint Serenity-Custom:Bourns_SRF2012_4T -> Serenity-Custom:X2Y_0805_4T; symbol Pilot:S_CMC-RS485 -> Pilot:S_X2Y-RS485; MPN SRF2012-121YA -> CX0805MRX7R0BB472
Connections:
- net GPS_RF is gone; now on net ETH_TXP: ETH1-PHY.11 (TD_P)
- net GPS_VCC_RF is gone; now on net ETH1-PHY_RBIAS: ETH1-PHY.14 (RBIAS)
- net +3V3: now also ETH1-PHY.19 (VDDIO), R-P2-AD0.1 (A), C-TPM1.1 (P); no longer ETH1-PHY.7 (V_IO), ETH1-PHY.8 (VCC), H2.1 (P)
- net +5V: now also C-485-1.1 (P)
- net CAN_H: now also CMC-CAN.1 (W1_IN); no longer X2Y-CAN.1 (W1_IN)
- net CAN_H_F: now also CMC-CAN.2 (W1_OUT), TVS-CAN.1 (IO1); no longer C-485-1.1 (IO1), X2Y-CAN.2 (W1_OUT)
- net CAN_L: now also CMC-CAN.4 (W2_IN); no longer X2Y-CAN.4 (W2_IN)
- net CAN_L_F: now also CMC-CAN.3 (W2_OUT), TVS-CAN.3 (IO2); no longer C-485-1.3 (IO2), X2Y-CAN.3 (W2_OUT)
- net ETH2_BS: now also R-BS2T.2 (B)
- net ETH2_LINE_CTX: now also R-BS2T.1 (A)
- net ETH_LINE_RXN: now also ETH1.4 (RXN); no longer R-BS2T.4 (RXN)
- net ETH_LINE_RXP: now also ETH1.3 (RXP); no longer R-BS2T.3 (RXP)
- net ETH_LINE_TXN: now also ETH1.2 (TXN); no longer R-BS2T.2 (TXN)
- net ETH_LINE_TXP: now also ETH1.1 (TXP); no longer R-BS2T.1 (TXP)
- net ETH_RXN: now also ETH1-PHY.7 (RD_M)
- net ETH_RXP: now also ETH1-PHY.8 (RD_P)
- net ETH_TXN: now also ETH1-PHY.10 (TD_M)
- net GND: now also C-485-1.2 (N), ETH1-PHY.21 (GND), ETH1-PHY.25 (EP), ETH1-PHY.9 (GND), X2Y-CAN.1 (A), X2Y-CAN.2 (B), X2Y-RS485.1 (A), X2Y-RS485.2 (B), C-TPM1.2 (N); no longer ETH1-PHY.1 (GND), ETH1-PHY.10 (GND), ETH1-PHY.12 (GND), H2.2 (N)
- net GND2_CAN: now also X2Y-CAN.3 (G1), X2Y-CAN.4 (G2), TVS-CAN.2 (GND); no longer C-485-1.2 (GND)
- net GND2_RS485: now also X2Y-RS485.3 (G1), X2Y-RS485.4 (G2), TVS-RS485.2 (GND); no longer ETH1.2 (GND)
- net MDC0: now also ETH1-PHY.16 (MDC)
- net MDIO0: now also ETH1-PHY.15 (MDIO)
- net PGND: now also ETH1.MP (SHIELD), H2.1 (PGND), H4.1 (PGND); no longer R-BS2T.MP (SHIELD), R-P2-AD0.1 (PGND)
- net PHY1_INTRN: now also ETH1-PHY.3 (INTR/PWRDN)
- net PHY1_RSTN: now also ETH1-PHY.5 (RST_N)
- net PHY_XI_25M: now also ETH1-PHY.13 (XI)
- net RMII0_CRS_DV: now also ETH1-PHY.20 (CRS_DV/PhyAdd1)
- net RMII0_REF_CLK: now also ETH1-PHY.2 (50MHzOut)
- net RMII0_RXD0: now also ETH1-PHY.18 (RX_D0/PhyAdd0)
- net RMII0_RXD1: now also ETH1-PHY.17 (RX_D1/Leader)
- net RMII0_RX_ER: now also ETH1-PHY.22 (RX_ER/A-MDIX)
- net RMII0_TXD0: now also ETH1-PHY.23 (TX_D0)
- net RMII0_TXD1: now also ETH1-PHY.24 (TX_D1)
- net RMII0_TX_EN: now also ETH1-PHY.1 (TX_EN)
- net RMII1_RXD0: now also R-P2-AD0.2 (B)
- net RS485_A: now also CMC-RS485.1 (W1_IN); no longer X2Y-RS485.1 (W1_IN)
- net RS485_A_F: now also CMC-RS485.2 (W1_OUT), TVS-RS485.1 (IO1); no longer ETH1.1 (IO1), X2Y-RS485.2 (W1_OUT)
- net RS485_B: now also CMC-RS485.4 (W2_IN); no longer X2Y-RS485.4 (W2_IN)
- net RS485_B_F: now also CMC-RS485.3 (W2_OUT), TVS-RS485.3 (IO2); no longer ETH1.3 (IO2), X2Y-RS485.3 (W2_OUT)
- net VCC2_CAN: now also TVS-CAN.5 (VCC); no longer C-485-1.5 (VCC)
- net VCC2_RS485: now also TVS-RS485.5 (VCC); no longer ETH1.5 (VCC)
- net GPS_RESETN: no longer names the net of PB2-P2.9 (P9)
- net GPS_RESETN: no longer ETH1-PHY.9 (RESET_N)
- net GPS_TIMEPULSE: no longer names the net of ETH1-PHY.4 (LED0/ANEG)
- net GPS_TIMEPULSE: no longer PB2-P2.10 (P10)
- net UART_GPS_RX: no longer names the net of PB2-P1.31 (P31)
- net UART_GPS_RX: no longer ETH1-PHY.3 (RXD)
- net UART_GPS_TX: no longer names the net of PB2-P1.32 (P32)
- net UART_GPS_TX: no longer ETH1-PHY.2 (TXD)
- no-connect marks 91 -> 89
Other:
- moved on the sheet: X2Y-CAN, X2Y-RS485

Commit message: feat(pilot): PB2-I re-map, TPSM828224 3V3, keep-copper re-floorplan, AM625/MSPM0 header capability docs
Pilot (branch pilot-refloorplan, owner S. Griffing decisions 2026-10-17; implemented by
Claude Opus 5.5):
- 3V3 rail -> TI TPSM828224SILR MicroSiP module [REF-PWR-008]; C-3V3 caps chosen on DC-bias
  curves (Taiyo Yuden MSASJ168BC6226MTNA01 [REF-PWR-011]); SIL0010D land + STEP.
- Keep-copper re-floorplan for ISOW1044/ISOW1412 sec 13.1 bubbles (iso_zones_pilot.py,
  refloorplan_pilot.py, refloorplan_keep_copper.sh); PCB DRC 0 / parity 0 / 107 unconnected
  at that point (PCB predates the header re-map below; re-sync pending in avionics/WBS.md).
- PB2-I header re-map from BeagleBoard sources [REF-SENSOR-021, REF-SENSOR-041 sec 4.2,
  REF-SENSOR-047]; TSM-DV-LC rail footprints mirrored so pin 1 lands on the official row
  on B.Cu; GNSS replaced by JST-GH expansion ports; Ethernet ring = DP83825I on RMII2 +
  USB NIC on USB1 (CH397A placeholder; AX88772E pending, WCH fails the AGENTS.md sec 5
  sourcing rule).

AM625 / MSPM0L1105 capability check (owner request 2026-10-17):
- New avionics/kicad/PB2I_AM625_HEADER_CAPABILITIES.md + extracted JSON from TI SPRSP58C
  Table 5-1 / sec 5.3.1 [REF-SENSOR-049], SPRUIV7C sec 1.4.12 [REF-SENSOR-050], MSPM0L1105
  SLASEX5C [REF-SENSOR-051] and SLAU847F sec 2.4.1.2 [REF-SENSOR-052]: CPSW3G has two
  external ports but only port 2 reaches the header; 3 CAN-FD reachable; 17 dual-ball
  header pins; 8 AIN pins also tied to the MSPM0 (SWCLK pull-down on P2-35 after POR).
- PB2_HEADER_PINMAP.md sec 1 second balls on P1-2/4/6 added and footnote corrected.
- Reviewed by ce-doc-review (coherence + feasibility subagents, Claude Haiku / Opus 5.5);
  findings applied. ce-compound-refresh: new learning
  docs/solutions/conventions/pb2-header-capability-from-soc-datasheet-not-srm-summary.md,
  two stale "Pilot still has 2.54 mm rails" notes updated, CONCEPTS.md "Shared Header Pin".

Not committed: avionics/datasheets/spruiv7c.pdf (129 MB, abov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
Parts:
- removed C-BST: 100nF, Capacitor_SMD:C_0402_1005Metric, symbol Pilot:S_C-BST
- removed C-P2-A1: 10nF, Capacitor_SMD:C_0201_0603Metric, symbol Pilot:S_C-P2-A1
- removed C-P2-A2: 100nF, Capacitor_SMD:C_0402_1005Metric, symbol Pilot:S_C-P2-A2
- removed C-P2-A3: 1uF, Capacitor_SMD:C_0402_1005Metric, symbol Pilot:S_C-P2-A3
- removed C-P2-CRD1: 100nF, Capacitor_SMD:C_0402_1005Metric, symbol Pilot:S_C-P2-CRD1
- removed C-P2-CRD2: 1uF, Capacitor_SMD:C_0402_1005Metric, symbol Pilot:S_C-P2-CRD2
- removed C-P2-CTD1: 100nF, Capacitor_SMD:C_0402_1005Metric, symbol Pilot:S_C-P2-CTD1
- removed C-P2-CTD2: 1uF, Capacitor_SMD:C_0402_1005Metric, symbol Pilot:S_C-P2-CTD2
- removed C-P2-IO1: 10nF, Capacitor_SMD:C_0201_0603Metric, symbol Pilot:S_C-P2-IO1
- removed C-P2-IO2: 100nF, Capacitor_SMD:C_0402_1005Metric, symbol Pilot:S_C-P2-IO2
- removed C-P2-IO3: 1uF, Capacitor_SMD:C_0402_1005Metric, symbol Pilot:S_C-P2-IO3
- removed C-SS: 10nF, Capacitor_SMD:C_0201_0603Metric, symbol Pilot:S_C-SS
- removed ETH2: SM04B-GHS-TB, Connector_JST:JST_GH_SM04B-GHS-TB_1x04-1MP_P1.25mm_Horizontal, symbol Pilot:S_ETH2
- removed L-3V3: 3.3uH 2.25A, Serenity-Custom:L_WE-MAPI_3015, symbol Pilot:S_L-3V3
- removed R-BS1T: 75R, Resistor_SMD:R_0402_1005Metric, symbol Pilot:S_R-BS1T
- removed R-EN3: 100k, Resistor_SMD:R_0201_0603Metric, symbol Pilot:S_R-EN3
- removed R-FB3H: 100k 1%, Resistor_SMD:R_0201_0603Metric, symbol Pilot:S_R-FB3H
- removed R-FB3L: 32.4k 1%, Resistor_SMD:R_0201_0603Metric, symbol Pilot:S_R-FB3L
- removed R-P2-AD0: 2.49k, Resistor_SMD:R_0201_0603Metric, symbol Pilot:S_R-P2-AD0
- removed R-P2-RBIAS: 6.49k 1%, Resistor_SMD:R_0201_0603Metric, symbol Pilot:S_R-P2-RBIAS
- added C-GPS5: 1uF 10V, Capacitor_SMD:C_0402_1005Metric, symbol Pilot:S_C-GPS5
- added C-SPI5: 1uF 10V, Capacitor_SMD:C_0402_1005Metric, symbol Pilot:S_C-SPI5
- added C-U2-A1: 1uF, Capacitor_SMD:C_0402_1005Metric, symbol Pilot:S_C-U2-A1
- added C-U2-AK: 1uF, Capacitor_SMD:C_0402_1005Metric, symbol Pilot:S_C-U2-AK
- added C-U2-CRD: 1uF, Capacitor_SMD:C_0402_1005Metric, symbol Pilot:S_C-U2-CRD
- added C-U2-CTD: 1uF, Capacitor_SMD:C_0402_1005Metric, symbol Pilot:S_C-U2-CTD
- added C-U2-DK: 100nF, Capacitor_SMD:C_0201_0603Metric, symbol Pilot:S_C-U2-DK
- added C-U2-IO: 100nF, Capacitor_SMD:C_0201_0603Metric, symbol Pilot:S_C-U2-IO
- added C-U2-V5A: 10uF 6.3V X6S, Capacitor_SMD:C_0603_1608Metric, symbol Pilot:S_C-U2-V5A
- added C-U2-V5B: 100nF, Capacitor_SMD:C_0201_0603Metric, symbol Pilot:S_C-U2-V5B
- added ESD-GPS: TPD4E05U06DQAR, Serenity-Custom:TI_DQA0010A_USON-10_2.5x1.0mm_P0.5mm, symbol Pilot:S_ESD-GPS
- added ESD-SPI: TPD4E05U06DQAR, Serenity-Custom:TI_DQA0010A_USON-10_2.5x1.0mm_P0.5mm, symbol Pilot:S_ESD-SPI
- added ESD-SS2: TPD1E05U06DYAR, Diode_SMD:D_SOD-523, symbol Pilot:S_ESD-SS2
- added F-GPS: MF-PSMF035X, Fuse:Fuse_0805_2012Metric, symbol Pilot:S_F-GPS
- added F-SPI: MF-PSMF035X, Fuse:Fuse_0805_2012Metric, symbol Pilot:S_F-SPI
- added J-GPS: SM06B-GHS-TB, Connector_JST:JST_GH_SM06B-GHS-TB_1x06-1MP_P1.25mm_Horizontal, symbol Pilot:S_J-GPS
- added J-SPI: SM07B-GHS-TB, Connector_JST:JST_GH_SM07B-GHS-TB_1x07-1MP_P1.25mm_Horizontal, symbol Pilot:S_J-SPI
- added R-I2C-SCL: 1.5k, Resistor_SMD:R_0201_0603Metric, symbol Pilot:S_R-I2C-SCL
- added R-I2C-SDA: 1.5k, Resistor_SMD:R_0201_0603Metric, symbol Pilot:S_R-I2C-SDA
- added RS-485: SM04B-GHS-TB, Connector_JST:JST_GH_SM04B-GHS-TB_1x04-1MP_P1.25mm_Horizontal, symbol Pilot:S_RS-485
- added X2Y-RS485: 4.7nF X2Y, Serenity-Custom:X2Y_0805_4T, symbol Pilot:S_X2Y-RS485
- C-3V3-IN: value 10uF 10V X5R -> 22uF 6.3V X6S; footprint Capacitor_SMD:C_0805_2012Metric -> Capacitor_SMD:C_0603_1608Metric; MPN (none) -> MSASJ168BC6226MTNA01
- C-3V3-O1, C-3V3-O2: value 22uF 6.3V X5R -> 22uF 6.3V X6S; footprint Capacitor_SMD:C_0805_2012Metric -> Capacitor_SMD:C_0603_1608Metric; MPN (none) -> MSASJ168BC6226MTNA01
- C-485-1, C-CAN1: footprint Capacitor_SMD:C_0201_0603Metric -> Capacitor_SMD:C_0402_1005Metric
- ETH2: renamed from RS-485; symbol Pilot:S_RS-485 -> Pilot:S_ETH2
- ETH2-USB: renamed from ETH2-PHY; value DP83825IRMQR -> CH397A; footprint Package_DFN_QFN:Texas_RMQ0024A_WQFN-24-1EP_3x3mm_P0.4mm_EP1.9x1.9mm -> Package_DFN_QFN:QFN-24-1EP_4x4mm_P0.5mm_EP2.8x2.8mm; symbol Pilot:S_ETH2-PHY -> Pilot:S_ETH2-USB; MPN DP83825IRMQR -> CH397A
- R-BS1T: renamed from X2Y-RS485; value 4.7nF X2Y -> 75R; footprint Serenity-Custom:X2Y_0805_4T -> Resistor_SMD:R_0402_1005Metric; symbol Pilot:S_X2Y-RS485 -> Pilot:S_R-BS1T; MPN CX0805MRX7R0BB472 -> (none)
- U-3V3: value TPS62933DRLR -> TPSM828224SILR; footprint Package_TO_SOT_SMD:SOT-583-8 -> Serenity-Custom:TI_SIL0010D_uSiP-10_2.0x2.5mm_P0.5mm; MPN TPS62933DRLR -> TPSM828224SILR
Connections:
- net BST_3V3 is gone; now on net +3V3: U-3V3.6 (VOUT)
- net FB_3V3 is gone; now on net +3V3: U-3V3.8 (FB)
- net SS_3V3 is gone; now on net +3V3: U-3V3.7 (VOUT)
- net SW_3V3 is gone; now on net +3V3: U-3V3.5 (VOUT)
- net U3V3_EN is gone; now on net +5V: U-3V3.2 (VIN)
- net +3V3: now also ETH2-USB.1 (AVDD33), ETH2-USB.10 (AVDD33), ETH2-USB.11 (V5), ETH2-USB.13 (VDDIO), ETH2-USB.18 (VDDIO), C-U2-A1.1 (P), C-U2-IO.1 (P), C-U2-V5A.1 (P), C-U2-V5B.1 (P), R-I2C-SCL.1 (A), R-I2C-SDA.1 (A); no longer ETH2-USB.19 (VDDIO), ETH2-USB.6 (VDDA3V3)
- net +5V: now also PB2-P1.1 (P1), PB2-P1.5 (P5), U-3V3.1 (VIN), F-GPS.1 (A), F-SPI.1 (A); no longer PB2-P1.35 (P35), PB2-P2.35 (P35)
- net BARO_INT: now also PB2-P2.18 (P18); no longer PB2-P1.17 (P17)
- net CAN_STB: now also PB2-P2.10 (P10); no longer PB2-P1.14 (P14)
- net DSHOT0: now also PB2-P1.23 (P23); no longer PB2-P1.6 (P6)
- net DSHOT1: now also PB2-P1.13 (P13); no longer PB2-P1.5 (P5)
- net DSHOT2: now also PB2-P1.29 (P29); no longer PB2-P1.4 (P4)
- net DSHOT3: now also PB2-P1.21 (P21); no longer PB2-P1.3 (P3)
- net ETH2_CRD: now also C-U2-CRD.1 (P)
- net ETH2_CTD: now also C-U2-CTD.1 (P)
- net ETH2_LINE_RXN: now also ETH2.4 (RXN)
- net ETH2_LINE_RXP: now also ETH2.3 (RXP)
- net ETH2_LINE_TXN: now also ETH2.2 (TXN)
- net ETH2_LINE_TXP: now also ETH2.1 (TXP)
- net ETH2_RXN: now also ETH2-USB.5 (MDIRN); no longer ETH2-USB.7 (RD_M)
- net ETH2_RXP: now also ETH2-USB.4 (MDIRP); no longer ETH2-USB.8 (RD_P)
- net ETH2_TXN: now also ETH2-USB.3 (MDITN); no longer ETH2-USB.10 (TD_M)
- net ETH2_TXP: now also ETH2-USB.2 (MDITP); no longer ETH2-USB.11 (TD_P)
- net ETH_BS: now also R-BS1T.2 (B)
- net ETH_LINE_CTX: now also R-BS1T.1 (A)
- net GND: now also ETH2-USB.24 (GND), ETH2-USB.6 (GND), PB2-P1.15 (P15), PB2-P1.16 (P16), PB2-P1.22 (P22), PB2-P2.15 (P15), PB2-P2.21 (P21), U-3V3.10 (GND), U-3V3.9 (GND), C-GPS5.2 (N), C-SPI5.2 (N), C-U2-A1.2 (N), C-U2-AK.2 (N), C-U2-CRD.2 (N), C-U2-CTD.2 (N), C-U2-DK.2 (N), C-U2-IO.2 (N), C-U2-V5A.2 (N), C-U2-V5B.2 (N), ESD-GPS.3 (GND), ESD-GPS.8 (GND), ESD-SPI.3 (GND), ESD-SPI.8 (GND), ESD-SS2.2 (GND), J-GPS.6 (GND), J-SPI.7 (GND), X2Y-RS485.1 (A), X2Y-RS485.2 (B); no longer ETH2-USB.21 (GND), ETH2-USB.9 (GND), PB2-P1.1 (P1), PB2-P1.2 (P2), PB2-P1.36 (P36), PB2-P2.36 (P36), R-BS1T.1 (A), R-BS1T.2 (B), U-3V3.1 (RT), U-3V3.4 (GND)
- net GND2_RS485: now also RS-485.1 (GND), X2Y-RS485.3 (G1), X2Y-RS485.4 (G2); no longer ETH2.1 (GND), R-BS1T.3 (G1), R-BS1T.4 (G2)
- net IMU_INT1: now also PB2-P2.19 (P19); no longer PB2-P1.19 (P19)
- net IMU_INT2: now also PB2-P2.22 (P22); no longer PB2-P1.18 (P18)
- net M1553_IRQN: now also PB2-P2.17 (P17); no longer PB2-P1.7 (P7)
- net M1553_MRN: now also PB2-P2.6 (P6); no longer PB2-P1.8 (P8)
- net M1553_TX_INH: now also PB2-P2.8 (P8); no longer PB2-P1.9 (P9)
- net MCAN0_RX: now also PB2-P2.7 (P7); no longer PB2-P1.15 (P15)
- net MCAN0_TX: now also PB2-P2.5 (P5); no longer PB2-P1.16 (P16)
- net MDC0: now also PB2-P2.1 (P1); no longer PB2-P2.18 (P18)
- net MDIO0: now also PB2-P2.3 (P3); no longer PB2-P2.17 (P17)
- net PGND: now also J-GPS.MP (SHIELD), J-SPI.MP (SHIELD), RS-485.MP (SHIELD)
- net PHY1_INTRN: now also PB2-P2.28 (P28); no longer PB2-P2.16 (P16)
- net PHY1_RSTN: now also PB2-P2.20 (P20); no longer PB2-P2.15 (P15)
- net RS485_A_F: now also RS-485.2 (A); no longer ETH2.2 (A)
- net RS485_B_F: now also RS-485.3 (B); no longer ETH2.3 (B)
- net RS485_DE: now also PB2-P2.32 (P32); no longer PB2-P1.11 (P11)
- net RS485_RX: now also PB2-P2.24 (P24); no longer PB2-P1.12 (P12)
- net RS485_TX: now also PB2-P2.33 (P33); no longer PB2-P1.13 (P13)
- net SPI0_CLK: now also PB2-P2.29 (P29); no longer PB2-P1.25 (P25)
- net SPI0_CS_1553: now also PB2-P2.9 (P9); no longer PB2-P1.20 (P20)
- net SPI0_CS_BARO: now also PB2-P2.11 (P11); no longer PB2-P1.22 (P22)
- net SPI0_CS_IMU: now also PB2-P1.3 (P3); no longer PB2-P1.26 (P26)
- net SPI0_CS_TPM: now also PB2-P1.26 (P26); no longer PB2-P1.21 (P21)
- net SPI0_MISO: now also PB2-P2.27 (P27); no longer PB2-P1.23 (P23)
- net SPI0_MOSI: now also PB2-P2.25 (P25); no longer PB2-P1.24 (P24)
- net TPM_IRQN: now also PB2-P1.20 (P20); no longer PB2-P1.29 (P29)
- net VCC2_RS485: now also RS-485.4 (VCC); no longer ETH2.4 (VCC)
- net EXT_SPI_MISO: now reaches PB2-P1.10 (P10)
- net EXT_SPI_MISO: now also ESD-SPI.2 (D1-), J-SPI.3 (MISO)
- net RMII2_RXD0: now reaches PB2-P1.27 (P27)
- net RMII2_RXD0: now also ETH1-PHY.18 (RX_D0/PhyAdd0), R-P1-AD0.2 (B)
- net EXT_SPI_SS2: now reaches PB2-P1.31 (P31)
- net EXT_SPI_SS2: now also ESD-SS2.1 (IO), J-SPI.6 (SS2)
- net EXT_UART_TX: now reaches PB2-P2.4 (P4)
- net EXT_UART_TX: now also ESD-GPS.1 (D1+), J-GPS.2 (TX)
- net +3V3_PB2 renamed EXT_I2C_SDA
- net EXT_I2C_SDA: now also ESD-GPS.5 (D2-), J-GPS.5 (SDA), R-I2C-SDA.2 (B); no longer PB2-P1.34 (P34)
- net ETH2-PHY_RBIAS: no longer names the net of ETH2-USB.14 (GPIO6)
- net MDC1: no longer names the net of ETH2-USB.16 (NC)
- net MDC1: no longer PB2-P2.2 (P2)
- net MDIO1: no longer names the net of ETH2-USB.15 (LED0)
- net MDIO1: no longer PB2-P2.1 (P1)
- net PHY2_INTRN: no longer names the net of PB2-P2.14 (P14)
- net PHY2_INTRN: no longer ETH2-USB.3 (INTR/PWRDN)
- net PHY2_RSTN: no longer names the net of PB2-P2.13 (P13)
- net PHY2_RSTN: no longer ETH2-USB.5 (RST_N)
- net PHY_XI_25M renamed XI_25M
- net XI_25M: now also ETH2-USB.21 (XI); no longer ETH2-USB.13 (XI)
- net RMII0_CRS_DV renamed RMII2_CRS_DV
- net RMII2_CRS_DV: now also PB2-P1.35 (P35); no longer PB2-P2.29 (P29)
- net RMII0_REF_CLK renamed RMII2_REF_CLK
- net RMII2_REF_CLK: now also PB2-P1.34 (P34); no longer PB2-P2.27 (P27)
- removed net RMII0_RXD0: ETH1-PHY.18 (RX_D0/PhyAdd0), PB2-P2.31 (P31), R-P1-AD0.2 (B)
- net RMII0_RXD1: no longer names the net of PB2-P2.30 (P30)
- net RMII0_RXD1: no longer ETH1-PHY.17 (RX_D1/Leader)
- net RMII0_RX_ER renamed RMII2_RX_ER
- net RMII2_RX_ER: now also PB2-P1.19 (P19); no longer PB2-P2.28 (P28)
- net RMII0_TXD0: no longer names the net of PB2-P2.34 (P34)
- net RMII0_TXD0: no longer ETH1-PHY.23 (TX_D0)
- net RMII0_TXD1 renamed RMII2_TXD1
- net RMII2_TXD1: now also PB2-P2.31 (P31); no longer PB2-P2.33 (P33)
- net RMII0_TX_EN renamed RMII2_TX_EN
- net RMII2_TX_EN: now also PB2-P1.2 (P2); no longer PB2-P2.32 (P32)
- net RMII1_CRS_DV: no longer names the net of ETH2-USB.20 (NC)
- net RMII1_CRS_DV: no longer PB2-P2.21 (P21)
- removed net RMII1_REF_CLK: ETH2-USB.2 (50MHzOut), PB2-P2.19 (P19)
- net RMII1_RXD0: no longer names the net of PB2-P2.23 (P23)
- net RMII1_RXD0: no longer ETH2-USB.18 (RX_D0/PhyAdd0)
- net RMII1_RXD1: no longer names the net of ETH2-USB.17 (LED1)
- net RMII1_RXD1: no longer PB2-P2.22 (P22)
- net RMII1_RX_ER: no longer names the net of ETH2-USB.22 (XO)
- net RMII1_RX_ER: no longer PB2-P2.20 (P20)
- net RMII1_TXD0: no longer names the net of PB2-P2.26 (P26)
- net RMII1_TXD0: no longer ETH2-USB.23 (TX_D0)
- removed net RMII1_TXD1: ETH2-USB.24 (TX_D1), PB2-P2.25 (P25)
- removed net RMII1_TX_EN: ETH2-USB.1 (TX_EN), PB2-P2.24 (P24)
- new net ETH2-USB_AVDDK: C-U2-AK.1 (P), ETH2-USB.23 (AVDDK)
- new net ETH2-USB_DVDDK: C-U2-DK.1 (P), ETH2-USB.9 (DVDDK)
- new net EXT_GPS_5V: C-GPS5.1 (P), F-GPS.2 (B), J-GPS.1 (VCC)
- new net EXT_I2C_SCL: ESD-GPS.4 (D2+), J-GPS.4 (SCL), PB2-P1.36 (P36), R-I2C-SCL.2 (B)
- new net EXT_SPI_5V: C-SPI5.1 (P), F-SPI.2 (B), J-SPI.1 (VCC)
- new net EXT_SPI_MOSI: ESD-SPI.4 (D2+), J-SPI.4 (MOSI), PB2-P1.12 (P12)
- new net EXT_SPI_SCK: ESD-SPI.1 (D1+), J-SPI.2 (SCK), PB2-P1.8 (P8)
- new net EXT_SPI_SS1: ESD-SPI.5 (D2-), J-SPI.5 (SS1), PB2-P1.6 (P6)
- new net EXT_UART_RX: ESD-GPS.2 (D1-), J-GPS.3 (RX), PB2-P2.2 (P2)
- new net RMII2_RXD1: ETH1-PHY.17 (RX_D1/Leader), PB2-P1.25 (P25)
- new net RMII2_TXD0: ETH1-PHY.23 (TX_D0), PB2-P1.4 (P4)
- new net USB1_DM: ETH2-USB.7 (UDM), PB2-P1.9 (P9)
- new net USB1_DP: ETH2-USB.8 (UDP), PB2-P1.11 (P11)
- no-connect marks 89 -> 106
Other:
- moved on the sheet: ETH2, ETH2-USB

Commit message: refactor(avionics): align Pilot + TACCO header pins and Ethernet names to BeagleBoard / TI naming
Owner decisions 2026-10-17 (S. Griffing; implemented by Claude Opus 5.5):
- REJECTED: second/third CAN-FD bus (the fleet's four buses already cover the need) and
  moving RMII2/DSHOT off the MSPM0-shared AIN pins (RMII2 has no other balls, SPRSP58C
  Table 5-5 [REF-SENSOR-049]; free PRU pins sit under the P2 isolation band).
- PB2 header symbol pins P1..P36 -> BeagleBoard SRM designators P1.01..P2.36
  [REF-SENSOR-041 sec 4.2] on both boards.
- Ethernet ring parts/nets -> TI interface names [REF-SENSOR-049 sec 5.3.1]: PHY-RMII2,
  T-RMII2, ETH_RMII2_*, RMII2_PHY_RSTN/INTRN, C-/R-RMII2-* (both boards); NIC-USB1, T-USB1,
  ETH_USB1_*, C-USB1-*, J-ETH-RMII2 / J-ETH-USB1 (Pilot).
- New avionics/kicad/align_pb2_ti_names.py does the exact-token rename across generators,
  schematics, symbol libraries, PCBs, netlists, project netclasses and scripts. Pilot's
  schematic was regenerated from the edited generator and matched the text rename
  (modulo UUIDs). ERC / DRC / schematic-parity counts unchanged and the Pilot parity item
  set is identical after renaming (Pilot 0 / 43 / 112 pre-existing, PCB re-sync pending;
  TACCO 0 / 5 / 0).
- Refdes-prefix parent tables made specific so the Bob-Smith parts stay with their
  transformer/connector. Unused imports removed in gen_pilot_pcb.py / gen_tacco_pcb.py.

Co-Authored-By: Claude Opus 5.5 <noreply@anthropic.com>
Parts:
- C-RMII2-A1: renamed from C-P1-A1; symbol Pilot:S_C-P1-A1 -> Pilot:S_C-RMII2-A1
- C-RMII2-A2: renamed from C-P1-A2; symbol Pilot:S_C-P1-A2 -> Pilot:S_C-RMII2-A2
- C-RMII2-A3: renamed from C-P1-A3; symbol Pilot:S_C-P1-A3 -> Pilot:S_C-RMII2-A3
- C-RMII2-BS: renamed from C-BS1; symbol Pilot:S_C-BS1 -> Pilot:S_C-RMII2-BS
- C-RMII2-CRD1: renamed from C-P1-CRD1; symbol Pilot:S_C-P1-CRD1 -> Pilot:S_C-RMII2-CRD1
- C-RMII2-CRD2: renamed from C-P1-CRD2; symbol Pilot:S_C-P1-CRD2 -> Pilot:S_C-RMII2-CRD2
- C-RMII2-CTD1: renamed from C-P1-CTD1; symbol Pilot:S_C-P1-CTD1 -> Pilot:S_C-RMII2-CTD1
- C-RMII2-CTD2: renamed from C-P1-CTD2; symbol Pilot:S_C-P1-CTD2 -> Pilot:S_C-RMII2-CTD2
- C-RMII2-IO1: renamed from C-P1-IO1; symbol Pilot:S_C-P1-IO1 -> Pilot:S_C-RMII2-IO1
- C-RMII2-IO2: renamed from C-P1-IO2; symbol Pilot:S_C-P1-IO2 -> Pilot:S_C-RMII2-IO2
- C-RMII2-IO3: renamed from C-P1-IO3; symbol Pilot:S_C-P1-IO3 -> Pilot:S_C-RMII2-IO3
- C-USB1-A1: renamed from C-U2-A1; symbol Pilot:S_C-U2-A1 -> Pilot:S_C-USB1-A1
- C-USB1-AK: renamed from C-U2-AK; symbol Pilot:S_C-U2-AK -> Pilot:S_C-USB1-AK
- C-USB1-BS: renamed from C-BS2; symbol Pilot:S_C-BS2 -> Pilot:S_C-USB1-BS
- C-USB1-CRD: renamed from C-U2-CRD; symbol Pilot:S_C-U2-CRD -> Pilot:S_C-USB1-CRD
- C-USB1-CTD: renamed from C-U2-CTD; symbol Pilot:S_C-U2-CTD -> Pilot:S_C-USB1-CTD
- C-USB1-DK: renamed from C-U2-DK; symbol Pilot:S_C-U2-DK -> Pilot:S_C-USB1-DK
- C-USB1-IO: renamed from C-U2-IO; symbol Pilot:S_C-U2-IO -> Pilot:S_C-USB1-IO
- C-USB1-V5A: renamed from C-U2-V5A; symbol Pilot:S_C-U2-V5A -> Pilot:S_C-USB1-V5A
- C-USB1-V5B: renamed from C-U2-V5B; symbol Pilot:S_C-U2-V5B -> Pilot:S_C-USB1-V5B
- J-ETH-RMII2: renamed from ETH1; symbol Pilot:S_ETH1 -> Pilot:S_J-ETH-RMII2
- J-ETH-USB1: renamed from ETH2; symbol Pilot:S_ETH2 -> Pilot:S_J-ETH-USB1
- NIC-USB1: renamed from ETH2-USB; symbol Pilot:S_ETH2-USB -> Pilot:S_NIC-USB1
- PHY-RMII2: renamed from ETH1-PHY; symbol Pilot:S_ETH1-PHY -> Pilot:S_PHY-RMII2
- R-RMII2-AD0: renamed from R-P1-AD0; symbol Pilot:S_R-P1-AD0 -> Pilot:S_R-RMII2-AD0
- R-RMII2-BSR: renamed from R-BS1R; symbol Pilot:S_R-BS1R -> Pilot:S_R-RMII2-BSR
- R-RMII2-BST: renamed from R-BS1T; symbol Pilot:S_R-BS1T -> Pilot:S_R-RMII2-BST
- R-RMII2-RBIAS: renamed from R-P1-RBIAS; symbol Pilot:S_R-P1-RBIAS -> Pilot:S_R-RMII2-RBIAS
- R-USB1-BSR: renamed from R-BS2R; symbol Pilot:S_R-BS2R -> Pilot:S_R-USB1-BSR
- R-USB1-BST: renamed from R-BS2T; symbol Pilot:S_R-BS2T -> Pilot:S_R-USB1-BST
- T-RMII2: renamed from T-ETH; symbol Pilot:S_T-ETH -> Pilot:S_T-RMII2
- T-USB1: renamed from T-ETH2; symbol Pilot:S_T-ETH2 -> Pilot:S_T-USB1
Connections:
- net ETH1-PHY_RBIAS renamed PHY-RMII2_RBIAS
- net ETH2-USB_AVDDK renamed NIC-USB1_AVDDK
- net ETH2-USB_DVDDK renamed NIC-USB1_DVDDK
- net ETH2_BS renamed ETH_USB1_BS
- net ETH2_CRD renamed ETH_USB1_CRD
- net ETH2_CTD renamed ETH_USB1_CTD
- net ETH2_LINE_CRX renamed ETH_USB1_LINE_CRX
- net ETH2_LINE_CTX renamed ETH_USB1_LINE_CTX
- net ETH2_LINE_RXN renamed ETH_USB1_LINE_RXN
- net ETH2_LINE_RXP renamed ETH_USB1_LINE_RXP
- net ETH2_LINE_TXN renamed ETH_USB1_LINE_TXN
- net ETH2_LINE_TXP renamed ETH_USB1_LINE_TXP
- net ETH2_RXN renamed ETH_USB1_RXN
- net ETH2_RXP renamed ETH_USB1_RXP
- net ETH2_TXN renamed ETH_USB1_TXN
- net ETH2_TXP renamed ETH_USB1_TXP
- net ETH_BS renamed ETH_RMII2_BS
- net ETH_CRD renamed ETH_RMII2_CRD
- net ETH_CTD renamed ETH_RMII2_CTD
- net ETH_LINE_CRX renamed ETH_RMII2_LINE_CRX
- net ETH_LINE_CTX renamed ETH_RMII2_LINE_CTX
- net ETH_LINE_RXN renamed ETH_RMII2_LINE_RXN
- net ETH_LINE_RXP renamed ETH_RMII2_LINE_RXP
- net ETH_LINE_TXN renamed ETH_RMII2_LINE_TXN
- net ETH_LINE_TXP renamed ETH_RMII2_LINE_TXP
- net ETH_RXN renamed ETH_RMII2_RXN
- net ETH_RXP renamed ETH_RMII2_RXP
- net ETH_TXN renamed ETH_RMII2_TXN
- net ETH_TXP renamed ETH_RMII2_TXP
- net PHY1_INTRN renamed RMII2_PHY_INTRN
- net PHY1_RSTN renamed RMII2_PHY_RSTN
