File: avionics/kicad/Pilot/kicads/Pilot.kicad_sch (KiCad schematic)
At the start: 118 parts, among them X2Y-CAN 4.7nF X2Y, X2Y-RS485 4.7nF X2Y

Commit message: feat(pilot): single 6-pin J-SPI expansion port; compliant field-port TVS
Schematic only (ERC 0, 118 -> 111 parts); the PCB re-sync waits for the
AX88772E swap so the board is re-placed and re-routed once.

Owner decisions (S. Griffing, 2026-10-17), implemented by Claude Opus 5.5:

- One JST-GH expansion port: J-SPI becomes a 6-pin SM06B-GHS-TB (5V, SCK,
  MISO, MOSI, !SS1, GND; Pixhawk DS-009 "SPI port" order without !SS2,
  [REF-CONN-002]). The SPI2 balls also mux to UART1/UART6 (SPRSP58C
  Table 5-1 [REF-SENSOR-049], PB2I_AM625_HEADER_CAPABILITIES.md sec 4).
  J-GPS, F-GPS, C-GPS5, R-I2C-SCL/SDA, ESD-GPS and ESD-SS2 removed;
  P1-31/33/36 and P2-2/4 are spare.
- AGENTS.md sec 5 sourcing rule: the Nexperia (Wingtech, PRC) PRTR5V0U2X is
  replaced. It was also a 5 V rail-referenced clamp, holding CAN and RS-485
  lines inside 0..5 V.
    TVS-CAN    -> TI ESD2CAN24DCKRQ1, SC-70, +/-24 V, 3 pF
                  (SLVSFW5D Table 4-1, sec 5.7) [REF-SENSOR-053];
                  ISOW1044 bus pins are rated +/-58 V [REF-SENSOR-009].
    TVS-RS485  -> Bourns CDSOT23-SM712, SOT-23, -7/+12 V VWM [REF-SENSOR-054];
                  ISOW1412 bus pins are rated -12..+15 V [REF-SENSOR-010].
    TVS-1553P/N -> Bourns SMAJ33CA [REF-SENSOR-055]. The old local SMAJ PDF
                  names no manufacturer.
- The generator gains an optional `mfr` flag that emits a `Manufacturer`
  schematic property, so generic part numbers name their maker of record.
- REFERENCES.md adds REF-SENSOR-053..056 (056 = the owner-supplied ASIX
  AX88772E datasheet v1.03; no confidentiality marking; 0-70 C accepted by
  the owner, since -40..85 C is the PB2-I module's rating, not a board
  requirement). REF-SENSOR-038 is marked as failing the sourcing rule.
- WBS items closed and avionics/TODO.md regenerated; Pilot.md update block;
  CLAUDE-MEMORY.md mirror refreshed.

Verification: kicad-cli 9.0.2 sch erc = 0 violations. The netlist diff
against the unchanged-generator output shows exactly the 7 parts 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
Parts:
- removed C-25M: 100nF, Capacitor_SMD:C_0402_1005Metric, symbol Pilot:S_C-25M
- removed C-50M: 100nF, Capacitor_SMD:C_0402_1005Metric, symbol Pilot:S_C-50M
- removed C-GPS5: 1uF 10V, Capacitor_SMD:C_0402_1005Metric, symbol Pilot:S_C-GPS5
- removed C-IMU1: 100nF, Capacitor_SMD:C_0402_1005Metric, symbol Pilot:S_C-IMU1
- removed ESD-GPS: TPD4E05U06DQAR, Serenity-Custom:TI_DQA0010A_USON-10_2.5x1.0mm_P0.5mm, symbol Pilot:S_ESD-GPS
- removed ESD-SS2: TPD1E05U06DYAR, Diode_SMD:D_SOD-523, symbol Pilot:S_ESD-SS2
- removed F-GPS: MF-PSMF035X, Fuse:Fuse_0805_2012Metric, symbol Pilot:S_F-GPS
- removed J-GPS: SM06B-GHS-TB, Connector_JST:JST_GH_SM06B-GHS-TB_1x06-1MP_P1.25mm_Horizontal, symbol Pilot:S_J-GPS
- removed R-1553P: 55R 2%, Resistor_SMD:R_0603_1608Metric, symbol Pilot:S_R-1553P
- removed R-I2C-SCL: 1.5k, Resistor_SMD:R_0201_0603Metric, symbol Pilot:S_R-I2C-SCL
- removed R-I2C-SDA: 1.5k, Resistor_SMD:R_0201_0603Metric, symbol Pilot:S_R-I2C-SDA
- removed R-RMII2-AD0: 2.49k, Resistor_SMD:R_0201_0603Metric, symbol Pilot:S_R-RMII2-AD0
- added C-USB1-BS: 10nF 2kV, Capacitor_SMD:C_1808_4520Metric, symbol Pilot:S_C-USB1-BS
- added H2: M2.5 PGND, Serenity-Custom:MountingHole_2.7mm_M2.5_PGND_Ring, symbol Pilot:S_H2
- added R-1553IRQ: 10k, Resistor_SMD:R_0402_1005Metric, symbol Pilot:S_R-1553IRQ
- added X-25M: 25MHz 3.3V, Oscillator:Oscillator_SMD_ECS_2520MV-xxx-xx-4Pin_2.5x2.0mm, symbol Pilot:S_X-25M
- added X-50M: 50MHz 3.3V, Oscillator:Oscillator_SMD_ECS_2520MV-xxx-xx-4Pin_2.5x2.0mm, symbol Pilot:S_X-50M
- C-25M: renamed from C-USB1-BS; value 10nF 2kV -> 100nF; footprint Capacitor_SMD:C_1808_4520Metric -> Capacitor_SMD:C_0402_1005Metric; symbol Pilot:S_C-USB1-BS -> Pilot:S_C-25M
- C-50M: renamed from R-1553IRQ; value 10k -> 100nF; footprint Resistor_SMD:R_0402_1005Metric -> Capacitor_SMD:C_0402_1005Metric; symbol Pilot:S_R-1553IRQ -> Pilot:S_C-50M
- C-IMU1: renamed from X-50M; value 50MHz 3.3V -> 100nF; footprint Oscillator:Oscillator_SMD_ECS_2520MV-xxx-xx-4Pin_2.5x2.0mm -> Capacitor_SMD:C_0402_1005Metric; symbol Pilot:S_X-50M -> Pilot:S_C-IMU1; MPN ECS-2520MV-500-BN-TR -> (none)
- J-SPI: value SM07B-GHS-TB -> SM06B-GHS-TB; footprint Connector_JST:JST_GH_SM07B-GHS-TB_1x07-1MP_P1.25mm_Horizontal -> Connector_JST:JST_GH_SM06B-GHS-TB_1x06-1MP_P1.25mm_Horizontal; MPN SM07B-GHS-TB(LF)(SN) -> SM06B-GHS-TB(LF)(SN)
- R-1553P: renamed from X-25M; value 25MHz 3.3V -> 55R 2%; footprint Oscillator:Oscillator_SMD_ECS_2520MV-xxx-xx-4Pin_2.5x2.0mm -> Resistor_SMD:R_0603_1608Metric; symbol Pilot:S_X-25M -> Pilot:S_R-1553P; MPN ECS-2520MV-250-BN-TR -> (none)
- R-RMII2-AD0: renamed from H2; value M2.5 PGND -> 2.49k; footprint Serenity-Custom:MountingHole_2.7mm_M2.5_PGND_Ring -> Resistor_SMD:R_0201_0603Metric; symbol Pilot:S_H2 -> Pilot:S_R-RMII2-AD0
- TVS-1553N, TVS-1553P: Manufacturer (none) -> Bourns
- TVS-CAN: value PRTR5V0U2X -> ESD2CAN24-Q1; footprint Package_TO_SOT_SMD:SOT-363_SC-70-6 -> Package_TO_SOT_SMD:SOT-323_SC-70; MPN PRTR5V0U2X,115 -> ESD2CAN24DCKRQ1; Manufacturer (none) -> Texas Instruments
- TVS-RS485: value PRTR5V0U2X -> CDSOT23-SM712; footprint Package_TO_SOT_SMD:SOT-363_SC-70-6 -> Package_TO_SOT_SMD:SOT-23; MPN PRTR5V0U2X,115 -> CDSOT23-SM712; Manufacturer (none) -> Bourns
Connections:
- net +3V3: now also C-25M.1 (P), C-IMU1.1 (P), R-RMII2-AD0.1 (A), R-1553IRQ.1 (A), X-25M.4 (VDD), X-50M.4 (VDD); no longer C-IMU1.4 (VDD), R-1553P.4 (VDD)
- net BUS_1553_P: now also R-1553P.2 (B)
- net CAN_L_F: now also TVS-CAN.2 (IO2); no longer TVS-CAN.3 (IO2)
- net ETH_USB1_BS: now also C-USB1-BS.1 (P); no longer C-25M.1 (P)
- net GND: now also C-25M.2 (N), C-50M.2 (N), J-SPI.6 (GND), X-25M.2 (GND), X-50M.2 (GND); no longer J-SPI.7 (GND), R-1553P.2 (GND)
- net GND2_CAN: now also TVS-CAN.3 (GND); no longer TVS-CAN.2 (GND)
- net GND2_RS485: now also TVS-RS485.3 (COM); no longer TVS-RS485.2 (GND)
- net M1553_IRQN: now also R-1553IRQ.2 (B); no longer C-50M.2 (B)
- net M1553_MCLK: now also X-50M.3 (OUT); no longer C-IMU1.3 (OUT)
- net M1553_SEC_P: now also R-1553P.1 (A)
- net PGND: now also C-USB1-BS.2 (N), H2.1 (PGND); no longer C-25M.2 (N), R-RMII2-AD0.1 (PGND)
- net RMII2_RXD0: now also R-RMII2-AD0.2 (B)
- net RS485_B_F: now also TVS-RS485.2 (IO2); no longer TVS-RS485.3 (IO2)
- net VCC2_CAN: no longer TVS-CAN.5 (VCC)
- net VCC2_RS485: no longer TVS-RS485.5 (VCC)
- net XI_25M: now also X-25M.3 (OUT); no longer R-1553P.3 (OUT)
- net EXT_I2C_SCL: no longer names the net of PB2-P1.36 (P1.36)
- net EXT_I2C_SDA: no longer names the net of PB2-P1.33 (P1.33)
- net EXT_SPI_SS2: no longer names the net of PB2-P1.31 (P1.31)
- net EXT_SPI_SS2: no longer J-SPI.6 (SS2)
- net EXT_UART_RX: no longer names the net of PB2-P2.2 (P2.02)
- net EXT_UART_TX: no longer names the net of PB2-P2.4 (P2.04)
- no-connect marks 106 -> 103
Other:
- moved on the sheet: C-25M, C-50M

Commit message: feat(pilot): replace CH397A USB NIC with ASIX AX88772E per ASIX demo board
Schematic only (ERC 0, 111 -> 134 parts). The PCB re-sync is still pending.

The WCH CH397A (PRC-domiciled, AGENTS.md sec 5) is replaced by the ASIX
AX88772EQF [REF-SENSOR-056] (owner selection 2026-10-17). The circuit
follows the ASIX demo board V1.01 sheet 2 [REF-SENSOR-058], its BOM
[REF-SENSOR-060] and the Application Design Note v1.10 [REF-SENSOR-057].
Owner documents supplied 2026-10-18; implemented by Claude Opus 5.5.

- Own 20 MHz crystal. The part does not support an external oscillator
  (app note sec 5 note 2), so X-25M now clocks only the DP83825I.
  Y-USB1 = ECS ECS-200-20-33-AGM-TR [REF-SENSOR-059]: CL 20 pF, +/-25 ppm
  tolerance, +/-30 ppm stability, ESR 60 ohm max. It has 15 pF load caps
  and a 200 ohm series resistor, as on the demo. The demo's "NSK 20M
  CRYSTAL" has no part number or identifiable maker.
- On-die 1.1 V buck: LX -> L-USB1 2.2 uH -> DVDD11, then a bead to
  AVDD11; the 3.3 V analog pins sit behind a bead from +3V3. The beads
  reuse the vetted Murata BLM15EX331SN1D [REF-SENSOR-043]. Every power pin
  has a 0.1 uF (app note sec 8 item 5).
- VBUS (owner 2026-10-18): 4.7 k pull-up to +3V3 plus PB2-I P1-31
  GPIO0_59, so the NIC attaches without firmware and Linux can force a
  detach.
- RSET 24 k 1 %; PU and PME pulled up with 4.7 k. RST_N, GPIO2/3/4 and
  the LED pins are left open, as on the demo's default fit.
- Land: KiCad QFN-32-1EP_4x4mm_P0.4mm_EP2.9x2.9mm matches the data sheet
  sec 6 recommended footprint to 0.02 mm.
- refloorplan_pilot.py PARENT anchors cover the new *-USB1 parts and
  still do not match the Bob-Smith C-USB1-BS / R-USB1-BS* parts.

Open (avionics/WBS.md): the L-USB1 part number (the Darfon data sheet is
not on file; the land is a 2.0 x 1.6 mm placeholder); ECS option-code
availability; DTS for P1-31.

Verification: kicad-cli 9.0.2 sch erc = 0. The netlist was checked pin
by pin for every NIC-USB1 net. flake8 reports no new findings (b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
Parts:
- removed C-1553D: 100nF, Capacitor_SMD:C_0402_1005Metric, symbol Pilot:S_C-1553D
- removed C-USB1-A1: 1uF, Capacitor_SMD:C_0402_1005Metric, symbol Pilot:S_C-USB1-A1
- removed C-USB1-AK: 1uF, Capacitor_SMD:C_0402_1005Metric, symbol Pilot:S_C-USB1-AK
- removed C-USB1-BS: 10nF 2kV, Capacitor_SMD:C_1808_4520Metric, symbol Pilot:S_C-USB1-BS
- removed C-USB1-DK: 100nF, Capacitor_SMD:C_0201_0603Metric, symbol Pilot:S_C-USB1-DK
- removed C-USB1-IO: 100nF, Capacitor_SMD:C_0201_0603Metric, symbol Pilot:S_C-USB1-IO
- removed C-USB1-V5A: 10uF 6.3V X6S, Capacitor_SMD:C_0603_1608Metric, symbol Pilot:S_C-USB1-V5A
- removed C-USB1-V5B: 100nF, Capacitor_SMD:C_0201_0603Metric, symbol Pilot:S_C-USB1-V5B
- removed H2: M2.5 PGND, Serenity-Custom:MountingHole_2.7mm_M2.5_PGND_Ring, symbol Pilot:S_H2
- removed R-1553IRQ: 10k, Resistor_SMD:R_0402_1005Metric, symbol Pilot:S_R-1553IRQ
- removed R-USB1-BSR: 75R, Resistor_SMD:R_0402_1005Metric, symbol Pilot:S_R-USB1-BSR
- removed X-25M: 25MHz 3.3V, Oscillator:Oscillator_SMD_ECS_2520MV-xxx-xx-4Pin_2.5x2.0mm, symbol Pilot:S_X-25M
- removed X-50M: 50MHz 3.3V, Oscillator:Oscillator_SMD_ECS_2520MV-xxx-xx-4Pin_2.5x2.0mm, symbol Pilot:S_X-50M
- added C-25M: 100nF, Capacitor_SMD:C_0402_1005Metric, symbol Pilot:S_C-25M
- added C-50M: 100nF, Capacitor_SMD:C_0402_1005Metric, symbol Pilot:S_C-50M
- added C-IMU1: 100nF, Capacitor_SMD:C_0402_1005Metric, symbol Pilot:S_C-IMU1
- added C-IMU2: 10nF, Capacitor_SMD:C_0201_0603Metric, symbol Pilot:S_C-IMU2
- added C-RMII2-A1: 10nF, Capacitor_SMD:C_0201_0603Metric, symbol Pilot:S_C-RMII2-A1
- added C-USB1-A11B: 10uF 6.3V X5R, Capacitor_SMD:C_0603_1608Metric, symbol Pilot:S_C-USB1-A11B
- added C-USB1-A11H1: 100nF, Capacitor_SMD:C_0201_0603Metric, symbol Pilot:S_C-USB1-A11H1
- added C-USB1-A11H2: 100nF, Capacitor_SMD:C_0201_0603Metric, symbol Pilot:S_C-USB1-A11H2
- added C-USB1-A33B: 4.7uF 10V X5R, Capacitor_SMD:C_0603_1608Metric, symbol Pilot:S_C-USB1-A33B
- added C-USB1-A33H1: 100nF, Capacitor_SMD:C_0201_0603Metric, symbol Pilot:S_C-USB1-A33H1
- added C-USB1-A33H2: 100nF, Capacitor_SMD:C_0201_0603Metric, symbol Pilot:S_C-USB1-A33H2
- added C-USB1-A33H3: 100nF, Capacitor_SMD:C_0201_0603Metric, symbol Pilot:S_C-USB1-A33H3
- added C-USB1-A33H4: 100nF, Capacitor_SMD:C_0201_0603Metric, symbol Pilot:S_C-USB1-A33H4
- added C-USB1-BKB: 4.7uF 10V X5R, Capacitor_SMD:C_0603_1608Metric, symbol Pilot:S_C-USB1-BKB
- added C-USB1-BKH: 100nF, Capacitor_SMD:C_0201_0603Metric, symbol Pilot:S_C-USB1-BKH
- added C-USB1-D04: 100nF, Capacitor_SMD:C_0201_0603Metric, symbol Pilot:S_C-USB1-D04
- added C-USB1-D10: 100nF, Capacitor_SMD:C_0201_0603Metric, symbol Pilot:S_C-USB1-D10
- added C-USB1-D11: 100nF, Capacitor_SMD:C_0201_0603Metric, symbol Pilot:S_C-USB1-D11
- added C-USB1-D22: 100nF, Capacitor_SMD:C_0201_0603Metric, symbol Pilot:S_C-USB1-D22
- added C-USB1-IO18: 100nF, Capacitor_SMD:C_0201_0603Metric, symbol Pilot:S_C-USB1-IO18
- added C-USB1-IO5: 100nF, Capacitor_SMD:C_0201_0603Metric, symbol Pilot:S_C-USB1-IO5
- added C-USB1-LXB: 10uF 6.3V X5R, Capacitor_SMD:C_0603_1608Metric, symbol Pilot:S_C-USB1-LXB
- added C-USB1-LXH: 100nF, Capacitor_SMD:C_0201_0603Metric, symbol Pilot:S_C-USB1-LXH
- added C-USB1-XI: 15pF C0G, Capacitor_SMD:C_0402_1005Metric, symbol Pilot:S_C-USB1-XI
- added C-USB1-XO: 15pF C0G, Capacitor_SMD:C_0402_1005Metric, symbol Pilot:S_C-USB1-XO
- added FB-USB1-A11: 330R@100MHz, Inductor_SMD:L_0402_1005Metric, symbol Pilot:S_FB-USB1-A11
- added FB-USB1-A33: 330R@100MHz, Inductor_SMD:L_0402_1005Metric, symbol Pilot:S_FB-USB1-A33
- added L-USB1: 2.2uH, Inductor_SMD:L_Murata_DFE201610P, symbol Pilot:S_L-USB1
- added R-1553N: 55R 2%, Resistor_SMD:R_0603_1608Metric, symbol Pilot:S_R-1553N
- added R-1553P: 55R 2%, Resistor_SMD:R_0603_1608Metric, symbol Pilot:S_R-1553P
- added R-USB1-PME: 4.7k, Resistor_SMD:R_0201_0603Metric, symbol Pilot:S_R-USB1-PME
- added R-USB1-PU: 4.7k, Resistor_SMD:R_0201_0603Metric, symbol Pilot:S_R-USB1-PU
- added R-USB1-RSET: 24k 1%, Resistor_SMD:R_0402_1005Metric, symbol Pilot:S_R-USB1-RSET
- added R-USB1-VBUS: 4.7k, Resistor_SMD:R_0201_0603Metric, symbol Pilot:S_R-USB1-VBUS
- added R-USB1-XO: 200R, Resistor_SMD:R_0402_1005Metric, symbol Pilot:S_R-USB1-XO
- added Y-USB1: 20MHz CL20pF, Crystal:Crystal_SMD_3225-4Pin_3.2x2.5mm, symbol Pilot:S_Y-USB1
- C-1553D: renamed from C-50M; symbol Pilot:S_C-50M -> Pilot:S_C-1553D
- C-USB1-BS: renamed from R-1553P; value 55R 2% -> 10nF 2kV; footprint Resistor_SMD:R_0603_1608Metric -> Capacitor_SMD:C_1808_4520Metric; symbol Pilot:S_R-1553P -> Pilot:S_C-USB1-BS
- C-USB1-CRD, C-USB1-CTD: value 1uF -> 100nF
- H2: renamed from C-RMII2-A1; value 10nF -> M2.5 PGND; footprint Capacitor_SMD:C_0201_0603Metric -> Serenity-Custom:MountingHole_2.7mm_M2.5_PGND_Ring; symbol Pilot:S_C-RMII2-A1 -> Pilot:S_H2
- NIC-USB1: value CH397A -> AX88772EQF; footprint Package_DFN_QFN:QFN-24-1EP_4x4mm_P0.5mm_EP2.8x2.8mm -> Package_DFN_QFN:QFN-32-1EP_4x4mm_P0.4mm_EP2.9x2.9mm; MPN CH397A -> AX88772EQF
- R-1553IRQ: renamed from C-IMU1; value 100nF -> 10k; footprint Capacitor_SMD:C_0402_1005Metric -> Resistor_SMD:R_0402_1005Metric; symbol Pilot:S_C-IMU1 -> Pilot:S_R-1553IRQ
- R-USB1-BSR: renamed from C-25M; value 100nF -> 75R; footprint Capacitor_SMD:C_0402_1005Metric -> Resistor_SMD:R_0402_1005Metric; symbol Pilot:S_C-25M -> Pilot:S_R-USB1-BSR
- X-25M: renamed from R-1553N; value 55R 2% -> 25MHz 3.3V; footprint Resistor_SMD:R_0603_1608Metric -> Oscillator:Oscillator_SMD_ECS_2520MV-xxx-xx-4Pin_2.5x2.0mm; symbol Pilot:S_R-1553N -> Pilot:S_X-25M; MPN (none) -> ECS-2520MV-250-BN-TR
- X-50M: renamed from C-IMU2; value 10nF -> 50MHz 3.3V; footprint Capacitor_SMD:C_0201_0603Metric -> Oscillator:Oscillator_SMD_ECS_2520MV-xxx-xx-4Pin_2.5x2.0mm; symbol Pilot:S_C-IMU2 -> Pilot:S_X-50M; MPN (none) -> ECS-2520MV-500-BN-TR
Connections:
- net +3V3: now also NIC-USB1.5 (DVDD33), X-25M.4 (VDD), X-50M.4 (VDD), C-25M.1 (P), C-50M.1 (P), C-IMU1.1 (P), C-IMU2.1 (P), C-RMII2-A1.1 (P), C-USB1-BKB.1 (P), C-USB1-BKH.1 (P), C-USB1-IO18.1 (P), C-USB1-IO5.1 (P), FB-USB1-A33.1 (A), R-USB1-PME.1 (A), R-USB1-PU.1 (A), R-USB1-VBUS.1 (A); no longer H2.1 (P), NIC-USB1.1 (AVDD33), NIC-USB1.10 (AVDD33), NIC-USB1.11 (V5), R-USB1-BSR.1 (P), X-50M.1 (P)
- net BUS_1553_N: now also R-1553N.2 (B); no longer X-25M.2 (B)
- net BUS_1553_P: now also R-1553P.2 (B); no longer C-USB1-BS.2 (B)
- net ETH_USB1_BS: now also C-USB1-BS.1 (P), R-USB1-BSR.2 (B)
- net ETH_USB1_LINE_CRX: now also R-USB1-BSR.1 (A)
- net ETH_USB1_RXN: now also NIC-USB1.31 (MDIN1); no longer NIC-USB1.5 (MDIRN)
- net ETH_USB1_RXP: now also NIC-USB1.30 (MDIP1); no longer NIC-USB1.4 (MDIRP)
- net ETH_USB1_TXN: now also NIC-USB1.28 (MDIN0); no longer NIC-USB1.3 (MDITN)
- net ETH_USB1_TXP: now also NIC-USB1.27 (MDIP0); no longer NIC-USB1.2 (MDITP)
- net GND: now also NIC-USB1.14 (AVSS33_BUCK), NIC-USB1.33 (EP), X-25M.2 (GND), C-25M.2 (N), C-50M.2 (N), C-IMU1.2 (N), C-IMU2.2 (N), C-RMII2-A1.2 (N), C-USB1-A11B.2 (N), C-USB1-A11H1.2 (N), C-USB1-A11H2.2 (N), C-USB1-A33B.2 (N), C-USB1-A33H1.2 (N), C-USB1-A33H2.2 (N), C-USB1-A33H3.2 (N), C-USB1-A33H4.2 (N), C-USB1-BKB.2 (N), C-USB1-BKH.2 (N), C-USB1-D04.2 (N), C-USB1-D10.2 (N), C-USB1-D11.2 (N), C-USB1-D22.2 (N), C-USB1-IO18.2 (N), C-USB1-IO5.2 (N), C-USB1-LXB.2 (N), C-USB1-LXH.2 (N), C-USB1-XI.2 (N), C-USB1-XO.2 (N), R-USB1-RSET.2 (B), Y-USB1.2 (GND), Y-USB1.4 (GND); no longer H2.2 (N), NIC-USB1.24 (GND), NIC-USB1.25 (EP), NIC-USB1.6 (GND), R-1553IRQ.2 (N), R-USB1-BSR.2 (N)
- net M1553_IRQN: now also R-1553IRQ.2 (B)
- net M1553_MCLK: now also X-50M.3 (OUT)
- net M1553_SEC_N: now also R-1553N.1 (A); no longer X-25M.1 (A)
- net M1553_SEC_P: now also R-1553P.1 (A); no longer C-USB1-BS.1 (A)
- net PGND: now also C-USB1-BS.2 (N), H2.1 (PGND)
- net USB1_DM: now also NIC-USB1.3 (USB_DM); no longer NIC-USB1.7 (UDM)
- net USB1_DP: now also NIC-USB1.2 (USB_DP); no longer NIC-USB1.8 (UDP)
- net XI_25M: now also X-25M.3 (OUT); no longer NIC-USB1.21 (XI)
- net NIC-USB1_LX: now reaches NIC-USB1.12 (LX)
- net NIC-USB1_LX: now also L-USB1.1 (A)
- net NIC-USB1_DVDD11: now reaches NIC-USB1.22 (DVDD11)
- net NIC-USB1_DVDD11: now also NIC-USB1.10 (DVDD11), NIC-USB1.11 (DVDD11), NIC-USB1.4 (DVDD11), C-USB1-D04.1 (P), C-USB1-D10.1 (P), C-USB1-D11.1 (P), C-USB1-D22.1 (P), C-USB1-LXB.1 (P), C-USB1-LXH.1 (P), FB-USB1-A11.1 (A), L-USB1.2 (B)
- net NIC-USB1_VBUS: now reaches PB2-P1.31 (P1.31)
- net NIC-USB1_VBUS: now also NIC-USB1.6 (VBUS), R-USB1-VBUS.2 (B)
- net NIC-USB1_AVDDK renamed NIC-USB1_XI
- net NIC-USB1_XI: now also C-USB1-XI.1 (P), Y-USB1.1 (X1)
- net NIC-USB1_DVDDK: no longer names the net of NIC-USB1.9 (NC)
- new net NIC-USB1_AVDD11: C-USB1-A11B.1 (P), C-USB1-A11H1.1 (P), C-USB1-A11H2.1 (P), FB-USB1-A11.2 (B), NIC-USB1.32 (AVDD11_GBE)
- new net NIC-USB1_AVDD33: C-USB1-A33B.1 (P), C-USB1-A33H1.1 (P), C-USB1-A33H2.1 (P), C-USB1-A33H3.1 (P), C-USB1-A33H4.1 (P), FB-USB1-A33.2 (B), NIC-USB1.1 (AVDD33_USB), NIC-USB1.25 (AVDD33_XTAL), NIC-USB1.29 (AVDD33_GBE)
- new net NIC-USB1_PME: NIC-USB1.8 (GPIO_8/PME), R-USB1-PME.2 (B)
- new net NIC-USB1_PU: NIC-USB1.7 (PU), R-USB1-PU.2 (B)
- new net NIC-USB1_RSET: NIC-USB1.26 (RSET), R-USB1-RSET.1 (A)
- new net NIC-USB1_XO: NIC-USB1.24 (XTAL_OUT), R-USB1-XO.1 (A)
- new net NIC-USB1_XO_R: C-USB1-XO.1 (P), R-USB1-XO.2 (B), Y-USB1.3 (X2)
- no-connect marks 103 -> 101
Other:
- moved on the sheet: C-1553D, C-USB1-BS, R-1553IRQ, R-USB1-BSR
